File: cad/cad.kicad_sch (KiCad schematic)
At the start: 23 parts

Commit message: I love KiCad
Parts:
- removed U12, U13, U8, U9: ~, symbol custom_symbol_lib:rising_edge_8_bit_latch
- removed U19: ~, symbol custom_symbol_lib:quad_and
- added U12: (no value), Package_DIP:DIP-48_W15.24mm, symbol custom_symbol_lib:2x8_bit_latch
- added U13: ~, Package_DIP:DIP-14_W7.62mm, symbol custom_symbol_lib:quad_and
- added U19: ~, Package_DIP:DIP-14_W7.62mm, symbol custom_symbol_lib:6xNOT
- added U8: ~, Package_DIP:DIP-48_W15.24mm, symbol custom_symbol_lib:2x8_bit_latch
- added U9: ~, Package_DIP:DIP-14_W7.62mm, symbol custom_symbol_lib:quad_OR
- U1, U14, U15, U16, U17, U2, U20, U21, U22, U23, U3, U4: footprint (none) -> Package_DIP:DIP-16_W7.62mm
- U10, U11: footprint (none) -> Package_DIP:DIP-28_W15.24mm
- U18, U6, U7: footprint (none) -> Package_DIP:DIP-20_W7.62mm
- U5: footprint (none) -> custom_footprint_library:bus_connector
Connections:
- new net: U12.1 (OE_A#), U12.24 (OE_B#), U12.4 (GND), U13.7 (GND), U14.8 (GND), U15.8 (GND), U16.8 (GND), U17.8 (GND), U18.10 (GND), U19.7 (GND), U5.11 (GND), U9. (GND)
- new net: U12.36 (DB0), U5.4 (WRITE_0), U9.1 (0A)
- new net: U5.1 (READ_0), U9.2 (0B), U9.5 (1A)
- new net: U12.33 (DB2), U8.25 (CLK2), U8.48 (CLK1), U9.3 (Q0)
- new net: U12.30 (DB4), U9.4 (Q1)
- new net: U5.2 (READ_1), U9.6 (1B)
- new net: U1.6 (B0), U1.7 (C_IN), U1.8 (GND), U2.8 (GND), U3.8 (GND), U4.8 (GND), U6.10 (GND), U7.10 (GND), U8.1 (OE1#), U8.24 (OE2#), U8.4 (GND)
- new net: U2.14 (A2), U8.11 (QA6)
- new net: U2.12 (A3), U8.12 (QA7)
- new net: U3.5 (A0), U8.13 (QB0)
- new net: U3.3 (A1), U8.14 (QB1)
- new net: U3.14 (A2), U8.16 (QB2)
- new net: U3.12 (A3), U8.17 (QB3)
- new net: U4.5 (A0), U8.19 (QB4)
- new net: U1.5 (A0), U8.2 (QA0)
- new net: U4.3 (A1), U8.20 (QB5)
- new net: U4.14 (A2), U8.22 (QB6)
- new net: U4.12 (A3), U8.23 (QB7)
- new net: U17.12 (A3), U23.11 (A3), U7.19 (Q7), U8.26 (DB7)
- new net: U17.14 (A2), U23.14 (A2), U7.16 (Q6), U8.27 (DB6)
- new net: U17.3 (A1), U23.5 (A1), U7.15 (Q5), U8.29 (DB5)
- new net: U1.3 (A1), U8.3 (QA1)
- new net: U17.5 (A0), U23.2 (A0), U7.12 (Q4), U8.30 (DB4)
- new net: U16.12 (A3), U22.11 (A3), U7.9 (Q3), U8.32 (DB3)
- new net: U16.14 (A2), U22.14 (A2), U7.6 (Q2), U8.33 (DB2)
- new net: U16.3 (A1), U22.5 (A1), U7.5 (Q1), U8.35 (DB1)
- new net: U16.5 (A0), U22.2 (A0), U7.2 (Q0), U8.36 (DB0)
- new net: U15.12 (A3), U21.11 (A3), U6.19 (Q7), U8.37 (DA7)
- new net: U15.14 (A2), U21.14 (A2), U6.16 (Q6), U8.38 (DA6)
- new net: U15.3 (A1), U21.5 (A1), U6.15 (Q5), U8.40 (DA5)
- new net: U15.5 (A0), U21.2 (A0), U6.12 (Q4), U8.41 (DA4)
- new net: U14.12 (A3), U20.11 (A3), U6.9 (Q3), U8.43 (DA3)
- new net: U14.14 (A2), U20.14 (A2), U6.6 (Q2), U8.44 (DA2)
- new net: U14.3 (A1), U20.5 (A1), U6.5 (Q1), U8.46 (DA1)
- new net: U14.5 (A0), U20.2 (A0), U6.2 (Q0), U8.47 (DA0)
- new net: U1.14 (A2), U8.5 (QA2)
- new net: U1.12 (A3), U8.6 (QA3)
- new net: U1.16 (V+), U12.7 (V+), U13.14 (V+), U14.16 (V+), U14.7 (C_IN), U15.16 (V+), U16.11 (B3), U16.15 (B2), U16.16 (V+), U16.2 (B1), U16.6 (B0), U17.11 (B3), U17.15 (B2), U17.16 (V+), U17.2 (B1), U17.6 (B0), U18.1 (CLEAR#), U18.20 (V+), U19.14 (V+), U2.16 (V+), U3.16 (V+), U5.10 (V+), U6.1 (CLEAR#), U6.20 (V+), U7.20 (V+), U8.7 (V+)
- new net: U2.5 (A0), U8.8 (QA4)
- new net: U2.3 (A1), U8.9 (QA5)
- new net: U4.1 (Σ1), U7.14 (D5)
- new net: U4.10 (Σ3), U7.18 (D7)
- new net: U1.11 (B3), U1.15 (B2), U1.2 (B1), U12.14 (QB1), U2.11 (B3), U2.15 (B2), U2.2 (B1), U2.6 (B0), U3.11 (B3), U3.15 (B2), U3.2 (B1), U3.6 (B0), U4.11 (B3), U4.15 (B2), U4.2 (B1), U4.6 (B0)
- new net: U4.13 (Σ2), U7.17 (D6)
- new net: U4.4 (Σ0), U7.13 (D4)
- new net: U3.9 (C_OUT), U4.7 (C_IN)
- new net: U12.22 (QB6), U13.1 (1A)
- new net: U12.25 (CLK_B), U13.2 (1B), U5.9 (CLK_B)
- new net: U12.17 (QB3), U13.4 (2A)
- new net: U12.48 (CLK_A), U13.5 (2B), U5.8 (CLK_A)
- new net: U13.6 (2Q), U6.11 (CLK), U7.11 (CLK)
- new net: U14.10 (Σ3), U20.10 (B3)
- new net: U10.10 (A0), U10.7 (A3), U10.8 (A2), U10.9 (A1), U11.10 (A0), U11.7 (A3), U11.8 (A2), U11.9 (A1), U20.12 (Q2), U20.4 (Q0), U20.7 (Q1), U20.9 (Q3)
- new net: U14.13 (Σ2), U20.13 (B2)
- new net: U20.15 (E#), U20.8 (GND)
- new net: U20.16 (V+), U21.16 (V+), U22.16 (V+), U23.16 (V+)
- new net: U14.4 (Σ0), U20.3 (B0)
- new net: U14.1 (Σ1), U20.6 (B1)
- new net: U3.1 (Σ1), U7.4 (D1)
- new net: U3.10 (Σ3), U7.8 (D3)
- new net: U3.13 (Σ2), U7.7 (D2)
- new net: U3.4 (Σ0), U7.3 (D0)
- new net: U2.9 (C_OUT), U3.7 (C_IN)
- new net: U12.13 (QB0), U12.47 (DA0)
- new net: U12.16 (QB2), U12.46 (DA1)
- new net: U12.19 (QB4), U12.44 (DA2)
- new net: U12.2 (QA0), U12.35 (DB1)
- new net: U12.20 (QB5), U12.43 (DA3)
- new net: U12.27 (DB6), U12.6 (QA3)
- new net: U12.29 (DB5), U12.5 (QA2)
- new net: U12.3 (QA1), U12.32 (DB3)
- new net: U10.11 (D0), U11.11 (D0), U18.3 (D0), U5.12 (D0)
- new net: U10.12 (D1), U11.12 (D1), U18.4 (D1), U5.13 (D1)
- new net: U10.13 (D2), U11.13 (D2), U18.7 (D2), U5.14 (D2)
- new net: U10.15 (D3), U11.15 (D3), U18.8 (D3), U5.15 (D3)
- new net: U10.16 (D4), U11.16 (D4), U18.13 (D4), U5.16 (D4)
- new net: U10.17 (D5), U11.17 (D5), U18.14 (D5), U5.17 (D5)
- new net: U10.18 (D6), U11.18 (D6), U18.17 (D6), U5.18 (D6)
- new net: U10.19 (D7), U11.19 (D7), U18.18 (D7), U5.19 (D7)
- new net: U2.1 (Σ1), U6.14 (D5)
- new net: U2.10 (Σ3), U6.18 (D7)
- new net: U2.13 (Σ2), U6.17 (D6)
- new net: U2.4 (Σ0), U6.13 (D4)
- new net: U1.9 (C_OUT), U2.7 (C_IN)
- new net: U10.1 (A14), U11.1 (A14), U23.12 (Q2)
- new net: U10.2 (A12), U11.2 (A12), U23.4 (Q0)
- new net: U10.21 (A10), U11.21 (A10), U22.12 (Q2)
- new net: U10.23 (A11), U11.23 (A11), U22.9 (Q3)
- new net: U10.24 (A9), U11.24 (A9), U22.7 (Q1)
- new net: U10.25 (A8), U11.25 (A8), U22.4 (Q0)
- new net: U10.26 (A13), U11.26 (A13), U23.7 (Q1)
- new net: U10.3 (A7), U11.3 (A7), U21.9 (Q3)
- new net: U10.4 (A6), U11.4 (A6), U21.12 (Q2)
- new net: U10.5 (A5), U11.5 (A5), U21.7 (Q1)
- new net: U10.6 (A4), U11.6 (A4), U21.4 (Q0)
- new net: U1.1 (Σ1), U6.4 (D1)
- new net: U1.10 (Σ3), U6.8 (D3)
- new net: U1.13 (Σ2), U6.7 (D2)
- new net: U1.4 (Σ0), U6.3 (D0)
- new net: U14.11 (B3), U18.9 (Q3)
- new net: U14.15 (B2), U18.6 (Q2)
- new net: U14.2 (B1), U18.5 (Q1)
- new net: U14.6 (B0), U18.2 (Q0)
- new net: U14.9 (C_OUT), U15.7 (C_IN)
- new net: U15.1 (Σ1), U21.6 (B1)
- new net: U15.10 (Σ3), U21.10 (B3)
- new net: U15.11 (B3), U18.19 (Q7)
- new net: U15.13 (Σ2), U21.13 (B2)
- new net: U15.15 (B2), U18.16 (Q6)
- new net: U15.2 (B1), U18.15 (Q5)
- new net: U15.4 (Σ0), U21.3 (B0)
- new net: U15.6 (B0), U18.12 (Q4)
- new net: U15.9 (C_OUT), U16.7 (C_IN)
- new net: U21.15 (E#), U21.8 (GND)
- new net: U16.10 (Σ3), U22.10 (B3)
- new net: U16.13 (Σ2), U22.13 (B2)
- new net: U22.15 (E#), U22.8 (GND)
- new net: U16.4 (Σ0), U22.3 (B0)
- new net: U16.1 (Σ1), U22.6 (B1)
- new net: U16.9 (C_OUT), U17.7 (C_IN)
- new net: U17.10 (Σ3), U23.10 (B3)
- new net: U17.13 (Σ2), U23.13 (B2)
- new net: U23.15 (E#), U23.8 (GND)
- new net: U17.4 (Σ0), U23.3 (B0)
- new net: U17.1 (Σ1), U23.6 (B1)
Other:
- note added: "Decrement (for pop)"
- note added: "Load new value"
- note added: "WRITE 2: (unused) WRITE 1: OFFSET-READ WRITE 0: STACK-POP READ 2: SET-STACK-OFFSET READ 1: OFFSET-WRITE READ 0: STACK-PUSH"
- note added: "Write"
