File: kicad/ALU/ALU.kicad_sch (KiCad schematic)
At the start: 17 parts

Commit message: Done w/ ALU schematic
Parts:
- added R1, R2, R3, R4, R5: 10k, custom_footprint_library:0.4_pitch_resistor, symbol Device:R
- added U18, U19, U52: ~, Package_DIP:DIP-14_W7.62mm, symbol custom_symbol_lib:6xNOT
- added U20, U22, U26, U29, U38, U43, U44, U45: ~, Package_DIP:DIP-20_W7.62mm, symbol custom_symbol_lib:8_bit_transparent_latch
- added U21, U23: ~, Package_DIP:DIP-14_W7.62mm, symbol custom_symbol_lib:quad_OR
- added U24, U25, U42, U50, U53, U54: ~, Package_DIP:DIP-14_W7.62mm, symbol custom_symbol_lib:quad_and
- added U27, U28, U39, U40: ~, Package_DIP:DIP-14_W7.62mm, symbol custom_symbol_lib:4x_XNOR
- added U30, U31, U32, U33, U34, U35, U36, U37: ~, Package_DIP:DIP-16_W7.62mm, symbol custom_symbol_lib:multiplexer_8_bit
- added U41: ~, Package_DIP:DIP-14_W7.62mm, symbol custom_symbol_lib:2x_4_input_AND
- added U46, U47, U48, U49: ~, custom_footprint_library:jumper, symbol custom_symbol_lib:jumper
- added U51: ~, Package_DIP:DIP-14_W7.62mm, symbol custom_symbol_lib:dual_latch
- U16, U17, U6: symbol custom_symbol_lib:rising_edge_8_bit_latch -> custom_symbol_lib:8_bit_transparent_latch
Connections:
- net at U13.5 (A0), U3.1 (A0), U4.19 (Q0): now also U18.1 (I0), U21.1 (0A), U24.1 (1A), U27.1 (1A), U30.4 (D0), U31.3 (D1), U32.2 (D2), U33.1 (D3), U34.15 (D4), U35.14 (D5), U36.13 (D6), U37.12 (D7), U39.1 (1A), U44.2 (D0)
- net at U13.2 (B1), U3.10 (B1), U5.18 (Q1): now also U21.6 (1B), U24.5 (2B), U27.6 (2B), U30.10 (A1), U31.10 (A1), U32.10 (A1), U33.10 (A1), U34.10 (A1), U35.10 (A1), U36.10 (A1), U37.10 (A1), U39.6 (2B), U45.3 (D1)
- net at U13.15 (B2), U3.11 (B2), U5.17 (Q2): now also U21.9 (2B), U24.12 (3B), U27.9 (3B), U30.9 (A2), U31.9 (A2), U32.9 (A2), U33.9 (A2), U34.9 (A2), U35.9 (A2), U36.9 (A2), U37.9 (A2), U39.9 (3B), U45.4 (D2)
- net at U13.11 (B3), U3.12 (B3), U5.16 (Q3): now also U21.13 (3B), U24.9 (4B), U27.13 (4B), U39.13 (4B), U45.5 (D3)
- net at U15.6 (B0), U3.13 (B4), U5.15 (Q4): now also U23.2 (0B), U25.2 (1B), U28.2 (1B), U40.2 (1B), U45.6 (D4)
- net at U15.2 (B1), U3.14 (B5), U5.14 (Q5): now also U23.6 (1B), U25.5 (2B), U28.6 (2B), U40.6 (2B), U45.7 (D5)
- net at U15.15 (B2), U3.15 (B6), U5.13 (Q6): now also U23.9 (2B), U25.12 (3B), U28.9 (3B), U40.9 (3B), U45.8 (D6)
- net at U15.11 (B3), U3.16 (B7), U5.12 (Q7): now also U23.13 (3B), U25.9 (4B), U28.13 (4B), U40.13 (4B), U45.9 (D7)
- net at U13.3 (A1), U3.2 (A1), U4.18 (Q1): now also U18.3 (I1), U21.5 (1A), U24.4 (2A), U27.5 (2A), U30.12 (D7), U31.4 (D0), U32.3 (D1), U33.2 (D2), U34.1 (D3), U35.15 (D4), U36.14 (D5), U37.13 (D6), U39.5 (2A), U44.3 (D1)
- net at U13.8 (GND), U15.8 (GND), U16.10 (GND)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: now also U10.7 (GND), U11.11 (I4), U11.7 (GND), U12.7 (GND), U14.1 (OE#), U14.10 (GND), U2.13 (GND), U3.30 (GND), U4.10 (GND), U6.10 (GND), U7.8 (GND), U8.5 (E3#), U8.8 (GND), U9.7 (GND), R1.1, R2.1, R3.1, R4.1, R5.1, U18.7 (GND), U19.11 (I4), U19.13 (I5), U19.5 (I2), U19.7 (GND), U19.9 (I3), U20.10 (GND), U21.7 (GND), U22.10 (GND), U23.7 (GND), U24.7 (GND), U25.7 (GND), U26.10 (GND), U27.7 (GND), U28.7 (GND), U29.10 (GND), U30.7 (OE#), U30.8 (GND), U31.7 (OE#), U31.8 (GND), U32.7 (OE#), U32.8 (GND), U33.7 (OE#), U33.8 (GND), U34.7 (OE#), U34.8 (GND), U35.7 (OE#), U35.8 (GND), U36.7 (OE#), U36.8 (GND), U37.7 (OE#), U37.8 (GND), U38.10 (GND), U39.7 (GND), U40.7 (GND), U41.7 (GND), U42.10 (4A), U42.12 (3B), U42.13 (3A), U42.4 (2A), U42.5 (2B), U42.7 (GND), U42.9 (4B), U43.10 (GND), U43.3 (D1), U43.4 (D2), U43.5 (D3), U43.6 (D4), U43.7 (D5), U43.8 (D6), U43.9 (D7), U44.10 (GND), U45.10 (GND), U46.2 (GND), U47.2 (GND), U48.2 (GND), U49.2 (GND), U50.1 (1A), U50.2 (1B), U50.4 (2A), U50.5 (2B), U50.7 (GND), U51.10 (1RESET), U51.11 (1CLK), U51.4 (0RESET), U51.6 (0SET), U51.7 (GND), U51.8 (1SET), U51.9 (1D), U52.1 (I0), U52.11 (I4), U52.3 (I1), U52.5 (I2), U52.7 (GND), U52.9 (I3), U53.12 (3B), U53.13 (3A), U53.7 (GND), U54.10 (4A), U54.12 (3B), U54.13 (3A), U54.4 (2A), U54.5 (2B), U54.7 (GND), U54.9 (4B); no longer U12.14 (V+), U12.5 (1D), U3.29 (V+), U6.20 (V+)
- net at U13.14 (A2), U3.3 (A2), U4.17 (Q2): now also U18.5 (I2), U21.8 (2A), U24.13 (3A), U27.8 (3A), U30.13 (D6), U31.12 (D7), U32.4 (D0), U33.3 (D1), U34.2 (D2), U35.1 (D3), U36.15 (D4), U37.14 (D5), U39.8 (3A), U44.4 (D2)
- net at U12.12 (2C), U12.13 (2D), U13.16 (V+)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: now also U10.14 (V+), U11.14 (V+), U12.14 (V+), U14.20 (V+), U16.11 (CLK), U17.11 (CLK), U2.12 (V+), U3.29 (V+), U4.20 (V+), U5.20 (V+), U6.11 (CLK), U6.20 (V+), U7.16 (V+), U7.6 (E1), U8.16 (V+), U18.14 (V+), U19.14 (V+), U20.11 (CLK), U20.20 (V+), U21.14 (V+), U22.11 (CLK), U22.20 (V+), U23.14 (V+), U24.14 (V+), U25.14 (V+), U26.11 (CLK), U26.20 (V+), U27.14 (V+), U28.14 (V+), U29.11 (CLK), U29.20 (V+), U30.16 (V+), U31.16 (V+), U32.16 (V+), U33.16 (V+), U34.16 (V+), U35.16 (V+), U36.16 (V+), U37.16 (V+), U38.11 (CLK), U38.20 (V+), U39.14 (V+), U40.14 (V+), U41.14 (V+), U42.14 (V+), U43.11 (CLK), U43.20 (V+), U44.11 (CLK), U44.20 (V+), U45.11 (CLK), U45.20 (V+), U50.14 (V+), U51.14 (V+), U52.14 (V+), U53.14 (V+), U54.14 (V+); no longer U12.10 (2B), U12.7 (GND), U12.9 (2A), U3.30 (GND), U6.10 (GND)
- net at U13.12 (A3), U3.4 (A3), U4.16 (Q3): now also U18.9 (I3), U21.12 (3A), U24.10 (4A), U27.12 (4A), U30.14 (D5), U31.13 (D6), U32.12 (D7), U33.4 (D0), U34.3 (D1), U35.2 (D2), U36.1 (D3), U37.15 (D4), U39.12 (4A), U44.5 (D3)
- net at U15.5 (A0), U3.5 (A4), U4.15 (Q4): now also U18.11 (I4), U23.1 (0A), U25.1 (1A), U28.1 (1A), U30.15 (D4), U31.14 (D5), U32.13 (D6), U33.12 (D7), U34.4 (D0), U35.3 (D1), U36.2 (D2), U37.1 (D3), U40.1 (1A), U44.6 (D4)
- net at U15.3 (A1), U3.6 (A5), U4.14 (Q5): now also U18.13 (I5), U23.5 (1A), U25.4 (2A), U28.5 (2A), U30.1 (D3), U31.15 (D4), U32.14 (D5), U33.13 (D6), U34.12 (D7), U35.4 (D0), U36.3 (D1), U37.2 (D2), U40.5 (2A), U44.7 (D5)
- net at U15.14 (A2), U3.7 (A6), U4.13 (Q6): now also U19.1 (I0), U23.8 (2A), U25.13 (3A), U28.8 (3A), U30.2 (D2), U31.1 (D3), U32.15 (D4), U33.14 (D5), U34.13 (D6), U35.12 (D7), U36.4 (D0), U37.3 (D1), U40.8 (3A), U44.8 (D6)
- net at U15.12 (A3), U3.8 (A7), U4.12 (Q7): now also U19.3 (I1), U23.12 (3A), U25.10 (4A), U28.12 (4A), U30.3 (D1), U31.2 (D2), U32.1 (D3), U33.15 (D4), U34.14 (D5), U35.13 (D6), U36.12 (D7), U37.4 (D0), U40.12 (4A), U44.9 (D7)
- net at U13.6 (B0), U3.9 (B0), U5.19 (Q0): now also U21.2 (0B), U24.2 (1B), U27.2 (1B), U30.11 (A0), U31.11 (A0), U32.11 (A0), U33.11 (A0), U34.11 (A0), U35.11 (A0), U36.11 (A0), U37.11 (A0), U39.2 (1B), U45.2 (D0)
- net at U12.1 (1A): now also U10.10 (O4); no longer U11.8 (03)
- net at U12.2 (1B): now also U10.12 (O5); no longer U11.6 (O2)
- net at U12.4 (1C): now also U11.2 (O0); no longer U10.10 (O4)
- net at U12.6 (1Q): now also U54.1 (1A); no longer U6.1 (OE#)
- net at U12.8 (2Q): now also U54.2 (1B)
- net at U14.9 (D7), U16.12 (Q7), U17.12 (Q7)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: now also U20.12 (Q7), U22.12 (Q7), U26.12 (Q7), U29.12 (Q7), U38.12 (Q7), U43.12 (Q7), U44.12 (Q7), U45.12 (Q7)
- net at U14.8 (D6), U16.13 (Q6), U17.13 (Q6)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: now also U20.13 (Q6), U22.13 (Q6), U26.13 (Q6), U29.13 (Q6), U38.13 (Q6), U43.13 (Q6), U44.13 (Q6), U45.13 (Q6)
- net at U14.7 (D5), U16.14 (Q5), U17.14 (Q5)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: now also U20.14 (Q5), U22.14 (Q5), U26.14 (Q5), U29.14 (Q5), U38.14 (Q5), U43.14 (Q5), U44.14 (Q5), U45.14 (Q5)
- net at U14.6 (D4), U16.15 (Q4), U17.15 (Q4)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: now also U20.15 (Q4), U22.15 (Q4), U26.15 (Q4), U29.15 (Q4), U38.15 (Q4), U43.15 (Q4), U44.15 (Q4), U45.15 (Q4)
- net at U14.5 (D3), U16.16 (Q3), U17.16 (Q3)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: now also U20.16 (Q3), U22.16 (Q3), U26.16 (Q3), U29.16 (Q3), U38.16 (Q3), U43.16 (Q3), U44.16 (Q3), U45.16 (Q3)
- net at U14.4 (D2), U16.17 (Q2), U17.17 (Q2)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: now also U20.17 (Q2), U22.17 (Q2), U26.17 (Q2), U29.17 (Q2), U38.17 (Q2), U43.17 (Q2), U44.17 (Q2), U45.17 (Q2)
- net at U14.3 (D1), U16.18 (Q1), U17.18 (Q1)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: now also U20.18 (Q1), U22.18 (Q1), U26.18 (Q1), U29.18 (Q1), U38.18 (Q1), U43.18 (Q1), U44.18 (Q1), U45.18 (Q1)
- net at U14.2 (D0), U16.19 (Q0), U17.19 (Q0)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: now also U20.19 (Q0), U22.19 (Q0), U26.19 (Q0), U29.19 (Q0), U38.19 (Q0), U43.19 (Q0), U44.19 (Q0), U45.19 (Q0)
- net at U4.11 (CLK): now also U46.3 (OUT)
- net at U10.2 (O0): now also U38.1 (OE#)
- net at U10.4 (O1): now also U43.1 (OE#)
- net at U10.6 (O2): now also U44.1 (OE#)
- net at U10.8 (03): now also U45.1 (OE#)
- net at U5.11 (CLK): now also U47.3 (OUT)
- net at U14.11 (CLK): now also U48.3 (OUT)
- net at U9.10 (O4): now also U26.1 (OE#)
- net at U9.12 (O5): now also U29.1 (OE#)
- net at U9.6 (O2): now also U20.1 (OE#)
- net at U9.8 (03): now also U22.1 (OE#)
- net at U2.1 (READ_0): now also R1.2, U53.1 (1A)
- net at U2.10 (CLK_A): now also U53.2 (1B), U53.5 (2B), U53.9 (4B)
- net at U2.11 (CLK_B): now also U51.3 (0CLK)
- net at U2.2 (READ_1): now also R2.2, U53.4 (2A)
- net at U2.23 (ENABLE): now also R5.2, U50.12 (3B)
- net at U2.3 (READ_2): now also R3.2, U53.10 (4A)
- net at U2.5 (WRITE_0): now also R4.2, U50.10 (4A)
- net at U2.9 (READ_READY): now also U11.13 (I5), U49.3 (OUT)
- net at U11.12 (O5): now also U7.5 (E3#), U8.4 (E2#)
- net at U11.4 (O1): now also U12.5 (1D)
- new net: U30.5 (Q), U38.2 (D0)
- new net: U31.5 (Q), U38.3 (D1)
- new net: U32.5 (Q), U38.4 (D2)
- new net: U33.5 (Q), U38.5 (D3)
- new net: U34.5 (Q), U38.6 (D4)
- new net: U35.5 (Q), U38.7 (D5)
- new net: U36.5 (Q), U38.8 (D6)
- new net: U37.5 (Q), U38.9 (D7)
- new net: U11.8 (03), U12.10 (2B)
- new net: U11.6 (O2), U12.9 (2A)
- new net: U24.3 (1Q), U26.2 (D0)
- new net: U24.6 (2Q), U26.3 (D1)
- new net: U24.11 (3Q), U26.4 (D2)
- new net: U24.8 (4Q), U26.5 (D3)
- new net: U25.3 (1Q), U26.6 (D4)
- new net: U25.6 (2Q), U26.7 (D5)
- new net: U25.11 (3Q), U26.8 (D6)
- new net: U25.8 (4Q), U26.9 (D7)
- new net: U46.1 (IN), U53.3 (1Q)
- new net: U54.3 (1Q), U6.1 (OE#)
- new net: U21.3 (Q0), U22.2 (D0)
- new net: U21.4 (Q1), U22.3 (D1)
- new net: U21.10 (Q2), U22.4 (D2)
- new net: U21.11 (Q3), U22.5 (D3)
- new net: U22.6 (D4), U23.3 (Q0)
- new net: U22.7 (D5), U23.4 (Q1)
- new net: U22.8 (D6), U23.10 (Q2)
- new net: U22.9 (D7), U23.11 (Q3)
- new net: U27.10 (3Q), U29.4 (D2)
- new net: U27.11 (4Q), U29.5 (D3)
- new net: U27.3 (1Q), U29.2 (D0)
- new net: U27.4 (2Q), U29.3 (D1)
- new net: U49.1 (IN), U50.11 (3Q), U52.13 (I5)
- new net: U50.13 (3A), U51.1 (0Q)
- new net: U50.8 (4Q), U51.5 (0D)
- new net: U50.9 (4B), U52.12 (O5)
- new net: U19.2 (O0), U20.8 (D6)
- new net: U19.4 (O1), U20.9 (D7)
- new net: U47.1 (IN), U53.6 (2Q)
- new net: U48.1 (IN), U53.8 (4Q)
- new net: U41.6 (1Q), U42.1 (1A)
- new net: U41.8 (2Q), U42.2 (1B)
- new net: U42.3 (1Q), U43.2 (D0)
- new net: U39.3 (1Q), U41.1 (1A)
- new net: U40.4 (2Q), U41.10 (2B)
- new net: U40.10 (3Q), U41.12 (2C)
- new net: U40.11 (4Q), U41.13 (2D)
- new net: U39.4 (2Q), U41.2 (1B)
- new net: U39.10 (3Q), U41.4 (1C)
- new net: U39.11 (4Q), U41.5 (1D)
- new net: U40.3 (1Q), U41.9 (2A)
- new net: U28.10 (3Q), U29.8 (D6)
- new net: U28.11 (4Q), U29.9 (D7)
- new net: U28.3 (1Q), U29.6 (D4)
- new net: U28.4 (2Q), U29.7 (D5)
- new net: U18.10 (O4), U20.6 (D4)
- new net: U18.12 (O5), U20.7 (D5)
- new net: U18.2 (O0), U20.2 (D0)
- new net: U18.4 (O1), U20.3 (D1)
- new net: U18.6 (O2), U20.4 (D2)
- new net: U18.8 (03), U20.5 (D3)
- no-connect marks 1 -> 42
Other:
- note added: "A & B"
- note added: "ADD & ADD-C"
- note added: "ALU - - -"
- note added: "ALU-A ALU-B ALU-C-IN -"
- note added: "AND"
- note added: "EQ"
- note added: "NOT"
- note added: "OR"
- note added: "Opcodes 10 - 15 Not yet implemented"
- note added: "SHIFT"
- note added: "XNOR"
- note removed: "#10 (GREATER-THEN) #14 & 15 (MULT- A & B)"
- moved on the sheet: U1, U10, U11, U12, U13, U14, U15, U16, U17, U2, U3, U4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
