File: kicad/ALU/ALU.kicad_pcb (KiCad board)
At the start: 2 copper layers, 59 parts

Commit message: Finished IO controller schematic
Parts:
- moved U6 82.2 mm to (80.0, 154.4)
- moved U3 72.8 mm to (146.2, 188.5)
- moved U12 64.6 mm to (110.6, 167.2), turned to -90 degrees
- moved U54 59.4 mm to (134.6, 168.2), turned to -90 degrees
- moved U9 43.1 mm to (154.5, 150.9)
- moved U10 43.1 mm to (165.4, 150.9)
- moved U11 43.1 mm to (176.2, 150.9)
- moved U40 32.6 mm to (569.2, 150.4)
- moved U39 32.6 mm to (558.4, 150.4)
- moved U41 32.6 mm to (580.0, 150.4)
- moved U42 32.6 mm to (590.9, 150.4)
- moved U7 12.4 mm to (119.2, 137.4)
- moved U8 12.4 mm to (130.0, 137.4)
- moved U1 4.69 mm to (73.0, 68.9)
- moved U2 2.75 mm to (73.0, 93.8)
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
Commit message: Almost done with prog mem schematic
Parts:
- moved U45 423.3 mm to (199.4, 104.2), turned to -90 degrees
- moved U44 376.2 mm to (235.7, 104.4), turned to -90 degrees
- moved U40 365.5 mm to (208.6, 90.6), turned to 180 degrees
- moved U41 354.6 mm to (230.6, 90.2), turned to 180 degrees
- moved U42 337.2 mm to (259.2, 90.0), turned to -90 degrees
- moved U39 323.0 mm to (242.8, 81.0), turned to 90 degrees
- moved U43 315.2 mm to (265.2, 103.4), turned to -90 degrees
- moved U37 223.7 mm to (283.0, 99.8), turned to 180 degrees
- moved U33 196.5 mm to (277.3, 72.0), turned to 90 degrees
- moved U36 195.3 mm to (301.2, 100.8), turned to 180 degrees
- moved U38 190.0 mm to (300.4, 113.2), turned to -90 degrees
- moved U35 169.6 mm to (317.0, 100.8), turned to 180 degrees
- moved U32 161.1 mm to (305.6, 72.2), turned to 90 degrees
- moved U1 161.0 mm to (174.4, 194.0), turned to 90 degrees
- moved U34 142.2 mm to (335.0, 101.1), turned to 180 degrees
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Routing:
- net Net-(U10-V+): track 0.00 -> 1445.4 mm, vias 0 -> 15
- net Net-(U10-GND): track 0.00 -> 1389.0 mm, vias 0 -> 15
- net Net-(U13-A2): track 0.00 -> 801.6 mm, vias 0 -> 8
- net Net-(U13-A3): track 0.00 -> 784.5 mm, vias 0 -> 9
- net Net-(U15-A2): track 0.00 -> 762.7 mm, vias 0 -> 6
- net Net-(U15-A1): track 0.00 -> 758.7 mm, vias 0 -> 13
- net Net-(U13-B1): track 0.00 -> 737.4 mm, vias 0 -> 4
- net Net-(U15-A3): track 0.00 -> 733.5 mm, vias 0 -> 15
- net Net-(U13-B0): track 0.00 -> 725.7 mm, vias 0 -> 9
- net Net-(U13-B2): track 0.00 -> 722.7 mm, vias 0 -> 10
- net Net-(U15-A0): track 0.00 -> 721.5 mm, vias 0 -> 13
- net Net-(U13-A1): track 0.00 -> 689.7 mm, vias 0 -> 6
- net Net-(U13-A0): track 0.00 -> 641.9 mm, vias 0 -> 11
- net Net-(U13-B3): track 0.00 -> 580.7 mm, vias 0 -> 8
- net Net-(U15-B1): track 0.00 -> 563.9 mm, vias 0 -> 7
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- added copper zone on B.Cu, net Net-(U10-GND)
- added copper zone on F.Cu, net Net-(U10-V+)
Other:
- board outline added: 296 x 139 mm
- board text added: "30 ALU EXTENSION 1"
- board text added: "OPCODE 0 .... 3"
