File: kicad/gpram/gpram.kicad_sch (KiCad schematic)
At the start: 17 parts

Commit message: Working on GPRAM schematic
Parts:
- removed U6: ~, Package_DIP:DIP-16_W7.62mm, symbol custom_symbol_lib:4bit_adder
- added R1, R2, R3, R4, R5, R6, R7, R8, R9: 10k, custom_footprint_library:0.4_pitch_resistor, symbol Device:R
- added U18, U19, U20, U21, U22, U23, U27, U28, U29, U30, U31, U32, U33: ~, custom_footprint_library:jumper, symbol custom_symbol_lib:jumper
- added U24: ~, Package_DIP:DIP-14_W7.62mm, symbol custom_symbol_lib:quad_and
- added U25, U26: ~, Package_DIP:DIP-20_W7.62mm, symbol custom_symbol_lib:rising_edge_8_bit_latch
- added U34, U6: ~, Package_DIP:DIP-14_W7.62mm, symbol custom_symbol_lib:6xNOT
Connections:
- net at U14.1 (OE#): now also U34.2 (O0)
- net at U10.1 (OE#), U10.10 (GND), U11.11 (B3)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: now also U17.14 (GND), U2.14 (GND), U18.2 (GND), U19.2 (GND), U20.2 (GND), U21.2 (GND), U22.2 (GND), U23.2 (GND), U24.12 (3B), U24.13 (3A), U24.7 (GND), U25.10 (GND), U26.10 (GND), U27.2 (GND), U28.2 (GND), U29.2 (GND), U30.2 (GND), U31.2 (GND), U32.2 (GND), U33.2 (GND), U34.7 (GND), U6.7 (GND)
- net at U14.11 (CLK): now also U9.1 (OE#), U32.3 (OUT), U34.1 (I0)
- net at U1.14 (D0), U14.2 (D0), U15.2 (D0)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: now also U25.9 (D7), U26.12 (Q7); no longer U17.11 (D0), U2.11 (D0)
- net at U10.20 (V+), U14.20 (V+), U15.20 (V+)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: now also U11.16 (V+), U12.16 (V+), U17.28 (V+), U2.28 (V+), U8.16 (V+), U24.14 (V+), U25.20 (V+), U26.20 (V+), U34.14 (V+), U6.14 (V+); no longer U11.7 (C_IN), U12.9 (C_OUT), U13.20 (V+)
- net at U1.15 (D1), U14.3 (D1), U15.3 (D1)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: now also U25.8 (D6), U26.13 (Q6); no longer U17.12 (D1), U2.12 (D1)
- net at U1.16 (D2), U14.4 (D2), U15.4 (D2)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: now also U25.7 (D5), U26.14 (Q5); no longer U17.13 (D2), U2.13 (D2)
- net at U1.17 (D3), U14.5 (D3), U15.5 (D3)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: now also U25.6 (D4), U26.15 (Q4); no longer U17.15 (D3), U2.15 (D3)
- net at U1.18 (D4), U14.6 (D4), U15.6 (D4)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: now also U25.5 (D3), U26.16 (Q3); no longer U17.16 (D4), U2.16 (D4)
- net at U1.19 (D5), U14.7 (D5), U15.7 (D5)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: now also U25.4 (D2), U26.17 (Q2); no longer U17.17 (D5), U2.17 (D5)
- net at U1.20 (D6), U14.8 (D6), U15.8 (D6)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: now also U25.3 (D1), U26.18 (Q1); no longer U17.18 (D6), U2.18 (D6)
- net at U1.21 (D7), U14.9 (D7), U15.9 (D7)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: now also U25.2 (D0), U26.19 (Q0); no longer U17.19 (D7), U2.19 (D7)
- net at U15.1 (OE#): now also U34.4 (O1)
- net at U15.11 (CLK): now also U13.1 (OE#), U33.3 (OUT), U34.3 (I1)
- net at U16.1 (OE#): now also U34.8 (03)
- net at U10.12 (Q7), U11.12 (A3), U16.9 (D7): now also U2.20 (CE#), U6.1 (I0)
- net at U10.11 (CLK): now also U28.3 (OUT)
- net at U1.1 (READ_0): now also R1.1
- net at U1.13 (GND): now also R1.2, R2.2, R3.2, R4.2, R5.2, R6.2, R7.2, R8.2, R9.1
- net at U1.2 (READ_1): now also R2.1
- net at U1.23 (ENABLE): now also R9.2
- net at U1.3 (READ_2): now also R3.1
- net at U1.4 (READ_3): now also R4.1
- net at U1.5 (WRITE_0): now also R5.1
- net at U1.6 (WRITE_1): now also R6.1
- net at U1.7 (WRITE_2): now also R7.1
- net at U1.8 (WRITE_2): now also R8.1
- net at U5.11 (CLK): now also U27.3 (OUT)
- net at U12.7 (C_IN): now also U8.9 (C_OUT); no longer U12.16 (V+)
- net at U2.22 (OE#): now also U17.22 (OE#), U6.4 (O1)
- net at U2.27 (WE#): now also U17.27 (WE#), U6.6 (O2)
- net at U3.1 (OE#): now also U34.6 (O2)
- net at U13.11 (CLK): now also U9.11 (CLK), U29.3 (OUT)
- net at U17.20 (CE#): now also U6.2 (O0)
- new net: U20.3 (OUT), U26.11 (CLK)
- new net: U25.1 (OE#), U6.10 (O4)
- new net: U24.6 (2Q), U6.11 (I4)
- new net: U24.5 (2B), U24.9 (4B), U6.12 (O5)
- new net: U24.3 (1Q), U6.13 (I5)
- new net: U24.8 (4Q), U6.3 (I1)
- new net: U18.3 (OUT), U6.5 (I2)
- new net: U26.1 (OE#), U6.8 (03)
- new net: U21.3 (OUT), U6.9 (I3)
- new net: U11.7 (C_IN), U12.9 (C_OUT), U13.20 (V+)
- new net: U30.3 (OUT), U34.5 (I2)
- new net: U19.3 (OUT), U24.1 (1A), U24.10 (4A)
- new net: U23.3 (OUT), U24.2 (1B), U24.4 (2A)
- new net: U22.3 (OUT), U25.11 (CLK)
- new net: U17.19 (D7), U2.19 (D7), U25.12 (Q7), U26.9 (D7)
- new net: U17.18 (D6), U2.18 (D6), U25.13 (Q6), U26.8 (D6)
- new net: U17.17 (D5), U2.17 (D5), U25.14 (Q5), U26.7 (D5)
- new net: U17.16 (D4), U2.16 (D4), U25.15 (Q4), U26.6 (D4)
- new net: U17.15 (D3), U2.15 (D3), U25.16 (Q3), U26.5 (D3)
- new net: U17.13 (D2), U2.13 (D2), U25.17 (Q2), U26.4 (D2)
- new net: U17.12 (D1), U2.12 (D1), U25.18 (Q1), U26.3 (D1)
- new net: U17.11 (D0), U2.11 (D0), U25.19 (Q0), U26.2 (D0)
- new net: U31.3 (OUT), U34.9 (I3)
- no-connect marks 1 -> 2
Other:
- note added: "A OE to bus"
- note added: "B OE to bus"
- moved on the sheet: U17, U2

Commit message: Working on GPRAM schematic
Parts:
- added U35, U38, U41, U44: ~, Package_DIP:DIP-14_W7.62mm, symbol custom_symbol_lib:quad_OR
- added U36, U37, U42, U45, U46: ~, Package_DIP:DIP-14_W7.62mm, symbol custom_symbol_lib:quad_and
- added U39, U40: ~, Package_DIP:DIP-20_W7.62mm, symbol custom_symbol_lib:rising_edge_8_bit_latch
- added U43: ~, custom_footprint_library:jumper, symbol custom_symbol_lib:jumper
- added U47: ~, Package_DIP:DIP-14_W7.62mm, symbol custom_symbol_lib:6xNOT
Connections:
- net at U10.1 (OE#), U10.10 (GND), U11.11 (B3)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: now also R1.2, R2.2, R3.2, R4.2, R5.2, R6.2, R7.2, R8.2, R9.1, U1.13 (GND), U4.10 (1RESET), U4.4 (0RESET), U4.6 (0SET), U4.7 (GND), U4.8 (1SET), U35.7 (GND), U36.7 (GND), U37.7 (GND), U38.12 (3A), U38.13 (3B), U38.5 (1A), U38.6 (1B), U38.7 (GND), U38.8 (2A), U38.9 (2B), U39.1 (OE#), U39.10 (GND), U40.1 (OE#), U40.10 (GND), U41.7 (GND), U42.7 (GND), U43.2 (GND), U44.7 (GND), U45.7 (GND), U46.12 (3B), U46.13 (3A), U46.7 (GND), U47.1 (I0), U47.3 (I1), U47.5 (I2), U47.7 (GND), U47.9 (I3)
- net at U10.20 (V+), U11.16 (V+), U12.16 (V+)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: now also U1.12 (V+), U13.20 (V+), U4.14 (V+), U35.14 (V+), U36.14 (V+), U37.14 (V+), U38.14 (V+), U39.20 (V+), U40.20 (V+), U41.14 (V+), U42.14 (V+), U44.14 (V+), U45.14 (V+), U46.14 (V+), U47.14 (V+)
- net at R9.2, U1.23 (ENABLE): now also U37.10 (4A), U37.13 (3A)
- net at U27.1 (IN): now also U35.3 (Q0)
- net at U4.1 (0Q): now also U37.2 (1B)
- net at U4.11 (1CLK): now also U44.11 (Q3)
- net at U4.12 (1Q3): now also U36.1 (1A), U45.1 (1A)
- net at U4.13 (1Q): now also U36.4 (2A), U45.4 (2A)
- net at U4.3 (0CLK): now also U46.8 (4Q)
- net at U4.5 (0D): now also U44.3 (Q0)
- net at U4.9 (1D): now also U44.10 (Q2)
- net at U20.1 (IN): now also U21.1 (IN), U37.8 (4Q)
- net at U24.3 (1Q), U6.13 (I5): now also U1.22 (FAULT)
- net at R8.1, U1.8 (WRITE_2): now also U41.1 (0A), U44.9 (2B)
- net at U32.1 (IN): now also U36.12 (3B), U45.3 (1Q)
- net at R7.1, U1.7 (WRITE_2): now also U41.2 (0B)
- net at R1.1, U1.1 (READ_0): now also U41.13 (3B)
- net at U1.10 (CLK_A): now also U39.11 (CLK), U46.10 (4A), U47.11 (I4)
- net at U1.11 (CLK_B): now also U37.5 (2B), U40.11 (CLK), U47.13 (I5)
- net at R2.1, U1.2 (READ_1): now also U41.12 (3A), U44.1 (0A)
- net at R3.1, U1.3 (READ_2): now also U41.9 (2B)
- net at R4.1, U1.4 (READ_3): now also U41.8 (2A), U44.8 (2A)
- net at R5.1, U1.5 (WRITE_0): now also U41.6 (1B)
- net at R6.1, U1.6 (WRITE_1): now also U41.5 (1A), U44.2 (0B)
- net at U1.9 (READ_READY): now also U43.3 (OUT)
- net at U28.1 (IN): now also U35.4 (Q1)
- net at U11.7 (C_IN), U12.9 (C_OUT): no longer U13.20 (V+)
- net at U33.1 (IN): now also U36.9 (4B), U45.6 (2Q)
- net at U18.1 (IN): now also U37.6 (2Q)
- net at U30.1 (IN): now also U36.3 (1Q)
- net at U29.1 (IN): now also U35.10 (Q2)
- net at U23.1 (IN): now also U22.1 (IN), U37.4 (2A), U39.18 (Q1), U40.5 (D3)
- net at U19.1 (IN): now also U41.4 (Q1), U42.1 (1A)
- net at U34.10 (O4): now also U42.5 (2B)
- net at U34.11 (I4): now also U37.12 (3B), U40.17 (Q2)
- net at U34.12 (O5): now also U42.2 (1B)
- net at U34.13 (I5): now also U35.12 (3A), U37.9 (4B), U39.2 (D0), U40.19 (Q0)
- net at U31.1 (IN): now also U36.6 (2Q)
- new net: U40.2 (D0), U42.3 (1Q)
- new net: U41.3 (Q0), U42.4 (2A), U46.2 (1B)
- new net: U40.4 (D2), U42.6 (2Q)
- new net: U44.12 (3A), U46.3 (1Q)
- new net: U44.13 (3B), U46.6 (2Q)
- new net: U44.4 (Q1), U46.9 (4B)
- new net: U35.11 (Q3), U43.1 (IN), U44.5 (1A)
- new net: U39.3 (D1), U41.11 (Q3), U44.6 (1B)
- new net: U46.1 (1A), U47.10 (O4)
- new net: U46.4 (2A), U47.12 (O5)
- new net: U39.5 (D3), U41.10 (Q2), U46.5 (2B)
- new net: U39.16 (Q3), U40.6 (D4), U45.2 (1B), U45.5 (2B)
- new net: U38.2 (0B), U39.17 (Q2)
- new net: U35.8 (2A), U39.19 (Q0), U40.3 (D1)
- new net: U35.9 (2B), U39.4 (D2), U40.16 (Q3)
- new net: U35.1 (0A), U36.11 (3Q)
- new net: U35.13 (3B), U36.2 (1B), U36.5 (2B), U37.11 (3Q)
- new net: U35.2 (0B), U35.6 (1B), U37.3 (1Q)
- new net: U35.5 (1A), U36.8 (4Q)
- new net: U37.1 (1A), U38.3 (Q0)
- new net: U36.10 (4A), U36.13 (3A), U40.15 (Q4)
- new net: U38.1 (0A), U40.18 (Q1)
- no-connect marks 2 -> 6
Other:
- note added: "++addr enable"
- note added: "<- Enable <-"
- note added: "A(0)/B(1) select"
- note added: "GPRAM-ADDR-B GPRAM-ADDR-A GPRAM-INC-ADDR GPRAM"
- note added: "Read ready"
- note added: "Write addr Write Read addr Read"
- moved on the sheet: R1, R2, R3, R4, R5, R6, R7, R8, R9, U1, U27, U28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

Commit message: Verified GPRAM schematic
Parts:
- removed U45: ~, Package_DIP:DIP-14_W7.62mm, symbol custom_symbol_lib:quad_and
Connections:
- net at R1.2, R2.2, R3.2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: now also U39.6 (D4), U39.7 (D5), U39.8 (D6), U39.9 (D7), U40.7 (D5), U40.8 (D6), U40.9 (D7)
- net at U42.10 (4A): now also U36.4 (2A), U4.13 (1Q)
- net at U42.11 (3Q): now also U32.1 (IN), U36.12 (3B)
- net at U42.12 (3B): now also U39.16 (Q3), U40.6 (D4), U42.9 (4B)
- net at U42.13 (3A): now also U36.1 (1A), U4.12 (1Q3)
- net at U42.8 (4Q): now also U33.1 (IN), U36.9 (4B)
- no-connect marks 6 -> 18

Commit message: Finished GPRAM PCB
Changed lines of the file:
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@@
 	(wire
 		(pts
-			(xy 363.22 76.2) (xy 302.26 76.2)
+			(xy 302.26 76.2) (xy 374.65 76.2)
 		)
 		(stroke
@@
 	(wire
 		(pts
-			(xy 374.65 92.71) (xy 363.22 92.71)
-		)
-		(stroke
-			(width 0)
-			(type default)
-		)
-	)
-	(wire
-		(pts
 			(xy 351.79 100.33) (xy 369.57 100.33)
 		)
@@
 	(wire
 		(pts
+			(xy 374.65 76.2) (xy 374.65 106.68)
+		)
+		(stroke
+			(width 0)
+			(type default)
+		)
+	)
+	(wire
+		(pts
 			(xy 440.69 55.88) (xy 405.13 55.88)
 		)
@@
 	(wire
 		(pts
-			(xy 374.65 106.68) (xy 374.65 92.71)
-		)
-		(stroke
-			(width 0)
-			(type default)
-		)
-	)
-	(wire
-		(pts
 			(xy 223.52 142.24) (xy 153.67 142.24)
 		)
@@
 		)
 		(stroke
-			(width 0)
-			(type default)
-		)
-	)
-	(wire
-		(pts
-			(xy 363.22 92.71) (xy 363.22 76.2)
-		)
-		(stroke
