File: kicad/call_stack/call_stack.kicad_pcb (KiCad board)
At the start: 2 copper layers, 100 x 100 mm, 27 parts

Commit message: Finished some more PCBs and uploaded to JLCPCB
Parts:
- U6, U7: moved to F.Cu
- moved U25 230.8 mm to (275.1, 129.7), turned to -90 degrees
- moved U21 214.7 mm to (176.9, 138.8), turned to 90 degrees
- moved U24 199.9 mm to (202.9, 122.4)
- moved U27 197.8 mm to (144.2, 124.4)
- moved U26 194.6 mm to (159.2, 124.4)
- moved U22 194.3 mm to (191.6, 116.7), turned to -90 degrees
- moved U5 191.2 mm to (221.0, 62.6), turned to 90 degrees
- moved U4 181.0 mm to (221.5, 132.6), turned to 90 degrees
- moved U3 162.3 mm to (177.8, 103.5), turned to 90 degrees
- moved U12 117.8 mm to (160.1, 51.7)
- moved U14 117.8 mm to (160.1, 67.0)
- moved U15 117.8 mm to (160.1, 74.7)
- moved U19 117.8 mm to (160.1, 105.5)
- moved U20 117.8 mm to (160.1, 113.2)
- moved U13 117.8 mm to (160.1, 59.3)
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Routing:
- net Net-(U1-GND): track 0.00 -> 667.3 mm, vias 0 -> 1
- net Net-(U1-V+): track 0.00 -> 425.2 mm, vias 0 -> 3
- net Net-(U1-Pop): track 0.00 -> 234.6 mm, vias 0 -> 1
- net Net-(U11-Q2): track 0.00 -> 213.4 mm
- net Net-(U11-Q0): track 0.00 -> 208.3 mm, vias 0 -> 2
- net Net-(U11-Q1): track 0.00 -> 206.5 mm, vias 0 -> 3
- net Net-(U11-Q3): track 0.00 -> 197.9 mm
- net Net-(U1-Push): track 0.00 -> 197.2 mm
- net Net-(U11-Q4): track 0.00 -> 184.0 mm
- net Net-(U11-Q5): track 0.00 -> 165.3 mm, vias 0 -> 2
- net Net-(U1-B_CLK): track 0.00 -> 160.2 mm, vias 0 -> 1
- net Net-(U1-OE): track 0.00 -> 159.8 mm
- net Net-(U11-Q6): track 0.00 -> 154.2 mm
- net Net-(U1-A_CLK): track 0.00 -> 151.5 mm, vias 0 -> 2
- net Net-(U21-O5): track 0.00 -> 150.2 mm, vias 0 -> 2
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- added copper zone on B.Cu, net Net-(U1-GND)
- added copper zone on F.Cu, net Net-(U1-V+)
Other:
- board size 100 x 100 mm -> 140.5 x 100 mm
- board text added: "CALL STACK MEMORY"
