File: kicad/startup_controller/startup_controller.kicad_pcb (KiCad board)
At the start: 2 copper layers, 73.7 x 43.8 mm, 16 parts

Commit message: Finished some more PCBs and uploaded to JLCPCB
Parts:
- moved D3 7.41 mm to (133.0, 109.0), turned to 90 degrees
- moved D5 6.00 mm to (133.1, 81.6)
- moved D4 2.02 mm to (133.3, 96.0), turned to 90 degrees
Routing:
- net Net-(D1-K): track 165.6 -> 175.8 mm
- net Net-(D5-A): track 129.4 -> 133.1 mm
- net Net-(D4-A): track 42.4 -> 39.3 mm
- net Net-(D3-A): track 32.7 -> 35.0 mm, vias 0 -> 1
Other:
- board text added: "ENABLE"
- board text added: "POWER"
- board text added: "R"
- board text added: "S"
- board text added: "START"
