File: kicad/version_1/stack_controller/stack_controller.kicad_sch (KiCad schematic)
At the start: 53 parts

Commit message: Lots of stuff
Connections:
- no-connect marks 16 -> 21
Changed lines of the file:
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@@
 	)
 	(no_connect
+		(at 166.37 313.69)
+	)
+	(no_connect
 		(at 167.64 279.4)
 	)
@@
 	)
 	(no_connect
+		(at 163.83 314.96)
+	)
+	(no_connect
 		(at 287.02 326.39)
 	)
@@
 	)
 	(no_connect
+		(at 171.45 294.64)
+	)
+	(no_connect
 		(at 269.24 257.81)
 	)
@@
 	)
 	(no_connect
+		(at 247.65 264.16)
+	)
+	(no_connect
 		(at 88.9 247.65)
 	)
@@
 		(at 245.11 316.23)
 	)
+	(no_connect
+		(at 227.33 298.45)
+	)
 	(wire
 		(pts
@@
 		)
 	)
+	(polyline
+		(pts
+			(xy 170.18 292.1) (xy 171.45 292.1)
+		)
+		(stroke
+			(width 0)
+			(type default)
+		)
+	)
 	(wire
 		(pts
@@
 		)
 	)
+	(polyline
+		(pts
+			(xy 170.18 300.99) (xy 170.18 292.1)
+		)
+		(stroke
+			(width 0)
+			(type default)
+		)
+	)
 	(wire
 		(pts
@@
 		)
 	)
+	(polyline
+		(pts
+			(xy 228.6 290.83) (xy 228.6 298.45)
+		)
+		(stroke
+			(width 0)
+			(type default)
+		)
+	)
 	(wire
 		(pts
@@
 		)
 	)
+	(polyline
+		(pts
+			(xy 161.29 314.96) (xy 161.29 316.23)
+		)
+		(stroke
+			(width 0)
+			(type default)
+		)
+	)
 	(wire
 		(pts
@@
 		)
 	)
+	(polyline
+		(pts
+			(xy 228.6 262.89) (xy 228.6 290.83)
+		)
+		(stroke
+			(width 0)
+			(type default)
+		)
+	)
 	(wire
 		(pts
@@
 		)
 	)
+	(polyline
+		(pts
+			(xy 166.37 316.23) (xy 161.29 316.23)
+		)
+		(stroke
+			(width 0)
+			(type default)
+		)
+	)
 	(wire
 		(pts
@@
 		)
 		(stroke
+			(width 0)
+			(type default)
+		)
+	)
+	(polyline
+		(pts
+			(xy 247.65 262.89) (xy 228.6 262.89)
+		)
+		(stroke
