File: kicad/version_2/stack_controller/stack_controller.kicad_sch (KiCad schematic)
At the start: 53 parts

Commit message: Lots of stuff
Connections:
- net at U24.1 (1A): now also U26.18 (Q1); no longer U28.11 (3Q)
- net at U24.10 (4A): no longer U9.14 (Q5)
- net at U24.12 (3B), U24.4 (2A), U28.5 (2B)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: no longer U24.9 (4B)
- net at U24.5 (2B): now also U26.5 (D3), U9.17 (Q2); no longer U9.16 (Q3)
- net at U24.8 (4Q): no longer U27.8 (2A)
- net at R6.1, U47.2 (1B): now also U5.23 (ENABLE)
- net at U26.19 (Q0), U31.1 (I0), U47.1 (1A)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: now also U27.13 (3B), U43.1 (IN); no longer U28.10 (4A)
- net at U26.11 (CLK), U28.13 (3A), U5.11 (CLK_B): no longer U28.9 (4B)
- net at U26.13 (Q6): no longer U27.6 (1B)
- net at U26.14 (Q5): now also U27.6 (1B); no longer U9.9 (D7)
- net at U26.15 (Q4): now also U27.8 (2A); no longer U9.7 (D5)
- net at U26.17 (Q2), U9.4 (D2): now also U42.1 (IN)
- net at U28.12 (3B): no longer U26.18 (Q1)
- net at U26.8 (D6): no longer U9.12 (Q7)
- now unconnected: U26.16 (Q3), U28.8 (4Q), U9.5 (D3)
Other:
- note added: "<- This AND gate no longer used"
- note added: "A-B"
- note added: "Main write sequence (B-A-B) AND POP"
- note added: "Mem write"
- note added: "OFF-READ | POP"
- note added: "Offset write offset address select sequence 2(B)"
- note added: "PUSH | OFF-WRITE 1(A)"
- note added: "Push address CLK 1(A)"
- note added: "Push address CLK 2(B)"
- note added: "Push or offset write to be ANDed w/ A CLK"
