File: kicad/version_2/prog_mem/prog_mem.kicad_sch (KiCad schematic)
At the start: 37 parts

Commit message: Fixed prog mem and updated PCB
Parts:
- removed U5: ~, Package_DIP:DIP-20_W7.62mm, symbol custom_symbol_lib:8_bit_transparent_latch
- added U16: ~, Package_DIP:DIP-20_W7.62mm, symbol custom_symbol_lib:8_bit_transparent_latch
- added U21, U5: ~, Package_DIP:DIP-20_W7.62mm, symbol custom_symbol_lib:rising_edge_8_bit_latch
Connections:
- net at R1.1, R10.1, R2.1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: now also U16.10 (GND), U21.10 (GND), U5.10 (GND); no longer U12.9 (I3)
- net at U15.3 (OUT), U25.1 (IN), U6.5 (2B): now also U12.9 (I3)
- net at D1.1 (K), R8.1, U1.32 (V+)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: now also U16.11 (CLK), U16.20 (V+), U21.20 (V+), U5.20 (V+)
- net at U1.12 (A0), U11.19 (Q0), U19.1 (0)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: now also U8.19 (Q0)
- net at U1.26 (A9), U10.18 (Q1), U19.10 (9)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: now also U16.18 (Q1); no longer U8.18 (Q1)
- net at U1.23 (A10), U10.17 (Q2), U19.11 (10)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: now also U16.17 (Q2); no longer U8.17 (Q2)
- net at U1.25 (A11), U10.16 (Q3), U19.12 (11)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: now also U16.16 (Q3); no longer U8.16 (Q3)
- net at U1.4 (A12), U10.15 (Q4), U19.13 (12)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: now also U16.15 (Q4); no longer U8.15 (Q4)
- net at U1.28 (A13), U10.14 (Q5), U19.14 (13)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: now also U16.14 (Q5); no longer U8.14 (Q5)
- net at U1.29 (A14), U10.13 (Q6), U19.15 (14)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: now also U16.13 (Q6); no longer U8.13 (Q6)
- net at U1.3 (A15), U10.12 (Q7), U19.16 (15)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: now also U16.12 (Q7); no longer U8.12 (Q7)
- net at U1.11 (A1), U11.18 (Q1), U19.2 (1)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: now also U8.18 (Q1)
- net at U1.10 (A2), U11.17 (Q2), U19.3 (2)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: now also U8.17 (Q2)
- net at U1.9 (A3), U11.16 (Q3), U19.4 (3)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: now also U8.16 (Q3)
- net at U1.8 (A4), U11.15 (Q4), U19.5 (4)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: now also U8.15 (Q4)
- net at U1.7 (A5), U11.14 (Q5), U19.6 (5)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: now also U8.14 (Q5)
- net at U1.6 (A6), U11.13 (Q6), U19.7 (6)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: now also U8.13 (Q6)
- net at U1.5 (A7), U11.12 (Q7), U19.8 (7)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: now also U8.12 (Q7)
- net at U1.27 (A8), U10.19 (Q0), U19.9 (8)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: now also U16.19 (Q0); no longer U8.19 (Q0)
- net at U1.24 (OE#), U12.4 (O1), U7.24 (OE#)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: now also U16.1 (OE#)
- net at U12.8 (03): now also U21.1 (OE#), U5.1 (OE#)
- net at U1.13 (DQ0), U14.19 (Q0): now also U21.2 (D0); no longer U2.32 (D8)
- net at U1.14 (DQ1), U14.18 (Q1): now also U21.3 (D1); no longer U2.33 (D9)
- net at U1.15 (DQ2), U14.17 (Q2): now also U21.4 (D2); no longer U2.34 (D10)
- net at U1.17 (DQ3), U14.16 (Q3): now also U21.5 (D3); no longer U2.35 (D11)
- net at U1.18 (DQ4), U14.15 (Q4): now also U21.6 (D4); no longer U2.36 (D12)
- net at U1.19 (DQ5), U14.14 (Q5): now also U21.7 (D5); no longer U2.37 (D13)
- net at U1.20 (DQ6), U14.13 (Q6): now also U21.8 (D6); no longer U2.38 (D14)
- net at U1.21 (DQ7), U14.12 (Q7): now also U21.9 (D7); no longer U2.39 (D15)
- net at U2.10 (A2): now also U8.4 (D2)
- net at U2.11 (A3): now also U8.5 (D3)
- net at U2.12 (A4): now also U8.6 (D4)
- net at U2.13 (A5): now also U8.7 (D5)
- net at U2.14 (A6): now also U8.8 (D6)
- net at U2.15 (A7): now also U8.9 (D7)
- net at U8.2 (D0): now also U2.8 (A0); no longer U2.16 (A8)
- net at U8.3 (D1): now also U2.9 (A1); no longer U2.17 (A9)
- net at U2.18 (A10): now also U16.4 (D2); no longer U8.4 (D2)
- net at U2.19 (A11): now also U16.5 (D3); no longer U8.5 (D3)
- net at U2.20 (A12): now also U16.6 (D4); no longer U8.6 (D4)
- net at U2.21 (A13): now also U16.7 (D5); no longer U8.7 (D5)
- net at U2.22 (A14): now also U16.8 (D6); no longer U8.8 (D6)
- net at U2.23 (A15): now also U16.9 (D7); no longer U8.9 (D7)
- net at U13.19 (Q0), U7.13 (DQ0): now also U5.2 (D0); no longer U2.24 (D0)
- net at U13.18 (Q1), U7.14 (DQ1): now also U5.3 (D1); no longer U2.25 (D1)
- net at U13.17 (Q2), U7.15 (DQ2): now also U5.4 (D2); no longer U2.26 (D2)
- net at U13.16 (Q3), U7.17 (DQ3): now also U5.5 (D3); no longer U2.27 (D3)
- net at U13.15 (Q4), U7.18 (DQ4): now also U5.6 (D4); no longer U2.28 (D4)
- net at U13.14 (Q5), U7.19 (DQ5): now also U5.7 (D5); no longer U2.29 (D5)
- net at U13.13 (Q6), U7.20 (DQ6): now also U5.8 (D6); no longer U2.30 (D6)
- net at U13.12 (Q7), U7.21 (DQ7): now also U5.9 (D7); no longer U2.31 (D7)
- net at U2.6 (Done), U6.6 (2Q): now also U21.11 (CLK), U5.11 (CLK)
- new net: U2.39 (D15), U21.12 (Q7)
- new net: U2.38 (D14), U21.13 (Q6)
- new net: U2.37 (D13), U21.14 (Q5)
- new net: U2.36 (D12), U21.15 (Q4)
- new net: U2.35 (D11), U21.16 (Q3)
- new net: U2.34 (D10), U21.17 (Q2)
- new net: U2.33 (D9), U21.18 (Q1)
- new net: U2.32 (D8), U21.19 (Q0)
- new net: U16.2 (D0), U2.16 (A8)
- new net: U16.3 (D1), U2.17 (A9)
- new net: U2.24 (D0), U5.19 (Q0)
- new net: U2.25 (D1), U5.18 (Q1)
- new net: U2.26 (D2), U5.17 (Q2)
- new net: U2.27 (D3), U5.16 (Q3)
- new net: U2.28 (D4), U5.15 (Q4)
- new net: U2.29 (D5), U5.14 (Q5)
- new net: U2.30 (D6), U5.13 (Q6)
- new net: U2.31 (D7), U5.12 (Q7)
- no-connect marks 8 -> 7
Other:
- moved on the sheet: D1, R1, R10, R2, R3, R4, R5, R6, R7, R8, R9, U1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
