File: kicad/version_2/led_matrix/led_matrix.kicad_sch (KiCad schematic)
At the start: 1302 parts

Commit message: Led matrix progress
Parts:
- removed D1, D10, D100, D1000, D1001, D1002, D1003, D1004, D1005, D1006, D1007, D1008, D1009, D101, D1010, D1011, D1012, D1013, D1014, D1015, D1016, D1017, D1018, D1019, D102, D1020, D1021, D1022, D1023, D1024, D1025, D1026, D1027, D1028, D1029, D103, D1030, D1031, D1032, D1033, D1034, D1035, D1036, D1037, D1038, D1039, D104, D1040, D1041, D1042, D1043, D1044, D1045, D1046, D1047, D1048, D1049, D105, D1050, D1051, D1052, D1053, D1054, D1055, D1056, D1057, D1058, D1059, D106, D1060, D1061, D1062, D1063, D1064, D1065, D1066, D1067, D1068, D1069, D107, D1070, D1071, D1072, D1073, D1074, D1075, D1076, D1077, D1078, D1079, D108, D1080, D1081, D1082, D1083, D1084, D1085, D1086, D1087, D1088, D1089, D109, D1090, D1091, D1092, D1093, D1094, D1095, D1096, D1097, D1098, D1099, D11, D110, D1100, D1101, D1102, D1103, D1104, D1105, D1106, D1107, D1108, D1109, D111, D1110, D1111, D1112, D1113, D1114, D1115, D1116, D1117, D1118, D1119, D112, D1120, D1121, D1122, D1123, D1124, D1125, D1126, D1127, D1128, D1129, D113, D1130, D1131, D1132, D1133, D1134, D1135, D1136, D1137, D1138, D1139, D114, D1140, D1141, D1142, D1143, D1144, D1145, D1146, D1147, D1148, D1149, D115, D1150, D1151, D1152, D1153, D1154, D1155, D1156, D1157, D1158, D1159, D116, D1160, D1161, D1162, D1163, D1164, D1165, D1166, D1167, D1168, D1169, D117, D1170, D1171, D1172, D1173, D1174, D1175, D1176, D1177, D1178, D1179, D118, D1180, D1181, D1182, D1183, D1184, D1185, D1186, D1187, D1188, D1189, D119, D1190, D1191, D1192, D1193, D1194, D1195, D1196, D1197, D1198, D1199, D12, D120, D1200, D1201, D1202, D1203, D1204, D1205, D1206, D1207, D1208, D1209, D121, D1210, D1211, D1212, D1213, D1214, D1215, D1216, D1217, D1218, D1219, D122, D1220, D1221, D1222, D1223, D1224, D1225, D1226, D1227, D1228, D1229, D123, D1230, D1231, D1232, D1233, D1234, D1235, D1236, D1237, D1238, D1239, D124, D1240, D1241, D1242, D1243, D1244, D1245, D1246, D1247, D1248, D1249, D125, D1250, D1251, D1252, D1253, D1254, D1255, D1256, D1257, D1258, D1259, D126, D1260, D1261, D1262, D1263, D1264, D1265, D1266, D1267, D1268, D1269, D127, D1270, D1271, D1272, D1273, D1274, D1275, D1276, D1277, D1278, D1279, D128, D1280, D129, D13, D130, D131, D132, D133, D134, D135, D136, D137, D138, D139, D14, D140, D141, D142, D143, D144, D145, D146, D147, D148, D149, D15, D150, D151, D152, D153, D154, D155, D156, D157, D158, D159, D16, D160, D161, D162, D163, D164, D165, D166, D167, D168, D169, D17, D170, D171, D172, D173, D174, D175, D176, D177, D178, D179, D18, D180, D181, D182, D183, D184, D185, D186, D187, D188, D189, D19, D190, D191, D192, D193, D194, D195, D196, D197, D198, D199, D2, D20, D200, D201, D202, D203, D204, D205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: LED, LED_THT:LED_D3.0mm, symbol Device:LED
- removed U11, U5, U7, U9: ~, Package_DIP:DIP-24_W7.62mm, symbol custom_symbol_lib:led_sink_16_bit
- added R10, R11, R12, R13, R5, R6, R8, R9: R, symbol Device:R
- added U11, U20, U21, U22, U23, U5, U7, U9: ~, custom_footprint_library:led_block_16_x_8, symbol custom_symbol_lib:led_block_16_x_8
- added U18, U19: ~, Package_DIP:DIP-24_W7.62mm, symbol custom_symbol_lib:led_sink_16_bit
Connections:
- net at U8.7 (O2): now also U9.3 (C2)
- net at U13.6 (O1): now also U21.2 (C1)
- net at U8.18 (O13): now also U9.14 (C13)
- net at U12.17 (O12): now also U20.13 (C12)
- net at U6.7 (O2): now also U7.3 (C2)
- net at U8.8 (O3): now also U9.4 (C3)
- net at U12.9 (O4): now also U20.5 (C4)
- net at U12.18 (O13): now also U20.14 (C13)
- net at U6.16 (O11): now also U7.12 (C11)
- net at U8.9 (O4): now also U9.5 (C4)
- net at U6.19 (O14): now also U7.15 (C14)
- net at U10.14 (O9): now also U11.10 (C9)
- net at U4.5 (O0): now also U5.1 (C0)
- net at U8.16 (O11): now also U9.12 (C11)
- net at U4.8 (O3): now also U5.4 (C3)
- net at U6.6 (O1): now also U7.2 (C1)
- net at U6.17 (O12): now also U7.13 (C12)
- net at U10.11 (O6): now also U11.7 (C6)
- net at U10.15 (O10): now also U11.11 (C10)
- net at U6.18 (O13): now also U7.14 (C13)
- net at U10.6 (O1): now also U11.2 (C1)
- net at U12.16 (O11): now also U20.12 (C11)
- net at U12.20 (O15): now also U20.16 (C15)
- net at U8.11 (O6): now also U9.7 (C6)
- net at U10.16 (O11): now also U11.12 (C11)
- net at U13.16 (O11): now also U21.12 (C11)
- net at U8.20 (O15): now also U9.16 (C15)
- net at U13.8 (O3): now also U21.4 (C3)
- net at U13.17 (O12): now also U21.13 (C12)
- net at U10.12 (O7): now also U11.8 (C7)
- net at U4.17 (O12): now also U5.13 (C12)
- net at U8.6 (O1): now also U9.2 (C1)
- net at U12.6 (O1): now also U20.2 (C1)
- net at U4.16 (O11): now also U5.12 (C11)
- net at U12.13 (O8): now also U20.9 (C8)
- net at U6.15 (O10): now also U7.11 (C10)
- net at U4.20 (O15): now also U5.16 (C15)
- net at U6.20 (O15): now also U7.16 (C15)
- net at U4.6 (O1): now also U5.2 (C1)
- net at U8.13 (O8): now also U9.9 (C8)
- net at U4.15 (O10): now also U5.11 (C10)
- net at U12.19 (O14): now also U20.15 (C14)
- net at U12.8 (O3): now also U20.4 (C3)
- net at U8.5 (O0): now also U9.1 (C0)
- net at U13.19 (O14): now also U21.15 (C14)
- net at U13.9 (O4): now also U21.5 (C4)
- net at U4.10 (O5): now also U5.6 (C5)
- net at U10.20 (O15): now also U11.16 (C15)
- net at U13.15 (O10): now also U21.11 (C10)
- net at U13.12 (O7): now also U21.8 (C7)
- net at U6.9 (O4): now also U7.5 (C4)
- net at U4.11 (O6): now also U5.7 (C6)
- net at U10.8 (O3): now also U11.4 (C3)
- net at U10.10 (O5): now also U11.6 (C5)
- net at U4.19 (O14): now also U5.15 (C14)
- net at U10.18 (O13): now also U11.14 (C13)
- net at U13.18 (O13): now also U21.14 (C13)
- net at U4.13 (O8): now also U5.9 (C8)
- net at U13.11 (O6): now also U21.7 (C6)
- net at U8.12 (O7): now also U9.8 (C7)
- net at U12.7 (O2): now also U20.3 (C2)
- net at U12.5 (O0): now also U20.1 (C0)
- net at U13.7 (O2): now also U21.3 (C2)
- net at U10.7 (O2): now also U11.3 (C2)
- net at U13.5 (O0): now also U21.1 (C0)
- net at U8.15 (O10): now also U9.11 (C10)
- net at U13.10 (O5): now also U21.6 (C5)
- net at U13.20 (O15): now also U21.16 (C15)
- net at U13.13 (O8): now also U21.9 (C8)
- net at U8.17 (O12): now also U9.13 (C12)
- net at U6.13 (O8): now also U7.9 (C8)
- net at U4.9 (O4): now also U5.5 (C4)
- net at U10.19 (O14): now also U11.15 (C14)
- net at U4.12 (O7): now also U5.8 (C7)
- net at U6.5 (O0): now also U7.1 (C0)
- net at U12.11 (O6): now also U20.7 (C6)
- net at U4.7 (O2): now also U5.3 (C2)
- net at U4.18 (O13): now also U5.14 (C13)
- net at U12.15 (O10): now also U20.11 (C10)
- net at U8.14 (O9): now also U9.10 (C9)
- net at U6.12 (O7): now also U7.8 (C7)
- net at U10.13 (O8): now also U11.9 (C8)
- net at U10.9 (O4): now also U11.5 (C4)
- net at U12.14 (O9): now also U20.10 (C9)
- net at U10.17 (O12): now also U11.13 (C12)
- net at U4.14 (O9): now also U5.10 (C9)
- net at U12.10 (O5): now also U20.6 (C5)
- net at U10.5 (O0): now also U11.1 (C0)
- net at U8.1 (GND): now also U10.1 (GND), U10.21 (OE#), U12.1 (GND), U12.21 (OE#), U13.1 (GND), U13.21 (OE#), U4.1 (GND), U4.21 (OE#), U6.1 (GND), U6.21 (OE#), U8.21 (OE#), R10.2, R11.2, R12.2, R13.2, R5.2, R6.2, R8.2, R9.2, U18.1 (GND), U18.21 (OE#), U19.1 (GND), U19.21 (OE#)
- net at U8.10 (O5): now also U9.6 (C5)
- net at U8.19 (O14): now also U9.15 (C14)
- net at U8.2 (D_in): now also U10.2 (D_in), U12.2 (D_in), U13.2 (D_in), U4.2 (D_in), U6.2 (D_in), U18.2 (D_in), U19.2 (D_in)
- net at U8.23 (SET): now also R8.1
- net at U8.24 (V+): now also U10.24 (V+), U12.24 (V+), U13.24 (V+), U4.24 (V+), U6.24 (V+), U18.24 (V+), U19.24 (V+)
- net at U8.3 (CLK): now also U10.3 (CLK), U12.3 (CLK), U13.3 (CLK), U4.3 (CLK), U6.3 (CLK), U18.3 (CLK), U19.3 (CLK)
- net at U6.14 (O9): now also U7.10 (C9)
- net at U13.14 (O9): now also U21.10 (C9)
- net at U6.8 (O3): now also U7.4 (C3)
- net at U6.11 (O6): now also U7.7 (C6)
- net at U12.12 (O7): now also U20.8 (C7)
- net at U13.23 (SET): now also R11.1
- net at U6.10 (O5): now also U7.6 (C5)
- net at U6.23 (SET): now also R6.1
- net at U12.23 (SET): now also R10.1
- net at U4.23 (SET): now also R5.1
- net at U10.23 (SET): now also R9.1
- new net: U11.17 (R0), U20.17 (R0), U21.17 (R0), U22.17 (R0), U23.17 (R0), U5.17 (R0), U7.17 (R0), U9.17 (R0)
- new net: U11.18 (R1), U20.18 (R1), U21.18 (R1), U22.18 (R1), U23.18 (R1), U5.18 (R1), U7.18 (R1), U9.18 (R1)
- new net: U11.19 (R2), U20.19 (R2), U21.19 (R2), U22.19 (R2), U23.19 (R2), U5.19 (R2), U7.19 (R2), U9.19 (R2)
- new net: U11.20 (R3), U20.20 (R3), U21.20 (R3), U22.20 (R3), U23.20 (R3), U5.20 (R3), U7.20 (R3), U9.20 (R3)
- new net: U11.21 (R4), U20.21 (R4), U21.21 (R4), U22.21 (R4), U23.21 (R4), U5.21 (R4), U7.21 (R4), U9.21 (R4)
- new net: U11.22 (R5), U20.22 (R5), U21.22 (R5), U22.22 (R5), U23.22 (R5), U5.22 (R5), U7.22 (R5), U9.22 (R5)
- new net: U11.23 (R6), U20.23 (R6), U21.23 (R6), U22.23 (R6), U23.23 (R6), U5.23 (R6), U7.23 (R6), U9.23 (R6)
- new net: U11.24 (R7), U20.24 (R7), U21.24 (R7), U22.24 (R7), U23.24 (R7), U5.24 (R7), U7.24 (R7), U9.24 (R7)
- new net: U18.5 (O0), U22.1 (C0)
- new net: U18.14 (O9), U22.10 (C9)
- new net: U18.15 (O10), U22.11 (C10)
- new net: U18.16 (O11), U22.12 (C11)
- new net: U18.17 (O12), U22.13 (C12)
- new net: U18.18 (O13), U22.14 (C13)
- new net: U18.19 (O14), U22.15 (C14)
- new net: U18.20 (O15), U22.16 (C15)
- new net: U18.6 (O1), U22.2 (C1)
- new net: U18.7 (O2), U22.3 (C2)
- new net: U18.8 (O3), U22.4 (C3)
- new net: U18.9 (O4), U22.5 (C4)
- new net: U18.10 (O5), U22.6 (C5)
- new net: U18.11 (O6), U22.7 (C6)
- new net: U18.12 (O7), U22.8 (C7)
- new net: U18.13 (O8), U22.9 (C8)
- new net: R12.1, U18.23 (SET)
- new net: R13.1, U19.23 (SET)
- new net: U19.10 (O5), U23.6 (C5)
- new net: U19.11 (O6), U23.7 (C6)
- new net: U19.12 (O7), U23.8 (C7)
- new net: U19.13 (O8), U23.9 (C8)
- new net: U19.14 (O9), U23.10 (C9)
- new net: U19.15 (O10), U23.11 (C10)
- new net: U19.16 (O11), U23.12 (C11)
- new net: U19.17 (O12), U23.13 (C12)
- new net: U19.18 (O13), U23.14 (C13)
- new net: U19.19 (O14), U23.15 (C14)
- new net: U19.20 (O15), U23.16 (C15)
- new net: U19.5 (O0), U23.1 (C0)
- new net: U19.6 (O1), U23.2 (C1)
- new net: U19.7 (O2), U23.3 (C2)
- new net: U19.8 (O3), U23.4 (C3)
- new net: U19.9 (O4), U23.5 (C4)
- no-connect marks 3 -> 11

Commit message: Sick new LED block footprints
Parts:
- removed U11, U20, U21, U22, U23, U5, U7, U9: ~, custom_footprint_library:led_block_16_x_8, symbol custom_symbol_lib:led_block_16_x_8
- added U11, U5, U7, U9: ~, custom_footprint_library:led_block_16_x_8_left, symbol custom_symbol_lib:led_block_16_x_8_left
- added U20, U21, U22, U23: ~, custom_footprint_library:led_block_16_x_8_right, symbol custom_symbol_lib:led_block_16_x_8_right
Connections:
- net at U8.5 (O0): now also U7.1 (C0)
- net at U8.14 (O9): now also U7.10 (C9)
- net at U8.15 (O10): now also U7.11 (C10)
- net at U8.16 (O11): now also U7.12 (C11)
- net at U8.17 (O12): now also U7.13 (C12)
- net at U8.18 (O13): now also U7.14 (C13)
- net at U8.19 (O14): now also U7.15 (C14)
- net at U8.20 (O15): now also U7.16 (C15)
- net at U8.6 (O1): now also U7.2 (C1)
- net at U8.7 (O2): now also U7.3 (C2)
- net at U8.8 (O3): now also U7.4 (C3)
- net at U8.9 (O4): now also U7.5 (C4)
- net at U8.10 (O5): now also U7.6 (C5)
- net at U8.11 (O6): now also U7.7 (C6)
- net at U8.12 (O7): now also U7.8 (C7)
- net at U8.13 (O8): now also U7.9 (C8)
- net at U13.10 (O5): now also U22.6 (C5)
- net at U13.11 (O6): now also U22.7 (C6)
- net at U13.12 (O7): now also U22.8 (C7)
- net at U13.13 (O8): now also U22.9 (C8)
- net at U13.14 (O9): now also U22.10 (C9)
- net at U13.15 (O10): now also U22.11 (C10)
- net at U13.16 (O11): now also U22.12 (C11)
- net at U13.17 (O12): now also U22.13 (C12)
- net at U13.18 (O13): now also U22.14 (C13)
- net at U13.19 (O14): now also U22.15 (C14)
- net at U13.20 (O15): now also U22.16 (C15)
- net at U13.5 (O0): now also U22.1 (C0)
- net at U13.6 (O1): now also U22.2 (C1)
- net at U13.7 (O2): now also U22.3 (C2)
- net at U13.8 (O3): now also U22.4 (C3)
- net at U13.9 (O4): now also U22.5 (C4)
- net at U12.10 (O5): now also U9.6 (C5)
- net at U12.11 (O6): now also U9.7 (C6)
- net at U12.12 (O7): now also U9.8 (C7)
- net at U12.13 (O8): now also U9.9 (C8)
- net at U12.14 (O9): now also U9.10 (C9)
- net at U12.15 (O10): now also U9.11 (C10)
- net at U12.16 (O11): now also U9.12 (C11)
- net at U12.17 (O12): now also U9.13 (C12)
- net at U12.18 (O13): now also U9.14 (C13)
- net at U12.19 (O14): now also U9.15 (C14)
- net at U12.20 (O15): now also U9.16 (C15)
- net at U12.5 (O0): now also U9.1 (C0)
- net at U12.6 (O1): now also U9.2 (C1)
- net at U12.7 (O2): now also U9.3 (C2)
- net at U12.8 (O3): now also U9.4 (C3)
- net at U12.9 (O4): now also U9.5 (C4)
- net at U6.5 (O0): now also U20.1 (C0)
- net at U6.14 (O9): now also U20.10 (C9)
- net at U6.15 (O10): now also U20.11 (C10)
- net at U6.16 (O11): now also U20.12 (C11)
- net at U6.17 (O12): now also U20.13 (C12)
- net at U6.18 (O13): now also U20.14 (C13)
- net at U6.19 (O14): now also U20.15 (C14)
- net at U6.20 (O15): now also U20.16 (C15)
- net at U6.6 (O1): now also U20.2 (C1)
- net at U6.7 (O2): now also U20.3 (C2)
- net at U6.8 (O3): now also U20.4 (C3)
- net at U6.9 (O4): now also U20.5 (C4)
- net at U6.10 (O5): now also U20.6 (C5)
- net at U6.11 (O6): now also U20.7 (C6)
- net at U6.12 (O7): now also U20.8 (C7)
- net at U6.13 (O8): now also U20.9 (C8)
- net at U4.5 (O0): now also U5.1 (C0)
- net at U4.14 (O9): now also U5.10 (C9)
- net at U4.15 (O10): now also U5.11 (C10)
- net at U4.16 (O11): now also U5.12 (C11)
- net at U4.17 (O12): now also U5.13 (C12)
- net at U4.18 (O13): now also U5.14 (C13)
- net at U4.19 (O14): now also U5.15 (C14)
- net at U4.20 (O15): now also U5.16 (C15)
- net at U4.6 (O1): now also U5.2 (C1)
- net at U4.7 (O2): now also U5.3 (C2)
- net at U4.8 (O3): now also U5.4 (C3)
- net at U4.9 (O4): now also U5.5 (C4)
- net at U4.10 (O5): now also U5.6 (C5)
- net at U4.11 (O6): now also U5.7 (C6)
- net at U4.12 (O7): now also U5.8 (C7)
- net at U4.13 (O8): now also U5.9 (C8)
- net at U10.10 (O5): now also U21.6 (C5)
- net at U10.11 (O6): now also U21.7 (C6)
- net at U10.12 (O7): now also U21.8 (C7)
- net at U10.13 (O8): now also U21.9 (C8)
- net at U10.14 (O9): now also U21.10 (C9)
- net at U10.15 (O10): now also U21.11 (C10)
- net at U10.16 (O11): now also U21.12 (C11)
- net at U10.17 (O12): now also U21.13 (C12)
- net at U10.18 (O13): now also U21.14 (C13)
- net at U10.19 (O14): now also U21.15 (C14)
- net at U10.20 (O15): now also U21.16 (C15)
- net at U10.5 (O0): now also U21.1 (C0)
- net at U10.6 (O1): now also U21.2 (C1)
- net at U10.7 (O2): now also U21.3 (C2)
- net at U10.8 (O3): now also U21.4 (C3)
- net at U10.9 (O4): now also U21.5 (C4)
- net at U18.5 (O0): now also U11.1 (C0)
- net at U18.14 (O9): now also U11.10 (C9)
- net at U18.15 (O10): now also U11.11 (C10)
- net at U18.16 (O11): now also U11.12 (C11)
- net at U18.17 (O12): now also U11.13 (C12)
- net at U18.18 (O13): now also U11.14 (C13)
- net at U18.19 (O14): now also U11.15 (C14)
- net at U18.20 (O15): now also U11.16 (C15)
- net at U18.6 (O1): now also U11.2 (C1)
- net at U18.7 (O2): now also U11.3 (C2)
- net at U18.8 (O3): now also U11.4 (C3)
- net at U18.9 (O4): now also U11.5 (C4)
- net at U18.10 (O5): now also U11.6 (C5)
- net at U18.11 (O6): now also U11.7 (C6)
- net at U18.12 (O7): now also U11.8 (C7)
- net at U18.13 (O8): now also U11.9 (C8)
- net at U19.10 (O5): now also U23.6 (C5)
- net at U19.11 (O6): now also U23.7 (C6)
- net at U19.12 (O7): now also U23.8 (C7)
- net at U19.13 (O8): now also U23.9 (C8)
- net at U19.14 (O9): now also U23.10 (C9)
- net at U19.15 (O10): now also U23.11 (C10)
- net at U19.16 (O11): now also U23.12 (C11)
- net at U19.17 (O12): now also U23.13 (C12)
- net at U19.18 (O13): now also U23.14 (C13)
- net at U19.19 (O14): now also U23.15 (C14)
- net at U19.20 (O15): now also U23.16 (C15)
- net at U19.5 (O0): now also U23.1 (C0)
- net at U19.6 (O1): now also U23.2 (C1)
- net at U19.7 (O2): now also U23.3 (C2)
- net at U19.8 (O3): now also U23.4 (C3)
- net at U19.9 (O4): now also U23.5 (C4)
- new net: U11.17 (R0), U20.17 (R0), U21.17 (R0), U22.17 (R0), U23.17 (R0), U5.17 (R0), U7.17 (R0), U9.17 (R0)
- new net: U11.18 (R1), U20.18 (R1), U21.18 (R1), U22.18 (R1), U23.18 (R1), U5.18 (R1), U7.18 (R1), U9.18 (R1)
- new net: U11.19 (R2), U20.19 (R2), U21.19 (R2), U22.19 (R2), U23.19 (R2), U5.19 (R2), U7.19 (R2), U9.19 (R2)
- new net: U11.20 (R3), U20.20 (R3), U21.20 (R3), U22.20 (R3), U23.20 (R3), U5.20 (R3), U7.20 (R3), U9.20 (R3)
- new net: U11.21 (R4), U20.21 (R4), U21.21 (R4), U22.21 (R4), U23.21 (R4), U5.21 (R4), U7.21 (R4), U9.21 (R4)
- new net: U11.22 (R5), U20.22 (R5), U21.22 (R5), U22.22 (R5), U23.22 (R5), U5.22 (R5), U7.22 (R5), U9.22 (R5)
- new net: U11.23 (R6), U20.23 (R6), U21.23 (R6), U22.23 (R6), U23.23 (R6), U5.23 (R6), U7.23 (R6), U9.23 (R6)
- new net: U11.24 (R7), U20.24 (R7), U21.24 (R7), U22.24 (R7), U23.24 (R7), U5.24 (R7), U7.24 (R7), U9.24 (R7)

Commit message: Almost done with led matrix schematic
Parts:
- added C2: C, Capacitor_THT:CP_Radial_D4.0mm_P2.00mm, symbol Device:C
- added D1, D2, D3: LED, LED_THT:LED_D3.0mm, symbol Device:LED
- added Q1, Q2, Q3, Q4, Q5, Q6, Q7, Q9: IRF540N, Package_TO_SOT_THT:TO-220-3_Vertical, symbol Transistor_FET:IRF540N
- added R14, R15, R16, R17, R18, R19, R20, R7: R, custom_footprint_library:0.4_pitch_resistor, symbol Device:R
- added SW1: SW_DIP_x01, Button_Switch_THT:SW_DIP_SPSTx01_Slide_6.7x4.1mm_W7.62mm_P2.54mm_LowProfile, symbol Switch:SW_DIP_x01
- added U24, U33: ~, Package_DIP:DIP-16_W7.62mm, symbol custom_symbol_lib:3_to_8_demultiplexer
- added U25: ~, Package_DIP:DIP-16_W7.62mm, symbol custom_symbol_lib:8_bit_counter
- added U26: ~, Package_DIP:DIP-28_W15.24mm, symbol custom_symbol_lib:32Kx8_sram
- added U27, U28: ~, Package_DIP:DIP-16_W7.62mm, symbol custom_symbol_lib:multiplexer_8_bit
- added U29: ~, Package_DIP:DIP-14_W7.62mm, symbol custom_symbol_lib:4x_XOR
- added U30, U46: ~, Package_DIP:DIP-14_W7.62mm, symbol custom_symbol_lib:6xNOT
- added U31: ~, Package_DIP:DIP-20_W7.62mm, symbol custom_symbol_lib:8_bit_transparent_latch
- added U32, U43, U44, U51, U52: ~, Package_DIP:DIP-20_W7.62mm, symbol custom_symbol_lib:rising_edge_8_bit_latch
- added U34: ~, Package_DIP:DIP-14_W7.62mm, symbol custom_symbol_lib:OP_AMP_quad
- added U35, U36, U37, U38, U39, U40, U41, U42, U48: ~, custom_footprint_library:jumper, symbol custom_symbol_lib:jumper
- added U45, U47: ~, Package_DIP:DIP-14_W7.62mm, symbol custom_symbol_lib:quad_and
- added U49: ~, Package_DIP:DIP-14_W7.62mm, symbol custom_symbol_lib:dual_latch
- added U50: ~, Package_DIP:DIP-14_W7.62mm, symbol custom_symbol_lib:quad_OR
- R10, R11, R12, R13, R5, R6, R8, R9: footprint (none) -> custom_footprint_library:0.4_pitch_resistor
Connections:
- net at U10.2 (D_in), U12.2 (D_in), U13.2 (D_in)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: now also U29.3 (1Q)
- net at U10.3 (CLK), U12.3 (CLK), U13.3 (CLK)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: now also U39.3 (OUT)
- net at U13.4 (LE): now also U24.10 (Y5)
- net at U12.4 (LE): now also U24.11 (Y4)
- net at R3.1, R4.1, U15.1 (OUT_1): now also U17.13 (RCLK), U25.13 (RCLK), U30.3 (I1), U47.10 (4A)
- net at U10.4 (LE): now also U24.12 (Y3)
- net at U11.17 (R0), U20.17 (R0), U21.17 (R0)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: now also Q9.3 (S)
- net at U11.18 (R1), U20.18 (R1), U21.18 (R1)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: now also Q1.3 (S)
- net at U11.19 (R2), U20.19 (R2), U21.19 (R2)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: now also Q2.3 (S)
- net at U11.20 (R3), U20.20 (R3), U21.20 (R3)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: now also Q3.3 (S)
- net at U11.21 (R4), U20.21 (R4), U21.21 (R4)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: now also Q4.3 (S)
- net at U11.22 (R5), U20.22 (R5), U21.22 (R5)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: now also Q5.3 (S)
- net at U11.23 (R6), U20.23 (R6), U21.23 (R6)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: now also Q6.3 (S)
- net at U11.24 (R7), U20.24 (R7), U21.24 (R7)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: now also Q7.3 (S)
- net at U17.1 (Q1): now also U27.10 (A1), U28.10 (A1)
- net at U17.10 (CCLR#): now also U17.16 (V+), U25.10 (CCLR#), U25.16 (V+)
- net at U17.11 (CCLK): now also U25.11 (CCLK), U38.3 (OUT)
- net at U17.12 (CCKEN#): now also U17.14 (OE#), U17.8 (GND), U25.14 (OE#), U25.8 (GND)
- net at U17.15 (Q0): now also U27.11 (A0), U28.11 (A0)
- net at U17.2 (Q2): now also U27.9 (A2), U28.9 (A2)
- net at U17.3 (Q3): now also U27.7 (OE#), U30.1 (I0)
- net at U17.4 (Q4): now also U24.1 (A0), U31.2 (D0)
- net at U17.5 (Q5): now also U24.2 (A1), U31.6 (D4)
- net at U17.6 (Q6): now also U24.3 (A2), U31.7 (D5)
- net at U17.7 (Q7): now also R19.1, U31.3 (D1), U33.3 (A2)
- net at U17.9 (RCO#): now also U25.12 (CCKEN#)
- net at U16.1 (OE#): now also U30.10 (O4); no longer U16.10 (GND)
- net at U16.11 (CLK), U2.3 (CLK), U3.11 (CLK): now also U32.11 (CLK)
- net at U16.12 (Q7): now also U14.19 (D7), U44.9 (D7)
- net at U16.13 (Q6): now also U14.18 (D6), U44.8 (D6)
- net at U16.14 (Q5): now also U14.17 (D5), U44.7 (D5)
- net at U16.15 (Q4): now also U14.16 (D4), U44.6 (D4)
- net at U16.16 (Q3): now also U14.15 (D3), U44.5 (D3)
- net at U16.17 (Q2): now also U14.13 (D2), U44.4 (D2)
- net at U16.18 (Q1): now also U14.12 (D1), U44.3 (D1)
- net at U16.19 (Q0): now also U14.11 (D0), U44.2 (D0)
- net at U1.9 (8), U16.2 (D0): now also U32.2 (D0)
- net at U1.10 (9), U16.3 (D1): now also U32.3 (D1)
- net at U1.11 (10), U16.4 (D2): now also U32.4 (D2)
- net at U1.12 (11), U16.5 (D3): now also U32.5 (D3)
- net at U1.13 (12), U16.6 (D4): now also U32.6 (D4)
- net at U1.14 (13), U16.7 (D5): now also U32.7 (D5)
- net at U1.15 (14), U16.8 (D6): now also U32.8 (D6)
- net at U1.16 (15), U16.9 (D7): now also U32.9 (D7)
- net at U18.4 (LE): now also U24.9 (Y6)
- net at U8.4 (LE): now also U24.13 (Y2)
- net at U19.4 (LE): now also U24.7 (Y7)
- net at U3.1 (OE#): now also U30.8 (03); no longer U3.10 (GND)
- net at U3.13 (Q6): now also U14.5 (A5), U26.5 (A5), U31.14 (Q5)
- net at U3.14 (Q5): now also U14.6 (A4), U26.6 (A4), U31.15 (Q4)
- net at U3.15 (Q4): now also U14.7 (A3), U26.7 (A3), U31.16 (Q3)
- net at U3.16 (Q3): now also U14.8 (A2), U26.8 (A2), U31.17 (Q2)
- net at U3.17 (Q2): now also U14.9 (A1), U26.9 (A1), U31.18 (Q1)
- net at U3.18 (Q1): now also U14.10 (A0), U26.10 (A0), U31.19 (Q0)
- net at U3.19 (Q0): now also U45.10 (4A), U46.1 (I0)
- net at U6.4 (LE): now also U24.14 (Y1)
- net at U14.1 (A14): now also U14.14 (GND), U14.2 (A12), U14.20 (CE#), U14.21 (A10), U14.23 (A11), U14.24 (A9), U14.25 (A8), U14.26 (A13), U14.3 (A7), U14.4 (A6), U26.1 (A14), U26.14 (GND), U26.2 (A12), U26.20 (CE#), U26.21 (A10), U26.23 (A11), U26.24 (A9), U26.25 (A8), U26.26 (A13), U26.3 (A7), U26.4 (A6)
- net at U14.22 (OE#): now also U26.22 (OE#), U30.6 (O2)
- net at U14.27 (WE#): now also U46.4 (O1)
- net at U4.4 (LE): now also U24.15 (Y0)
- new net: U30.11 (I4), U45.6 (2Q), U47.1 (1A)
- new net: U30.12 (O5), U32.1 (OE#)
- new net: U30.13 (I5), U45.8 (4Q), U47.13 (3A)
- new net: U28.7 (OE#), U30.2 (O0), U47.5 (2B)
- new net: U30.4 (O1), U45.1 (1A)
- new net: U30.5 (I2), U35.3 (OUT)
- new net: U30.9 (I3), U31.1 (OE#), U41.3 (OUT), U45.5 (2B), U45.9 (4B)
- new net: U24.4 (E2#), U24.5 (E3#), U24.8 (GND)
- new net: U24.6 (E1), U40.3 (OUT)
- new net: Q1.1 (G), U33.14 (Y1)
- new net: Q1.2 (D), Q2.2 (D), Q3.2 (D), Q4.2 (D), Q5.2 (D), Q6.2 (D), Q7.2 (D), Q9.2 (D), SW1.2, U33.16 (V+)
- new net: D1.1 (K), D2.1 (K), D3.1 (K), R20.2, U33.5 (E3#), U33.8 (GND)
- new net: D1.2 (A), R17.2
- new net: U47.4 (2A), U47.9 (4B), U49.1 (0Q), U49.2 (0Q#), U49.5 (0D), U51.2 (D0)
- new net: U49.10 (1RESET), U49.11 (1CLK), U49.4 (0RESET), U49.6 (0SET), U49.7 (GND), U49.8 (1SET), U49.9 (1D)
- new net: U49.3 (0CLK), U50.3 (Q0)
- new net: Q5.1 (G), U33.10 (Y5)
- new net: Q2.1 (G), U33.13 (Y2)
- new net: Q3.1 (G), U33.12 (Y3)
- new net: R14.2, R15.1, R16.2, U34.3 (IN+_1)
- new net: C2.2, R15.2, U34.10 (IN+_3), U34.11 (GND), U34.12 (IN+_4), U34.13 (IN-_4), U34.5 (IN+_2), U34.6 (IN-_2), U34.9 (IN-_3)
- new net: U37.3 (OUT), U45.2 (1B)
- new net: U38.1 (IN), U45.3 (1Q)
- new net: U45.4 (2A), U46.2 (O0)
- new net: U46.5 (I2), U47.11 (3Q)
- new net: U42.3 (OUT), U47.12 (3B), U47.2 (1B)
- new net: U46.3 (I1), U47.3 (1Q)
- new net: U47.6 (2Q), U50.1 (0A)
- new net: U47.8 (4Q), U50.2 (0B)
- new net: Q7.1 (G), U33.7 (Y7)
- new net: R20.1, SW1.1, U33.6 (E1)
- new net: U51.1 (OE#), U51.10 (GND), U51.6 (D4), U51.7 (D5), U51.8 (D6), U51.9 (D7), U52.1 (OE#), U52.10 (GND), U52.6 (D4), U52.7 (D5), U52.8 (D6), U52.9 (D7)
- new net: U51.16 (Q3), U52.5 (D3)
- new net: U51.17 (Q2), U52.4 (D2)
- new net: U51.18 (Q1), U52.3 (D1)
- new net: U51.19 (Q0), U52.2 (D0)
- new net: U51.20 (V+), U52.20 (V+)
- new net: U51.3 (D1), U52.19 (Q0)
- new net: U51.4 (D2), U52.18 (Q1)
- new net: U51.5 (D3), U52.17 (Q2)
- new net: C2.1, R7.2, U34.2 (IN-_1)
- new net: U35.2 (GND), U36.2 (GND), U37.2 (GND), U38.2 (GND), U39.2 (GND), U40.2 (GND), U41.2 (GND), U42.2 (GND), U48.2 (GND)
- new net: U36.3 (OUT), U43.11 (CLK), U44.11 (CLK)
- new net: U33.4 (E2#), U48.3 (OUT)
- new net: U44.1 (OE#), U44.10 (GND)
- new net: U27.12 (D7), U44.12 (Q7)
- new net: U27.13 (D6), U44.13 (Q6)
- new net: U27.14 (D5), U44.14 (Q5)
- new net: U27.15 (D4), U44.15 (Q4)
- new net: U27.1 (D3), U44.16 (Q3)
- new net: U27.2 (D2), U44.17 (Q2)
- new net: U27.3 (D1), U44.18 (Q1)
- new net: U27.4 (D0), U44.19 (Q0)
- new net: R17.1, U25.1 (Q1), U31.5 (D3), U33.1 (A0)
- new net: Q4.1 (G), U33.11 (Y4)
- new net: Q9.1 (G), U33.15 (Y0)
- new net: R18.1, U25.15 (Q0), U31.4 (D2), U33.2 (A1)
- new net: Q6.1 (G), U33.9 (Y6)
- new net: D3.2 (A), R19.2
- new net: U27.5 (Q), U29.1 (1A)
- new net: U31.10 (GND), U31.8 (D6), U31.9 (D7)
- new net: U31.11 (CLK), U31.20 (V+)
- new net: D2.2 (A), R18.2
- new net: U43.1 (OE#), U43.10 (GND)
- new net: U28.12 (D7), U43.12 (Q7)
- new net: U28.13 (D6), U43.13 (Q6)
- new net: U28.14 (D5), U43.14 (Q5)
- new net: U28.15 (D4), U43.15 (Q4)
- new net: U28.1 (D3), U43.16 (Q3)
- new net: U28.2 (D2), U43.17 (Q2)
- new net: U28.3 (D1), U43.18 (Q1)
- new net: U28.4 (D0), U43.19 (Q0)
- new net: U26.11 (D0), U32.19 (Q0), U43.2 (D0)
- new net: U26.12 (D1), U32.18 (Q1), U43.3 (D1)
- new net: U26.13 (D2), U32.17 (Q2), U43.4 (D2)
- new net: U26.15 (D3), U32.16 (Q3), U43.5 (D3)
- new net: U26.16 (D4), U32.15 (Q4), U43.6 (D4)
- new net: U26.17 (D5), U32.14 (Q5), U43.7 (D5)
- new net: U26.18 (D6), U32.13 (Q6), U43.8 (D6)
- new net: U26.19 (D7), U32.12 (Q7), U43.9 (D7)
- new net: U28.5 (Q), U29.2 (1B)
- new net: R16.1, R7.1, U34.1 (OUT_1)
- new net: R14.1, U34.4 (V+)
- new net: U26.27 (WE#), U46.6 (O2)
- no-connect marks 11 -> 36
Other:
- note added: "Address"
- note added: "Data even columns"
- note added: "Data odd columns"
- moved on the sheet: C1, R1, R10, R11, R12, R13, R2, R3, R4, R5, R6, R8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

Commit message: Schematic probably done
Parts:
- removed C2: C, Capacitor_THT:CP_Radial_D4.0mm_P2.00mm, symbol Device:C
- removed R14, R15, R16, R7: R, custom_footprint_library:0.4_pitch_resistor, symbol Device:R
- removed U29: ~, Package_DIP:DIP-14_W7.62mm, symbol custom_symbol_lib:4x_XOR
- removed U34: ~, Package_DIP:DIP-14_W7.62mm, symbol custom_symbol_lib:OP_AMP_quad
- removed U48: ~, custom_footprint_library:jumper, symbol custom_symbol_lib:jumper
- added U29: ~, Package_DIP:DIP-14_W7.62mm, symbol custom_symbol_lib:quad_OR
- added U48, U53: ~, Package_DIP:DIP-14_W7.62mm, symbol custom_symbol_lib:dual_4_input_OR
- added U54: ~, Package_DIP:DIP-14_W7.62mm, symbol custom_symbol_lib:quad_and
Connections:
- net at U30.14 (V+): now also Q1.2 (D), Q2.2 (D), Q3.2 (D), Q4.2 (D), Q5.2 (D), Q6.2 (D), Q7.2 (D), Q9.2 (D), R2.1, SW1.2, U10.24 (V+), U12.24 (V+), U13.24 (V+), U14.28 (V+), U15.4 (V+), U16.20 (V+), U17.10 (CCLR#), U17.16 (V+), U18.24 (V+), U19.24 (V+), U2.1 (V+), U24.16 (V+), U25.10 (CCLR#), U25.16 (V+), U26.28 (V+), U27.16 (V+), U28.16 (V+), U3.20 (V+), U31.11 (CLK), U31.20 (V+), U32.20 (V+), U33.16 (V+), U4.24 (V+), U43.20 (V+), U44.20 (V+), U45.14 (V+), U46.14 (V+), U47.14 (V+), U49.14 (V+), U50.14 (V+), U51.20 (V+), U52.20 (V+), U6.24 (V+), U8.24 (V+), U29.14 (V+), U48.14 (V+), U48.2 (A0), U53.14 (V+), U53.9 (B0), U54.14 (V+)
- net at R3.1, R4.1, U15.1 (OUT_1)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: now also U52.11 (CLK)
- net at U30.4 (O1), U45.1 (1A): now also U51.11 (CLK), U54.13 (3A)
- net at U30.7 (GND): now also C1.2, D1.1 (K), D2.1 (K), D3.1 (K), R1.2, R10.2, R11.2, R12.2, R13.2, R20.2, R5.2, R6.2, R8.2, R9.2, U10.1 (GND), U10.21 (OE#), U12.1 (GND), U12.21 (OE#), U13.1 (GND), U13.21 (OE#), U14.1 (A14), U14.14 (GND), U14.2 (A12), U14.20 (CE#), U14.21 (A10), U14.23 (A11), U14.24 (A9), U14.25 (A8), U14.26 (A13), U14.3 (A7), U14.4 (A6), U15.10 (IN+_3), U15.11 (GND), U15.12 (IN+_4), U15.13 (IN-_4), U15.5 (IN+_2), U15.6 (IN-_2), U15.9 (IN-_3), U16.10 (GND), U17.12 (CCKEN#), U17.14 (OE#), U17.8 (GND), U18.1 (GND), U18.21 (OE#), U19.1 (GND), U19.21 (OE#), U2.2 (GND), U24.4 (E2#), U24.5 (E3#), U24.8 (GND), U25.14 (OE#), U25.8 (GND), U26.1 (A14), U26.14 (GND), U26.2 (A12), U26.20 (CE#), U26.21 (A10), U26.23 (A11), U26.24 (A9), U26.25 (A8), U26.26 (A13), U26.3 (A7), U26.4 (A6), U27.8 (GND), U28.8 (GND), U3.10 (GND), U31.10 (GND), U31.8 (D6), U31.9 (D7), U32.10 (GND), U33.4 (E2#), U33.5 (E3#), U33.8 (GND), U4.1 (GND), U4.21 (OE#), U43.1 (OE#), U43.10 (GND), U44.1 (OE#), U44.10 (GND), U45.7 (GND), U46.11 (I4), U46.7 (GND), U47.7 (GND), U49.10 (1RESET), U49.11 (1CLK), U49.4 (0RESET), U49.6 (0SET), U49.7 (GND), U49.8 (1SET), U49.9 (1D), U50.12 (3A), U50.13 (3B), U50.5 (1A), U50.6 (1B), U50.7 (GND), U50.8 (2A), U50.9 (2B), U51.1 (OE#), U51.10 (GND), U51.6 (D4), U51.7 (D5), U51.8 (D6), U51.9 (D7), U52.1 (OE#), U52.10 (GND), U52.6 (D4), U52.7 (D5), U52.8 (D6), U52.9 (D7), U6.1 (GND), U6.21 (OE#), U8.1 (GND), U8.21 (OE#), U29.5 (1A), U29.6 (1B), U29.7 (GND), U29.8 (2A), U29.9 (2B), U48.10 (B1), U48.11 (B2), U48.12 (B3), U48.7 (GND), U48.9 (B0), U53.7 (GND), U54.7 (GND)
- net at U10.2 (D_in), U12.2 (D_in), U13.2 (D_in)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: now also U29.3 (Q0)
- net at U47.9 (4B), U49.1 (0Q), U51.2 (D0): now also U40.1 (IN), U53.2 (A0); no longer U47.4 (2A), U49.2 (0Q#), U49.5 (0D)
- net at U45.11 (3Q): now also U42.1 (IN)
- net at U45.12 (3B): now also U51.19 (Q0), U52.2 (D0), U53.3 (A1)
- net at U45.13 (3A): now also U52.16 (Q3)
- net at U45.4 (2A), U46.2 (O0): now also U14.27 (WE#)
- net at U51.17 (Q2), U52.4 (D2): now also U53.11 (B2)
- net at U51.18 (Q1), U52.3 (D1): now also U48.4 (A2), U53.5 (A3)
- net at U51.3 (D1), U52.19 (Q0): now also U48.3 (A1), U53.4 (A2)
- net at U51.4 (D2), U52.18 (Q1): now also U36.1 (IN), U29.13 (3B), U48.5 (A3), U53.10 (B1)
- net at U51.5 (D3), U52.17 (Q2): now also U53.12 (B3)
- net at U39.1 (IN): now also U54.11 (3Q)
- net at U41.1 (IN): now also U53.13 (OB)
- net at U27.5 (Q): now also U29.1 (0A)
- net at U35.1 (IN): now also U48.1 (OA)
- net at U28.5 (Q): now also U29.2 (0B)
- net at U37.1 (IN): now also U46.8 (03)
- net at U46.4 (O1): no longer U14.27 (WE#)
- net at U46.12 (O5): now also U54.12 (3B)
- net at U46.13 (I5): now also U29.12 (3A), U53.1 (OA)
- net at U46.9 (I3): now also U29.11 (Q3)
- new net: U47.4 (2A), U49.2 (0Q#), U49.5 (0D)
- no-connect marks 36 -> 40
Other:
- note added: "CLK"
- note added: "CLK#"
- moved on the sheet: Q1, Q2, Q3, Q4, Q5, Q6, Q7, Q9, U46, U51, U52
