File: kicad/version_2/led_matrix/led_matrix.kicad_pcb (KiCad board)
At the start: 2 copper layers, 447 x 370.8 mm, 28 parts

Commit message: Sick new LED block footprints
Parts:
- removed C1: C, Capacitor_THT:CP_Radial_D4.0mm_P2.00mm
- removed R1, R2, R3, R4: R, custom_footprint_library:0.4_pitch_resistor
- removed U1: ~, Connector_PinHeader_2.54mm:PinHeader_1x16_P2.54mm_Vertical
- removed U10, U12, U13, U18, U19, U4, U6, U8: ~, Package_DIP:DIP-24_W7.62mm
- removed U11, U20, U21, U22, U23, U5, U7, U9: ~, custom_footprint_library:led_block_16_x_8
- removed U14: ~, Package_DIP:DIP-28_W15.24mm
- removed U15: ~, Package_DIP:DIP-14_W7.62mm
- removed U16, U3: ~, Package_DIP:DIP-20_W7.62mm
- removed U17: ~, Package_DIP:DIP-16_W7.62mm
- removed U2: ~, Connector_PinHeader_2.54mm:PinHeader_1x03_P2.54mm_Vertical
Other:
- board outline removed

Commit message: Almost done with led matrix schematic
Parts:
- added C1: C, Capacitor_THT:CP_Radial_D4.0mm_P2.00mm, F.Cu at (429.4, 471.9)
- added R1: R, custom_footprint_library:0.4_pitch_resistor, F.Cu at (424.8, 462.3)
- added R10: R, custom_footprint_library:0.4_pitch_resistor, F.Cu at (453.9, 462.3)
- added R11: R, custom_footprint_library:0.4_pitch_resistor, F.Cu at (457.5, 462.3)
- added R12: R, custom_footprint_library:0.4_pitch_resistor, F.Cu at (461.2, 462.3)
- added R13: R, custom_footprint_library:0.4_pitch_resistor, F.Cu at (464.8, 462.3)
- added R2: R, custom_footprint_library:0.4_pitch_resistor, F.Cu at (428.4, 462.3)
- added R3: R, custom_footprint_library:0.4_pitch_resistor, F.Cu at (432.1, 462.3)
- added R4: R, custom_footprint_library:0.4_pitch_resistor, F.Cu at (435.7, 462.3)
- added R5: R, custom_footprint_library:0.4_pitch_resistor, F.Cu at (439.3, 462.3)
- added R6: R, custom_footprint_library:0.4_pitch_resistor, F.Cu at (443.0, 462.3)
- added R8: R, custom_footprint_library:0.4_pitch_resistor, F.Cu at (446.6, 462.3)
- added R9: R, custom_footprint_library:0.4_pitch_resistor, F.Cu at (450.3, 462.3)
- added U1: ~, Connector_PinHeader_2.54mm:PinHeader_1x16_P2.54mm_Vertical, F.Cu at (680.7, 454.7)
- added U10: ~, Package_DIP:DIP-24_W7.62mm, F.Cu at (564.1, 472.4)
- added U11: ~, custom_footprint_library:led_block_16_x_8_left, F.Cu at (489.6, 336.6)
- added U12: ~, Package_DIP:DIP-24_W7.62mm, F.Cu at (575.0, 472.4)
- added U13: ~, Package_DIP:DIP-24_W7.62mm, F.Cu at (585.8, 472.4)
- added U14: ~, Package_DIP:DIP-28_W15.24mm, F.Cu at (716.3, 383.5)
- added U15: ~, Package_DIP:DIP-14_W7.62mm, F.Cu at (650.9, 472.4)
- added U16: ~, Package_DIP:DIP-20_W7.62mm, F.Cu at (629.2, 472.4)
- added U17: ~, Package_DIP:DIP-16_W7.62mm, F.Cu at (640.1, 472.4)
- added U18: ~, Package_DIP:DIP-24_W7.62mm, F.Cu at (596.7, 472.4)
- added U19: ~, Package_DIP:DIP-24_W7.62mm, F.Cu at (607.5, 472.4)
- added U2: ~, Connector_PinHeader_2.54mm:PinHeader_1x03_P2.54mm_Vertical, F.Cu at (425.3, 471.5)
- added U20: ~, custom_footprint_library:led_block_16_x_8_right, F.Cu at (615.3, 154.3)
- added U21: ~, custom_footprint_library:led_block_16_x_8_right, F.Cu at (615.3, 215.3)
- added U22: ~, custom_footprint_library:led_block_16_x_8_right, F.Cu at (615.3, 276.2)
- added U23: ~, custom_footprint_library:led_block_16_x_8_right, F.Cu at (615.3, 337.2)
- added U24: ~, Package_DIP:DIP-16_W7.62mm, F.Cu at (525.6, 422.9)
- added U25: ~, Package_DIP:DIP-16_W7.62mm, F.Cu at (536.5, 422.9)
- added U26: ~, Package_DIP:DIP-28_W15.24mm, F.Cu at (507.2, 395.9)
- added U27: ~, Package_DIP:DIP-16_W7.62mm, F.Cu at (547.3, 422.9)
- added U28: ~, Package_DIP:DIP-16_W7.62mm, F.Cu at (558.2, 422.9)
- added U29: ~, Package_DIP:DIP-14_W7.62mm, F.Cu at (547.3, 395.9)
- added U3: ~, Package_DIP:DIP-20_W7.62mm, F.Cu at (618.4, 472.4)
- added U30: ~, Package_DIP:DIP-14_W7.62mm, F.Cu at (558.2, 395.9)
- added U31: ~, Package_DIP:DIP-20_W7.62mm, F.Cu at (525.6, 395.9)
- added U32: ~, Package_DIP:DIP-20_W7.62mm, F.Cu at (536.5, 395.9)
- added U4: ~, Package_DIP:DIP-24_W7.62mm, F.Cu at (366.4, 133.3)
- added U5: ~, custom_footprint_library:led_block_16_x_8_left, F.Cu at (489.6, 153.7)
- added U6: ~, Package_DIP:DIP-24_W7.62mm, F.Cu at (542.4, 472.4)
- added U7: ~, custom_footprint_library:led_block_16_x_8_left, F.Cu at (489.6, 214.6)
- added U8: ~, Package_DIP:DIP-24_W7.62mm, F.Cu at (553.3, 472.4)
- added U9: ~, custom_footprint_library:led_block_16_x_8_left, F.Cu at (489.6, 275.6)

Commit message: Schematic probably done
Parts:
- added D1: LED, LED_THT:LED_D3.0mm, F.Cu at (447.7, 413.1)
- added D2: LED, LED_THT:LED_D3.0mm, F.Cu at (447.7, 418.6)
- added D3: LED, LED_THT:LED_D3.0mm, F.Cu at (447.7, 424.2)
- added Q1: IRF540N, Package_TO_SOT_THT:TO-220-3_Vertical, F.Cu at (383.4, 414.2)
- added Q2: IRF540N, Package_TO_SOT_THT:TO-220-3_Vertical, F.Cu at (383.4, 420.2)
- added Q3: IRF540N, Package_TO_SOT_THT:TO-220-3_Vertical, F.Cu at (383.4, 426.1)
- added Q4: IRF540N, Package_TO_SOT_THT:TO-220-3_Vertical, F.Cu at (383.4, 432.1)
- added Q5: IRF540N, Package_TO_SOT_THT:TO-220-3_Vertical, F.Cu at (383.4, 438.1)
- added Q6: IRF540N, Package_TO_SOT_THT:TO-220-3_Vertical, F.Cu at (383.4, 444.0)
- added Q7: IRF540N, Package_TO_SOT_THT:TO-220-3_Vertical, F.Cu at (383.4, 450.0)
- added Q9: IRF540N, Package_TO_SOT_THT:TO-220-3_Vertical, F.Cu at (383.4, 455.9)
- added R17: R, custom_footprint_library:0.4_pitch_resistor, F.Cu at (393.6, 444.2)
- added R18: R, custom_footprint_library:0.4_pitch_resistor, F.Cu at (397.2, 444.2)
- added R19: R, custom_footprint_library:0.4_pitch_resistor, F.Cu at (400.9, 444.2)
- added R20: R, custom_footprint_library:0.4_pitch_resistor, F.Cu at (404.5, 444.2)
- added SW1: SW_DIP_x01, Button_Switch_THT:SW_DIP_SPSTx01_Slide_6.7x4.1mm_W7.62mm_P2.54mm_LowProfile, F.Cu at (393.4, 454.0)
- added U29: ~, Package_DIP:DIP-14_W7.62mm, F.Cu at (366.6, 393.0)
- added U33: ~, Package_DIP:DIP-16_W7.62mm, F.Cu at (436.8, 412.4)
- added U35: ~, custom_footprint_library:jumper, F.Cu at (371.3, 418.5)
- added U36: ~, custom_footprint_library:jumper, F.Cu at (371.3, 427.4)
- added U37: ~, custom_footprint_library:jumper, F.Cu at (371.3, 436.3)
- added U38: ~, custom_footprint_library:jumper, F.Cu at (371.3, 445.2)
- added U39: ~, custom_footprint_library:jumper, F.Cu at (371.3, 454.2)
- added U40: ~, custom_footprint_library:jumper, F.Cu at (371.3, 463.1)
- added U41: ~, custom_footprint_library:jumper, F.Cu at (371.3, 472.0)
- added U42: ~, custom_footprint_library:jumper, F.Cu at (371.3, 480.9)
- added U43: ~, Package_DIP:DIP-20_W7.62mm, F.Cu at (393.4, 412.4)
- added U44: ~, Package_DIP:DIP-20_W7.62mm, F.Cu at (404.2, 412.4)
- added U45: ~, Package_DIP:DIP-14_W7.62mm, F.Cu at (377.5, 393.0)
- added U46: ~, Package_DIP:DIP-14_W7.62mm, F.Cu at (388.3, 393.0)
- added U47: ~, Package_DIP:DIP-14_W7.62mm, F.Cu at (399.2, 393.0)
- added U48: ~, Package_DIP:DIP-14_W7.62mm, F.Cu at (410.0, 393.0)
- added U49: ~, Package_DIP:DIP-14_W7.62mm, F.Cu at (420.9, 393.0)
- added U50: ~, Package_DIP:DIP-14_W7.62mm, F.Cu at (431.7, 393.0)
- added U51: ~, Package_DIP:DIP-20_W7.62mm, F.Cu at (415.1, 412.4)
- added U52: ~, Package_DIP:DIP-20_W7.62mm, F.Cu at (425.9, 412.4)
- added U53: ~, Package_DIP:DIP-14_W7.62mm, F.Cu at (442.6, 393.0)
- added U54: ~, Package_DIP:DIP-14_W7.62mm, F.Cu at (453.4, 393.0)
Connections:
- C1 pad 2: Net-(U15-GND) -> Net-(D1-K)
- R1 pad 2: Net-(U15-GND) -> Net-(D1-K)
- R10 pad 2: Net-(U10-GND) -> Net-(D1-K)
- R11 pad 2: Net-(U10-GND) -> Net-(D1-K)
- R12 pad 2: Net-(U10-GND) -> Net-(D1-K)
- R13 pad 2: Net-(U10-GND) -> Net-(D1-K)
- R2 pad 1: Net-(U15-V+) -> Net-(Q1-D)
- R5 pad 2: Net-(U10-GND) -> Net-(D1-K)
- R6 pad 2: Net-(U10-GND) -> Net-(D1-K)
- R8 pad 2: Net-(U10-GND) -> Net-(D1-K)
- R9 pad 2: Net-(U10-GND) -> Net-(D1-K)
- U10 pad 1: Net-(U10-GND) -> Net-(D1-K)
- U10 pad 21: Net-(U10-GND) -> Net-(D1-K)
- U10 pad 24: Net-(U10-V+) -> Net-(Q1-D)
- U12 pad 1: Net-(U10-GND) -> Net-(D1-K)
- U12 pad 21: Net-(U10-GND) -> Net-(D1-K)
- U12 pad 24: Net-(U10-V+) -> Net-(Q1-D)
- U13 pad 1: Net-(U10-GND) -> Net-(D1-K)
- U13 pad 21: Net-(U10-GND) -> Net-(D1-K)
- U13 pad 24: Net-(U10-V+) -> Net-(Q1-D)
- U14 pad 1: Net-(U14-A10) -> Net-(D1-K)
- U14 pad 14: Net-(U14-A10) -> Net-(D1-K)
- U14 pad 2: Net-(U14-A10) -> Net-(D1-K)
- U14 pad 20: unconnected-(U14-CE#-Pad20) -> Net-(D1-K)
- U14 pad 21: Net-(U14-A10) -> Net-(D1-K)
- U14 pad 22: unconnected-(U14-OE#-Pad22) -> Net-(U14-OE#)
- U14 pad 23: Net-(U14-A10) -> Net-(D1-K)
- U14 pad 24: Net-(U14-A10) -> Net-(D1-K)
- U14 pad 25: Net-(U14-A10) -> Net-(D1-K)
- U14 pad 26: Net-(U14-A10) -> Net-(D1-K)
- U14 pad 27: unconnected-(U14-WE#-Pad27) -> Net-(U14-WE#)
- U14 pad 28: unconnected-(U14-V+-Pad28) -> Net-(Q1-D)
- U14 pad 3: Net-(U14-A10) -> Net-(D1-K)
- U14 pad 4: Net-(U14-A10) -> Net-(D1-K)
- U15 pad 10: Net-(U15-GND) -> Net-(D1-K)
- U15 pad 11: Net-(U15-GND) -> Net-(D1-K)
- U15 pad 12: Net-(U15-GND) -> Net-(D1-K)
- U15 pad 13: Net-(U15-GND) -> Net-(D1-K)
- U15 pad 4: Net-(U15-V+) -> Net-(Q1-D)
- U15 pad 5: Net-(U15-GND) -> Net-(D1-K)
- U15 pad 6: Net-(U15-GND) -> Net-(D1-K)
- U15 pad 9: Net-(U15-GND) -> Net-(D1-K)
- U16 pad 1: unconnected-(U16-OE#-Pad1) -> Net-(U16-OE#)
- U16 pad 10: unconnected-(U16-GND-Pad10) -> Net-(D1-K)
- U16 pad 20: unconnected-(U16-V+-Pad20) -> Net-(Q1-D)
- U17 pad 10: unconnected-(U17-CCLR#-Pad10) -> Net-(Q1-D)
- U17 pad 11: unconnected-(U17-CCLK-Pad11) -> Net-(U17-CCLK)
- U17 pad 12: unconnected-(U17-CCKEN#-Pad12) -> Net-(D1-K)
- U17 pad 13: unconnected-(U17-RCLK-Pad13) -> Net-(U15-OUT_1)
- U17 pad 14: unconnected-(U17-OE#-Pad14) -> Net-(D1-K)
- U17 pad 16: unconnected-(U17-V+-Pad16) -> Net-(Q1-D)
- U17 pad 7: unconnected-(U17-Q7-Pad7) -> Net-(U17-Q7)
- U17 pad 8: unconnected-(U17-GND-Pad8) -> Net-(D1-K)
- U17 pad 9: unconnected-(U17-RCO#-Pad9) -> Net-(U17-RCO#)
- U18 pad 1: Net-(U10-GND) -> Net-(D1-K)
- U18 pad 21: Net-(U10-GND) -> Net-(D1-K)
- U18 pad 24: Net-(U10-V+) -> Net-(Q1-D)
- U19 pad 1: Net-(U10-GND) -> Net-(D1-K)
- U19 pad 21: Net-(U10-GND) -> Net-(D1-K)
- U19 pad 24: Net-(U10-V+) -> Net-(Q1-D)
- U2 pad 1: unconnected-(U2-V+-Pad1) -> Net-(Q1-D)
- U2 pad 2: unconnected-(U2-GND-Pad2) -> Net-(D1-K)
- U24 pad 16: unconnected-(U24-V+-Pad16) -> Net-(Q1-D)
- U24 pad 4: Net-(U24-E2#) -> Net-(D1-K)
- U24 pad 5: Net-(U24-E2#) -> Net-(D1-K)
- U24 pad 6: unconnected-(U24-E1-Pad6) -> Net-(U24-E1)
- U24 pad 8: Net-(U24-E2#) -> Net-(D1-K)
- U25 pad 1: unconnected-(U25-Q1-Pad1) -> Net-(U25-Q1)
- U25 pad 10: unconnected-(U25-CCLR#-Pad10) -> Net-(Q1-D)
- U25 pad 11: unconnected-(U25-CCLK-Pad11) -> Net-(U17-CCLK)
- U25 pad 12: unconnected-(U25-CCKEN#-Pad12) -> Net-(U17-RCO#)
- U25 pad 13: unconnected-(U25-RCLK-Pad13) -> Net-(U15-OUT_1)
- U25 pad 14: unconnected-(U25-OE#-Pad14) -> Net-(D1-K)
- U25 pad 15: unconnected-(U25-Q0-Pad15) -> Net-(U25-Q0)
- U25 pad 16: unconnected-(U25-V+-Pad16) -> Net-(Q1-D)
- U25 pad 8: unconnected-(U25-GND-Pad8) -> Net-(D1-K)
- U26 pad 1: Net-(U26-A10) -> Net-(D1-K)
- U26 pad 14: Net-(U26-A10) -> Net-(D1-K)
- U26 pad 2: Net-(U26-A10) -> Net-(D1-K)
- U26 pad 20: unconnected-(U26-CE#-Pad20) -> Net-(D1-K)
- U26 pad 21: Net-(U26-A10) -> Net-(D1-K)
- U26 pad 22: unconnected-(U26-OE#-Pad22) -> Net-(U14-OE#)
- U26 pad 23: Net-(U26-A10) -> Net-(D1-K)
- U26 pad 24: Net-(U26-A10) -> Net-(D1-K)
- U26 pad 25: Net-(U26-A10) -> Net-(D1-K)
- U26 pad 26: Net-(U26-A10) -> Net-(D1-K)
- U26 pad 27: unconnected-(U26-WE#-Pad27) -> Net-(U26-WE#)
- U26 pad 28: unconnected-(U26-V+-Pad28) -> Net-(Q1-D)
- U26 pad 3: Net-(U26-A10) -> Net-(D1-K)
- U26 pad 4: Net-(U26-A10) -> Net-(D1-K)
- U27 pad 1: Net-(U14-D3) -> Net-(U27-D3)
- U27 pad 12: Net-(U14-D7) -> Net-(U27-D7)
- U27 pad 13: Net-(U14-D6) -> Net-(U27-D6)
- U27 pad 14: Net-(U14-D5) -> Net-(U27-D5)
- U27 pad 15: Net-(U14-D4) -> Net-(U27-D4)
- U27 pad 16: unconnected-(U27-V+-Pad16) -> Net-(Q1-D)
- U27 pad 2: Net-(U14-D2) -> Net-(U27-D2)
- U27 pad 3: Net-(U14-D1) -> Net-(U27-D1)
- U27 pad 4: Net-(U14-D0) -> Net-(U27-D0)
- U27 pad 5: unconnected-(U27-Q-Pad5) -> Net-(U27-Q)
- U27 pad 8: unconnected-(U27-GND-Pad8) -> Net-(D1-K)
- U28 pad 1: Net-(U26-D3) -> Net-(U28-D3)
- U28 pad 12: Net-(U26-D7) -> Net-(U28-D7)
- U28 pad 13: Net-(U26-D6) -> Net-(U28-D6)
- U28 pad 14: Net-(U26-D5) -> Net-(U28-D5)
- U28 pad 15: Net-(U26-D4) -> Net-(U28-D4)
- U28 pad 16: unconnected-(U28-V+-Pad16) -> Net-(Q1-D)
- U28 pad 2: Net-(U26-D2) -> Net-(U28-D2)
- U28 pad 3: Net-(U26-D1) -> Net-(U28-D1)
- U28 pad 4: Net-(U26-D0) -> Net-(U28-D0)
- U28 pad 5: unconnected-(U28-Q-Pad5) -> Net-(U28-Q)
- U28 pad 8: unconnected-(U28-GND-Pad8) -> Net-(D1-K)
- U3 pad 1: unconnected-(U3-OE#-Pad1) -> Net-(U3-OE#)
- U3 pad 10: unconnected-(U3-GND-Pad10) -> Net-(D1-K)
- U3 pad 13: unconnected-(U3-Q6-Pad13) -> Net-(U14-A5)
- U3 pad 14: Net-(U14-A5) -> Net-(U14-A4)
- U3 pad 15: Net-(U14-A4) -> Net-(U14-A3)
- U3 pad 16: Net-(U14-A3) -> Net-(U14-A2)
- U3 pad 17: Net-(U14-A2) -> Net-(U14-A1)
- U3 pad 18: Net-(U14-A1) -> Net-(U14-A0)
- U3 pad 19: Net-(U14-A0) -> Net-(U3-Q0)
- U3 pad 20: unconnected-(U3-V+-Pad20) -> Net-(Q1-D)
- U30 pad 10: unconnected-(U30-O4-Pad10) -> Net-(U16-OE#)
- U30 pad 11: unconnected-(U30-I4-Pad11) -> Net-(U30-I4)
- U30 pad 12: unconnected-(U30-O5-Pad12) -> Net-(U30-O5)
- U30 pad 13: unconnected-(U30-I5-Pad13) -> Net-(U30-I5)
- U30 pad 14: unconnected-(U30-V+-Pad14) -> Net-(Q1-D)
- U30 pad 3: unconnected-(U30-I1-Pad3) -> Net-(U15-OUT_1)
- U30 pad 4: unconnected-(U30-O1-Pad4) -> Net-(U30-O1)
- U30 pad 5: unconnected-(U30-I2-Pad5) -> Net-(U30-I2)
- U30 pad 6: unconnected-(U30-O2-Pad6) -> Net-(U14-OE#)
- U30 pad 7: unconnected-(U30-GND-Pad7) -> Net-(D1-K)
- U30 pad 8: unconnected-(U30-03-Pad8) -> Net-(U3-OE#)
- U30 pad 9: unconnected-(U30-I3-Pad9) -> Net-(U30-I3)
- U31 pad 1: unconnected-(U31-OE#-Pad1) -> Net-(U30-I3)
- U31 pad 10: unconnected-(U31-GND-Pad10) -> Net-(D1-K)
- U31 pad 11: Net-(U31-CLK) -> Net-(Q1-D)
- U31 pad 2: unconnected-(U31-D0-Pad2) -> Net-(U17-Q4)
- U31 pad 20: Net-(U31-CLK) -> Net-(Q1-D)
- U31 pad 3: unconnected-(U31-D1-Pad3) -> Net-(U17-Q7)
- U31 pad 4: unconnected-(U31-D2-Pad4) -> Net-(U25-Q0)
- U31 pad 5: unconnected-(U31-D3-Pad5) -> Net-(U25-Q1)
- U31 pad 6: unconnected-(U31-D4-Pad6) -> Net-(U17-Q5)
- U31 pad 7: unconnected-(U31-D5-Pad7) -> Net-(U17-Q6)
- U31 pad 8: unconnected-(U31-D6-Pad8) -> Net-(D1-K)
- U31 pad 9: unconnected-(U31-D7-Pad9) -> Net-(D1-K)
- U32 pad 1: unconnected-(U32-OE#-Pad1) -> Net-(U30-O5)
- U32 pad 10: unconnected-(U32-GND-Pad10) -> Net-(D1-K)
- U32 pad 20: unconnected-(U32-V+-Pad20) -> Net-(Q1-D)
- U4 pad 1: Net-(U10-GND) -> Net-(D1-K)
- U4 pad 21: Net-(U10-GND) -> Net-(D1-K)
- U4 pad 24: Net-(U10-V+) -> Net-(Q1-D)
- U6 pad 1: Net-(U10-GND) -> Net-(D1-K)
- U6 pad 21: Net-(U10-GND) -> Net-(D1-K)
- U6 pad 24: Net-(U10-V+) -> Net-(Q1-D)
- U8 pad 1: Net-(U10-GND) -> Net-(D1-K)
- U8 pad 21: Net-(U10-GND) -> Net-(D1-K)
- U8 pad 24: Net-(U10-V+) -> Net-(Q1-D)
Other:
- board outline added: 436.2 x 400.7 mm

Commit message: LED matrix PCB done
Parts:
- removed the U29 at (366.6, 393.0)
- removed U50: ~, Package_DIP:DIP-14_W7.62mm
- added U34: ~, custom_footprint_library:jumper, F.Cu at (687.1, 478.2)
- moved R6 409.1 mm to (687.1, 134.0), turned to -90 degrees
- moved R9 356.7 mm to (687.1, 195.6), turned to -90 degrees
- moved U6 356.4 mm to (682.6, 144.8)
- moved R5 332.9 mm to (408.9, 130.8), turned to -90 degrees
- moved U42 315.9 mm to (687.1, 470.5)
- moved U41 315.9 mm to (687.1, 462.9)
- moved U40 315.8 mm to (687.1, 455.3)
- moved U39 315.8 mm to (687.1, 447.7)
- moved U38 315.8 mm to (687.1, 440.1)
- moved U37 315.8 mm to (687.1, 432.4)
- moved U36 315.8 mm to (687.1, 424.8)
- moved U35 315.8 mm to (687.1, 417.2)
- moved U8 311.2 mm to (406.4, 198.1)
- moved R11 309.0 mm to (686.4, 254.6), turned to -90 degrees
- moved U10 292.1 mm to (683.3, 205.7)
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Connections:
- R17 pad 1: Net-(U25-Q1) -> Net-(U17-Q7)
- R19 pad 1: Net-(U17-Q7) -> Net-(U25-Q1)
- U17 pad 13: Net-(U15-OUT_1) -> Net-(U17-CCLK)
- U25 pad 13: Net-(U15-OUT_1) -> Net-(U17-CCLK)
- U27 pad 7: Net-(U17-Q3) -> Net-(U27-OE#)
- U28 pad 7: Net-(U28-OE#) -> Net-(U17-Q3)
- U29 pad 1: unconnected-(U29-1A-Pad1) -> Net-(U27-Q)
- U29 pad 11: unconnected-(U29-4Q-Pad11) -> Net-(U29-Q3)
- U29 pad 12: unconnected-(U29-4A-Pad12) -> Net-(U29-3A)
- U29 pad 13: unconnected-(U29-4B-Pad13) -> Net-(U29-3B)
- U29 pad 14: unconnected-(U29-V+-Pad14) -> Net-(Q1-D)
- U29 pad 2: unconnected-(U29-1B-Pad2) -> Net-(U28-Q)
- U29 pad 4: unconnected-(U29-2A-Pad4) -> Net-(U29-Q1)
- U29 pad 5: unconnected-(U29-2B-Pad5) -> Net-(U29-1A)
- U29 pad 6: unconnected-(U29-2Q-Pad6) -> Net-(U29-1B)
- U29 pad 7: unconnected-(U29-GND-Pad7) -> Net-(D1-K)
- U29 pad 8: unconnected-(U29-3Q-Pad8) -> Net-(D1-K)
- U29 pad 9: unconnected-(U29-3A-Pad9) -> Net-(D1-K)
- U30 pad 2: Net-(U28-OE#) -> Net-(U27-OE#)
- U30 pad 3: Net-(U15-OUT_1) -> Net-(U30-I1)
- U33 pad 1: Net-(U25-Q1) -> Net-(U17-Q7)
- U33 pad 3: Net-(U17-Q7) -> Net-(U25-Q1)
- U35 pad 2: Net-(U35-GND) -> Net-(D1-K)
- U36 pad 2: Net-(U35-GND) -> Net-(D1-K)
- U37 pad 2: Net-(U35-GND) -> Net-(D1-K)
- U38 pad 2: Net-(U35-GND) -> Net-(D1-K)
- U39 pad 2: Net-(U35-GND) -> Net-(D1-K)
- U40 pad 2: Net-(U35-GND) -> Net-(D1-K)
- U41 pad 2: Net-(U35-GND) -> Net-(D1-K)
- U42 pad 2: Net-(U35-GND) -> Net-(D1-K)
- U43 pad 2: Net-(U26-D0) -> Net-(U26-D7)
- U43 pad 3: Net-(U26-D1) -> Net-(U26-D6)
- U43 pad 4: Net-(U26-D2) -> Net-(U26-D5)
- U43 pad 5: Net-(U26-D3) -> Net-(U26-D4)
- U43 pad 6: Net-(U26-D4) -> Net-(U26-D3)
- U43 pad 7: Net-(U26-D5) -> Net-(U26-D2)
- U43 pad 8: Net-(U26-D6) -> Net-(U26-D1)
- U43 pad 9: Net-(U26-D7) -> Net-(U26-D0)
- U44 pad 2: Net-(U14-D0) -> Net-(U14-D7)
- U44 pad 3: Net-(U14-D1) -> Net-(U14-D6)
- U44 pad 4: Net-(U14-D2) -> Net-(U14-D5)
- U44 pad 5: Net-(U14-D3) -> Net-(U14-D4)
- U44 pad 6: Net-(U14-D4) -> Net-(U14-D3)
- U44 pad 7: Net-(U14-D5) -> Net-(U14-D2)
- U44 pad 8: Net-(U14-D6) -> Net-(U14-D1)
- U44 pad 9: Net-(U14-D7) -> Net-(U14-D0)
- U45 pad 1: Net-(U30-O1) -> Net-(U30-I1)
- U45 pad 12: Net-(U45-3B) -> Net-(U30-I1)
- U45 pad 4: Net-(U14-WE#) -> Net-(U45-2A)
- U46 pad 2: Net-(U14-WE#) -> Net-(U45-2A)
- U46 pad 4: unconnected-(U46-O1-Pad4) -> Net-(U14-WE#)
- U47 pad 10: Net-(U15-OUT_1) -> Net-(U30-I1)
- U47 pad 5: Net-(U28-OE#) -> Net-(U27-OE#)
- U47 pad 6: Net-(U47-2Q) -> Net-(U29-1A)
- U47 pad 8: Net-(U47-4Q) -> Net-(U29-1B)
- U48 pad 2: Net-(Q1-D) -> Net-(D1-K)
- U49 pad 3: Net-(U49-0CLK) -> Net-(U29-Q1)
- U51 pad 16: Net-(U51-Q3) -> Net-(U45-3A)
- U51 pad 19: Net-(U45-3B) -> Net-(U51-Q0)
- U52 pad 11: Net-(U15-OUT_1) -> Net-(U30-I1)
- U52 pad 16: Net-(U45-3A) -> Net-(U52-Q3)
- U52 pad 2: Net-(U45-3B) -> Net-(U51-Q0)
- U52 pad 5: Net-(U51-Q3) -> Net-(U45-3A)
- U53 pad 10: Net-(U29-3B) -> Net-(U51-D3)
- U53 pad 11: Net-(U51-Q2) -> Net-(U45-3A)
- U53 pad 12: Net-(U51-D3) -> Net-(U52-Q3)
- U53 pad 3: Net-(U45-3B) -> Net-(U51-Q0)
- U53 pad 9: Net-(Q1-D) -> Net-(D1-K)
- U54 pad 1: unconnected-(U54-1A-Pad1) -> Net-(D1-K)
- U54 pad 10: unconnected-(U54-4A-Pad10) -> Net-(D1-K)
- U54 pad 2: unconnected-(U54-1B-Pad2) -> Net-(D1-K)
- U54 pad 4: unconnected-(U54-2A-Pad4) -> Net-(D1-K)
- U54 pad 5: unconnected-(U54-2B-Pad5) -> Net-(D1-K)
- U54 pad 9: unconnected-(U54-4B-Pad9) -> Net-(D1-K)
Routing:
- net Net-(D1-K): track 0.00 -> 1787.7 mm, vias 0 -> 2
- net Net-(Q1-D): track 0.00 -> 1439.5 mm, vias 0 -> 10
- net Net-(U10-CLK): track 0.00 -> 858.6 mm, vias 0 -> 4
- net Net-(U10-D_in): track 0.00 -> 851.8 mm, vias 0 -> 7
- net Net-(U24-Y0): track 0.00 -> 556.0 mm, vias 0 -> 2
- net Net-(U24-Y2): track 0.00 -> 469.2 mm, vias 0 -> 5
- net Net-(U12-LE): track 0.00 -> 396.5 mm, vias 0 -> 1
- net Net-(U17-Q5): track 0.00 -> 381.3 mm, vias 0 -> 4
- net Net-(U36-OUT): track 0.00 -> 355.2 mm, vias 0 -> 2
- net Net-(U18-LE): track 0.00 -> 326.6 mm, vias 0 -> 1
- net Net-(U30-I3): track 0.00 -> 289.6 mm, vias 0 -> 1
- net Net-(U30-I1): track 0.00 -> 285.1 mm, vias 0 -> 3
- net Net-(U3-Q0): track 0.00 -> 284.6 mm, vias 0 -> 6
- net Net-(U17-Q6): track 0.00 -> 279.1 mm, vias 0 -> 1
- net Net-(U3-OE#): track 0.00 -> 278.3 mm, vias 0 -> 3
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- added copper zone on B.Cu, net Net-(D1-K)
- added copper zone on F.Cu, net Net-(Q1-D)
Other:
- board size 436.2 x 400.7 mm -> 315.6 x 367 mm
- board text added: "Row activation"

Commit message: Added failsafe to LED matrix and some other stuff
Connections:
- U35 pad 3: Net-(U30-I2) -> Net-(U35-OUT)
- U41 pad 3: Net-(U30-I3) -> Net-(U41-OUT)
- U46 pad 10: unconnected-(U46-O4-Pad10) -> Net-(U46-O4)
- U46 pad 11: Net-(D1-K) -> Net-(U46-I4)
- U54 pad 1: Net-(D1-K) -> Net-(U35-OUT)
- U54 pad 10: Net-(D1-K) -> Net-(U46-O4)
- U54 pad 2: Net-(D1-K) -> Net-(U41-OUT)
- U54 pad 3: unconnected-(U54-1Q-Pad3) -> Net-(U46-I4)
- U54 pad 4: Net-(D1-K) -> Net-(U46-O4)
- U54 pad 5: Net-(D1-K) -> Net-(U41-OUT)
- U54 pad 6: unconnected-(U54-2Q-Pad6) -> Net-(U30-I3)
- U54 pad 8: unconnected-(U54-4Q-Pad8) -> Net-(U30-I2)
- U54 pad 9: Net-(D1-K) -> Net-(U35-OUT)
Routing:
- net Net-(U46-O4): track 0.00 -> 174.8 mm, vias 0 -> 10
- net Net-(U46-I4): track 0.00 -> 166.4 mm, vias 0 -> 9
- net Net-(U35-OUT): track 0.00 -> 134.5 mm, vias 0 -> 4
- net Net-(U41-OUT): track 0.00 -> 108.3 mm, vias 0 -> 2
- net Net-(U30-I2): track 98.0 -> 24.2 mm, vias 1 -> 0
- net Net-(U30-I3): track 289.6 -> 259.7 mm, vias 1 -> 4
- net Net-(D1-K): track 1787.7 -> 1762.1 mm
- net Net-(U17-Q0): track 92.5 -> 90.0 mm
- net Net-(U29-1A): track 131.9 -> 132.9 mm
- net Net-(U3-OE#): track 278.3 -> 277.3 mm

Commit message: Improved readme
Parts:
- removed C1: C, Capacitor_THT:CP_Radial_D4.0mm_P2.00mm
- removed D1, D2, D3: LED, LED_THT:LED_D3.0mm
- removed R1, R17, R18, R19, R2, R3, R4: R, custom_footprint_library:0.4_pitch_resistor
- removed U14, U26: ~, Package_DIP:DIP-28_W15.24mm
- removed U15, U29, U30, U45, U46, U47, U48, U49, U53, U54: ~, Package_DIP:DIP-14_W7.62mm
- removed U16, U3, U31, U32, U43, U44, U51, U52: ~, Package_DIP:DIP-20_W7.62mm
- removed U17, U25, U27, U28: ~, Package_DIP:DIP-16_W7.62mm
- removed U2: ~, Connector_PinHeader_2.54mm:PinHeader_1x03_P2.54mm_Vertical
- removed U34, U35, U36, U37, U38, U39, U40, U41, U42: ~, custom_footprint_library:jumper
- U1: footprint Connector_PinHeader_2.54mm:PinHeader_1x16_P2.54mm_Vertical -> Connector_PinHeader_2.54mm:PinHeader_1x13_P2.54mm_Vertical
- moved U1 266.1 mm to (664.9, 403.9), turned to 90 degrees
- moved U33 77.6 mm to (617.9, 405.1)
- moved R20 66.3 mm to (639.4, 400.1), turned to 0 degrees
- moved SW1 54.4 mm to (645.2, 404.5)
Connections:
- R10 pad 2: Net-(D1-K) -> Net-(U10-GND)
- R11 pad 2: Net-(D1-K) -> Net-(U10-GND)
- R12 pad 2: Net-(D1-K) -> Net-(U10-GND)
- R13 pad 2: Net-(D1-K) -> Net-(U10-GND)
- R20 pad 2: Net-(D1-K) -> Net-(U10-GND)
- R5 pad 2: Net-(D1-K) -> Net-(U10-GND)
- R6 pad 2: Net-(D1-K) -> Net-(U10-GND)
- R8 pad 2: Net-(D1-K) -> Net-(U10-GND)
- R9 pad 2: Net-(D1-K) -> Net-(U10-GND)
- U1 pad 1: Net-(U1-0) -> Net-(Q1-D)
- U1 pad 10: Net-(U1-9) -> Net-(U1-Row_A1)
- U1 pad 11: Net-(U1-10) -> Net-(U1-Row_A2)
- U1 pad 12: Net-(U1-11) -> Net-(U10-GND)
- U1 pad 13: Net-(U1-12) -> Net-(U10-GND)
- U1 pad 2: Net-(U1-1) -> Net-(Q1-D)
- U1 pad 3: Net-(U1-2) -> Net-(U1-Data)
- U1 pad 4: Net-(U1-3) -> Net-(U1-CLK)
- U1 pad 5: Net-(U1-4) -> Net-(U1-Driver_LE)
- U1 pad 6: Net-(U1-5) -> Net-(U1-Driver_A0)
- U1 pad 7: Net-(U1-6) -> Net-(U1-Driver_A1)
- U1 pad 8: Net-(U1-7) -> Net-(U1-Driver_A2)
- U1 pad 9: Net-(U1-8) -> Net-(U1-Row_A0)
- U10 pad 1: Net-(D1-K) -> Net-(U10-GND)
- U10 pad 2: Net-(U10-D_in) -> Net-(U1-Data)
- U10 pad 21: Net-(D1-K) -> Net-(U10-GND)
- U10 pad 3: Net-(U10-CLK) -> Net-(U1-CLK)
- U12 pad 1: Net-(D1-K) -> Net-(U10-GND)
- U12 pad 2: Net-(U10-D_in) -> Net-(U1-Data)
- U12 pad 21: Net-(D1-K) -> Net-(U10-GND)
- U12 pad 3: Net-(U10-CLK) -> Net-(U1-CLK)
- U13 pad 1: Net-(D1-K) -> Net-(U10-GND)
- U13 pad 2: Net-(U10-D_in) -> Net-(U1-Data)
- U13 pad 21: Net-(D1-K) -> Net-(U10-GND)
- U13 pad 3: Net-(U10-CLK) -> Net-(U1-CLK)
- U18 pad 1: Net-(D1-K) -> Net-(U10-GND)
- U18 pad 2: Net-(U10-D_in) -> Net-(U1-Data)
- U18 pad 21: Net-(D1-K) -> Net-(U10-GND)
- U18 pad 3: Net-(U10-CLK) -> Net-(U1-CLK)
- U19 pad 1: Net-(D1-K) -> Net-(U10-GND)
- U19 pad 2: Net-(U10-D_in) -> Net-(U1-Data)
- U19 pad 21: Net-(D1-K) -> Net-(U10-GND)
- U19 pad 3: Net-(U10-CLK) -> Net-(U1-CLK)
- U24 pad 1: Net-(U17-Q4) -> Net-(U1-Driver_A0)
- U24 pad 2: Net-(U17-Q5) -> Net-(U1-Driver_A1)
- U24 pad 3: Net-(U17-Q6) -> Net-(U1-Driver_A2)
- U24 pad 4: Net-(D1-K) -> Net-(U10-GND)
- U24 pad 5: Net-(D1-K) -> Net-(U10-GND)
- U24 pad 6: Net-(U24-E1) -> Net-(U1-Driver_LE)
- U24 pad 8: Net-(D1-K) -> Net-(U10-GND)
- U33 pad 1: Net-(U17-Q7) -> Net-(U1-Row_A0)
- U33 pad 2: Net-(U25-Q0) -> Net-(U1-Row_A1)
- U33 pad 3: Net-(U25-Q1) -> Net-(U1-Row_A2)
- U33 pad 4: Net-(D1-K) -> Net-(U10-GND)
- U33 pad 5: Net-(D1-K) -> Net-(U10-GND)
- U33 pad 8: Net-(D1-K) -> Net-(U10-GND)
- U4 pad 1: Net-(D1-K) -> Net-(U10-GND)
- U4 pad 2: Net-(U10-D_in) -> Net-(U1-Data)
- U4 pad 21: Net-(D1-K) -> Net-(U10-GND)
- U4 pad 3: Net-(U10-CLK) -> Net-(U1-CLK)
- U6 pad 1: Net-(D1-K) -> Net-(U10-GND)
- U6 pad 2: Net-(U10-D_in) -> Net-(U1-Data)
- U6 pad 21: Net-(D1-K) -> Net-(U10-GND)
- U6 pad 3: Net-(U10-CLK) -> Net-(U1-CLK)
- U8 pad 1: Net-(D1-K) -> Net-(U10-GND)
- U8 pad 2: Net-(U10-D_in) -> Net-(U1-Data)
- U8 pad 21: Net-(D1-K) -> Net-(U10-GND)
- U8 pad 3: Net-(U10-CLK) -> Net-(U1-CLK)
Routing:
- net Net-(D1-K): track 1762.1 -> 0.00 mm, vias 2 -> 0
- net Net-(U10-GND): track 0.00 -> 1286.9 mm, vias 0 -> 7
- net Net-(U10-CLK): track 858.6 -> 0.00 mm, vias 4 -> 0
- net Net-(U10-D_in): track 851.8 -> 0.00 mm, vias 7 -> 0
- net Net-(U1-CLK): track 0.00 -> 819.9 mm, vias 0 -> 5
- net Net-(U1-Data): track 0.00 -> 806.3 mm, vias 0 -> 8
- net Net-(Q1-D): track 1439.5 -> 973.0 mm, vias 10 -> 7
- net Net-(U17-Q5): track 381.3 -> 0.00 mm, vias 4 -> 0
- net Net-(U36-OUT): track 355.2 -> 0.00 mm, vias 2 -> 0
- net Net-(U30-I1): track 285.1 -> 0.00 mm, vias 3 -> 0
- net Net-(U3-Q0): track 284.6 -> 0.00 mm, vias 6 -> 0
- net Net-(U17-Q6): track 279.1 -> 0.00 mm, vias 1 -> 0
- net Net-(U17-CCLK): track 278.3 -> 0.00 mm, vias 3 -> 0
- net Net-(U14-OE#): track 277.9 -> 0.00 mm, vias 6 -> 0
- net Net-(U3-OE#): track 277.3 -> 0.00 mm, vias 3 -> 0
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- removed copper zone on B.Cu, net Net-(D1-K)
- removed copper zone on F.Cu, net Net-(Q1-D)
Other:
- board size 315.6 x 367 mm -> 314.3 x 295.3 mm
- board text removed: "Row activation"
