File: kicad/version_2/led_matrix/led_matrix.kicad_pcb (KiCad board)
At the start: 2 copper layers, 314.3 x 295.3 mm, 37 parts, among them Q1 IRF540N, Q2 IRF540N, Q3 IRF540N, Q4 IRF540N, Q5 IRF540N, Q6 IRF540N, Q7 IRF540N, Q9 IRF540N, SW1 SW_DIP_x01

Commit message: Fixed led matrix board
Parts:
- moved U24 17.9 mm to (672.5, 394.3), turned to 90 degrees
- moved R5 3.42 mm to (412.1, 129.5)
- moved R13 2.84 mm to (685.2, 318.1)
- moved R11 2.84 mm to (685.2, 257.2)
- moved U19 2.84 mm to (682.6, 327.7)
- moved R6 2.29 mm to (685.2, 135.3)
- moved R9 2.01 mm to (685.2, 196.2)
- moved R8 2.01 mm to (412.1, 190.5)
- moved U12 2.01 mm to (407.0, 261.0)
- moved U4 2.01 mm to (407.0, 139.1)
- moved U8 2.01 mm to (407.0, 200.0)
- moved U18 2.01 mm to (407.0, 321.9)
- moved U13 1.90 mm to (682.6, 266.7)
- moved R12 1.42 mm to (412.1, 312.4)
- moved R10 1.42 mm to (412.1, 251.5)
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Connections:
- U10 pad 3: Net-(U1-CLK) -> Net-(U10-CLK)
- U10 pad 4: Net-(U10-LE) -> Net-(U1-Driver_LE)
- U12 pad 3: Net-(U1-CLK) -> Net-(U12-CLK)
- U12 pad 4: Net-(U12-LE) -> Net-(U1-Driver_LE)
- U13 pad 3: Net-(U1-CLK) -> Net-(U13-CLK)
- U13 pad 4: Net-(U13-LE) -> Net-(U1-Driver_LE)
- U18 pad 3: Net-(U1-CLK) -> Net-(U18-CLK)
- U18 pad 4: Net-(U18-LE) -> Net-(U1-Driver_LE)
- U19 pad 3: Net-(U1-CLK) -> Net-(U19-CLK)
- U19 pad 4: Net-(U19-LE) -> Net-(U1-Driver_LE)
- U24 pad 10: Net-(U13-LE) -> Net-(U13-CLK)
- U24 pad 11: Net-(U12-LE) -> Net-(U12-CLK)
- U24 pad 12: Net-(U10-LE) -> Net-(U10-CLK)
- U24 pad 6: Net-(U1-Driver_LE) -> Net-(U1-CLK)
- U24 pad 7: Net-(U19-LE) -> Net-(U19-CLK)
- U24 pad 9: Net-(U18-LE) -> Net-(U18-CLK)
- U4 pad 3: Net-(U1-CLK) -> Net-(U24-Y0)
- U4 pad 4: Net-(U24-Y0) -> Net-(U1-Driver_LE)
- U6 pad 3: Net-(U1-CLK) -> Net-(U24-Y1)
- U6 pad 4: Net-(U24-Y1) -> Net-(U1-Driver_LE)
- U8 pad 3: Net-(U1-CLK) -> Net-(U24-Y2)
- U8 pad 4: Net-(U24-Y2) -> Net-(U1-Driver_LE)
Routing:
- net Net-(U1-Driver_LE): track 32.0 -> 876.7 mm, vias 0 -> 10
- net Net-(U1-CLK): track 819.9 -> 19.2 mm, vias 5 -> 1
- net Net-(U10-GND): track 1286.9 -> 1898.5 mm, vias 7 -> 10
- net Net-(U12-CLK): track 0.00 -> 399.4 mm, vias 0 -> 3
- net Net-(U12-LE): track 396.5 -> 0.00 mm, vias 1 -> 0
- net Net-(U18-CLK): track 0.00 -> 336.1 mm, vias 0 -> 2
- net Net-(U18-LE): track 326.6 -> 0.00 mm, vias 1 -> 0
- net Net-(U10-LE): track 219.4 -> 0.00 mm, vias 2 -> 0
- net Net-(U10-CLK): track 0.00 -> 180.1 mm, vias 0 -> 1
- net Net-(U13-LE): track 154.9 -> 0.00 mm, vias 3 -> 0
- net Net-(U13-CLK): track 0.00 -> 117.0 mm
- net Net-(U1-Data): track 806.3 -> 923.0 mm, vias 8 -> 17
- net Net-(U19-CLK): track 0.00 -> 82.5 mm
- net Net-(Q1-D): track 973.0 -> 1040.6 mm, vias 7 -> 12
- net Net-(U19-LE): track 57.8 -> 0.00 mm
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Other:
- board size 314.3 x 295.3 mm -> 301.6 x 295.3 mm

Commit message: Added new led matrix board for the 8x8 displays
Parts:
- removed R10, R11, R12, R13, R9: R, custom_footprint_library:0.4_pitch_resistor
- added R1: R, custom_footprint_library:0.4_pitch_resistor, F.Cu at (623.0, 138.1)
- added R2: R, custom_footprint_library:0.4_pitch_resistor, F.Cu at (419.0, 170.1)
- added R3: R, custom_footprint_library:0.4_pitch_resistor, F.Cu at (623.0, 170.1)
- added R4: R, custom_footprint_library:0.4_pitch_resistor, F.Cu at (419.0, 202.1)
- added R7: R, custom_footprint_library:0.4_pitch_resistor, F.Cu at (419.0, 234.1)
- added U14: ~, Package_DIP:DIP-24_W7.62mm, F.Cu at (424.1, 205.6)
- added U15: ~, Package_DIP:DIP-24_W7.62mm, F.Cu at (617.9, 198.0)
- added U16: ~, custom_footprint_library:8_x_8_led_matrix_KWM-30881CVB, F.Cu at (505.0, 202.0)
- added U17: ~, custom_footprint_library:8_x_8_led_matrix_KWM-30881CVB, F.Cu at (569.0, 202.0)
- added U2: ~, custom_footprint_library:8_x_8_led_matrix_KWM-30881CVB, F.Cu at (505.0, 138.0)
- added U25: ~, custom_footprint_library:8_x_8_led_matrix_KWM-30881CVB, F.Cu at (473.0, 234.0)
- added U26: ~, custom_footprint_library:8_x_8_led_matrix_KWM-30881CVB, F.Cu at (537.0, 234.0)
- added U3: ~, custom_footprint_library:8_x_8_led_matrix_KWM-30881CVB, F.Cu at (473.0, 138.0)
- U10, U12, U13, U18, U19, U6: footprint Package_DIP:DIP-24_W7.62mm -> custom_footprint_library:8_x_8_led_matrix_KWM-30881CVB
- U11, U7: footprint custom_footprint_library:led_block_16_x_8_left -> custom_footprint_library:8_x_8_led_matrix_KWM-30881CVB
- U20, U21: footprint custom_footprint_library:led_block_16_x_8_right -> Package_DIP:DIP-24_W7.62mm
- U22, U23: footprint custom_footprint_library:led_block_16_x_8_right -> custom_footprint_library:8_x_8_led_matrix_KWM-30881CVB
- U5, U9: footprint custom_footprint_library:led_block_16_x_8_left -> Package_DIP:DIP-24_W7.62mm
- moved R8 215.3 mm to (623.0, 234.1), turned to 180 degrees
- moved U20 208.6 mm to (424.1, 237.6), turned to 90 degrees
- moved U19 192.3 mm to (537.0, 202.0), turned to -90 degrees
- moved U11 184.5 mm to (569.0, 170.0), turned to -90 degrees
- moved U10 181.2 mm to (505.0, 170.0), turned to -90 degrees
- moved U13 174.8 mm to (537.0, 170.0), turned to -90 degrees
- moved U9 168.8 mm to (617.9, 166.0), turned to -90 degrees
- moved SW1 158.0 mm to (549.3, 278.9)
- moved R20 155.9 mm to (542.9, 277.6)
- moved U33 155.7 mm to (535.3, 273.1), turned to -90 degrees
- moved U1 155.0 mm to (569.0, 282.0)
- moved Q5 153.7 mm to (446.4, 272.5)
- moved Q1 153.7 mm to (494.7, 272.5)
- moved Q3 153.7 mm to (470.5, 272.5)
- moved Q6 153.7 mm to (434.3, 272.5)
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Connections:
- R20 pad 2: Net-(U10-GND) -> Net-(U14-GND)
- R5 pad 2: Net-(U10-GND) -> Net-(U14-GND)
- R6 pad 1: Net-(U6-SET) -> Net-(U15-SET)
- R6 pad 2: Net-(U10-GND) -> Net-(U14-GND)
- R8 pad 1: Net-(U8-SET) -> Net-(U21-SET)
- R8 pad 2: Net-(U10-GND) -> Net-(U14-GND)
- U1 pad 12: Net-(U10-GND) -> Net-(U14-GND)
- U1 pad 13: Net-(U10-GND) -> Net-(U14-GND)
- U10 pad 1: Net-(U10-GND) -> Net-(U10-R4)
- U10 pad 10: Net-(U10-O5) -> Net-(Q3-S)
- U10 pad 11: Net-(U10-O6) -> Net-(Q5-S)
- U10 pad 12: Net-(U10-O7) -> Net-(U10-R3)
- U10 pad 13: Net-(U10-O8) -> Net-(Q9-S)
- U10 pad 14: Net-(U10-O9) -> Net-(U10-R1)
- U10 pad 15: Net-(U10-O10) -> Net-(Q6-S)
- U10 pad 16: Net-(U10-O11) -> Net-(Q7-S)
- U10 pad 2: Net-(U1-Data) -> Net-(U10-R6)
- U10 pad 3: Net-(U10-CLK) -> Net-(Q1-S)
- U10 pad 4: Net-(U1-Driver_LE) -> Net-(Q2-S)
- U10 pad 5: Net-(U10-O0) -> Net-(U10-R7)
- U10 pad 6: Net-(U10-O1) -> Net-(Q4-S)
- U10 pad 7: Net-(U10-O2) -> Net-(U10-R5)
- U10 pad 8: Net-(U10-O3) -> Net-(U10-R2)
- U10 pad 9: Net-(U10-O4) -> Net-(U10-R0)
- U11 pad 1: Net-(U11-C0) -> Net-(U11-R4)
- U11 pad 10: Net-(U11-C9) -> Net-(Q3-S)
- U11 pad 11: Net-(U11-C10) -> Net-(Q5-S)
- U11 pad 12: Net-(U11-C11) -> Net-(U11-R3)
- U11 pad 13: Net-(U11-C12) -> Net-(Q9-S)
- U11 pad 14: Net-(U11-C13) -> Net-(U11-R1)
- U11 pad 15: Net-(U11-C14) -> Net-(Q6-S)
- U11 pad 16: Net-(U11-C15) -> Net-(Q7-S)
- U11 pad 2: Net-(U11-C1) -> Net-(U11-R6)
- U11 pad 3: Net-(U11-C2) -> Net-(Q1-S)
- U11 pad 4: Net-(U11-C3) -> Net-(Q2-S)
- U11 pad 5: Net-(U11-C4) -> Net-(U11-R7)
- U11 pad 6: Net-(U11-C5) -> Net-(Q4-S)
- U11 pad 7: Net-(U11-C6) -> Net-(U11-R5)
- U11 pad 8: Net-(U11-C7) -> Net-(U11-R2)
- U11 pad 9: Net-(U11-C8) -> Net-(U11-R0)
- U12 pad 1: Net-(U10-GND) -> Net-(U12-R4)
- U12 pad 10: Net-(U12-O5) -> Net-(Q3-S)
- U12 pad 11: Net-(U12-O6) -> Net-(Q5-S)
- U12 pad 12: Net-(U12-O7) -> Net-(U12-R3)
- U12 pad 13: Net-(U12-O8) -> Net-(Q9-S)
- U12 pad 14: Net-(U12-O9) -> Net-(U12-R1)
- U12 pad 15: Net-(U12-O10) -> Net-(Q6-S)
- U12 pad 16: Net-(U12-O11) -> Net-(Q7-S)
- U12 pad 2: Net-(U1-Data) -> Net-(U12-R6)
- U12 pad 3: Net-(U12-CLK) -> Net-(Q1-S)
- U12 pad 4: Net-(U1-Driver_LE) -> Net-(Q2-S)
- U12 pad 5: Net-(U12-O0) -> Net-(U12-R7)
- U12 pad 6: Net-(U12-O1) -> Net-(Q4-S)
- U12 pad 7: Net-(U12-O2) -> Net-(U12-R5)
- U12 pad 8: Net-(U12-O3) -> Net-(U12-R2)
- U12 pad 9: Net-(U12-O4) -> Net-(U12-R0)
- U13 pad 1: Net-(U10-GND) -> Net-(U13-R4)
- U13 pad 10: Net-(U13-O5) -> Net-(Q3-S)
- U13 pad 11: Net-(U13-O6) -> Net-(Q5-S)
- U13 pad 12: Net-(U13-O7) -> Net-(U13-R3)
- U13 pad 13: Net-(U13-O8) -> Net-(Q9-S)
- U13 pad 14: Net-(U13-O9) -> Net-(U13-R1)
- U13 pad 15: Net-(U13-O10) -> Net-(Q6-S)
- U13 pad 16: Net-(U13-O11) -> Net-(Q7-S)
- U13 pad 2: Net-(U1-Data) -> Net-(U13-R6)
- U13 pad 3: Net-(U13-CLK) -> Net-(Q1-S)
- U13 pad 4: Net-(U1-Driver_LE) -> Net-(Q2-S)
- U13 pad 5: Net-(U13-O0) -> Net-(U13-R7)
- U13 pad 6: Net-(U13-O1) -> Net-(Q4-S)
- U13 pad 7: Net-(U13-O2) -> Net-(U13-R5)
- U13 pad 8: Net-(U13-O3) -> Net-(U13-R2)
- U13 pad 9: Net-(U13-O4) -> Net-(U13-R0)
- U18 pad 1: Net-(U10-GND) -> Net-(U14-O3)
- U18 pad 10: Net-(U11-C5) -> Net-(Q3-S)
- U18 pad 11: Net-(U11-C6) -> Net-(Q5-S)
- U18 pad 12: Net-(U11-C7) -> Net-(U14-O4)
- U18 pad 13: Net-(U11-C8) -> Net-(Q9-S)
- U18 pad 14: Net-(U11-C9) -> Net-(U14-O6)
- U18 pad 15: Net-(U11-C10) -> Net-(Q6-S)
- U18 pad 16: Net-(U11-C11) -> Net-(Q7-S)
- U18 pad 2: Net-(U1-Data) -> Net-(U14-O1)
- U18 pad 3: Net-(U18-CLK) -> Net-(Q1-S)
- U18 pad 4: Net-(U1-Driver_LE) -> Net-(Q2-S)
- U18 pad 5: Net-(U11-C0) -> Net-(U14-O0)
- U18 pad 6: Net-(U11-C1) -> Net-(Q4-S)
- U18 pad 7: Net-(U11-C2) -> Net-(U14-O2)
- U18 pad 8: Net-(U11-C3) -> Net-(U14-O5)
- U18 pad 9: Net-(U11-C4) -> Net-(U14-O7)
- U19 pad 1: Net-(U10-GND) -> Net-(U15-O3)
- U19 pad 10: Net-(U19-O5) -> Net-(Q3-S)
- U19 pad 11: Net-(U19-O6) -> Net-(Q5-S)
- U19 pad 12: Net-(U19-O7) -> Net-(U15-O4)
- U19 pad 13: Net-(U19-O8) -> Net-(Q9-S)
- U19 pad 14: Net-(U19-O9) -> Net-(U15-O6)
- U19 pad 15: Net-(U19-O10) -> Net-(Q6-S)
- U19 pad 16: Net-(U19-O11) -> Net-(Q7-S)
- U19 pad 2: Net-(U1-Data) -> Net-(U15-O1)
- U19 pad 3: Net-(U19-CLK) -> Net-(Q1-S)
- U19 pad 4: Net-(U1-Driver_LE) -> Net-(Q2-S)
- U19 pad 5: Net-(U19-O0) -> Net-(U15-O0)
- U19 pad 6: Net-(U19-O1) -> Net-(Q4-S)
- U19 pad 7: Net-(U19-O2) -> Net-(U15-O2)
- U19 pad 8: Net-(U19-O3) -> Net-(U15-O5)
- U19 pad 9: Net-(U19-O4) -> Net-(U15-O7)
- U20 pad 1: Net-(U20-C0) -> Net-(U14-GND)
- U20 pad 10: Net-(U20-C9) -> Net-(U20-O5)
- U20 pad 11: Net-(U20-C10) -> Net-(U20-O6)
- U20 pad 12: Net-(U20-C11) -> Net-(U20-O7)
- U20 pad 13: Net-(U20-C12) -> Net-(U20-O8)
- U20 pad 14: Net-(U20-C13) -> Net-(U20-O9)
- U20 pad 15: Net-(U20-C14) -> Net-(U20-O10)
- U20 pad 16: Net-(U20-C15) -> Net-(U20-O11)
- U20 pad 17: Net-(Q9-S) -> Net-(U20-O12)
- U20 pad 18: Net-(Q1-S) -> Net-(U20-O13)
- U20 pad 19: Net-(Q2-S) -> Net-(U20-O14)
- U20 pad 2: Net-(U20-C1) -> Net-(U1-Data)
- U20 pad 20: Net-(Q3-S) -> Net-(U20-O15)
- U20 pad 21: Net-(Q4-S) -> Net-(U14-GND)
- U20 pad 22: Net-(Q5-S) -> unconnected-(U20-D_out-Pad22)
- U20 pad 23: Net-(Q6-S) -> Net-(U20-SET)
- U20 pad 24: Net-(Q7-S) -> Net-(Q1-D)
- U20 pad 3: Net-(U20-C2) -> Net-(U20-CLK)
- U20 pad 4: Net-(U20-C3) -> Net-(U1-Driver_LE)
- U20 pad 5: Net-(U20-C4) -> Net-(U20-O0)
- U20 pad 6: Net-(U20-C5) -> Net-(U20-O1)
- U20 pad 7: Net-(U20-C6) -> Net-(U20-O2)
- U20 pad 8: Net-(U20-C7) -> Net-(U20-O3)
- U20 pad 9: Net-(U20-C8) -> Net-(U20-O4)
- U21 pad 1: Net-(U10-O0) -> Net-(U14-GND)
- U21 pad 10: Net-(U10-O9) -> Net-(U21-O5)
- U21 pad 11: Net-(U10-O10) -> Net-(U21-O6)
- U21 pad 12: Net-(U10-O11) -> Net-(U21-O7)
- U21 pad 13: Net-(U10-O12) -> Net-(U21-O8)
- U21 pad 14: Net-(U10-O13) -> Net-(U21-O9)
- U21 pad 15: Net-(U10-O14) -> Net-(U21-O10)
- U21 pad 16: Net-(U10-O15) -> Net-(U21-O11)
- U21 pad 17: Net-(Q9-S) -> Net-(U21-O12)
- U21 pad 18: Net-(Q1-S) -> Net-(U21-O13)
- U21 pad 19: Net-(Q2-S) -> Net-(U21-O14)
- U21 pad 2: Net-(U10-O1) -> Net-(U1-Data)
- U21 pad 20: Net-(Q3-S) -> Net-(U21-O15)
- U21 pad 21: Net-(Q4-S) -> Net-(U14-GND)
- U21 pad 22: Net-(Q5-S) -> unconnected-(U21-D_out-Pad22)
- U21 pad 23: Net-(Q6-S) -> Net-(U21-SET)
- U21 pad 24: Net-(Q7-S) -> Net-(Q1-D)
- U21 pad 3: Net-(U10-O2) -> Net-(U21-CLK)
- U21 pad 4: Net-(U10-O3) -> Net-(U1-Driver_LE)
- U21 pad 5: Net-(U10-O4) -> Net-(U21-O0)
- U21 pad 6: Net-(U10-O5) -> Net-(U21-O1)
- U21 pad 7: Net-(U10-O6) -> Net-(U21-O2)
- U21 pad 8: Net-(U10-O7) -> Net-(U21-O3)
- U21 pad 9: Net-(U10-O8) -> Net-(U21-O4)
- U22 pad 1: Net-(U13-O0) -> Net-(U20-O11)
- U22 pad 10: Net-(U13-O9) -> Net-(Q3-S)
- U22 pad 11: Net-(U13-O10) -> Net-(Q5-S)
- U22 pad 12: Net-(U13-O11) -> Net-(U20-O12)
- U22 pad 13: Net-(U13-O12) -> Net-(Q9-S)
- U22 pad 14: Net-(U13-O13) -> Net-(U20-O14)
- U22 pad 15: Net-(U13-O14) -> Net-(Q6-S)
- U22 pad 16: Net-(U13-O15) -> Net-(Q7-S)
- U22 pad 2: Net-(U13-O1) -> Net-(U20-O9)
- U22 pad 3: Net-(U13-O2) -> Net-(Q1-S)
- U22 pad 4: Net-(U13-O3) -> Net-(Q2-S)
- U22 pad 5: Net-(U13-O4) -> Net-(U20-O8)
- U22 pad 6: Net-(U13-O5) -> Net-(Q4-S)
- U22 pad 7: Net-(U13-O6) -> Net-(U20-O10)
- U22 pad 8: Net-(U13-O7) -> Net-(U20-O13)
- U22 pad 9: Net-(U13-O8) -> Net-(U20-O15)
- U23 pad 1: Net-(U19-O0) -> Net-(U21-O11)
- U23 pad 10: Net-(U19-O9) -> Net-(Q3-S)
- U23 pad 11: Net-(U19-O10) -> Net-(Q5-S)
- U23 pad 12: Net-(U19-O11) -> Net-(U21-O12)
- U23 pad 13: Net-(U19-O12) -> Net-(Q9-S)
- U23 pad 14: Net-(U19-O13) -> Net-(U21-O14)
- U23 pad 15: Net-(U19-O14) -> Net-(Q6-S)
- U23 pad 16: Net-(U19-O15) -> Net-(Q7-S)
- U23 pad 2: Net-(U19-O1) -> Net-(U21-O9)
- U23 pad 3: Net-(U19-O2) -> Net-(Q1-S)
- U23 pad 4: Net-(U19-O3) -> Net-(Q2-S)
- U23 pad 5: Net-(U19-O4) -> Net-(U21-O8)
- U23 pad 6: Net-(U19-O5) -> Net-(Q4-S)
- U23 pad 7: Net-(U19-O6) -> Net-(U21-O10)
- U23 pad 8: Net-(U19-O7) -> Net-(U21-O13)
- U23 pad 9: Net-(U19-O8) -> Net-(U21-O15)
- U24 pad 10: Net-(U13-CLK) -> Net-(U15-CLK)
- U24 pad 11: Net-(U12-CLK) -> Net-(U14-CLK)
- U24 pad 12: Net-(U10-CLK) -> Net-(U24-Y3)
- U24 pad 4: Net-(U10-GND) -> Net-(U14-GND)
- U24 pad 5: Net-(U10-GND) -> Net-(U14-GND)
- U24 pad 7: Net-(U19-CLK) -> Net-(U21-CLK)
- U24 pad 8: Net-(U10-GND) -> Net-(U14-GND)
- U24 pad 9: Net-(U18-CLK) -> Net-(U20-CLK)
- U33 pad 4: Net-(U10-GND) -> Net-(U14-GND)
- U33 pad 5: Net-(U10-GND) -> Net-(U14-GND)
- U33 pad 8: Net-(U10-GND) -> Net-(U14-GND)
- U4 pad 1: Net-(U10-GND) -> Net-(U14-GND)
- U4 pad 10: Net-(U4-O5) -> Net-(U3-R2)
- U4 pad 11: Net-(U4-O6) -> Net-(U3-R1)
- U4 pad 12: Net-(U4-O7) -> Net-(U3-R0)
- U4 pad 13: Net-(U4-O8) -> Net-(U2-R7)
- U4 pad 14: Net-(U4-O9) -> Net-(U2-R6)
- U4 pad 15: Net-(U4-O10) -> Net-(U2-R5)
- U4 pad 16: Net-(U4-O11) -> Net-(U2-R4)
- U4 pad 17: Net-(U4-O12) -> Net-(U2-R3)
- U4 pad 18: Net-(U4-O13) -> Net-(U2-R2)
- U4 pad 19: Net-(U4-O14) -> Net-(U2-R1)
- U4 pad 20: Net-(U4-O15) -> Net-(U2-R0)
- U4 pad 21: Net-(U10-GND) -> Net-(U14-GND)
- U4 pad 5: Net-(U4-O0) -> Net-(U3-R7)
- U4 pad 6: Net-(U4-O1) -> Net-(U3-R6)
- U4 pad 7: Net-(U4-O2) -> Net-(U3-R5)
- U4 pad 8: Net-(U4-O3) -> Net-(U3-R4)
- U4 pad 9: Net-(U4-O4) -> Net-(U3-R3)
- U5 pad 1: Net-(U4-O0) -> Net-(U14-GND)
- U5 pad 10: Net-(U4-O9) -> Net-(U5-O5)
- U5 pad 11: Net-(U4-O10) -> Net-(U5-O6)
- U5 pad 12: Net-(U4-O11) -> Net-(U5-O7)
- U5 pad 13: Net-(U4-O12) -> Net-(U5-O8)
- U5 pad 14: Net-(U4-O13) -> Net-(U5-O9)
- U5 pad 15: Net-(U4-O14) -> Net-(U5-O10)
- U5 pad 16: Net-(U4-O15) -> Net-(U5-O11)
- U5 pad 17: Net-(Q9-S) -> Net-(U5-O12)
- U5 pad 18: Net-(Q1-S) -> Net-(U5-O13)
- U5 pad 19: Net-(Q2-S) -> Net-(U5-O14)
- U5 pad 2: Net-(U4-O1) -> Net-(U1-Data)
- U5 pad 20: Net-(Q3-S) -> Net-(U5-O15)
- U5 pad 21: Net-(Q4-S) -> Net-(U14-GND)
- U5 pad 22: Net-(Q5-S) -> unconnected-(U5-D_out-Pad22)
- U5 pad 23: Net-(Q6-S) -> Net-(U5-SET)
- U5 pad 24: Net-(Q7-S) -> Net-(Q1-D)
- U5 pad 3: Net-(U4-O2) -> Net-(U24-Y1)
- U5 pad 4: Net-(U4-O3) -> Net-(U1-Driver_LE)
- U5 pad 5: Net-(U4-O4) -> Net-(U5-O0)
- U5 pad 6: Net-(U4-O5) -> Net-(U5-O1)
- U5 pad 7: Net-(U4-O6) -> Net-(U5-O2)
- U5 pad 8: Net-(U4-O7) -> Net-(U5-O3)
- U5 pad 9: Net-(U4-O8) -> Net-(U5-O4)
- U6 pad 1: Net-(U10-GND) -> Net-(U5-O11)
- U6 pad 10: Net-(U20-C5) -> Net-(Q3-S)
- U6 pad 11: Net-(U20-C6) -> Net-(Q5-S)
- U6 pad 12: Net-(U20-C7) -> Net-(U5-O12)
- U6 pad 13: Net-(U20-C8) -> Net-(Q9-S)
- U6 pad 14: Net-(U20-C9) -> Net-(U5-O14)
- U6 pad 15: Net-(U20-C10) -> Net-(Q6-S)
- U6 pad 16: Net-(U20-C11) -> Net-(Q7-S)
- U6 pad 2: Net-(U1-Data) -> Net-(U5-O9)
- U6 pad 3: Net-(U24-Y1) -> Net-(Q1-S)
- U6 pad 4: Net-(U1-Driver_LE) -> Net-(Q2-S)
- U6 pad 5: Net-(U20-C0) -> Net-(U5-O8)
- U6 pad 6: Net-(U20-C1) -> Net-(Q4-S)
- U6 pad 7: Net-(U20-C2) -> Net-(U5-O10)
- U6 pad 8: Net-(U20-C3) -> Net-(U5-O13)
- U6 pad 9: Net-(U20-C4) -> Net-(U5-O15)
- U7 pad 1: Net-(U7-C0) -> Net-(U5-O3)
- U7 pad 10: Net-(U7-C9) -> Net-(Q3-S)
- U7 pad 11: Net-(U7-C10) -> Net-(Q5-S)
- U7 pad 12: Net-(U7-C11) -> Net-(U5-O4)
- U7 pad 13: Net-(U7-C12) -> Net-(Q9-S)
- U7 pad 14: Net-(U7-C13) -> Net-(U5-O6)
- U7 pad 15: Net-(U7-C14) -> Net-(Q6-S)
- U7 pad 16: Net-(U7-C15) -> Net-(Q7-S)
- U7 pad 2: Net-(U7-C1) -> Net-(U5-O1)
- U7 pad 3: Net-(U7-C2) -> Net-(Q1-S)
- U7 pad 4: Net-(U7-C3) -> Net-(Q2-S)
- U7 pad 5: Net-(U7-C4) -> Net-(U5-O0)
- U7 pad 6: Net-(U7-C5) -> Net-(Q4-S)
- U7 pad 7: Net-(U7-C6) -> Net-(U5-O2)
- U7 pad 8: Net-(U7-C7) -> Net-(U5-O5)
- U7 pad 9: Net-(U7-C8) -> Net-(U5-O7)
- U8 pad 1: Net-(U10-GND) -> Net-(U14-GND)
- U8 pad 10: Net-(U7-C5) -> Net-(U12-R2)
- U8 pad 11: Net-(U7-C6) -> Net-(U12-R1)
- U8 pad 12: Net-(U7-C7) -> Net-(U12-R0)
- U8 pad 13: Net-(U7-C8) -> Net-(U10-R7)
- U8 pad 14: Net-(U7-C9) -> Net-(U10-R6)
- U8 pad 15: Net-(U7-C10) -> Net-(U10-R5)
- U8 pad 16: Net-(U7-C11) -> Net-(U10-R4)
- U8 pad 17: Net-(U7-C12) -> Net-(U10-R3)
- U8 pad 18: Net-(U7-C13) -> Net-(U10-R2)
- U8 pad 19: Net-(U7-C14) -> Net-(U10-R1)
- U8 pad 20: Net-(U7-C15) -> Net-(U10-R0)
- U8 pad 21: Net-(U10-GND) -> Net-(U14-GND)
- U8 pad 5: Net-(U7-C0) -> Net-(U12-R7)
- U8 pad 6: Net-(U7-C1) -> Net-(U12-R6)
- U8 pad 7: Net-(U7-C2) -> Net-(U12-R5)
- U8 pad 8: Net-(U7-C3) -> Net-(U12-R4)
- U8 pad 9: Net-(U7-C4) -> Net-(U12-R3)
- U9 pad 1: Net-(U12-O0) -> Net-(U14-GND)
- U9 pad 10: Net-(U12-O9) -> Net-(U13-R2)
- U9 pad 11: Net-(U12-O10) -> Net-(U13-R1)
- U9 pad 12: Net-(U12-O11) -> Net-(U13-R0)
- U9 pad 13: Net-(U12-O12) -> Net-(U11-R7)
- U9 pad 14: Net-(U12-O13) -> Net-(U11-R6)
- U9 pad 15: Net-(U12-O14) -> Net-(U11-R5)
- U9 pad 16: Net-(U12-O15) -> Net-(U11-R4)
- U9 pad 17: Net-(Q9-S) -> Net-(U11-R3)
- U9 pad 18: Net-(Q1-S) -> Net-(U11-R2)
- U9 pad 19: Net-(Q2-S) -> Net-(U11-R1)
- U9 pad 2: Net-(U12-O1) -> Net-(U1-Data)
- U9 pad 20: Net-(Q3-S) -> Net-(U11-R0)
- U9 pad 21: Net-(Q4-S) -> Net-(U14-GND)
- U9 pad 22: Net-(Q5-S) -> unconnected-(U9-D_out-Pad22)
- U9 pad 23: Net-(Q6-S) -> Net-(U9-SET)
- U9 pad 24: Net-(Q7-S) -> Net-(Q1-D)
- U9 pad 3: Net-(U12-O2) -> Net-(U24-Y3)
- U9 pad 4: Net-(U12-O3) -> Net-(U1-Driver_LE)
- U9 pad 5: Net-(U12-O4) -> Net-(U13-R7)
- U9 pad 6: Net-(U12-O5) -> Net-(U13-R6)
- U9 pad 7: Net-(U12-O6) -> Net-(U13-R5)
- U9 pad 8: Net-(U12-O7) -> Net-(U13-R4)
- U9 pad 9: Net-(U12-O8) -> Net-(U13-R3)
Routing:
- net Net-(U10-GND): track 1898.5 -> 0.00 mm, vias 10 -> 0
- net Net-(U14-GND): track 0.00 -> 1665.0 mm, vias 0 -> 7
- net Net-(Q7-S): track 153.4 -> 963.7 mm, vias 2 -> 20
- net Net-(Q6-S): track 167.5 -> 931.8 mm, vias 2 -> 20
- net Net-(Q5-S): track 181.8 -> 835.7 mm, vias 2 -> 20
- net Net-(Q2-S): track 224.5 -> 815.8 mm, vias 2 -> 20
- net Net-(Q1-S): track 238.8 -> 804.9 mm, vias 2 -> 20
- net Net-(Q9-S): track 254.7 -> 795.2 mm, vias 2 -> 20
- net Net-(Q3-S): track 210.3 -> 750.2 mm, vias 2 -> 20
- net Net-(Q4-S): track 196.0 -> 639.7 mm, vias 2 -> 20
- net Net-(U1-Data): track 923.0 -> 499.0 mm, vias 17 -> 7
- net Net-(U12-CLK): track 399.4 -> 0.00 mm, vias 3 -> 0
- net Net-(U18-CLK): track 336.1 -> 0.00 mm, vias 2 -> 0
- net Net-(U1-Driver_LE): track 876.7 -> 553.0 mm, vias 10 -> 3
- net Net-(Q1-D): track 1040.6 -> 783.1 mm, vias 12 -> 10
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Other:
- board size 301.6 x 295.3 mm -> 220 x 172 mm
- board text added: "+5V +5V DATA CLK DRIVER LE DRIVER A0 DRIVER A1 DRIVER A2 ROW A0 ROW A1 ROW A2 GND GND"
- board text added: "32 X 32 LED DISPLAY 1:8 MULTIPLEXED"
