File: kicad/version_2/control_panel/control_panel.kicad_sch (KiCad schematic)
At the start: 41 parts, among them J1 Conn_01x01_Pin, J2 Conn_01x01_Pin, J3 Conn_01x01_Pin, J4 Conn_01x01_Pin, SW1 SW_Push

Commit message: Improved control panel and fixed music program
Parts:
- U17: footprint custom_footprint_library:manual_clock_switch -> custom_footprint_library:manual_clock_switch_side
Changed lines of the file:
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@@
 			)
 		)
-		(property "Footprint" "custom_footprint_library:manual_clock_switch"
+		(property "Footprint" "custom_footprint_library:manual_clock_switch_side"
 			(at 230.632 39.878 0)
 			(effects

Commit message: Finished control panel
Parts:
- added R10, R11, R12, R13, R8, R9: R, custom_footprint_library:0.4_pitch_resistor, symbol Device:R
- added SW2, SW3, SW4, SW5, SW6, SW7: SW_Push, Button_Switch_THT:SW_PUSH_6mm, symbol Switch:SW_Push
- added U20, U22: ~, Connector_PinHeader_2.54mm:PinHeader_1x08_P2.54mm_Vertical, symbol custom_symbol_lib:connector_8_bit
- added U21: ~, Connector_PinHeader_2.54mm:PinHeader_1x10_P2.54mm_Horizontal, symbol custom_symbol_lib:prog_mem_interface_write
- C2, C3, C4, C5, C6: footprint Capacitor_THT:C_Rect_L10.3mm_W4.5mm_P7.50mm_MKS4 -> Capacitor_THT:C_Rect_L11.0mm_W4.2mm_P10.00mm_MKT
Connections:
- net at C2.1, C3.1, C4.1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: now also SW2.2, SW3.2, SW4.2, SW5.2, SW6.2, SW7.2
- net at C1.2, C2.2, C3.2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: now also R10.2, R11.2, R12.2, R13.2, R8.2, R9.2
- net at U1.2 (B), U12.2 (B), U13.2 (B)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: now also U4.11 (CCLK), U4.13 (RCLK)
- new net: R8.1, SW2.1, U20.1 (0)
- new net: R9.1, SW3.1, U20.2 (1)
- new net: R10.1, SW4.1, U20.3 (2)
- new net: R11.1, SW5.1, U20.4 (3)
- new net: R12.1, SW6.1, U20.5 (4)
- new net: R13.1, SW7.1, U20.6 (5)
Other:
- note added: "Inputs"
- note added: "Outputs"

Commit message: before using copilot
Parts:
- SW2, SW3, SW4, SW5, SW6, SW7: footprint Button_Switch_THT:SW_PUSH_6mm -> custom_footprint_library:2_pin_button
Changed lines of the file:
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@@
 			)
 		)
-		(property "Footprint" "Button_Switch_THT:SW_PUSH_6mm"
+		(property "Footprint" "custom_footprint_library:2_pin_button"
 			(at 140.97 128.27 0)
 			(effects
@@
 			)
 		)
-		(property "Footprint" "Button_Switch_THT:SW_PUSH_6mm"
+		(property "Footprint" "custom_footprint_library:2_pin_button"
 			(at 140.97 123.19 0)
 			(effects
@@
 			)
 		)
-		(property "Footprint" "Button_Switch_THT:SW_PUSH_6mm"
+		(property "Footprint" "custom_footprint_library:2_pin_button"
 			(at 140.97 125.73 0)
 			(effects
@@
 			)
 		)
-		(property "Footprint" "Button_Switch_THT:SW_PUSH_6mm"
+		(property "Footprint" "custom_footprint_library:2_pin_button"
 			(at 140.97 118.11 0)
 			(effects
@@
 			)
 		)
-		(property "Footprint" "Button_Switch_THT:SW_PUSH_6mm"
+		(property "Footprint" "custom_footprint_library:2_pin_button"
 			(at 140.97 130.81 0)
 			(effects
@@
 			)
 		)
-		(property "Footprint" "Button_Switch_THT:SW_PUSH_6mm"
+		(property "Footprint" "custom_footprint_library:2_pin_button"
 			(at 140.97 120.65 0)
 			(effects
