File: kicad/vector_digital_controller/vector_digital_controller.kicad_sch (KiCad schematic)
At the start: 41 parts

Commit message: Working on vector controller
Parts:
- removed U18, U32: ~, Package_DIP:DIP-20_W7.62mm, symbol custom_symbol_lib:8_bit_transparent_latch
- added R1, R10, R11, R12, R13, R14, R15, R2, R3, R4, R5, R6, R7, R8, R9: R, custom_footprint_library:0.4_pitch_resistor, symbol Device:R
- added U18: ~, Connector_PinHeader_2.54mm:PinHeader_1x10_P2.54mm_Vertical, symbol custom_symbol_lib:vector_CRT
- added U24, U27: ~, Package_DIP:DIP-14_W7.62mm, symbol custom_symbol_lib:4x_XNOR
- added U25, U26: ~, Package_DIP:DIP-14_W7.62mm, symbol custom_symbol_lib:quad_and
- added U28: ~, Package_DIP:DIP-16_W7.62mm, symbol custom_symbol_lib:8_bit_counter
- added U29, U30: ~, Package_DIP:DIP-14_W7.62mm, symbol custom_symbol_lib:quad_OR
- added U31: ~, Package_DIP:DIP-20_W7.62mm, symbol custom_symbol_lib:8_bit_transparent_latch
- added U32, U44, U51, U52: ~, Package_DIP:DIP-24_W7.62mm, symbol custom_symbol_lib:MAX503_10_bit_dac_DIP_pkg
Connections:
- net 0: now also U11.19 (Q0), U38.19 (Q0), U8.19 (Q0), R1.1, U31.19 (Q0)
- net 1: now also U11.18 (Q1), U38.18 (Q1), U8.18 (Q1), R2.1, U31.18 (Q1)
- net 10: now also U10.17 (Q2), U37.17 (Q2), U5.12 (Q7), R11.1
- net 11: now also U10.16 (Q3), U37.16 (Q3), U7.16 (Q3), R12.1, U31.5 (D3)
- net 12: now also U10.15 (Q4), U37.15 (Q4), U7.15 (Q4), R13.1, U31.6 (D4)
- net 13: now also U10.14 (Q5), U37.14 (Q5), U7.14 (Q5), R14.1, U31.7 (D5)
- net 14: now also U10.13 (Q6), U37.13 (Q6), U7.13 (Q6), R15.1, U31.8 (D6)
- net 15: no longer U21.9 (D7)
- net 2: now also U11.17 (Q2), U38.17 (Q2), U8.17 (Q2), R3.1, U31.17 (Q2)
- net 3: now also U11.16 (Q3), U38.16 (Q3), U5.19 (Q0), U8.16 (Q3), R4.1
- net 4: now also U11.15 (Q4), U38.15 (Q4), U5.18 (Q1), U8.15 (Q4), R5.1
- net 5: now also U11.14 (Q5), U38.14 (Q5), U5.17 (Q2), U8.14 (Q5), R6.1
- net 6: now also U11.13 (Q6), U38.13 (Q6), U5.16 (Q3), U8.13 (Q6), R7.1
- net 7: now also U11.12 (Q7), U38.12 (Q7), U5.15 (Q4), U8.12 (Q7), R8.1
- net 8: now also U10.19 (Q0), U37.19 (Q0), U5.14 (Q5), R9.1
- net 9: now also U10.18 (Q1), U37.18 (Q1), U5.13 (Q6), R10.1
- net at U17.1 (Σ1): now also R14.2
- net at U17.11 (B3), U17.15 (B2), U17.2 (B1)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: now also U17.12 (A3)
- net at U33.12 (Q7): no longer U17.12 (A3)
- net at U17.13 (Σ2): now also R15.2
- net at U17.4 (Σ0): now also R13.2
- net at U21.10 (GND): now also U21.9 (D7)
- net at U48.16 (V+), U48.7 (C_IN): now also U48.5 (A0)
- net at U16.19 (Q0): no longer U48.5 (A0)
- net at U35.14 (OE#): now also U45.1 (OE#)
- net at U9.1 (Σ1): now also R6.2
- net at U9.10 (Σ3): now also R8.2
- net at U9.13 (Σ2): now also R7.2
- net at U9.4 (Σ0): now also R5.2
- net at U4.1 (Σ1): now also R2.2
- net at U4.10 (Σ3): now also R4.2
- net at U4.13 (Σ2): now also R3.2
- net at U4.4 (Σ0): now also R1.2
- net at U39.13 (Q6): now also U27.5 (2A)
- net at U39.14 (Q5): now also U27.8 (3A)
- net at U39.15 (Q4): now also U27.12 (4A)
- net at U39.16 (Q3): now also U24.1 (1A)
- net at U39.17 (Q2): now also U24.5 (2A)
- net at U39.18 (Q1): now also U24.8 (3A)
- net at U39.19 (Q0): now also U24.12 (4A)
- net at U14.1 (Σ1): now also R10.2
- net at U14.10 (Σ3): now also R12.2
- net at U14.13 (Σ2): now also R11.2
- net at U14.4 (Σ0): now also R9.2
- net VectorMemX7: now reaches U13.12 (Q7)
- net VectorMemX7: now also U3.19 (D7)
- net VectorMemX6: now reaches U13.13 (Q6)
- net VectorMemX6: now also U3.18 (D6)
- net VectorMemX5: now reaches U13.14 (Q5)
- net VectorMemX5: now also U3.17 (D5)
- net VectorMemX4: now reaches U13.15 (Q4)
- net VectorMemX4: now also U3.16 (D4)
- net VectorMemX3: now reaches U13.16 (Q3)
- net VectorMemX3: now also U3.15 (D3)
- net VectorMemX2: now reaches U13.17 (Q2)
- net VectorMemX2: now also U3.13 (D2)
- net VectorMemX1: now reaches U13.18 (Q1)
- net VectorMemX1: now also U3.12 (D1)
- net VectorMemX0: now reaches U13.19 (Q0)
- net VectorMemX0: now also U3.11 (D0)
- net at U7.1 (OE#): now also U7.10 (GND)
- new net: U51.12 (DGND), U51.14 (AGND), U51.17 (REFGND), U51.19 (VSS), U51.22 (ROFS)
- new net: U51.13 (REFIN), U51.18 (REFOUT)
- new net: U51.15 (CLR#), U51.23 (VDD)
- new net: U18.3 (X1), U51.20 (VOUT), U51.21 (RFB)
- new net: U24.9 (3B), U28.1 (Q1), U29.1 (0A)
- new net: U24.13 (4B), U28.15 (Q0)
- new net: U24.6 (2B), U28.2 (Q2), U29.2 (0B)
- new net: U24.2 (1B), U28.3 (Q3), U29.5 (1A)
- new net: U27.13 (4B), U28.4 (Q4), U29.6 (1B)
- new net: U27.9 (3B), U28.5 (Q5), U29.8 (2A)
- new net: U27.6 (2B), U28.6 (Q6), U29.9 (2B)
- new net: U24.10 (3Q), U25.4 (2A)
- new net: U24.11 (4Q), U25.5 (2B)
- new net: U24.3 (1Q), U25.1 (1A)
- new net: U24.4 (2Q), U25.2 (1B)
- new net: U27.1 (1A), U27.2 (1B), U27.7 (GND)
- new net: U25.12 (3B), U27.10 (3Q)
- new net: U25.13 (3A), U27.11 (4Q)
- new net: U25.9 (4B), U27.4 (2Q)
- new net: U18.1 (X0), U32.20 (VOUT), U32.21 (RFB)
- new net: U18.2 (Y0), U44.20 (VOUT), U44.21 (RFB)
- new net: U18.4 (Y1), U52.20 (VOUT), U52.21 (RFB)
- new net: U52.12 (DGND), U52.14 (AGND), U52.17 (REFGND), U52.19 (VSS), U52.22 (ROFS)
- new net: U52.13 (REFIN), U52.18 (REFOUT)
- new net: U52.15 (CLR#), U52.23 (VDD)
- new net: U25.10 (4A), U25.11 (3Q)
- new net: U25.3 (1Q), U26.13 (3A)
- new net: U25.6 (2Q), U26.12 (3B)
- new net: U25.8 (4Q), U26.9 (4B)
- new net: U29.10 (Q2), U30.1 (0A)
- new net: U29.11 (Q3), U30.2 (0B)
- new net: U26.10 (4A), U26.11 (3Q)
- new net: U44.12 (DGND), U44.14 (AGND), U44.17 (REFGND), U44.19 (VSS), U44.22 (ROFS)
- new net: U44.13 (REFIN), U44.18 (REFOUT)
- new net: U44.15 (CLR#), U44.23 (VDD)
- new net: U32.12 (DGND), U32.14 (AGND), U32.17 (REFGND), U32.19 (VSS), U32.22 (ROFS)
- new net: U32.13 (REFIN), U32.18 (REFOUT)
- new net: U32.15 (CLR#), U32.23 (VDD)
- new net: U29.12 (3A), U29.4 (Q1)
- new net: U29.13 (3B), U29.3 (Q0)
- new net: U31.10 (GND), U31.9 (D7)
- no-connect marks 1 -> 9
Other:
- note added: "0: Vector address bits 8-14, enable flag"
- note added: "1: Vector address bits 0-7"
- note added: "2: Length bits 0-6 (7 bits), line flag MSB (0=point, 1=line)"
- note added: "3: Offset X"
- note added: "4: Offset Y"
- note added: "MSB Not needed"
- note added: "Ok to stop the clock?"
- note added: "Sprite finished comparison"
- note added: "Sprite frame"
- note added: "Sprite frame and MSB must always be enabled, so put transparent latch for rest of spreite addressing"
- note added: "Sprite limit comparison"
- moved on the sheet: U12, U14, U17, U19, U20, U21, U3, U33, U4, U9

Commit message: Progress on vectors
Parts:
- added U53: ~, Package_DIP:DIP-16_W7.62mm, symbol custom_symbol_lib:3_to_8_demultiplexer
- added U55, U56, U57, U66, U67, U72, U73, U74: ~, Package_DIP:DIP-16_W7.62mm, symbol custom_symbol_lib:4bit_adder
- added U58: ~, Package_DIP:DIP-14_W7.62mm, symbol custom_symbol_lib:6xNOT
- added U59, U61, U68, U69: ~, Package_DIP:DIP-14_W7.62mm, symbol custom_symbol_lib:quad_and
- added U60: ~, Package_DIP:DIP-14_W7.62mm, symbol custom_symbol_lib:quad_OR
- added U63, U64, U65: ~, Package_DIP:DIP-20_W7.62mm, symbol custom_symbol_lib:rising_edge_8_bit_latch
Connections:
- net VectorAddr10 is gone; now on net VectorAddress10: U3.21 (A10)
- net VectorAddr11 is gone; now on net VectorAddress11: U3.23 (A11)
- net VectorAddr12 is gone; now on net VectorAddress12: U3.2 (A12)
- net VectorAddr13 is gone; now on net VectorAddress13: U3.26 (A13)
- net VectorAddr14 is gone; now on net VectorAddress14: U3.1 (A14)
- net VectorAddr6 is gone; now on net VectorAddress6: U3.4 (A6)
- net VectorAddr7 is gone; now on net VectorAddress7: U3.3 (A7)
- net VectorAddr8 is gone; now on net VectorAddress8: U3.25 (A8)
- net VectorAddr9 is gone; now on net VectorAddress9: U3.24 (A9)
- net 0: no longer R1.1, U1.19 (Q0), U10.2 (D0), U11.19 (Q0), U11.2 (D0), U19.2 (D0), U20.19 (Q0), U20.2 (D0), U31.19 (Q0), U35.15 (Q0), U36.10 (A0), U36.11 (D0), U37.2 (D0), U38.19 (Q0), U38.2 (D0), U39.2 (D0), U40.2 (D0), U41.2 (D0), U5.2 (D0), U6.19 (Q0), U7.2 (D0), U8.19 (Q0)
- net 1: no longer R2.1, U1.18 (Q1), U10.3 (D1), U11.18 (Q1), U11.3 (D1), U19.3 (D1), U20.18 (Q1), U20.3 (D1), U31.18 (Q1), U35.1 (Q1), U36.12 (D1), U36.9 (A1), U37.3 (D1), U38.18 (Q1), U38.3 (D1), U39.3 (D1), U40.3 (D1), U41.3 (D1), U5.3 (D1), U6.18 (Q1), U7.3 (D1), U8.18 (Q1)
- net 2: no longer R3.1, U1.17 (Q2), U10.4 (D2), U11.17 (Q2), U11.4 (D2), U19.4 (D2), U20.17 (Q2), U20.4 (D2), U31.17 (Q2), U35.2 (Q2), U36.13 (D2), U36.8 (A2), U37.4 (D2), U38.17 (Q2), U38.4 (D2), U39.4 (D2), U40.4 (D2), U41.4 (D2), U5.4 (D2), U6.17 (Q2), U7.4 (D2), U8.17 (Q2)
- net 3: no longer R4.1, U1.16 (Q3), U10.5 (D3), U11.16 (Q3), U11.5 (D3), U19.5 (D3), U20.16 (Q3), U20.5 (D3), U36.15 (D3), U36.7 (A3), U37.5 (D3), U38.16 (Q3), U38.5 (D3), U39.5 (D3), U40.5 (D3), U41.5 (D3), U45.19 (Q0), U5.19 (Q0), U5.5 (D3), U6.16 (Q3), U7.5 (D3), U8.16 (Q3)
- net 4: no longer R5.1, U1.15 (Q4), U10.6 (D4), U11.15 (Q4), U11.6 (D4), U19.6 (D4), U20.15 (Q4), U20.6 (D4), U36.16 (D4), U36.6 (A4), U37.6 (D4), U38.15 (Q4), U38.6 (D4), U39.6 (D4), U40.6 (D4), U41.6 (D4), U45.18 (Q1), U5.18 (Q1), U5.6 (D4), U6.15 (Q4), U7.6 (D4), U8.15 (Q4)
- net 5: no longer R6.1, U1.14 (Q5), U10.7 (D5), U11.14 (Q5), U11.7 (D5), U19.7 (D5), U20.14 (Q5), U20.7 (D5), U36.17 (D5), U36.5 (A5), U37.7 (D5), U38.14 (Q5), U38.7 (D5), U39.7 (D5), U40.7 (D5), U41.7 (D5), U45.17 (Q2), U5.17 (Q2), U5.7 (D5), U6.14 (Q5), U7.7 (D5), U8.14 (Q5)
- net 6: no longer R7.1, U1.13 (Q6), U10.8 (D6), U11.13 (Q6), U11.8 (D6), U19.8 (D6), U20.13 (Q6), U20.8 (D6), U36.18 (D6), U36.4 (A6), U37.8 (D6), U38.13 (Q6), U38.8 (D6), U39.8 (D6), U40.8 (D6), U41.8 (D6), U45.16 (Q3), U5.16 (Q3), U5.8 (D6), U6.13 (Q6), U7.8 (D6), U8.13 (Q6)
- net 7: no longer R8.1, U1.12 (Q7), U10.9 (D7), U11.12 (Q7), U11.9 (D7), U19.9 (D7), U20.12 (Q7), U20.9 (D7), U36.19 (D7), U36.3 (A7), U37.9 (D7), U38.12 (Q7), U38.9 (D7), U39.9 (D7), U40.9 (D7), U41.9 (D7), U45.15 (Q4), U5.15 (Q4), U5.9 (D7), U6.12 (Q7), U7.9 (D7), U8.12 (Q7)
- net VectorMemX0: now also U22.5 (A0)
- net VectorMemX1: now also U22.3 (A1)
- net VectorMemX2: now also U22.14 (A2)
- net VectorMemX3: now also U22.12 (A3)
- net VectorMemX4: now also U23.5 (A0)
- net VectorMemX5: now also U23.3 (A1)
- net VectorMemX6: now also U23.14 (A2)
- net VectorMemX7: now also U23.12 (A3)
- net at U21.1 (OE#): now also U20.1 (OE#)
- net at U21.11 (CLK): now also U60.11 (Q3)
- net at U51.1 (D7/S1): now also U32.1 (D7/S1), U63.18 (Q1), U65.18 (Q1)
- net at U51.10 (WR#): now also U32.10 (WR#), U44.10 (WR#), U52.10 (WR#)
- net at U51.16 (LDAC#): now also U32.16 (LDAC#), U44.16 (LDAC#), U52.16 (LDAC#)
- net at U51.2 (D8/D0): now also U32.2 (D8/D0), U63.17 (Q2), U65.17 (Q2)
- net at U51.24 (D6/S0): now also U32.24 (D6/S0), U63.19 (Q0), U65.19 (Q0)
- net at U51.3 (D9/D1): now also U32.3 (D9/D1), U63.16 (Q3), U65.16 (Q3)
- net at U51.4 (D2): now also U32.4 (D2), U63.15 (Q4)
- net at U51.5 (D3): now also U32.5 (D3), U63.14 (Q5)
- net at U51.6 (D4): now also U32.6 (D4), U63.13 (Q6)
- net at U51.7 (D5): now also U32.7 (D5), U63.12 (Q7)
- net at U51.8 (A0): now also U32.8 (A0), U32.9 (A1), U44.8 (A0), U44.9 (A1), U51.9 (A1), U52.8 (A0), U52.9 (A1)
- net at U22.1 (Σ1): now also U55.3 (A1)
- net at U22.10 (Σ3): now also U55.12 (A3)
- net at U22.13 (Σ2): now also U55.14 (A2)
- net at U22.4 (Σ0): now also U55.5 (A0)
- net at U40.1 (OE#): now also U40.10 (GND)
- net at U40.11 (CLK): now also U53.12 (Y3)
- net at U40.12 (Q7): now also U23.11 (B3), U61.12 (3B)
- net at U40.13 (Q6): now also U23.15 (B2), U61.5 (2B)
- net at U40.14 (Q5): now also U23.2 (B1), U61.2 (1B)
- net at U40.15 (Q4): now also U23.6 (B0), U59.9 (4B)
- net at U40.16 (Q3): now also U22.11 (B3), U59.12 (3B)
- net at U40.17 (Q2): now also U22.15 (B2), U59.5 (2B)
- net at U40.18 (Q1): now also U22.2 (B1), U59.2 (1B)
- net at U40.19 (Q0): now also U22.6 (B0), U60.2 (0B)
- net at U16.19 (Q0): now also U58.1 (I0), U59.1 (1A), U59.10 (4A), U59.13 (3A), U59.4 (2A), U61.1 (1A), U61.13 (3A), U61.4 (2A), U68.1 (1A), U68.10 (4A), U68.13 (3A), U68.4 (2A), U69.1 (1A), U69.13 (3A), U69.4 (2A)
- net at U38.1 (OE#): now also U36.22 (OE#), U37.1 (OE#)
- net at U38.11 (CLK): now also U38.20 (V+)
- net at U23.1 (Σ1): now also U56.3 (A1)
- net at U23.10 (Σ3): now also U56.12 (A3)
- net at U23.13 (Σ2): now also U56.14 (A2)
- net at U23.4 (Σ0): now also U56.5 (A0)
- net at U23.9 (C_OUT): now also U57.5 (A0)
- net at U41.1 (OE#): now also U41.10 (GND)
- net at U41.11 (CLK): now also U53.11 (Y4)
- net at U41.12 (Q7): now also U67.11 (B3), U69.12 (3B)
- net at U41.13 (Q6): now also U67.15 (B2), U69.5 (2B)
- net at U41.14 (Q5): now also U67.2 (B1), U69.2 (1B)
- net at U41.15 (Q4): now also U67.6 (B0), U68.9 (4B)
- net at U41.16 (Q3): now also U66.11 (B3), U68.12 (3B)
- net at U41.17 (Q2): now also U66.15 (B2), U68.5 (2B)
- net at U41.18 (Q1): now also U66.2 (B1), U68.2 (1B)
- net at U41.19 (Q0): now also U60.6 (1B), U66.6 (B0)
- net at U39.1 (OE#): now also U39.10 (GND)
- net at U39.11 (CLK): now also U53.13 (Y2)
- net at U52.1 (D7/S1): now also U44.1 (D7/S1), U64.18 (Q1), U65.14 (Q5)
- net at U52.2 (D8/D0): now also U44.2 (D8/D0), U64.17 (Q2), U65.13 (Q6)
- net at U52.24 (D6/S0): now also U44.24 (D6/S0), U64.19 (Q0), U65.15 (Q4)
- net at U52.3 (D9/D1): now also U44.3 (D9/D1), U64.16 (Q3), U65.12 (Q7)
- net at U52.4 (D2): now also U44.4 (D2), U64.15 (Q4)
- net at U52.5 (D3): now also U44.5 (D3), U64.14 (Q5)
- net at U52.6 (D4): now also U44.6 (D4), U64.13 (Q6)
- net at U52.7 (D5): now also U44.7 (D5), U64.12 (Q7)
- net VectorMemY7: now reaches U15.12 (Q7)
- net VectorMemY7: now also U12.19 (D7), U67.12 (A3)
- net VectorMemY6: now reaches U15.13 (Q6)
- net VectorMemY6: now also U12.18 (D6), U67.14 (A2)
- net VectorMemY5: now reaches U15.14 (Q5)
- net VectorMemY5: now also U12.17 (D5), U67.3 (A1)
- net VectorMemY4: now reaches U15.15 (Q4)
- net VectorMemY4: now also U12.16 (D4), U67.5 (A0)
- net VectorMemY3: now reaches U15.16 (Q3)
- net VectorMemY3: now also U12.15 (D3), U66.12 (A3)
- net VectorMemY2: now reaches U15.17 (Q2)
- net VectorMemY2: now also U12.13 (D2), U66.14 (A2)
- net VectorMemY1: now reaches U15.18 (Q1)
- net VectorMemY1: now also U12.12 (D1), U66.3 (A1)
- net VectorMemY0: now reaches U15.19 (Q0)
- net VectorMemY0: now also U12.11 (D0), U66.5 (A0)
- net at U37.11 (CLK): now also U37.20 (V+)
- net at U20.11 (CLK): now also U60.10 (Q2)
- net at U7.17 (Q2): now also U31.4 (D2)
- net at U7.18 (Q1): now also U31.3 (D1)
- net at U7.19 (Q0): now also U31.2 (D0)
- net VectorAddress14: now reaches U12.1 (A14)
- net VectorAddress14: now also U10.13 (Q6), U21.13 (Q6), U33.8 (D6)
- net VectorAddress12: now reaches U12.2 (A12)
- net VectorAddress12: now also U10.15 (Q4), U21.15 (Q4), U33.6 (D4)
- net VectorAddress10: now reaches U12.21 (A10)
- net VectorAddress10: now also U10.17 (Q2), U21.17 (Q2), U33.4 (D2)
- net VectorAddress11: now reaches U12.23 (A11)
- net VectorAddress11: now also U10.16 (Q3), U21.16 (Q3), U33.5 (D3)
- net VectorAddress9: now reaches U12.24 (A9)
- net VectorAddress9: now also U10.18 (Q1), U21.18 (Q1), U33.3 (D1)
- net VectorAddress8: now reaches U12.25 (A8)
- net VectorAddress8: now also U10.19 (Q0), U21.19 (Q0), U33.2 (D0)
- net VectorAddress13: now reaches U12.26 (A13)
- net VectorAddress13: now also U10.14 (Q5), U21.14 (Q5), U33.7 (D5)
- net VectorAddress7: now reaches U12.3 (A7)
- net VectorAddress7: now also U11.12 (Q7), U19.9 (D7), U20.12 (Q7)
- net VectorAddress6: now reaches U12.4 (A6)
- net VectorAddress6: now also U11.13 (Q6), U19.8 (D6), U20.13 (Q6)
- removed net 10: R11.1, U10.17 (Q2), U21.17 (Q2), U21.4 (D2), U33.4 (D2), U36.21 (A10), U37.17 (Q2), U45.12 (Q7), U5.12 (Q7)
- removed net 11: R12.1, U10.16 (Q3), U21.16 (Q3), U21.5 (D3), U31.5 (D3), U33.5 (D3), U36.23 (A11), U37.16 (Q3), U7.16 (Q3)
- removed net 12: R13.1, U10.15 (Q4), U21.15 (Q4), U21.6 (D4), U31.6 (D4), U33.6 (D4), U36.2 (A12), U37.15 (Q4), U7.15 (Q4)
- removed net 13: R14.1, U10.14 (Q5), U21.14 (Q5), U21.7 (D5), U31.7 (D5), U33.7 (D5), U36.26 (A13), U37.14 (Q5), U7.14 (Q5)
- removed net 14: R15.1, U10.13 (Q6), U21.13 (Q6), U21.8 (D6), U31.8 (D6), U33.8 (D6), U36.1 (A14), U37.13 (Q6), U7.13 (Q6)
- removed net 8: R9.1, U10.19 (Q0), U21.19 (Q0), U21.2 (D0), U33.2 (D0), U36.25 (A8), U37.19 (Q0), U45.14 (Q5), U5.14 (Q5)
- removed net 9: R10.1, U10.18 (Q1), U21.18 (Q1), U21.3 (D1), U33.3 (D1), U36.24 (A9), U37.18 (Q1), U45.13 (Q6), U5.13 (Q6)
- net VectorAddr0 renamed VectorAddress0
- net VectorAddress0: now also U11.19 (Q0), U19.2 (D0), U20.19 (Q0)
- net VectorAddr1 renamed VectorAddress1
- net VectorAddress1: now also U11.18 (Q1), U19.3 (D1), U20.18 (Q1)
- net VectorAddr2 renamed VectorAddress2
- net VectorAddress2: now also U11.17 (Q2), U19.4 (D2), U20.17 (Q2)
- net VectorAddr3 renamed VectorAddress3
- net VectorAddress3: now also U11.16 (Q3), U19.5 (D3), U20.16 (Q3)
- net VectorAddr4 renamed VectorAddress4
- net VectorAddress4: now also U11.15 (Q4), U19.6 (D4), U20.15 (Q4)
- net VectorAddr5 renamed VectorAddress5
- net VectorAddress5: now also U11.14 (Q5), U19.7 (D5), U20.14 (Q5)
- new net: U53.14 (Y1), U60.8 (2A)
- new net: U53.15 (Y0), U60.12 (3A)
- new net: U53.4 (E2#), U53.5 (E3#), U53.8 (GND)
- new net: U67.1 (Σ1), U73.3 (A1)
- new net: U67.10 (Σ3), U73.12 (A3)
- new net: U67.13 (Σ2), U73.14 (A2)
- new net: U67.4 (Σ0), U73.5 (A0)
- new net: U66.9 (C_OUT), U67.7 (C_IN)
- new net: U66.8 (GND), U67.8 (GND), U72.6 (B0), U72.8 (GND), U73.8 (GND), U74.11 (B3), U74.12 (A3), U74.14 (A2), U74.15 (B2), U74.2 (B1), U74.3 (A1), U74.8 (GND)
- new net: U67.9 (C_OUT), U74.5 (A0)
- new net: U22.8 (GND), U23.8 (GND), U55.6 (B0), U55.8 (GND), U56.8 (GND), U57.11 (B3), U57.12 (A3), U57.14 (A2), U57.15 (B2), U57.2 (B1), U57.3 (A1), U57.8 (GND)
- new net: U10.9 (D7), U6.12 (Q7), U7.9 (D7)
- new net: U10.8 (D6), U6.13 (Q6), U7.8 (D6)
- new net: U10.7 (D5), U6.14 (Q5), U7.7 (D5)
- new net: U10.6 (D4), U6.15 (Q4), U7.6 (D4)
- new net: U10.5 (D3), U6.16 (Q3), U7.5 (D3)
- new net: U10.4 (D2), U6.17 (Q2), U7.4 (D2)
- new net: U10.3 (D1), U6.18 (Q1), U7.3 (D1)
- new net: U10.2 (D0), U6.19 (Q0), U7.2 (D0)
- new net: U56.13 (Σ2), U65.2 (D0)
- new net: U56.10 (Σ3), U65.3 (D1)
- new net: U57.4 (Σ0), U65.4 (D2)
- new net: U57.1 (Σ1), U65.5 (D3)
- new net: U65.6 (D4), U73.13 (Σ2)
- new net: U65.7 (D5), U73.10 (Σ3)
- new net: U65.8 (D6), U74.4 (Σ0)
- new net: U65.9 (D7), U74.1 (Σ1)
- new net: U1.12 (Q7), U11.9 (D7), U5.9 (D7)
- new net: U1.13 (Q6), U11.8 (D6), U5.8 (D6)
- new net: U1.14 (Q5), U11.7 (D5), U5.7 (D5)
- new net: U1.15 (Q4), U11.6 (D4), U5.6 (D4)
- new net: U1.16 (Q3), U11.5 (D3), U5.5 (D3)
- new net: U1.17 (Q2), U11.4 (D2), U5.4 (D2)
- new net: U1.18 (Q1), U11.3 (D1), U5.3 (D1)
- new net: U1.19 (Q0), U11.2 (D0), U5.2 (D0)
- new net: U68.11 (3Q), U73.6 (B0)
- new net: U68.3 (1Q), U72.15 (B2)
- new net: U68.6 (2Q), U72.11 (B3)
- new net: U68.8 (4Q), U73.2 (B1)
- new net: U57.6 (B0), U61.11 (3Q)
- new net: U56.15 (B2), U61.3 (1Q)
- new net: U56.11 (B3), U61.6 (2Q)
- new net: U56.9 (C_OUT), U57.7 (C_IN)
- new net: U63.10 (GND), U63.2 (D0), U63.3 (D1)
- new net: U55.4 (Σ0), U63.4 (D2)
- new net: U55.1 (Σ1), U63.5 (D3)
- new net: U55.13 (Σ2), U63.6 (D4)
- new net: U55.10 (Σ3), U63.7 (D5)
- new net: U56.4 (Σ0), U63.8 (D6)
- new net: U56.1 (Σ1), U63.9 (D7)
- new net: U55.11 (B3), U59.6 (2Q)
- new net: U55.15 (B2), U59.3 (1Q)
- new net: U55.16 (V+), U55.7 (C_IN)
- new net: U55.2 (B1), U60.3 (Q0)
- new net: U55.9 (C_OUT), U56.7 (C_IN)
- new net: U64.5 (D3), U72.1 (Σ1)
- new net: U64.7 (D5), U72.10 (Σ3)
- new net: U66.10 (Σ3), U72.12 (A3)
- new net: U64.6 (D4), U72.13 (Σ2)
- new net: U66.13 (Σ2), U72.14 (A2)
- new net: U72.16 (V+), U72.7 (C_IN)
- new net: U60.4 (Q1), U72.2 (B1)
- new net: U66.1 (Σ1), U72.3 (A1)
- new net: U64.4 (D2), U72.4 (Σ0)
- new net: U66.4 (Σ0), U72.5 (A0)
- new net: U72.9 (C_OUT), U73.7 (C_IN)
- new net: U58.2 (O0), U60.1 (0A), U60.5 (1A)
- new net: U64.10 (GND), U64.2 (D0), U64.3 (D1)
- new net: U64.8 (D6), U73.4 (Σ0)
- new net: U64.9 (D7), U73.1 (Σ1)
- new net: U56.6 (B0), U59.11 (3Q)
- new net: U56.2 (B1), U59.8 (4Q)
- new net: U69.11 (3Q), U74.6 (B0)
- new net: U73.9 (C_OUT), U74.7 (C_IN)
- new net: U69.3 (1Q), U73.15 (B2)
- new net: U69.6 (2Q), U73.11 (B3)
- new net: U66.16 (V+), U66.7 (C_IN)
- new net: U60.13 (3B), U60.9 (2B)
- new net LoadVectorAddress0: R1.1, U20.2 (D0), U38.19 (Q0)
- new net LoadVectorAddress1: R2.1, U20.3 (D1), U38.18 (Q1)
- new net LoadVectorAddress10: R11.1, U21.4 (D2), U37.17 (Q2)
- new net LoadVectorAddress11: R12.1, U21.5 (D3), U37.16 (Q3)
- new net LoadVectorAddress12: R13.1, U21.6 (D4), U37.15 (Q4)
- new net LoadVectorAddress13: R14.1, U21.7 (D5), U37.14 (Q5)
- new net LoadVectorAddress14: R15.1, U21.8 (D6), U37.13 (Q6)
- new net LoadVectorAddress2: R3.1, U20.4 (D2), U38.17 (Q2)
- new net LoadVectorAddress3: R4.1, U20.5 (D3), U38.16 (Q3)
- new net LoadVectorAddress4: R5.1, U20.6 (D4), U38.15 (Q4)
- new net LoadVectorAddress5: R6.1, U20.7 (D5), U38.14 (Q5)
- new net LoadVectorAddress6: R7.1, U20.8 (D6), U38.13 (Q6)
- new net LoadVectorAddress7: R8.1, U20.9 (D7), U38.12 (Q7)
- new net LoadVectorAddress8: R9.1, U21.2 (D0), U37.19 (Q0)
- new net LoadVectorAddress9: R10.1, U21.3 (D1), U37.18 (Q1)
- new net SpriteData0: U36.11 (D0), U37.2 (D0), U38.2 (D0), U39.2 (D0), U40.2 (D0), U41.2 (D0), U8.19 (Q0)
- new net SpriteData1: U36.12 (D1), U37.3 (D1), U38.3 (D1), U39.3 (D1), U40.3 (D1), U41.3 (D1), U8.18 (Q1)
- new net SpriteData2: U36.13 (D2), U37.4 (D2), U38.4 (D2), U39.4 (D2), U40.4 (D2), U41.4 (D2), U8.17 (Q2)
- new net SpriteData3: U36.15 (D3), U37.5 (D3), U38.5 (D3), U39.5 (D3), U40.5 (D3), U41.5 (D3), U8.16 (Q3)
- new net SpriteData4: U36.16 (D4), U37.6 (D4), U38.6 (D4), U39.6 (D4), U40.6 (D4), U41.6 (D4), U8.15 (Q4)
- new net SpriteData5: U36.17 (D5), U37.7 (D5), U38.7 (D5), U39.7 (D5), U40.7 (D5), U41.7 (D5), U8.14 (Q5)
- new net SpriteData6: U36.18 (D6), U37.8 (D6), U38.8 (D6), U39.8 (D6), U40.8 (D6), U41.8 (D6), U8.13 (Q6)
- new net SpriteData7: U36.19 (D7), U37.9 (D7), U38.9 (D7), U39.9 (D7), U40.9 (D7), U41.9 (D7), U8.12 (Q7)
- new net SpriteMemAddr0: U31.19 (Q0), U35.15 (Q0), U36.10 (A0), U53.1 (A0)
- new net SpriteMemAddr1: U31.18 (Q1), U35.1 (Q1), U36.9 (A1), U53.2 (A1)
- new net SpriteMemAddr10: U36.21 (A10), U45.12 (Q7), U5.12 (Q7)
- new net SpriteMemAddr11: U31.5 (D3), U36.23 (A11), U7.16 (Q3)
- new net SpriteMemAddr12: U31.6 (D4), U36.2 (A12), U7.15 (Q4)
- new net SpriteMemAddr13: U31.7 (D5), U36.26 (A13), U7.14 (Q5)
- new net SpriteMemAddr14: U31.8 (D6), U36.1 (A14), U7.13 (Q6)
- new net SpriteMemAddr2: U31.17 (Q2), U35.2 (Q2), U36.8 (A2), U53.3 (A2)
- new net SpriteMemAddr3: U36.7 (A3), U45.19 (Q0), U5.19 (Q0)
- new net SpriteMemAddr4: U36.6 (A4), U45.18 (Q1), U5.18 (Q1)
- new net SpriteMemAddr5: U36.5 (A5), U45.17 (Q2), U5.17 (Q2)
- new net SpriteMemAddr6: U36.4 (A6), U45.16 (Q3), U5.16 (Q3)
- new net SpriteMemAddr7: U36.3 (A7), U45.15 (Q4), U5.15 (Q4)
- new net SpriteMemAddr8: U36.25 (A8), U45.14 (Q5), U5.14 (Q5)
- new net SpriteMemAddr9: U36.24 (A9), U45.13 (Q6), U5.13 (Q6)
- no-connect marks 9 -> 20
Other:
- note added: "NBH Loader for both X & Y"
- note added: "NBL & NBM Loader X"
- note added: "NBL & NBM Loader Y"
- note added: "Resolution"
- note added: "Vector address B (bits 8-14) (MSB=0) / Sprite set field address (MSB=1)"
- note removed: "Vector address B (bits 8-15) (MSB=0) / Sprite set field address (MSB=1)"
- moved on the sheet: R1, R10, R11, R12, R13, R14, R15, R2, R3, R4, R5, R6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

Commit message: KiCad progress
Parts:
- removed U72, U73: ~, Package_DIP:DIP-16_W7.62mm, symbol custom_symbol_lib:4bit_adder
- added U100, U104, U105, U106, U97: ~, Package_DIP:DIP-14_W7.62mm, symbol custom_symbol_lib:quad_and
- added U101, U107, U112, U99: ~, Package_DIP:DIP-14_W7.62mm, symbol custom_symbol_lib:quad_OR
- added U102, U103, U96: ~, Package_DIP:DIP-14_W7.62mm, symbol custom_symbol_lib:dual_latch
- added U108, U109, U110, U111, U54, U62, U70, U71, U75, U76, U77, U78, U79, U80, U81, U82, U83, U84, U85, U86, U87, U88, U89, U90, U91, U92: ~, custom_footprint_library:jumper, symbol custom_symbol_lib:jumper
- added U113, U98: ~, Package_DIP:DIP-14_W7.62mm, symbol custom_symbol_lib:6xNOT
- added U72: ~, custom_footprint_library:crystal_dip_14, symbol custom_symbol_lib:clock_8_mhz
- added U73, U95: ~, Package_DIP:DIP-20_W7.62mm, symbol custom_symbol_lib:rising_edge_8_bit_latch
- added U93, U94: ~, Package_DIP:DIP-16_W7.62mm, symbol custom_symbol_lib:4bit_adder
Connections:
- net at U2.1 (READ_0): now also U97.2 (1B)
- net at U2.10 (CLK_A): now also U97.1 (1A), U97.10 (4A), U97.13 (3A), U97.4 (2A)
- net at U2.2 (READ_1): now also U97.5 (2B)
- net at U2.3 (READ_2): now also U97.12 (3B)
- net at U2.4 (READ_3): now also U97.9 (4B)
- net at U67.1 (Σ1): now also U93.3 (A1)
- net at U67.10 (Σ3): now also U93.12 (A3)
- net at U41.12 (Q7), U67.11 (B3): now also U60.6 (1B); no longer U69.12 (3B)
- net at U67.13 (Σ2): now also U93.14 (A2)
- net at U41.13 (Q6), U67.15 (B2): now also U69.12 (3B); no longer U69.5 (2B)
- net at U41.14 (Q5), U67.2 (B1): now also U69.5 (2B); no longer U69.2 (1B)
- net at U67.4 (Σ0): now also U93.5 (A0)
- net at U41.15 (Q4), U67.6 (B0): now also U69.2 (1B); no longer U68.9 (4B)
- net at U74.5 (A0): now also U66.4 (Σ0); no longer U67.9 (C_OUT)
- net at U22.11 (B3), U40.16 (Q3): now also U59.9 (4B); no longer U59.12 (3B)
- net at U22.15 (B2), U40.17 (Q2): now also U59.12 (3B); no longer U59.5 (2B)
- net at U22.2 (B1), U40.18 (Q1): now also U59.5 (2B); no longer U59.2 (1B)
- net at U22.6 (B0), U40.19 (Q0): now also U59.2 (1B); no longer U60.2 (0B)
- net at U22.8 (GND), U23.8 (GND), U55.8 (GND)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: now also U57.6 (B0); no longer U55.6 (B0)
- net at U23.11 (B3), U40.12 (Q7): now also U60.2 (0B); no longer U61.12 (3B)
- net at U23.15 (B2), U40.13 (Q6): now also U61.12 (3B); no longer U61.5 (2B)
- net at U23.2 (B1), U40.14 (Q5): now also U61.5 (2B); no longer U61.2 (1B)
- net at U23.6 (B0), U40.15 (Q4): now also U61.2 (1B); no longer U59.9 (4B)
- net at U6.1 (OE#): now also U6.10 (GND)
- net at U6.11 (CLK): now also U101.2 (0B), U97.6 (2Q)
- net at U10.1 (OE#): now also U11.1 (OE#), U13.1 (OE#), U15.1 (OE#), U50.8 (03)
- net at U10.11 (CLK): now also U11.11 (CLK), U5.11 (CLK), U7.11 (CLK), U101.4 (Q1)
- net at U65.6 (D4): now also U93.13 (Σ2)
- net at U65.7 (D5): now also U93.10 (Σ3)
- net at U65.8 (D6): now also U94.4 (Σ0); no longer U74.4 (Σ0)
- net at U65.9 (D7): now also U94.1 (Σ1); no longer U74.1 (Σ1)
- net at U1.1 (OE#): now also U1.10 (GND)
- net at U1.11 (CLK): now also U101.1 (0A), U97.3 (1Q)
- net at U50.10 (O4): now also U104.1 (1A), U104.4 (2A)
- net at U50.11 (I4): now also U86.3 (OUT)
- net at U50.12 (O5): now also U104.10 (4A), U104.13 (3A)
- net at U50.13 (I5): now also U88.3 (OUT)
- net at U50.5 (I2): now also U7.12 (Q7), U105.10 (4A), U105.4 (2A)
- net at U50.6 (O2): now also U105.1 (1A), U105.13 (3A)
- net at U50.9 (I3): now also U108.3 (OUT)
- net at U28.10 (CCLR#): now also U58.10 (O4)
- net at U28.11 (CCLK): now also U28.13 (RCLK), U82.3 (OUT)
- net at U28.12 (CCKEN#): now also U28.14 (OE#), U28.8 (GND)
- net at U68.11 (3Q): now also U74.15 (B2)
- net at U41.16 (Q3), U66.11 (B3): now also U68.9 (4B); no longer U68.12 (3B)
- net at U41.18 (Q1), U66.2 (B1): now also U68.5 (2B); no longer U68.2 (1B)
- net at U68.3 (1Q): now also U74.6 (B0)
- net at U41.17 (Q2), U66.15 (B2): now also U68.12 (3B); no longer U68.5 (2B)
- net at U68.6 (2Q): now also U74.2 (B1)
- net at U68.8 (4Q): now also U74.11 (B3)
- net at U8.1 (OE#): now also U31.1 (OE#), U5.1 (OE#), U58.6 (O2)
- net at U13.11 (CLK), U8.11 (CLK): now also U101.9 (2B), U97.11 (3Q), U99.2 (0B)
- net at U15.11 (CLK), U16.11 (CLK): now also U101.8 (2A), U97.8 (4Q), U99.9 (2B)
- net at U61.11 (3Q): now also U56.15 (B2); no longer U57.6 (B0)
- net at U61.3 (1Q): now also U56.6 (B0); no longer U56.15 (B2)
- net at U61.6 (2Q): now also U56.2 (B1); no longer U56.11 (B3)
- net at U41.19 (Q0), U66.6 (B0): now also U68.2 (1B); no longer U60.6 (1B)
- net at U55.11 (B3): now also U59.8 (4Q); no longer U59.6 (2Q)
- net at U55.15 (B2): now also U59.11 (3Q); no longer U59.3 (1Q)
- net at U55.2 (B1): now also U59.6 (2Q); no longer U60.3 (Q0)
- net at U26.4 (2A): now also U106.10 (4A), U113.13 (I5)
- net at U26.8 (4Q): now also U92.1 (IN)
- net at U64.5 (D3): now also U74.1 (Σ1)
- net at U64.7 (D5): now also U74.10 (Σ3)
- net at U66.10 (Σ3): now also U74.12 (A3)
- net at U64.6 (D4): now also U74.13 (Σ2)
- net at U66.13 (Σ2): now also U74.14 (A2)
- net at U60.4 (Q1): now also U93.11 (B3)
- net at U66.1 (Σ1): now also U74.3 (A1)
- net at U64.4 (D2): now also U74.4 (Σ0)
- net at U58.11 (I4): now also U75.3 (OUT)
- net at U58.3 (I1): now also U109.3 (OUT)
- net at U58.4 (O1): now also U12.27 (WE#), U3.27 (WE#)
- net at U58.5 (I2): now also U110.3 (OUT)
- net at U58.8 (03): now also U36.27 (WE#)
- net at U58.9 (I3): now also U111.3 (OUT)
- net at U64.8 (D6): now also U93.4 (Σ0)
- net at U64.9 (D7): now also U93.1 (Σ1)
- net at U74.16 (V+): now also U74.7 (C_IN)
- net at U69.11 (3Q): now also U93.15 (B2); no longer U74.6 (B0)
- net at U74.9 (C_OUT): now also U93.7 (C_IN)
- net at U31.11 (CLK): now also U31.20 (V+)
- net at U69.3 (1Q): now also U93.6 (B0)
- net at U69.6 (2Q): now also U93.2 (B1)
- new net: U108.2 (GND), U109.2 (GND), U110.2 (GND), U111.2 (GND), U54.2 (GND), U62.2 (GND), U70.2 (GND), U71.2 (GND), U75.2 (GND), U76.2 (GND), U77.2 (GND), U78.2 (GND), U79.2 (GND), U80.2 (GND), U81.2 (GND), U82.2 (GND), U83.2 (GND), U84.2 (GND), U85.2 (GND), U86.2 (GND), U87.2 (GND), U88.2 (GND), U89.2 (GND), U90.2 (GND), U91.2 (GND), U92.2 (GND)
- new net: U105.5 (2B), U89.3 (OUT)
- new net: U66.8 (GND), U67.8 (GND), U74.8 (GND), U93.8 (GND), U94.11 (B3), U94.12 (A3), U94.14 (A2), U94.15 (B2), U94.2 (B1), U94.3 (A1), U94.6 (B0), U94.8 (GND)
- new net: U93.9 (C_OUT), U94.7 (C_IN)
- new net: U112.2 (0B), U81.3 (OUT)
- new net: U112.3 (Q0), U113.1 (I0)
- new net: U106.9 (4B), U113.12 (O5)
- new net: U112.5 (1A), U113.2 (O0)
- new net: U112.4 (Q1), U113.3 (I1)
- new net: U112.1 (0A), U113.4 (O1), U62.1 (IN)
- new net: U113.5 (I2), U62.3 (OUT)
- new net: U112.8 (2A), U113.6 (O2)
- new net: U72.1 (OE), U72.14 (V+)
- new net: U54.1 (IN), U72.8 (CLK)
- new net: U102.5 (0D), U105.11 (3Q)
- new net: U105.12 (3B), U105.9 (4B), U106.3 (1Q)
- new net: U105.2 (1B), U87.3 (OUT)
- new net: U101.13 (3B), U105.3 (1Q)
- new net: U101.12 (3A), U105.6 (2Q)
- new net: U102.9 (1D), U105.8 (4Q)
- new net: U104.8 (4Q), U110.1 (IN)
- new net: U104.11 (3Q), U111.1 (IN)
- new net: U104.12 (3B), U106.6 (2Q)
- new net: U104.2 (1B), U107.10 (Q2)
- new net: U104.3 (1Q), U108.1 (IN)
- new net: U104.5 (2B), U106.11 (3Q)
- new net: U104.6 (2Q), U109.1 (IN)
- new net: U104.9 (4B), U107.4 (Q1)
- new net: U103.1 (0Q), U106.12 (3B), U107.1 (0A), U107.9 (2B)
- new net: U103.13 (1Q), U106.4 (2A), U107.2 (0B), U107.6 (1B)
- new net: U107.3 (Q0), U98.11 (I4)
- new net: U102.13 (1Q), U103.9 (1D), U106.5 (2B), U107.5 (1A)
- new net: U102.1 (0Q), U103.5 (0D), U106.13 (3A), U107.8 (2A)
- new net: U67.9 (C_OUT), U94.5 (A0)
- new net: U98.1 (I0), U99.3 (Q0)
- new net: U106.2 (1B), U98.10 (O4)
- new net: U102.11 (1CLK), U103.3 (0CLK), U98.12 (O5)
- new net: U102.3 (0CLK), U103.11 (1CLK), U112.9 (2B), U54.3 (OUT), U98.13 (I5)
- new net: U98.2 (O0), U99.5 (1A)
- new net: U98.3 (I1), U99.4 (Q1)
- new net: U100.1 (1A), U98.4 (O1), U99.1 (0A)
- new net: U98.5 (I2), U99.10 (Q2)
- new net: U98.6 (O2), U99.12 (3A)
- new net: U100.4 (2A), U98.8 (03), U99.8 (2A)
- new net: U98.9 (I3), U99.11 (Q3)
- new net: U73.1 (OE#), U73.10 (GND), U95.10 (GND), U96.7 (GND)
- new net: U101.3 (Q0), U99.13 (3B), U99.6 (1B)
- new net: U55.6 (B0), U59.3 (1Q)
- new net: U73.11 (CLK), U96.3 (0CLK)
- new net: U79.1 (IN), U82.1 (IN)
- new net: U102.10 (1RESET), U102.4 (0RESET), U102.6 (0SET), U102.7 (GND), U102.8 (1SET), U103.10 (1RESET), U103.4 (0RESET), U103.6 (0SET), U103.7 (GND), U103.8 (1SET)
- new net: U112.10 (Q2), U70.1 (IN)
- new net: U106.8 (4Q), U112.6 (1B)
- new net: U100.2 (1B), U100.5 (2B), U101.10 (Q2)
- new net: U101.11 (Q3), U106.1 (1A)
- new net: U100.3 (1Q), U101.5 (1A)
- new net: U100.6 (2Q), U101.6 (1B)
- new net: U56.11 (B3), U60.3 (Q0)
- no-connect marks 20 -> 29
Other:
- note added: "APP CLK"
- note added: "APP CLK #"
- note added: "Clock enable latch"
- note added: "Counter 13"
- note added: "Encoder 1"
- note added: "G15"
- note added: "G16"
- note added: "G17"
- note added: "G18"
- note added: "Gate 0"
- note added: "Gate 10"
- note added: "Gate 11"
- note added: "Gate 12"
- note added: "Gate 14"
- note added: "Gate 2"
- note added: "Gate 3"
- note added: "Gate 4"
- note added: "Gate 5"
- note added: "Gate 6"
- note added: "Gate 7"
- note added: "Gate 8"
- note added: "Gate 9"
- note added: "Input corruption prevention SR latches"
- note added: "Q"
- note added: "R"
- note added: "Reset"
- note added: "S"
- note added: "Vec(0) / Sprite (1) write safe encoder"
- note removed: "Sprite limit comparison"
- moved on the sheet: R1, R10, R11, R12, R13, R14, R15, R2, R3, R4, R5, R6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

Commit message: Progress on vector thingy
Parts:
- removed U34, U35: ~, Package_DIP:DIP-16_W7.62mm, symbol custom_symbol_lib:8_bit_counter
- added U114: ~, Package_DIP:DIP-14_W7.62mm, symbol custom_symbol_lib:dual_latch
- added U115: ~, Package_DIP:DIP-14_W7.62mm, symbol custom_symbol_lib:quad_and
- added U116, U120: ~, Package_DIP:DIP-14_W7.62mm, symbol custom_symbol_lib:quad_OR
- added U117: ~, Package_DIP:DIP-14_W7.62mm, symbol custom_symbol_lib:6xNOT
- added U118, U122: ~, custom_footprint_library:jumper, symbol custom_symbol_lib:jumper
- added U119: ~, Connector_PinHeader_2.54mm:PinHeader_2x03_P2.54mm_Vertical, symbol custom_symbol_lib:Jumper_2x3
- added U121, U34: ~, Package_DIP:DIP-16_W7.62mm, symbol custom_symbol_lib:12_bit_counter_no_output_latch
- added U35: ~, Package_DIP:DIP-20_W7.62mm, symbol custom_symbol_lib:8_bit_transparent_latch
- U18: footprint Connector_PinHeader_2.54mm:PinHeader_1x10_P2.54mm_Vertical -> Connector_PinHeader_2.54mm:PinHeader_1x11_P2.54mm_Vertical
Connections:
- net SpriteMemAddr0: now also U35.19 (Q0)
- net SpriteMemAddr1: now also U35.18 (Q1)
- net SpriteMemAddr2: now also U35.17 (Q2)
- net at U108.2 (GND), U109.2 (GND), U110.2 (GND)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: now also U118.2 (GND), U122.2 (GND)
- net at U42.1 (1A), U45.6 (D4): now also U34.3 (Q4)
- net at U42.12 (4A), U45.9 (D7): now also U34.13 (Q7)
- net at U42.5 (2A), U45.7 (D5): now also U34.2 (Q5)
- net at U42.8 (3A), U45.8 (D6): now also U34.4 (Q6)
- net at U92.1 (IN): now also U30.3 (Q0); no longer U26.8 (4Q)
- net at U92.3 (OUT): now also U26.5 (2B)
- net at U51.11 (CS#): now also U52.11 (CS#), U58.12 (O5)
- net at U45.1 (OE#): now also U35.1 (OE#)
- net at U106.10 (4A), U113.13 (I5): now also U26.6 (2Q); no longer U26.4 (2A)
- net at U113.8 (03): now also U34.10 (CLK#)
- net at U113.9 (I3): now also U71.3 (OUT), U121.11 (Reset)
- net at U50.3 (I1): now also U76.3 (OUT); no longer U47.3 (1Q)
- net at U50.4 (O1): now also U121.10 (CLK#)
- net at U91.3 (OUT): now also U114.3 (0CLK), U117.9 (I3)
- net at U18.8 (Update_V0): now also U119.4 (In2)
- net at U18.9 (Update_V1): now also U119.3 (In1)
- net at U45.10 (GND): now also U121.8 (GND), U34.8 (GND), U35.10 (GND), U35.5 (D3), U35.6 (D4), U35.7 (D5), U35.8 (D6), U35.9 (D7)
- net at U45.2 (D0), U46.1 (1A): now also U34.9 (Q0)
- net at U45.3 (D1), U46.5 (2A): now also U34.7 (Q1)
- net at U45.4 (D2), U46.8 (3A): now also U34.6 (Q2)
- net at U45.5 (D3), U46.12 (4A): now also U34.5 (Q3)
- net at U30.4 (Q1): now also U26.4 (2A)
- net at U26.1 (1A): now also U117.6 (O2)
- net at U26.2 (1B): now also U117.5 (I2), U117.8 (03)
- net at U26.3 (1Q): now also U115.12 (3B), U115.9 (4B)
- net at U58.13 (I5): now also U32.11 (CS#), U44.11 (CS#), U118.3 (OUT)
- net at U36.14 (GND): now also U36.20 (CE#)
- net at U12.14 (GND): now also U12.20 (CE#)
- net at U3.14 (GND): now also U3.20 (CE#)
- new net: U114.1 (0Q), U115.8 (4Q)
- new net: U114.2 (0Q#), U115.11 (3Q)
- new net: U114.4 (0RESET), U114.6 (0SET), U114.7 (GND)
- new net: U114.5 (0D), U116.12 (3A), U117.2 (O0)
- new net: U116.10 (Q2), U117.1 (I0)
- new net: U116.11 (Q3), U117.3 (I1)
- new net: U116.8 (2A), U117.4 (O1), U118.1 (IN)
- new net: U119.1 (Out1_A), U120.6 (1B)
- new net: U119.2 (Out2_A), U120.5 (1A)
- new net: U119.5 (Out1_B), U120.2 (0B)
- new net: U119.6 (Out2_B), U120.1 (0A)
- new net: U115.10 (4A), U116.1 (0A)
- new net: U116.13 (3B), U116.4 (Q1)
- new net: U116.2 (0B), U120.3 (Q0)
- new net: U116.3 (Q0), U116.9 (2B)
- new net: U115.13 (3A), U116.5 (1A)
- new net: U116.6 (1B), U120.4 (Q1)
- new net: U121.16 (V+), U35.11 (CLK), U35.20 (V+)
- new net: U121.6 (Q2), U35.4 (D2)
- new net: U121.7 (Q1), U35.3 (D1)
- new net: U121.9 (Q0), U35.2 (D0)
- new net: U34.11 (Reset), U47.3 (1Q)
- no-connect marks 29 -> 42
Other:
- note added: "DAC update select latch"
- note added: "G19"
- note added: "G20"
- note added: "G21"
- note added: "G22"
- note added: "G23"
- note added: "G24"
- note added: "G26"
- note added: "G27"
- note added: "Latch 25"
- moved on the sheet: U108, U109, U110, U111, U71, U72, U75, U76, U77, U78, U79, U80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
