File: kicad/vector_digital_controller/vector_digital_controller.kicad_sch (KiCad schematic)
At the start: 137 parts

Commit message: Potentially finished kicad
Parts:
- removed U96: ~, Package_DIP:DIP-14_W7.62mm, symbol custom_symbol_lib:dual_latch
- added R16, R17, R18, R19: R, custom_footprint_library:0.4_pitch_resistor, symbol Device:R
- added U123: ~, Package_DIP:DIP-14_W7.62mm, symbol custom_symbol_lib:dual_latch
- added U124, U126, U129, U130, U132: ~, Package_DIP:DIP-14_W7.62mm, symbol custom_symbol_lib:quad_and
- added U127, U134, U136: ~, Package_DIP:DIP-14_W7.62mm, symbol custom_symbol_lib:6xNOT
- added U128, U131, U133, U135: ~, Package_DIP:DIP-14_W7.62mm, symbol custom_symbol_lib:quad_OR
- added U96: ~, Connector_PinHeader_2.54mm:PinHeader_1x02_P2.54mm_Vertical, symbol custom_symbol_lib:jumper_simple
Connections:
- net SpriteData7: now also U126.9 (4B), U127.3 (I1)
- net SpriteMemAddr11: no longer U31.5 (D3)
- net SpriteMemAddr12: no longer U31.6 (D4)
- net SpriteMemAddr13: no longer U31.7 (D5)
- net SpriteMemAddr14: no longer U31.8 (D6)
- net at U89.1 (IN): now also U134.12 (O5), U135.1 (0A)
- net at U108.2 (GND), U109.2 (GND), U110.2 (GND)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: now also U1.1 (OE#), U1.10 (GND), U10.10 (GND), U100.7 (GND), U101.7 (GND), U102.10 (1RESET), U102.4 (0RESET), U102.6 (0SET), U102.7 (GND), U102.8 (1SET), U103.10 (1RESET), U103.4 (0RESET), U103.6 (0SET), U103.7 (GND), U103.8 (1SET), U104.7 (GND), U105.7 (GND), U106.7 (GND), U107.7 (GND), U11.10 (GND), U112.7 (GND), U113.7 (GND), U114.10 (1RESET), U114.4 (0RESET), U114.6 (0SET), U114.7 (GND), U114.8 (1SET), U115.2 (1B), U115.3 (1Q), U115.5 (2B), U115.6 (2Q), U115.7 (GND), U116.7 (GND), U117.7 (GND), U12.14 (GND), U12.20 (CE#), U120.12 (3A), U120.13 (3B), U120.7 (GND), U120.8 (2A), U120.9 (2B), U121.8 (GND), U13.10 (GND), U14.11 (B3), U14.15 (B2), U14.2 (B1), U14.6 (B0), U14.8 (GND), U15.10 (GND), U16.1 (OE#), U16.10 (GND), U17.11 (B3), U17.12 (A3), U17.15 (B2), U17.2 (B1), U17.6 (B0), U17.8 (GND), U18.10 (GND), U19.1 (OE#), U19.10 (GND), U2.13 (GND), U20.10 (GND), U21.10 (GND), U21.9 (D7), U22.8 (GND), U23.8 (GND), U24.7 (GND), U25.7 (GND), U26.7 (GND), U27.1 (1A), U27.2 (1B), U27.7 (GND), U28.12 (CCKEN#), U28.14 (OE#), U28.8 (GND), U29.7 (GND), U3.14 (GND), U3.20 (CE#), U30.12 (3A), U30.13 (3B), U30.7 (GND), U30.8 (2A), U30.9 (2B), U31.10 (GND), U31.5 (D3), U31.6 (D4), U31.7 (D5), U31.8 (D6), U31.9 (D7), U32.12 (DGND), U32.14 (AGND), U32.17 (REFGND), U32.19 (VSS), U32.22 (ROFS), U33.1 (OE#), U33.10 (GND), U33.9 (D7), U34.8 (GND), U35.10 (GND), U35.5 (D3), U35.6 (D4), U35.7 (D5), U35.8 (D6), U35.9 (D7), U36.14 (GND), U36.20 (CE#), U37.10 (GND), U38.10 (GND), U39.1 (OE#), U39.10 (GND), U4.11 (B3), U4.15 (B2), U4.2 (B1), U4.6 (B0), U4.8 (GND), U40.1 (OE#), U40.10 (GND), U41.1 (OE#), U41.10 (GND), U42.7 (GND), U43.7 (GND), U44.12 (DGND), U44.14 (AGND), U44.17 (REFGND), U44.19 (VSS), U44.22 (ROFS), U45.10 (GND), U46.7 (GND), U47.7 (GND), U48.11 (B3), U48.15 (B2), U48.2 (B1), U48.6 (B0), U48.8 (GND), U49.11 (B3), U49.15 (B2), U49.2 (B1), U49.6 (B0), U49.8 (GND), U5.10 (GND), U50.7 (GND), U51.12 (DGND), U51.14 (AGND), U51.17 (REFGND), U51.19 (VSS), U51.22 (ROFS), U52.12 (DGND), U52.14 (AGND), U52.17 (REFGND), U52.19 (VSS), U52.22 (ROFS), U53.4 (E2#), U53.5 (E3#), U53.8 (GND), U55.8 (GND), U56.8 (GND), U57.11 (B3), U57.12 (A3), U57.14 (A2), U57.15 (B2), U57.2 (B1), U57.3 (A1), U57.6 (B0), U57.8 (GND), U58.7 (GND), U59.7 (GND), U6.1 (OE#), U6.10 (GND), U60.7 (GND), U61.7 (GND), U63.10 (GND), U63.2 (D0), U63.3 (D1), U64.10 (GND), U64.2 (D0), U64.3 (D1), U65.10 (GND), U66.8 (GND), U67.8 (GND), U68.7 (GND), U69.7 (GND), U7.1 (OE#), U7.10 (GND), U72.7 (GND), U73.1 (OE#), U73.10 (GND), U74.8 (GND), U8.10 (GND), U9.11 (B3), U9.15 (B2), U9.2 (B1), U9.6 (B0), U9.8 (GND), U93.8 (GND), U94.11 (B3), U94.12 (A3), U94.14 (A2), U94.15 (B2), U94.2 (B1), U94.3 (A1), U94.6 (B0), U94.8 (GND), U95.1 (OE#), U95.10 (GND), U97.7 (GND), U98.7 (GND), U99.7 (GND), R16.2, R17.2, R18.2, R19.2, U123.6 (0SET), U123.7 (GND), U123.8 (1SET), U124.7 (GND), U126.7 (GND), U127.7 (GND), U128.7 (GND), U129.7 (GND), U130.7 (GND), U131.12 (3A), U131.13 (3B), U131.7 (GND), U131.8 (2A), U131.9 (2B), U132.7 (GND), U133.7 (GND), U134.7 (GND), U135.7 (GND), U136.11 (I4), U136.13 (I5), U136.7 (GND), U136.9 (I3)
- net at U93.16 (V+): now also U1.20 (V+), U10.20 (V+), U100.14 (V+), U101.14 (V+), U102.14 (V+), U103.14 (V+), U104.14 (V+), U105.14 (V+), U106.14 (V+), U107.14 (V+), U11.20 (V+), U112.14 (V+), U113.14 (V+), U114.14 (V+), U115.14 (V+), U116.14 (V+), U117.14 (V+), U12.28 (V+), U120.14 (V+), U121.16 (V+), U13.20 (V+), U14.16 (V+), U15.20 (V+), U16.20 (V+), U17.16 (V+), U19.20 (V+), U2.12 (V+), U20.20 (V+), U21.20 (V+), U22.16 (V+), U22.7 (C_IN), U23.16 (V+), U24.14 (V+), U25.14 (V+), U26.14 (V+), U27.14 (V+), U28.16 (V+), U29.14 (V+), U3.28 (V+), U30.14 (V+), U31.11 (CLK), U31.20 (V+), U32.15 (CLR#), U32.23 (VDD), U33.20 (V+), U34.16 (V+), U35.11 (CLK), U35.20 (V+), U36.28 (V+), U37.11 (CLK), U37.20 (V+), U38.11 (CLK), U38.20 (V+), U39.20 (V+), U4.16 (V+), U4.7 (C_IN), U40.20 (V+), U41.20 (V+), U42.14 (V+), U43.14 (V+), U44.15 (CLR#), U44.23 (VDD), U45.11 (CLK), U45.20 (V+), U46.14 (V+), U47.14 (V+), U48.16 (V+), U48.5 (A0), U48.7 (C_IN), U49.16 (V+), U5.20 (V+), U50.14 (V+), U51.15 (CLR#), U51.23 (VDD), U52.15 (CLR#), U52.23 (VDD), U53.16 (V+), U55.16 (V+), U55.7 (C_IN), U56.16 (V+), U57.16 (V+), U58.14 (V+), U59.14 (V+), U6.20 (V+), U60.14 (V+), U61.14 (V+), U63.20 (V+), U64.20 (V+), U65.20 (V+), U66.16 (V+), U66.7 (C_IN), U67.16 (V+), U68.14 (V+), U69.14 (V+), U7.20 (V+), U72.1 (OE), U72.14 (V+), U73.20 (V+), U74.16 (V+), U74.7 (C_IN), U8.20 (V+), U9.16 (V+), U94.16 (V+), U95.20 (V+), U97.14 (V+), U98.14 (V+), U99.14 (V+), U123.14 (V+), U124.14 (V+), U126.14 (V+), U127.14 (V+), U128.14 (V+), U129.14 (V+), U130.14 (V+), U131.14 (V+), U132.14 (V+), U133.14 (V+), U134.14 (V+), U135.14 (V+), U136.14 (V+), U96.2 (B)
- net at U2.23 (ENABLE): now also U124.1 (1A), U124.9 (4B), U126.5 (2B), U130.2 (1B), U136.5 (I2)
- net at U53.6 (E1): now also U77.3 (OUT)
- net at U20.1 (OE#), U21.1 (OE#): now also U104.1 (1A), U104.4 (2A), U12.22 (OE#), U3.22 (OE#), U50.10 (O4)
- net at U30.3 (Q0), U92.1 (IN): now also U127.9 (I3)
- net at U32.10 (WR#), U44.10 (WR#), U51.10 (WR#)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: now also U117.10 (O4)
- net at U32.16 (LDAC#), U44.16 (LDAC#), U51.16 (LDAC#)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: now also U113.10 (O4)
- net at U32.8 (A0), U32.9 (A1), U44.8 (A0)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: now also U117.12 (O5), U63.1 (OE#), U64.1 (OE#)
- net at U81.1 (IN): now also U18.5 (Line_Done)
- net at U112.2 (0B), U81.3 (OUT): now also U132.4 (2A)
- net at U113.11 (I4): now also U85.3 (OUT)
- net at U78.1 (IN): now also U130.3 (1Q)
- net at U78.3 (OUT): now also U95.5 (D3)
- net at U19.11 (CLK): now also U28.11 (CCLK), U28.13 (RCLK), U33.11 (CLK), U79.3 (OUT)
- net at U114.11 (1CLK): now also U70.3 (OUT), U73.11 (CLK), U127.1 (I0), U129.2 (1B)
- net at U114.13 (1Q): now also U30.6 (1B), U128.6 (1B)
- net at U114.9 (1D): now also U132.11 (3Q)
- net at U117.11 (I4): now also U84.3 (OUT)
- net at U117.13 (I5): now also U65.1 (OE#), U83.3 (OUT)
- net at U119.1 (Out1_A), U120.6 (1B): now also R19.1
- net at U119.2 (Out2_A), U120.5 (1A): now also R17.1
- net at U119.5 (Out1_B), U120.2 (0B): now also R18.1
- net at U119.6 (Out2_B), U120.1 (0A): now also R16.1
- net at U65.11 (CLK): now also U63.11 (CLK), U64.11 (CLK), U82.3 (OUT)
- net at U121.6 (Q2), U35.4 (D2): now also U127.5 (I2), U129.9 (4B)
- net at U75.1 (IN): now also U73.18 (Q1), U95.3 (D1), U126.2 (1B), U133.9 (2B)
- net at U87.1 (IN): now also U133.1 (0A), U134.4 (O1)
- net at U88.1 (IN): now also U133.8 (2A), U134.8 (03)
- net at U91.1 (IN): now also U130.11 (3Q)
- net at U18.11 (+5V): now also U96.1 (A)
- net at U18.6 (Beam_Enable): now also U90.3 (OUT)
- net at U18.7 (Point_(0)_/_Line_(1)_Sel): now also U39.12 (Q7)
- net at U71.1 (IN): now also U126.3 (1Q)
- net at U107.11 (Q3): now also U124.10 (4A)
- net at U107.12 (3A): now also U112.11 (Q3)
- net at U107.13 (3B): now also U123.1 (0Q), U123.9 (1D)
- net at U90.1 (IN): now also U135.8 (2A), U136.4 (O1)
- net at U102.11 (1CLK), U103.3 (0CLK), U98.12 (O5): now also U123.3 (0CLK)
- net at U102.3 (0CLK), U103.11 (1CLK), U112.9 (2B)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: now also U124.13 (3A)
- net at U95.11 (CLK): now also U127.2 (O0), U129.5 (2B)
- net at U95.12 (Q7): now also U85.1 (IN), U132.12 (3B), U132.9 (4B)
- net at U95.13 (Q6): now also U73.9 (D7), U130.10 (4A)
- net at U95.14 (Q5): now also U73.8 (D6), U80.1 (IN), U127.11 (I4), U130.5 (2B), U131.2 (0B), U132.1 (1A)
- net at U95.15 (Q4): now also U73.7 (D5), U86.1 (IN)
- net at U95.16 (Q3): now also U73.6 (D4), U130.12 (3B), U133.6 (1B)
- net at U95.17 (Q2): now also U128.8 (2A), U129.10 (4A), U129.13 (3A)
- net at U95.18 (Q1): now also U126.10 (4A), U126.13 (3A), U135.13 (3B)
- net at U95.19 (Q0): now also U73.3 (D1), U126.1 (1A)
- net at U95.2 (D0): now also U30.5 (1A), U73.19 (Q0), U132.5 (2B)
- net at U95.4 (D2): now also U73.17 (Q2), U128.1 (0A)
- net at U95.6 (D4): now also U73.15 (Q4), U133.13 (3B), U135.2 (0B), U135.9 (2B)
- net at U95.7 (D5): now also U73.14 (Q5), U79.1 (IN), U82.1 (IN), U130.4 (2A), U131.1 (0A)
- net at U95.8 (D6): now also U73.13 (Q6)
- net at U95.9 (D7): now also U73.12 (Q7), U130.9 (4B)
- net at U122.1 (IN): now also U124.8 (4Q)
- net at U122.3 (OUT): now also U73.2 (D0)
- net at U77.1 (IN): now also U129.3 (1Q)
- net at U73.16 (Q3): now also U128.2 (0B), U128.5 (1A), U128.9 (2B)
- net at U73.4 (D2): now also U126.6 (2Q)
- net at U73.5 (D3): now also U129.8 (4Q)
- net at U76.1 (IN): now also U129.6 (2Q)
- net at U112.12 (3A): now also U126.11 (3Q)
- net at U112.13 (3B): now also U132.8 (4Q)
- net at U26.8 (4Q): now also U127.13 (I5), U132.10 (4A)
- net at U83.1 (IN): now also U131.3 (Q0)
- net at U80.3 (OUT): now also U60.13 (3B), U60.9 (2B)
- net at U84.1 (IN): now also U131.4 (Q1)
- new net: U135.10 (Q2), U136.1 (I0)
- new net: U135.12 (3A), U136.2 (O0)
- new net: U135.11 (Q3), U136.3 (I1)
- new net: U123.10 (1RESET), U123.4 (0RESET), U136.6 (O2)
- new net: U134.11 (I4), U135.3 (Q0)
- new net: U134.13 (I5), U135.4 (Q1)
- new net: U134.10 (O4), U135.5 (1A)
- new net: U132.6 (2Q), U135.6 (1B)
- new net: U128.3 (Q0), U129.1 (1A)
- new net: U128.12 (3A), U129.11 (3Q)
- new net: U127.6 (O2), U129.12 (3B)
- new net: U128.10 (Q2), U129.4 (2A)
- new net: U126.12 (3B), U127.4 (O1)
- new net: U126.4 (2A), U128.11 (Q3)
- new net: U126.8 (4Q), U128.13 (3B)
- new net: U133.3 (Q0), U134.1 (I0)
- new net: U133.5 (1A), U134.2 (O0)
- new net: U133.4 (Q1), U134.3 (I1)
- new net: U133.10 (Q2), U134.5 (I2)
- new net: U133.12 (3A), U134.6 (O2)
- new net: U133.11 (Q3), U134.9 (I3)
- new net: U127.12 (O5), U132.13 (3A)
- new net: U127.10 (O4), U132.2 (1B)
- new net: U132.3 (1Q), U133.2 (0B)
- new net: U128.4 (Q1), U130.1 (1A)
- new net: U130.6 (2Q), U131.5 (1A)
- new net: U130.8 (4Q), U131.6 (1B)
- new net: U123.11 (1CLK), U124.11 (3Q)
- new net: U123.12 (1Q#), U124.12 (3B), U124.2 (1B)
- new net: U124.3 (1Q), U124.4 (2A)
- new net: U123.2 (0Q#), U124.5 (2B)
- new net: U123.5 (0D), U124.6 (2Q)
- new net: U127.8 (03), U130.13 (3A)
- no-connect marks 42 -> 60
Other:
- note added: "0"
- note added: "1"
- note added: "Decoder 59"
- note added: "Decoder 60"
- note added: "Decoder 61"
- note added: "Falling"
- note added: "G29"
- note added: "G30"
- note added: "G31"
- note added: "G32"
- note added: "G33"
- note added: "G34"
- note added: "G35"
- note added: "G36"
- note added: "G37"
- note added: "G38"
- note added: "G39"
- note added: "G40"
- note added: "G41"
- note added: "G42"
- note added: "G43"
- note added: "G44"
- note added: "G45"
- note added: "G46"
- note added: "G47"
- note added: "G48"
- note added: "G49"
- note added: "G50"
- note added: "G51"
- note added: "G52"
- note added: "G53"
- note added: "G58"
- note added: "L27"
- note added: "L28"
- note added: "L54"
- note added: "L55"
- note added: "L56"
- note added: "L57"
- note added: "Pull down unconnected jumper pins"
- note added: "Rising"
- note added: "Rising 8"
- note removed: "APP CLK"
- note removed: "APP CLK #"
- moved on the sheet: U73, U95

Commit message: Satisfied ERC
Connections:
- net at R16.2, R17.2, R18.2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: now also U100.10 (4A), U100.12 (3B), U100.13 (3A), U100.9 (4B), U115.10 (4A), U115.12 (3B), U115.13 (3A), U115.14 (V+), U115.9 (4B), U61.10 (4A), U61.9 (4B), U69.10 (4A), U69.9 (4B); no longer U115.2 (1B), U115.3 (1Q), U115.5 (2B), U115.6 (2Q), U115.7 (GND)
- net at U1.20 (V+), U10.20 (V+), U100.14 (V+)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: now also U115.7 (GND); no longer U115.14 (V+)
- net at U114.1 (0Q): now also U115.1 (1A); no longer U115.8 (4Q)
- net at U114.2 (0Q#): now also U115.4 (2A); no longer U115.11 (3Q)
- net at U116.1 (0A): now also U115.3 (1Q); no longer U115.10 (4A)
- net at U116.5 (1A): now also U115.6 (2Q); no longer U115.13 (3A)
- net at U104.10 (4A), U104.13 (3A), U50.12 (O5): now also U35.1 (OE#), U36.22 (OE#), U37.1 (OE#), U38.1 (OE#), U45.1 (OE#)
- new net: U115.2 (1B), U115.5 (2B), U26.3 (1Q)
- no-connect marks 60 -> 68
Other:
- moved on the sheet: U115

Commit message: Bus loading fixed
Parts:
- removed U131: ~, Package_DIP:DIP-14_W7.62mm, symbol custom_symbol_lib:quad_OR
- removed U31: ~, Package_DIP:DIP-20_W7.62mm, symbol custom_symbol_lib:8_bit_transparent_latch
- added U125: ~, Package_DIP:DIP-14_W7.62mm, symbol custom_symbol_lib:6xNOT
- added U139, U140, U141: ~, Package_DIP:DIP-20_W7.62mm, symbol custom_symbol_lib:rising_edge_8_bit_latch
- added U31: ~, Package_DIP:DIP-14_W7.62mm, symbol custom_symbol_lib:quad_and
Connections:
- net 0: now also U139.2 (D0); no longer U13.2 (D0), U15.2 (D0)
- net 1: now also U139.3 (D1); no longer U13.3 (D1), U15.3 (D1)
- net 2: now also U139.4 (D2); no longer U13.4 (D2), U15.4 (D2)
- net 3: now also U139.5 (D3); no longer U13.5 (D3), U15.5 (D3)
- net 4: now also U139.6 (D4); no longer U13.6 (D4), U15.6 (D4)
- net 5: now also U139.7 (D5); no longer U13.7 (D5), U15.7 (D5)
- net 6: now also U139.8 (D6); no longer U13.8 (D6), U15.8 (D6)
- net 7: now also U100.2 (1B), U139.9 (D7); no longer U13.9 (D7), U15.9 (D7)
- net SpriteData0: now also U15.19 (Q0); no longer U8.19 (Q0)
- net SpriteData1: now also U15.18 (Q1); no longer U8.18 (Q1)
- net SpriteData2: now also U15.17 (Q2); no longer U8.17 (Q2)
- net SpriteData3: now also U15.16 (Q3); no longer U8.16 (Q3)
- net SpriteData4: now also U15.15 (Q4); no longer U8.15 (Q4)
- net SpriteData5: now also U15.14 (Q5); no longer U8.14 (Q5)
- net SpriteData6: now also U15.13 (Q6); no longer U8.13 (Q6)
- net SpriteData7: now also U15.12 (Q7); no longer U8.12 (Q7)
- net SpriteMemAddr0: now also U7.19 (Q0)
- net SpriteMemAddr1: now also U7.18 (Q1)
- net SpriteMemAddr11: now also U16.16 (Q3); no longer U7.16 (Q3)
- net SpriteMemAddr12: now also U16.15 (Q4); no longer U7.15 (Q4)
- net SpriteMemAddr13: now also U16.14 (Q5); no longer U7.14 (Q5)
- net SpriteMemAddr14: now also U16.13 (Q6); no longer U7.13 (Q6)
- net SpriteMemAddr2: now also U7.17 (Q2)
- net VectorMemY0: now also U140.19 (Q0); no longer U15.19 (Q0)
- net VectorMemY1: now also U140.18 (Q1); no longer U15.18 (Q1)
- net VectorMemY2: now also U140.17 (Q2); no longer U15.17 (Q2)
- net VectorMemY3: now also U140.16 (Q3); no longer U15.16 (Q3)
- net VectorMemY4: now also U140.15 (Q4); no longer U15.15 (Q4)
- net VectorMemY5: now also U140.14 (Q5); no longer U15.14 (Q5)
- net VectorMemY6: now also U140.13 (Q6); no longer U15.13 (Q6)
- net VectorMemY7: now also U140.12 (Q7); no longer U15.12 (Q7)
- net at R16.2, R17.2, R18.2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: now also U100.4 (2A), U100.5 (2B), U8.1 (OE#), U139.1 (OE#), U139.10 (GND), U140.10 (GND), U141.1 (OE#), U141.10 (GND), U31.7 (GND); no longer U100.10 (4A), U100.12 (3B), U100.13 (3A), U100.9 (4B), U115.10 (4A), U115.12 (3B), U115.13 (3A), U115.9 (4B), U120.12 (3A), U120.13 (3B), U120.8 (2A), U120.9 (2B), U136.11 (I4), U136.9 (I3), U7.1 (OE#)
- net at U1.20 (V+), U10.20 (V+), U100.14 (V+)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: now also U31.14 (V+); no longer U13.20 (V+), U15.20 (V+), U8.20 (V+), U98.14 (V+), U99.14 (V+)
- net at U48.12 (A3): now also U141.16 (Q3); no longer U16.16 (Q3)
- net at U48.14 (A2): now also U141.17 (Q2); no longer U16.17 (Q2)
- net at U48.3 (A1): now also U141.18 (Q1); no longer U16.18 (Q1)
- net at U101.2 (0B), U6.11 (CLK), U97.6 (2Q): now also U100.1 (1A)
- net at U10.9 (D7), U6.12 (Q7), U7.9 (D7): now also U105.10 (4A), U105.4 (2A), U50.5 (I2)
- net at U10.1 (OE#), U11.1 (OE#), U13.1 (OE#)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: now also U140.1 (OE#); no longer U15.1 (OE#)
- net at U108.3 (OUT), U50.9 (I3): now also U115.13 (3A), U136.9 (I3)
- net at U5.1 (OE#), U58.6 (O2): now also U15.1 (OE#), U7.1 (OE#); no longer U8.1 (OE#)
- net at U8.11 (CLK), U97.11 (3Q), U99.2 (0B): no longer U101.9 (2B), U13.11 (CLK)
- net at U16.12 (Q7): no longer U49.12 (A3)
- net at U49.14 (A2): now also U141.13 (Q6); no longer U16.13 (Q6)
- net at U49.3 (A1): now also U141.14 (Q5); no longer U16.14 (Q5)
- net at U49.5 (A0): now also U141.15 (Q4); no longer U16.15 (Q4)
- net at U58.1 (I0), U59.1 (1A), U59.10 (4A)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: now also U141.19 (Q0); no longer U16.19 (Q0)
- net at U110.3 (OUT), U58.5 (I2): now also U115.10 (4A), U136.11 (I4)
- net at U136.10 (O4): now also U115.9 (4B)
- net at U136.8 (03): now also U115.12 (3B)
- net at U98.4 (O1), U99.1 (0A): now also U100.10 (4A), U101.5 (1A), U31.4 (2A); no longer U100.1 (1A)
- net at U98.8 (03), U99.8 (2A): now also U101.6 (1B), U31.10 (4A), U31.13 (3A); no longer U100.4 (2A)
- net at U127.11 (I4), U130.5 (2B), U132.1 (1A)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: now also U120.9 (2B)
- net at U130.4 (2A), U73.14 (Q5), U79.1 (IN)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: now also U120.8 (2A)
- net at U120.10 (Q2): now also U83.1 (IN)
- net at U120.11 (Q3): now also U84.1 (IN)
- net at U115.11 (3Q): now also U100.9 (4B), U31.2 (1B), U31.9 (4B)
- net at U115.8 (4Q): now also U100.12 (3B), U31.12 (3B), U31.5 (2B)
- net at U100.3 (1Q): now also U16.11 (CLK); no longer U101.5 (1A)
- net at U100.6 (2Q): no longer U101.6 (1B)
- net at U130.6 (2Q): now also U120.12 (3A)
- net at U130.8 (4Q): now also U120.13 (3B)
- net at U100.11 (3Q): now also U5.11 (CLK), U7.11 (CLK)
- net at U100.8 (4Q): now also U13.11 (CLK)
- new net: U10.11 (CLK), U11.11 (CLK), U31.3 (1Q)
- new net: U13.9 (D7), U15.9 (D7), U8.12 (Q7)
- new net: U13.8 (D6), U15.8 (D6), U8.13 (Q6)
- new net: U13.7 (D5), U15.7 (D5), U8.14 (Q5)
- new net: U13.6 (D4), U15.6 (D4), U8.15 (Q4)
- new net: U13.5 (D3), U15.5 (D3), U8.16 (Q3)
- new net: U13.4 (D2), U15.4 (D2), U8.17 (Q2)
- new net: U13.3 (D1), U15.3 (D1), U8.18 (Q1)
- new net: U13.2 (D0), U15.2 (D0), U8.19 (Q0)
- new net: U15.20 (V+), U8.20 (V+)
- new net: U139.11 (CLK), U97.8 (4Q), U99.9 (2B)
- new net: U139.12 (Q7), U140.9 (D7), U141.9 (D7)
- new net: U139.13 (Q6), U140.8 (D6), U141.8 (D6)
- new net: U139.14 (Q5), U140.7 (D5), U141.7 (D5)
- new net: U139.15 (Q4), U140.6 (D4), U141.6 (D4)
- new net: U139.16 (Q3), U140.5 (D3), U141.5 (D3)
- new net: U139.17 (Q2), U140.4 (D2), U141.4 (D2)
- new net: U139.18 (Q1), U140.3 (D1), U141.3 (D1)
- new net: U139.19 (Q0), U140.2 (D0), U141.2 (D0)
- new net: U139.20 (V+), U141.20 (V+)
- new net: U98.14 (V+), U99.14 (V+)
- new net: U15.11 (CLK), U31.6 (2Q)
- new net: U141.11 (CLK), U31.11 (3Q)
- new net: U141.12 (Q7), U49.12 (A3)
- new net: U100.13 (3A), U101.4 (Q1), U31.1 (1A)
- new net: U140.11 (CLK), U31.8 (4Q)
- now unconnected: U101.10 (Q2), U101.8 (2A), U7.12 (Q7)
- no-connect marks 68 -> 63
Other:
- note added: "G62"
- note added: "G63"
- note added: "G64"
- note added: "G65"
- note added: "G66"
- note added: "G67"
- note added: "G68"
- note added: "G69"
- note added: "G70"
- note added: "G71"
- note added: "G72"
- note added: "G73"
- note added: "G74"
- note added: "G75"
- note added: "G76"
- note added: "G77"
- note added: "G78"
- note added: "G79"
- note added: "L81"
- note added: "L82"
- note removed: "Input corruption prevention SR latches"
- note removed: "Reset"
- note removed: "Sprite frame and MSB must always be enabled, so put transparent latch for rest of spreite addressing"
- moved on the sheet: R1, R10, R11, R12, R13, R14, R15, R16, R17, R18, R19, R2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

Commit message: Vector thingy almost completely verified except math and DAC stuff
Parts:
- removed U125: ~, Package_DIP:DIP-14_W7.62mm, symbol custom_symbol_lib:6xNOT
- removed U28: ~, Package_DIP:DIP-16_W7.62mm, symbol custom_symbol_lib:8_bit_counter
- added U28: ~, Package_DIP:DIP-16_W7.62mm, symbol custom_symbol_lib:12_bit_counter_no_output_latch
Connections:
- net at R16.2, R17.2, R18.2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: now also U101.8 (2A), U101.9 (2B), U28.8 (GND)
- net at U1.20 (V+), U10.20 (V+), U100.14 (V+)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: now also U13.20 (V+), U139.20 (V+), U140.20 (V+), U141.20 (V+), U15.20 (V+), U8.20 (V+), U98.14 (V+), U99.14 (V+), U28.16 (V+)
- net at U19.11 (CLK), U33.11 (CLK), U79.3 (OUT): now also U58.11 (I4)
- net at U24.9 (3B), U29.1 (0A): now also U28.7 (Q1)
- net at U58.10 (O4): now also U28.10 (CLK#)
- net at U24.13 (4B): now also U28.9 (Q0)
- net at U24.6 (2B), U29.2 (0B): now also U28.6 (Q2)
- net at U24.2 (1B), U29.5 (1A): now also U28.5 (Q3)
- net at U27.13 (4B), U29.6 (1B): now also U28.3 (Q4)
- net at U27.9 (3B), U29.8 (2A): now also U28.2 (Q5)
- net at U27.6 (2B), U29.9 (2B): now also U28.4 (Q6)
- net at U75.3 (OUT): now also U28.11 (Reset); no longer U58.11 (I4)
- no-connect marks 63 -> 68
Other:
- note added: "G10"
- note added: "G83"
- note added: "G84"
- note added: "G86"
- note removed: "Gate 10"
