File: kicad/vector_digital_controller/vector_digital_controller.kicad_sch (KiCad schematic)
At the start: 156 parts

Commit message: Vector graphics board finished
Parts:
- renumbered U15 to U420, U28 to U421, U38 to U422, U31 to U423, U13 to U424, U8 to U425
Changed lines of the file:
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@@
 		(dnp no)
 		(fields_autoplaced yes)
-		(property "Reference" "U38"
-			(at 436.5341 328.93 0)
+		(property "Reference" "U422"
+			(at 436.4833 327.66 0)
 			(effects
 				(font
@@
 		)
 		(property "Value" "~"
-			(at 436.5341 331.47 0)
+			(at 436.4833 330.2 0)
 			(effects
 				(font
@@
 			(project "vector_digital_controller"
 				(path "/efcfb5e8-5771-4082-b7fd-a57c87392461"
-					(reference "U38")
+					(reference "U422")
 					(unit 1)
 				)
@@
 		(dnp no)
 		(fields_autoplaced yes)
-		(property "Reference" "U8"
-			(at 177.4541 172.72 0)
+		(property "Reference" "U425"
+			(at 177.4033 171.45 0)
 			(effects
 				(font
@@
 		)
 		(property "Value" "~"
-			(at 177.4541 175.26 0)
+			(at 177.4033 173.99 0)
 			(effects
 				(font
@@
 			(project "vector_digital_controller"
 				(path "/efcfb5e8-5771-4082-b7fd-a57c87392461"
-					(reference "U8")
+					(reference "U425")
 					(unit 1)
 				)
@@
 		(dnp no)
 		(fields_autoplaced yes)
-		(property "Reference" "U15"
-			(at 214.2841 172.72 0)
+		(property "Reference" "U420"
+			(at 214.2333 171.45 0)
 			(effects
 				(font
@@
 		)
 		(property "Value" "~"
-			(at 214.2841 175.26 0)
+			(at 214.2333 173.99 0)
 			(effects
 				(font
@@
 			(project "vector_digital_controller"
 				(path "/efcfb5e8-5771-4082-b7fd-a57c87392461"
-					(reference "U15")
+					(reference "U420")
 					(unit 1)
 				)
@@
 		(on_board yes)
 		(dnp no)
-		(property "Reference" "U13"
+		(property "Reference" "U424"
 			(at 213.868 147.066 0)
 			(effects
@@
 			(project "vector_digital_controller"
 				(path "/efcfb5e8-5771-4082-b7fd-a57c87392461"
-					(reference "U13")
+					(reference "U424")
 					(unit 1)
 				)
@@
 		(dnp no)
 		(fields_autoplaced yes)
-		(property "Reference" "U31"
-			(at 182.5341 318.77 0)
+		(property "Reference" "U423"
+			(at 182.4833 317.5 0)
 			(effects
 				(font
@@
 		)
 		(property "Value" "~"
-			(at 182.5341 321.31 0)
+			(at 182.4833 320.04 0)
 			(effects
 				(font
@@
 			(project "vector_digital_controller"
 				(path "/efcfb5e8-5771-4082-b7fd-a57c87392461"
-					(reference "U31")
+					(reference "U423")
 					(unit 1)
 				)
@@
 		(dnp no)
 		(fields_autoplaced yes)
-		(property "Reference" "U28"
+		(property "Reference" "U421"
 			(at 599.8767 369.57 0)
 			(effects
@@
 			(project "vector_digital_controller"
 				(path "/efcfb5e8-5771-4082-b7fd-a57c87392461"
-					(reference "U28")
+					(reference "U421")
 					(unit 1)
 				)

Commit message: Moved rusty logic circuits into this repo
Parts:
- U18: footprint Connector_PinHeader_2.54mm:PinHeader_1x11_P2.54mm_Vertical -> Connector_PinHeader_2.54mm:PinHeader_1x12_P2.54mm_Vertical
Connections:
- net at U102.3 (0CLK), U103.11 (1CLK), U112.9 (2B)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: now also U18.12 (Digital_CLK)
