File: kicad/vector_digital_controller/vector_digital_controller.kicad_pcb (KiCad board)
At the start: 2 copper layers, 50 parts

Commit message: Progress on vector thingy
Parts:
- added R1: R, custom_footprint_library:0.4_pitch_resistor, F.Cu at (140.5, 84.3)
- added R10: R, custom_footprint_library:0.4_pitch_resistor, F.Cu at (173.3, 84.3)
- added R11: R, custom_footprint_library:0.4_pitch_resistor, F.Cu at (176.9, 84.3)
- added R12: R, custom_footprint_library:0.4_pitch_resistor, F.Cu at (180.5, 84.3)
- added R13: R, custom_footprint_library:0.4_pitch_resistor, F.Cu at (184.2, 84.3)
- added R14: R, custom_footprint_library:0.4_pitch_resistor, F.Cu at (187.8, 84.3)
- added R15: R, custom_footprint_library:0.4_pitch_resistor, F.Cu at (191.5, 84.3)
- added R2: R, custom_footprint_library:0.4_pitch_resistor, F.Cu at (144.1, 84.3)
- added R3: R, custom_footprint_library:0.4_pitch_resistor, F.Cu at (147.8, 84.3)
- added R4: R, custom_footprint_library:0.4_pitch_resistor, F.Cu at (151.4, 84.3)
- added R5: R, custom_footprint_library:0.4_pitch_resistor, F.Cu at (155.1, 84.3)
- added R6: R, custom_footprint_library:0.4_pitch_resistor, F.Cu at (158.7, 84.3)
- added R7: R, custom_footprint_library:0.4_pitch_resistor, F.Cu at (162.3, 84.3)
- added R8: R, custom_footprint_library:0.4_pitch_resistor, F.Cu at (166.0, 84.3)
- added R9: R, custom_footprint_library:0.4_pitch_resistor, F.Cu at (169.6, 84.3)
- added U100: ~, Package_DIP:DIP-14_W7.62mm, F.Cu at (43.2, 55.7)
- added U101: ~, Package_DIP:DIP-14_W7.62mm, F.Cu at (54.0, 55.7)
- added U102: ~, Package_DIP:DIP-14_W7.62mm, F.Cu at (64.8, 55.7)
- added U103: ~, Package_DIP:DIP-14_W7.62mm, F.Cu at (75.6, 55.7)
- added U104: ~, Package_DIP:DIP-14_W7.62mm, F.Cu at (86.4, 55.7)
- added U105: ~, Package_DIP:DIP-14_W7.62mm, F.Cu at (97.2, 55.7)
- added U106: ~, Package_DIP:DIP-14_W7.62mm, F.Cu at (107.9, 55.7)
- added U107: ~, Package_DIP:DIP-14_W7.62mm, F.Cu at (118.7, 55.7)
- added U108: ~, custom_footprint_library:jumper, F.Cu at (190.7, 32.0)
- added U109: ~, custom_footprint_library:jumper, F.Cu at (190.7, 41.0)
- added U110: ~, custom_footprint_library:jumper, F.Cu at (190.7, 49.9)
- added U111: ~, custom_footprint_library:jumper, F.Cu at (190.7, 58.8)
- added U112: ~, Package_DIP:DIP-14_W7.62mm, F.Cu at (129.5, 55.7)
- added U113: ~, Package_DIP:DIP-14_W7.62mm, F.Cu at (32.5, 75.1)
- added U114: ~, Package_DIP:DIP-14_W7.62mm, F.Cu at (43.2, 75.1)
- added U115: ~, Package_DIP:DIP-14_W7.62mm, F.Cu at (54.0, 75.1)
- added U116: ~, Package_DIP:DIP-14_W7.62mm, F.Cu at (64.8, 75.1)
- added U117: ~, Package_DIP:DIP-14_W7.62mm, F.Cu at (75.6, 75.1)
- added U118: ~, custom_footprint_library:jumper, F.Cu at (190.7, 67.7)
- added U119: ~, Connector_PinHeader_2.54mm:PinHeader_2x03_P2.54mm_Vertical, F.Cu at (80.9, 190.6)
- added U120: ~, Package_DIP:DIP-14_W7.62mm, F.Cu at (86.4, 75.1)
- added U51: ~, Package_DIP:DIP-24_W7.62mm, F.Cu at (54.0, 175.2)
- added U52: ~, Package_DIP:DIP-24_W7.62mm, F.Cu at (64.8, 175.2)
- added U53: ~, Package_DIP:DIP-16_W7.62mm, F.Cu at (172.6, 116.3)
- added U54: ~, custom_footprint_library:jumper, F.Cu at (145.0, 23.1)
- added U55: ~, Package_DIP:DIP-16_W7.62mm, F.Cu at (183.4, 116.3)
- added U56: ~, Package_DIP:DIP-16_W7.62mm, F.Cu at (194.2, 116.3)
- added U57: ~, Package_DIP:DIP-16_W7.62mm, F.Cu at (129.5, 138.1)
- added U58: ~, Package_DIP:DIP-14_W7.62mm, F.Cu at (43.2, 36.4)
- added U59: ~, Package_DIP:DIP-14_W7.62mm, F.Cu at (54.0, 36.4)
- added U60: ~, Package_DIP:DIP-14_W7.62mm, F.Cu at (64.8, 36.4)
- added U61: ~, Package_DIP:DIP-14_W7.62mm, F.Cu at (75.6, 36.4)
- added U62: ~, custom_footprint_library:jumper, F.Cu at (145.0, 32.0)
- added U63: ~, Package_DIP:DIP-20_W7.62mm, F.Cu at (64.8, 148.3)
- added U64: ~, Package_DIP:DIP-20_W7.62mm, F.Cu at (75.6, 148.3)
- added U65: ~, Package_DIP:DIP-20_W7.62mm, F.Cu at (86.4, 148.3)
- added U66: ~, Package_DIP:DIP-16_W7.62mm, F.Cu at (140.3, 138.1)
- added U67: ~, Package_DIP:DIP-16_W7.62mm, F.Cu at (151.1, 138.1)
- added U68: ~, Package_DIP:DIP-14_W7.62mm, F.Cu at (86.4, 36.4)
- added U69: ~, Package_DIP:DIP-14_W7.62mm, F.Cu at (97.2, 36.4)
- added U70: ~, custom_footprint_library:jumper, F.Cu at (145.0, 41.0)
- added U71: ~, custom_footprint_library:jumper, F.Cu at (145.0, 49.9)
- added U72: ~, custom_footprint_library:crystal_dip_14, F.Cu at (90.1, 180.7)
- added U73: ~, Package_DIP:DIP-20_W7.62mm, F.Cu at (97.2, 148.3)
- added U74: ~, Package_DIP:DIP-16_W7.62mm, F.Cu at (161.8, 138.1)
- added U75: ~, custom_footprint_library:jumper, F.Cu at (145.0, 58.8)
- added U76: ~, custom_footprint_library:jumper, F.Cu at (145.0, 67.7)
- added U77: ~, custom_footprint_library:jumper, F.Cu at (145.0, 76.6)
- added U78: ~, custom_footprint_library:jumper, F.Cu at (160.3, 23.1)
- added U79: ~, custom_footprint_library:jumper, F.Cu at (160.3, 32.0)
- added U80: ~, custom_footprint_library:jumper, F.Cu at (160.3, 41.0)
- added U81: ~, custom_footprint_library:jumper, F.Cu at (160.3, 49.9)
- added U82: ~, custom_footprint_library:jumper, F.Cu at (160.3, 58.8)
- added U83: ~, custom_footprint_library:jumper, F.Cu at (160.3, 67.7)
- added U84: ~, custom_footprint_library:jumper, F.Cu at (160.3, 76.6)
- added U85: ~, custom_footprint_library:jumper, F.Cu at (175.5, 23.1)
- added U86: ~, custom_footprint_library:jumper, F.Cu at (175.5, 32.0)
- added U87: ~, custom_footprint_library:jumper, F.Cu at (175.5, 41.0)
- added U88: ~, custom_footprint_library:jumper, F.Cu at (175.5, 49.9)
- added U89: ~, custom_footprint_library:jumper, F.Cu at (175.5, 58.8)
- added U90: ~, custom_footprint_library:jumper, F.Cu at (175.5, 67.7)
- added U91: ~, custom_footprint_library:jumper, F.Cu at (175.5, 76.6)
- added U92: ~, custom_footprint_library:jumper, F.Cu at (190.7, 23.1)
- added U93: ~, Package_DIP:DIP-16_W7.62mm, F.Cu at (172.6, 138.1)
- added U94: ~, Package_DIP:DIP-16_W7.62mm, F.Cu at (183.4, 138.1)
- added U95: ~, Package_DIP:DIP-20_W7.62mm, F.Cu at (107.9, 148.3)
- added U96: ~, Package_DIP:DIP-14_W7.62mm, F.Cu at (107.9, 36.4)
- added U97: ~, Package_DIP:DIP-14_W7.62mm, F.Cu at (118.7, 36.4)
- added U98: ~, Package_DIP:DIP-14_W7.62mm, F.Cu at (129.5, 36.4)
- added U99: ~, Package_DIP:DIP-14_W7.62mm, F.Cu at (32.5, 55.7)
- U18: footprint Package_DIP:DIP-20_W7.62mm -> Connector_PinHeader_2.54mm:PinHeader_1x11_P2.54mm_Vertical
- U22, U23, U28: footprint Package_DIP:DIP-20_W7.62mm -> Package_DIP:DIP-16_W7.62mm
- U24, U25, U26, U27, U29, U30: footprint Package_DIP:DIP-20_W7.62mm -> Package_DIP:DIP-14_W7.62mm
- U32, U44: footprint Package_DIP:DIP-20_W7.62mm -> Package_DIP:DIP-24_W7.62mm
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Connections:
- U1 pad 1: unconnected-(U1-OE#-Pad1) -> Net-(U1-GND)
- U1 pad 10: unconnected-(U1-GND-Pad10) -> Net-(U1-GND)
- U1 pad 11: unconnected-(U1-CLK-Pad11) -> Net-(U1-CLK)
- U1 pad 12: /7 -> Net-(U1-Q7)
- U1 pad 13: /6 -> Net-(U1-Q6)
- U1 pad 14: /5 -> Net-(U1-Q5)
- U1 pad 15: /4 -> Net-(U1-Q4)
- U1 pad 16: /3 -> Net-(U1-Q3)
- U1 pad 17: /2 -> Net-(U1-Q2)
- U1 pad 18: /1 -> Net-(U1-Q1)
- U1 pad 19: /0 -> Net-(U1-Q0)
- U10 pad 1: unconnected-(U10-OE#-Pad1) -> Net-(U10-OE#)
- U10 pad 11: unconnected-(U10-CLK-Pad11) -> Net-(U10-CLK)
- U10 pad 13: unconnected-(U10-Q6-Pad13) -> /VectorAddress14
- U10 pad 14: unconnected-(U10-Q5-Pad14) -> /VectorAddress13
- U10 pad 15: unconnected-(U10-Q4-Pad15) -> /VectorAddress12
- U10 pad 16: unconnected-(U10-Q3-Pad16) -> /VectorAddress11
- U10 pad 17: unconnected-(U10-Q2-Pad17) -> /VectorAddress10
- U10 pad 18: unconnected-(U10-Q1-Pad18) -> /VectorAddress9
- U10 pad 19: unconnected-(U10-Q0-Pad19) -> /VectorAddress8
- U10 pad 2: /0 -> Net-(U10-D0)
- U10 pad 3: /1 -> Net-(U10-D1)
- U10 pad 4: /2 -> Net-(U10-D2)
- U10 pad 5: /3 -> Net-(U10-D3)
- U10 pad 6: /4 -> Net-(U10-D4)
- U10 pad 7: /5 -> Net-(U10-D5)
- U10 pad 8: /6 -> Net-(U10-D6)
- U10 pad 9: /7 -> Net-(U10-D7)
- U11 pad 1: unconnected-(U11-OE#-Pad1) -> Net-(U10-OE#)
- U11 pad 11: unconnected-(U11-CLK-Pad11) -> Net-(U10-CLK)
- U11 pad 12: unconnected-(U11-Q7-Pad12) -> /VectorAddress7
- U11 pad 13: unconnected-(U11-Q6-Pad13) -> /VectorAddress6
- U11 pad 14: unconnected-(U11-Q5-Pad14) -> /VectorAddress5
- U11 pad 15: unconnected-(U11-Q4-Pad15) -> /VectorAddress4
- U11 pad 16: unconnected-(U11-Q3-Pad16) -> /VectorAddress3
- U11 pad 17: unconnected-(U11-Q2-Pad17) -> /VectorAddress2
- U11 pad 18: unconnected-(U11-Q1-Pad18) -> /VectorAddress1
- U11 pad 19: unconnected-(U11-Q0-Pad19) -> /VectorAddress0
- U11 pad 2: /0 -> Net-(U1-Q0)
- U11 pad 3: /1 -> Net-(U1-Q1)
- U11 pad 4: /2 -> Net-(U1-Q2)
- U11 pad 5: /3 -> Net-(U1-Q3)
- U11 pad 6: /4 -> Net-(U1-Q4)
- U11 pad 7: /5 -> Net-(U1-Q5)
- U11 pad 8: /6 -> Net-(U1-Q6)
- U11 pad 9: /7 -> Net-(U1-Q7)
- U12 pad 1: unconnected-(U12-A14-Pad1) -> /VectorAddress14
- U12 pad 10: unconnected-(U12-A0-Pad10) -> /VectorAddress0
- U12 pad 11: unconnected-(U12-D0-Pad11) -> /VectorMemY0
- U12 pad 12: unconnected-(U12-D1-Pad12) -> /VectorMemY1
- U12 pad 13: unconnected-(U12-D2-Pad13) -> /VectorMemY2
- U12 pad 15: unconnected-(U12-D3-Pad15) -> /VectorMemY3
- U12 pad 16: unconnected-(U12-D4-Pad16) -> /VectorMemY4
- U12 pad 17: unconnected-(U12-D5-Pad17) -> /VectorMemY5
- U12 pad 18: unconnected-(U12-D6-Pad18) -> /VectorMemY6
- U12 pad 19: unconnected-(U12-D7-Pad19) -> /VectorMemY7
- U12 pad 2: unconnected-(U12-A12-Pad2) -> /VectorAddress12
- U12 pad 21: unconnected-(U12-A10-Pad21) -> /VectorAddress10
- U12 pad 23: unconnected-(U12-A11-Pad23) -> /VectorAddress11
- U12 pad 24: unconnected-(U12-A9-Pad24) -> /VectorAddress9
- U12 pad 25: unconnected-(U12-A8-Pad25) -> /VectorAddress8
- U12 pad 26: unconnected-(U12-A13-Pad26) -> /VectorAddress13
- U12 pad 27: unconnected-(U12-WE#-Pad27) -> Net-(U12-WE#)
- U12 pad 3: unconnected-(U12-A7-Pad3) -> /VectorAddress7
- U12 pad 4: unconnected-(U12-A6-Pad4) -> /VectorAddress6
- U12 pad 5: unconnected-(U12-A5-Pad5) -> /VectorAddress5
- U12 pad 6: unconnected-(U12-A4-Pad6) -> /VectorAddress4
- U12 pad 7: unconnected-(U12-A3-Pad7) -> /VectorAddress3
- U12 pad 8: unconnected-(U12-A2-Pad8) -> /VectorAddress2
- U12 pad 9: unconnected-(U12-A1-Pad9) -> /VectorAddress1
- U13 pad 1: unconnected-(U13-OE#-Pad1) -> Net-(U10-OE#)
- U13 pad 11: unconnected-(U13-CLK-Pad11) -> Net-(U101-2B)
- U13 pad 12: unconnected-(U13-Q7-Pad12) -> /VectorMemX7
- U13 pad 13: unconnected-(U13-Q6-Pad13) -> /VectorMemX6
- U13 pad 14: unconnected-(U13-Q5-Pad14) -> /VectorMemX5
- U13 pad 15: unconnected-(U13-Q4-Pad15) -> /VectorMemX4
- U13 pad 16: unconnected-(U13-Q3-Pad16) -> /VectorMemX3
- U13 pad 17: unconnected-(U13-Q2-Pad17) -> /VectorMemX2
- U13 pad 18: unconnected-(U13-Q1-Pad18) -> /VectorMemX1
- U13 pad 19: unconnected-(U13-Q0-Pad19) -> /VectorMemX0
- U15 pad 1: unconnected-(U15-OE#-Pad1) -> Net-(U10-OE#)
- U15 pad 11: unconnected-(U15-CLK-Pad11) -> Net-(U101-2A)
- U15 pad 12: unconnected-(U15-Q7-Pad12) -> /VectorMemY7
- U15 pad 13: unconnected-(U15-Q6-Pad13) -> /VectorMemY6
- U15 pad 14: unconnected-(U15-Q5-Pad14) -> /VectorMemY5
- U15 pad 15: unconnected-(U15-Q4-Pad15) -> /VectorMemY4
- U15 pad 16: unconnected-(U15-Q3-Pad16) -> /VectorMemY3
- U15 pad 17: unconnected-(U15-Q2-Pad17) -> /VectorMemY2
- U15 pad 18: unconnected-(U15-Q1-Pad18) -> /VectorMemY1
- U15 pad 19: unconnected-(U15-Q0-Pad19) -> /VectorMemY0
- U16 pad 1: unconnected-(U16-OE#-Pad1) -> Net-(U16-GND)
- U16 pad 10: unconnected-(U16-GND-Pad10) -> Net-(U16-GND)
- U16 pad 11: unconnected-(U16-CLK-Pad11) -> Net-(U101-2A)
- U16 pad 12: unconnected-(U16-Q7-Pad12) -> Net-(U16-Q7)
- U16 pad 13: unconnected-(U16-Q6-Pad13) -> Net-(U16-Q6)
- U16 pad 14: unconnected-(U16-Q5-Pad14) -> Net-(U16-Q5)
- U16 pad 15: unconnected-(U16-Q4-Pad15) -> Net-(U16-Q4)
- U16 pad 16: unconnected-(U16-Q3-Pad16) -> Net-(U16-Q3)
- U16 pad 17: unconnected-(U16-Q2-Pad17) -> Net-(U16-Q2)
- U16 pad 18: unconnected-(U16-Q1-Pad18) -> Net-(U16-Q1)
- U16 pad 19: unconnected-(U16-Q0-Pad19) -> Net-(U16-Q0)
- U17 pad 10: Net-(U17-Σ3) -> unconnected-(U17-Σ3-Pad10)
- U17 pad 11: Net-(U17-B0) -> Net-(U17-A3)
- U17 pad 15: Net-(U17-B0) -> Net-(U17-A3)
- U17 pad 2: Net-(U17-B0) -> Net-(U17-A3)
- U17 pad 6: Net-(U17-B0) -> Net-(U17-A3)
- U17 pad 8: Net-(U17-B0) -> Net-(U17-A3)
- U18 pad 1: unconnected-(U18-OE#-Pad1) -> Net-(U18-X0)
- U18 pad 2: Net-(U14-Σ0) -> Net-(U18-Y0)
- U18 pad 3: Net-(U14-Σ1) -> Net-(U18-X1)
- U18 pad 4: Net-(U14-Σ2) -> Net-(U18-Y1)
- U18 pad 5: Net-(U14-Σ3) -> unconnected-(U18-Line_Done-Pad5)
- U18 pad 6: Net-(U17-Σ0) -> unconnected-(U18-Beam_Enable-Pad6)
- U18 pad 7: Net-(U17-Σ1) -> unconnected-(U18-Point_(0)_/_Line_(1)_Sel-Pad7)
- U18 pad 8: Net-(U17-Σ2) -> Net-(U119-In2)
- U18 pad 9: Net-(U17-Σ3) -> Net-(U119-In1)
- U19 pad 2: /0 -> /VectorAddress0
- U19 pad 3: /1 -> /VectorAddress1
- U19 pad 4: /2 -> /VectorAddress2
- U19 pad 5: /3 -> /VectorAddress3
- U19 pad 6: /4 -> /VectorAddress4
- U19 pad 7: /5 -> /VectorAddress5
- U19 pad 8: /6 -> /VectorAddress6
- U19 pad 9: /7 -> /VectorAddress7
- U2 pad 1: unconnected-(U2-READ_0-Pad1) -> Net-(U2-READ_0)
- U2 pad 10: unconnected-(U2-CLK_A-Pad10) -> Net-(U2-CLK_A)
- U2 pad 2: unconnected-(U2-READ_1-Pad2) -> Net-(U2-READ_1)
- U2 pad 3: unconnected-(U2-READ_2-Pad3) -> Net-(U2-READ_2)
- U2 pad 4: unconnected-(U2-READ_3-Pad4) -> Net-(U2-READ_3)
- U20 pad 1: unconnected-(U20-OE#-Pad1) -> Net-(U20-OE#)
- U20 pad 11: unconnected-(U20-CLK-Pad11) -> Net-(U20-CLK)
- U20 pad 12: /7 -> /VectorAddress7
- U20 pad 13: /6 -> /VectorAddress6
- U20 pad 14: /5 -> /VectorAddress5
- U20 pad 15: /4 -> /VectorAddress4
- U20 pad 16: /3 -> /VectorAddress3
- U20 pad 17: /2 -> /VectorAddress2
- U20 pad 18: /1 -> /VectorAddress1
- U20 pad 19: /0 -> /VectorAddress0
- U20 pad 2: /0 -> /LoadVectorAddress0
- U20 pad 3: /1 -> /LoadVectorAddress1
- U20 pad 4: /2 -> /LoadVectorAddress2
- U20 pad 5: /3 -> /LoadVectorAddress3
- U20 pad 6: /4 -> /LoadVectorAddress4
- U20 pad 7: /5 -> /LoadVectorAddress5
- U20 pad 8: /6 -> /LoadVectorAddress6
- U20 pad 9: /7 -> /LoadVectorAddress7
- U21 pad 1: unconnected-(U21-OE#-Pad1) -> Net-(U20-OE#)
- U21 pad 10: unconnected-(U21-GND-Pad10) -> Net-(U21-D7)
- U21 pad 11: unconnected-(U21-CLK-Pad11) -> Net-(U21-CLK)
- U21 pad 13: /14 -> /VectorAddress14
- U21 pad 14: /13 -> /VectorAddress13
- U21 pad 15: /12 -> /VectorAddress12
- U21 pad 16: /11 -> /VectorAddress11
- U21 pad 17: /10 -> /VectorAddress10
- U21 pad 18: /9 -> /VectorAddress9
- U21 pad 19: /8 -> /VectorAddress8
- U21 pad 2: /8 -> /LoadVectorAddress8
- U21 pad 3: /9 -> /LoadVectorAddress9
- U21 pad 4: /10 -> /LoadVectorAddress10
- U21 pad 5: /11 -> /LoadVectorAddress11
- U21 pad 6: /12 -> /LoadVectorAddress12
- U21 pad 7: /13 -> /LoadVectorAddress13
- U21 pad 8: /14 -> /LoadVectorAddress14
- U21 pad 9: /15 -> Net-(U21-D7)
- U22 pad 1: unconnected-(U22-OE#-Pad1) -> Net-(U22-Σ1)
- U22 pad 10: unconnected-(U22-GND-Pad10) -> Net-(U22-Σ3)
- U22 pad 11: unconnected-(U22-CLK-Pad11) -> Net-(U22-B3)
- U22 pad 12: Net-(U22-Q7) -> /VectorMemX3
- U22 pad 13: Net-(U22-Q6) -> Net-(U22-Σ2)
- U22 pad 14: Net-(U22-Q5) -> /VectorMemX2
- U22 pad 15: Net-(U22-Q4) -> Net-(U22-B2)
- U22 pad 16: Net-(U22-Q3) -> Net-(U22-C_IN)
- U22 pad 2: Net-(U22-D0) -> Net-(U22-B1)
- U22 pad 3: Net-(U22-D1) -> /VectorMemX1
- U22 pad 4: Net-(U22-D2) -> Net-(U22-Σ0)
- U22 pad 5: Net-(U22-D3) -> /VectorMemX0
- U22 pad 6: Net-(U22-D4) -> Net-(U22-B0)
- U22 pad 7: Net-(U22-D5) -> Net-(U22-C_IN)
- U22 pad 8: Net-(U22-D6) -> Net-(U22-GND)
- U22 pad 9: Net-(U22-D7) -> Net-(U22-C_OUT)
- U23 pad 1: unconnected-(U23-OE#-Pad1) -> Net-(U23-Σ1)
- U23 pad 10: unconnected-(U23-GND-Pad10) -> Net-(U23-Σ3)
- U23 pad 11: unconnected-(U23-CLK-Pad11) -> Net-(U23-B3)
- U23 pad 12: Net-(U23-Q7) -> /VectorMemX7
- U23 pad 13: Net-(U23-Q6) -> Net-(U23-Σ2)
- U23 pad 14: Net-(U23-Q5) -> /VectorMemX6
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
Commit message: Satisfied ERC
Parts:
- added R16: R, custom_footprint_library:0.4_pitch_resistor, F.Cu at (188.3, 96.4)
- added R17: R, custom_footprint_library:0.4_pitch_resistor, F.Cu at (192.0, 96.4)
- added R18: R, custom_footprint_library:0.4_pitch_resistor, F.Cu at (195.6, 96.4)
- added R19: R, custom_footprint_library:0.4_pitch_resistor, F.Cu at (199.2, 96.4)
- added U121: ~, Package_DIP:DIP-16_W7.62mm, F.Cu at (187.4, 160.7)
- added U122: ~, custom_footprint_library:jumper, F.Cu at (183.9, 53.1)
- added U123: ~, Package_DIP:DIP-14_W7.62mm, F.Cu at (79.6, 78.3)
- added U124: ~, Package_DIP:DIP-14_W7.62mm, F.Cu at (90.4, 78.3)
- added U126: ~, Package_DIP:DIP-14_W7.62mm, F.Cu at (101.1, 78.3)
- added U127: ~, Package_DIP:DIP-14_W7.62mm, F.Cu at (111.9, 78.3)
- added U128: ~, Package_DIP:DIP-14_W7.62mm, F.Cu at (122.7, 78.3)
- added U129: ~, Package_DIP:DIP-14_W7.62mm, F.Cu at (25.7, 97.6)
- added U130: ~, Package_DIP:DIP-14_W7.62mm, F.Cu at (36.5, 97.6)
- added U131: ~, Package_DIP:DIP-14_W7.62mm, F.Cu at (47.2, 97.6)
- added U132: ~, Package_DIP:DIP-14_W7.62mm, F.Cu at (58.0, 97.6)
- added U133: ~, Package_DIP:DIP-14_W7.62mm, F.Cu at (68.8, 97.6)
- added U134: ~, Package_DIP:DIP-14_W7.62mm, F.Cu at (79.6, 97.6)
- added U135: ~, Package_DIP:DIP-14_W7.62mm, F.Cu at (90.4, 97.6)
- added U136: ~, Package_DIP:DIP-14_W7.62mm, F.Cu at (101.1, 97.6)
- U35: footprint Package_DIP:DIP-16_W7.62mm -> Package_DIP:DIP-20_W7.62mm
- U96: footprint Package_DIP:DIP-14_W7.62mm -> Connector_PinHeader_2.54mm:PinHeader_1x02_P2.54mm_Vertical
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Connections:
- U1 pad 20: unconnected-(U1-V+-Pad20) -> Net-(U1-V+)
- U10 pad 10: unconnected-(U10-GND-Pad10) -> Net-(U1-GND)
- U10 pad 20: unconnected-(U10-V+-Pad20) -> Net-(U1-V+)
- U100 pad 14: unconnected-(U100-V+-Pad14) -> Net-(U1-V+)
- U100 pad 7: unconnected-(U100-GND-Pad7) -> Net-(U1-GND)
- U101 pad 14: unconnected-(U101-V+-Pad14) -> Net-(U1-V+)
- U101 pad 7: unconnected-(U101-GND-Pad7) -> Net-(U1-GND)
- U102 pad 10: Net-(U102-0RESET) -> Net-(U1-GND)
- U102 pad 14: unconnected-(U102-V+-Pad14) -> Net-(U1-V+)
- U102 pad 4: Net-(U102-0RESET) -> Net-(U1-GND)
- U102 pad 6: Net-(U102-0RESET) -> Net-(U1-GND)
- U102 pad 7: Net-(U102-0RESET) -> Net-(U1-GND)
- U102 pad 8: Net-(U102-0RESET) -> Net-(U1-GND)
- U103 pad 10: Net-(U102-0RESET) -> Net-(U1-GND)
- U103 pad 14: unconnected-(U103-V+-Pad14) -> Net-(U1-V+)
- U103 pad 4: Net-(U102-0RESET) -> Net-(U1-GND)
- U103 pad 6: Net-(U102-0RESET) -> Net-(U1-GND)
- U103 pad 7: Net-(U102-0RESET) -> Net-(U1-GND)
- U103 pad 8: Net-(U102-0RESET) -> Net-(U1-GND)
- U104 pad 14: unconnected-(U104-V+-Pad14) -> Net-(U1-V+)
- U104 pad 7: unconnected-(U104-GND-Pad7) -> Net-(U1-GND)
- U105 pad 14: unconnected-(U105-V+-Pad14) -> Net-(U1-V+)
- U105 pad 7: unconnected-(U105-GND-Pad7) -> Net-(U1-GND)
- U106 pad 14: unconnected-(U106-V+-Pad14) -> Net-(U1-V+)
- U106 pad 7: unconnected-(U106-GND-Pad7) -> Net-(U1-GND)
- U107 pad 11: unconnected-(U107-Q3-Pad11) -> Net-(U107-Q3)
- U107 pad 12: unconnected-(U107-3A-Pad12) -> Net-(U107-3A)
- U107 pad 13: unconnected-(U107-3B-Pad13) -> Net-(U107-3B)
- U107 pad 14: unconnected-(U107-V+-Pad14) -> Net-(U1-V+)
- U107 pad 7: unconnected-(U107-GND-Pad7) -> Net-(U1-GND)
- U108 pad 2: Net-(U108-GND) -> Net-(U1-GND)
- U109 pad 2: Net-(U108-GND) -> Net-(U1-GND)
- U11 pad 10: unconnected-(U11-GND-Pad10) -> Net-(U1-GND)
- U11 pad 20: unconnected-(U11-V+-Pad20) -> Net-(U1-V+)
- U110 pad 2: Net-(U108-GND) -> Net-(U1-GND)
- U111 pad 2: Net-(U108-GND) -> Net-(U1-GND)
- U112 pad 11: unconnected-(U112-Q3-Pad11) -> Net-(U107-3A)
- U112 pad 12: unconnected-(U112-3A-Pad12) -> Net-(U112-3A)
- U112 pad 13: unconnected-(U112-3B-Pad13) -> Net-(U112-3B)
- U112 pad 14: unconnected-(U112-V+-Pad14) -> Net-(U1-V+)
- U112 pad 7: unconnected-(U112-GND-Pad7) -> Net-(U1-GND)
- U113 pad 10: unconnected-(U113-O4-Pad10) -> Net-(U113-O4)
- U113 pad 11: unconnected-(U113-I4-Pad11) -> Net-(U113-I4)
- U113 pad 14: unconnected-(U113-V+-Pad14) -> Net-(U1-V+)
- U113 pad 7: unconnected-(U113-GND-Pad7) -> Net-(U1-GND)
- U113 pad 8: unconnected-(U113-03-Pad8) -> Net-(U113-03)
- U113 pad 9: unconnected-(U113-I3-Pad9) -> Net-(U113-I3)
- U114 pad 10: unconnected-(U114-1RESET-Pad10) -> Net-(U1-GND)
- U114 pad 11: unconnected-(U114-1CLK-Pad11) -> Net-(U114-1CLK)
- U114 pad 13: unconnected-(U114-1Q-Pad13) -> Net-(U114-1Q)
- U114 pad 14: unconnected-(U114-V+-Pad14) -> Net-(U1-V+)
- U114 pad 4: Net-(U114-0RESET) -> Net-(U1-GND)
- U114 pad 6: Net-(U114-0RESET) -> Net-(U1-GND)
- U114 pad 7: Net-(U114-0RESET) -> Net-(U1-GND)
- U114 pad 8: unconnected-(U114-1SET-Pad8) -> Net-(U1-GND)
- U114 pad 9: unconnected-(U114-1D-Pad9) -> Net-(U114-1D)
- U115 pad 14: unconnected-(U115-V+-Pad14) -> Net-(U1-V+)
- U115 pad 2: unconnected-(U115-1B-Pad2) -> Net-(U1-GND)
- U115 pad 3: unconnected-(U115-1Q-Pad3) -> Net-(U1-GND)
- U115 pad 5: unconnected-(U115-2B-Pad5) -> Net-(U1-GND)
- U115 pad 6: unconnected-(U115-2Q-Pad6) -> Net-(U1-GND)
- U115 pad 7: unconnected-(U115-GND-Pad7) -> Net-(U1-GND)
- U116 pad 14: unconnected-(U116-V+-Pad14) -> Net-(U1-V+)
- U116 pad 7: unconnected-(U116-GND-Pad7) -> Net-(U1-GND)
- U117 pad 10: unconnected-(U117-O4-Pad10) -> Net-(U117-O4)
- U117 pad 11: unconnected-(U117-I4-Pad11) -> Net-(U117-I4)
- U117 pad 12: unconnected-(U117-O5-Pad12) -> Net-(U117-O5)
- U117 pad 13: unconnected-(U117-I5-Pad13) -> Net-(U117-I5)
- U117 pad 14: unconnected-(U117-V+-Pad14) -> Net-(U1-V+)
- U117 pad 7: unconnected-(U117-GND-Pad7) -> Net-(U1-GND)
- U118 pad 2: Net-(U108-GND) -> Net-(U1-GND)
- U12 pad 14: unconnected-(U12-GND-Pad14) -> Net-(U1-GND)
- U12 pad 20: unconnected-(U12-CE#-Pad20) -> Net-(U1-GND)
- U12 pad 22: unconnected-(U12-OE#-Pad22) -> Net-(U104-1A)
- U12 pad 28: unconnected-(U12-V+-Pad28) -> Net-(U1-V+)
- U120 pad 12: unconnected-(U120-3A-Pad12) -> Net-(U1-GND)
- U120 pad 13: unconnected-(U120-3B-Pad13) -> Net-(U1-GND)
- U120 pad 14: unconnected-(U120-V+-Pad14) -> Net-(U1-V+)
- U120 pad 7: unconnected-(U120-GND-Pad7) -> Net-(U1-GND)
- U120 pad 8: unconnected-(U120-2A-Pad8) -> Net-(U1-GND)
- U120 pad 9: unconnected-(U120-2B-Pad9) -> Net-(U1-GND)
- U13 pad 10: unconnected-(U13-GND-Pad10) -> Net-(U1-GND)
- U13 pad 20: unconnected-(U13-V+-Pad20) -> Net-(U1-V+)
- U14 pad 11: Net-(U14-B0) -> Net-(U1-GND)
- U14 pad 15: Net-(U14-B0) -> Net-(U1-GND)
- U14 pad 16: unconnected-(U14-V+-Pad16) -> Net-(U1-V+)
- U14 pad 2: Net-(U14-B0) -> Net-(U1-GND)
- U14 pad 6: Net-(U14-B0) -> Net-(U1-GND)
- U14 pad 8: Net-(U14-B0) -> Net-(U1-GND)
- U15 pad 10: unconnected-(U15-GND-Pad10) -> Net-(U1-GND)
- U15 pad 20: unconnected-(U15-V+-Pad20) -> Net-(U1-V+)
- U16 pad 1: Net-(U16-GND) -> Net-(U1-GND)
- U16 pad 10: Net-(U16-GND) -> Net-(U1-GND)
- U16 pad 20: unconnected-(U16-V+-Pad20) -> Net-(U1-V+)
- U17 pad 11: Net-(U17-A3) -> Net-(U1-GND)
- U17 pad 12: Net-(U17-A3) -> Net-(U1-GND)
- U17 pad 15: Net-(U17-A3) -> Net-(U1-GND)
- U17 pad 16: unconnected-(U17-V+-Pad16) -> Net-(U1-V+)
- U17 pad 2: Net-(U17-A3) -> Net-(U1-GND)
- U17 pad 6: Net-(U17-A3) -> Net-(U1-GND)
- U17 pad 8: Net-(U17-A3) -> Net-(U1-GND)
- U18 pad 10: unconnected-(U18-GND-Pad10) -> Net-(U1-GND)
- U18 pad 11: unconnected-(U18-+5V-Pad11) -> Net-(U18-+5V)
- U18 pad 5: unconnected-(U18-Line_Done-Pad5) -> Net-(U18-Line_Done)
- U18 pad 6: unconnected-(U18-Beam_Enable-Pad6) -> Net-(U18-Beam_Enable)
- U18 pad 7: unconnected-(U18-Point_(0)_/_Line_(1)_Sel-Pad7) -> Net-(U18-Point_(0)_/_Line_(1)_Sel)
- U19 pad 1: unconnected-(U19-OE#-Pad1) -> Net-(U1-GND)
- U19 pad 10: unconnected-(U19-GND-Pad10) -> Net-(U1-GND)
- U19 pad 11: unconnected-(U19-CLK-Pad11) -> Net-(U19-CLK)
- U19 pad 20: unconnected-(U19-V+-Pad20) -> Net-(U1-V+)
- U2 pad 12: unconnected-(U2-V+-Pad12) -> Net-(U1-V+)
- U2 pad 13: unconnected-(U2-GND-Pad13) -> Net-(U1-GND)
- U2 pad 23: unconnected-(U2-ENABLE-Pad23) -> Net-(U124-1A)
- U20 pad 1: Net-(U20-OE#) -> Net-(U104-1A)
- U20 pad 10: unconnected-(U20-GND-Pad10) -> Net-(U1-GND)
- U20 pad 20: unconnected-(U20-V+-Pad20) -> Net-(U1-V+)
- U21 pad 1: Net-(U20-OE#) -> Net-(U104-1A)
- U21 pad 10: Net-(U21-D7) -> Net-(U1-GND)
- U21 pad 20: unconnected-(U21-V+-Pad20) -> Net-(U1-V+)
- U21 pad 9: Net-(U21-D7) -> Net-(U1-GND)
- U22 pad 16: Net-(U22-C_IN) -> Net-(U1-V+)
- U22 pad 7: Net-(U22-C_IN) -> Net-(U1-V+)
- U22 pad 8: Net-(U22-GND) -> Net-(U1-GND)
- U23 pad 16: unconnected-(U23-V+-Pad16) -> Net-(U1-V+)
- U23 pad 8: Net-(U22-GND) -> Net-(U1-GND)
- U24 pad 14: unconnected-(U24-V+-Pad14) -> Net-(U1-V+)
- U24 pad 7: unconnected-(U24-GND-Pad7) -> Net-(U1-GND)
- U25 pad 14: unconnected-(U25-V+-Pad14) -> Net-(U1-V+)
- U25 pad 7: unconnected-(U25-GND-Pad7) -> Net-(U1-GND)
- U26 pad 14: unconnected-(U26-V+-Pad14) -> Net-(U1-V+)
- U26 pad 7: unconnected-(U26-GND-Pad7) -> Net-(U1-GND)
- U26 pad 8: unconnected-(U26-4Q-Pad8) -> Net-(U127-I5)
- U27 pad 1: Net-(U27-1A) -> Net-(U1-GND)
- U27 pad 14: unconnected-(U27-V+-Pad14) -> Net-(U1-V+)
- U27 pad 2: Net-(U27-1A) -> Net-(U1-GND)
- U27 pad 7: Net-(U27-1A) -> Net-(U1-GND)
- U28 pad 11: Net-(U28-CCLK) -> Net-(U19-CLK)
- U28 pad 12: Net-(U28-CCKEN#) -> Net-(U1-GND)
- U28 pad 13: Net-(U28-CCLK) -> Net-(U19-CLK)
- U28 pad 14: Net-(U28-CCKEN#) -> Net-(U1-GND)
- U28 pad 16: unconnected-(U28-V+-Pad16) -> Net-(U1-V+)
- U28 pad 8: Net-(U28-CCKEN#) -> Net-(U1-GND)
- U29 pad 14: unconnected-(U29-V+-Pad14) -> Net-(U1-V+)
- U29 pad 7: unconnected-(U29-GND-Pad7) -> Net-(U1-GND)
- U3 pad 14: unconnected-(U3-GND-Pad14) -> Net-(U1-GND)
- U3 pad 20: unconnected-(U3-CE#-Pad20) -> Net-(U1-GND)
- U3 pad 22: unconnected-(U3-OE#-Pad22) -> Net-(U104-1A)
- U3 pad 28: unconnected-(U3-V+-Pad28) -> Net-(U1-V+)
- U30 pad 12: unconnected-(U30-3A-Pad12) -> Net-(U1-GND)
- U30 pad 13: unconnected-(U30-3B-Pad13) -> Net-(U1-GND)
- U30 pad 14: unconnected-(U30-V+-Pad14) -> Net-(U1-V+)
- U30 pad 5: unconnected-(U30-1A-Pad5) -> Net-(U132-2B)
- U30 pad 6: unconnected-(U30-1B-Pad6) -> Net-(U114-1Q)
- U30 pad 7: unconnected-(U30-GND-Pad7) -> Net-(U1-GND)
- U30 pad 8: unconnected-(U30-2A-Pad8) -> Net-(U1-GND)
- U30 pad 9: unconnected-(U30-2B-Pad9) -> Net-(U1-GND)
- U31 pad 10: Net-(U31-D7) -> Net-(U1-GND)
- U31 pad 11: Net-(U31-CLK) -> Net-(U1-V+)
- U31 pad 20: Net-(U31-CLK) -> Net-(U1-V+)
- U31 pad 5: /SpriteMemAddr11 -> Net-(U1-GND)
- U31 pad 6: /SpriteMemAddr12 -> Net-(U1-GND)
- U31 pad 7: /SpriteMemAddr13 -> Net-(U1-GND)
- U31 pad 8: /SpriteMemAddr14 -> Net-(U1-GND)
- U31 pad 9: Net-(U31-D7) -> Net-(U1-GND)
- U32 pad 10: Net-(U32-WR#) -> Net-(U117-O4)
- U32 pad 12: Net-(U32-AGND) -> Net-(U1-GND)
- U32 pad 14: Net-(U32-AGND) -> Net-(U1-GND)
- U32 pad 15: Net-(U32-CLR#) -> Net-(U1-V+)
- U32 pad 16: Net-(U32-LDAC#) -> Net-(U113-O4)
- U32 pad 17: Net-(U32-AGND) -> Net-(U1-GND)
- U32 pad 19: Net-(U32-AGND) -> Net-(U1-GND)
- U32 pad 22: Net-(U32-AGND) -> Net-(U1-GND)
- U32 pad 23: Net-(U32-CLR#) -> Net-(U1-V+)
- U32 pad 8: Net-(U32-A0) -> Net-(U117-O5)
- U32 pad 9: Net-(U32-A0) -> Net-(U117-O5)
- U33 pad 1: unconnected-(U33-OE#-Pad1) -> Net-(U1-GND)
- U33 pad 10: Net-(U33-D7) -> Net-(U1-GND)
- U33 pad 11: unconnected-(U33-CLK-Pad11) -> Net-(U19-CLK)
- U33 pad 20: unconnected-(U33-V+-Pad20) -> Net-(U1-V+)
- U33 pad 9: Net-(U33-D7) -> Net-(U1-GND)
- U34 pad 1: Net-(U34-Q1) -> unconnected-(U34-Q11-Pad1)
- U34 pad 10: Net-(U34-CCLR#) -> Net-(U113-03)
- U34 pad 11: Net-(U34-CCLK) -> Net-(U34-Reset)
- U34 pad 12: Net-(U34-CCKEN#) -> unconnected-(U34-Q8-Pad12)
- U34 pad 13: Net-(U34-CCLK) -> Net-(U34-Q7)
- U34 pad 14: Net-(U34-CCKEN#) -> unconnected-(U34-Q9-Pad14)
- U34 pad 15: Net-(U34-Q0) -> unconnected-(U34-Q10-Pad15)
- U34 pad 16: unconnected-(U34-V+-Pad16) -> Net-(U1-V+)
- U34 pad 2: Net-(U34-Q2) -> Net-(U34-Q5)
- U34 pad 3: Net-(U34-Q3) -> Net-(U34-Q4)
- U34 pad 4: Net-(U34-Q4) -> Net-(U34-Q6)
- U34 pad 5: Net-(U34-Q5) -> Net-(U34-Q3)
- U34 pad 6: Net-(U34-Q6) -> Net-(U34-Q2)
- U34 pad 7: Net-(U34-Q7) -> Net-(U34-Q1)
- U34 pad 8: Net-(U34-CCKEN#) -> Net-(U1-GND)
- U34 pad 9: unconnected-(U34-RCO#-Pad9) -> Net-(U34-Q0)
- U35 pad 1: /SpriteMemAddr1 -> Net-(U35-OE#)
- U35 pad 10: unconnected-(U35-CCLR#-Pad10) -> Net-(U1-GND)
- U35 pad 11: unconnected-(U35-CCLK-Pad11) -> Net-(U1-V+)
- U35 pad 14: Net-(U35-OE#) -> unconnected-(U35-Q5-Pad14)
- U35 pad 15: /SpriteMemAddr0 -> unconnected-(U35-Q4-Pad15)
- U35 pad 2: /SpriteMemAddr2 -> Net-(U121-Q0)
- U35 pad 3: unconnected-(U35-Q3-Pad3) -> Net-(U121-Q1)
- U35 pad 4: unconnected-(U35-Q4-Pad4) -> Net-(U121-Q2)
- U35 pad 5: unconnected-(U35-Q5-Pad5) -> Net-(U1-GND)
- U35 pad 6: unconnected-(U35-Q6-Pad6) -> Net-(U1-GND)
- U35 pad 7: unconnected-(U35-Q7-Pad7) -> Net-(U1-GND)
- U35 pad 8: unconnected-(U35-GND-Pad8) -> Net-(U1-GND)
- U35 pad 9: unconnected-(U35-RCO#-Pad9) -> Net-(U1-GND)
- U36 pad 14: unconnected-(U36-GND-Pad14) -> Net-(U1-GND)
- U36 pad 20: unconnected-(U36-CE#-Pad20) -> Net-(U1-GND)
- U36 pad 28: unconnected-(U36-V+-Pad28) -> Net-(U1-V+)
- U37 pad 10: unconnected-(U37-GND-Pad10) -> Net-(U1-GND)
- U37 pad 11: Net-(U37-CLK) -> Net-(U1-V+)
- U37 pad 20: Net-(U37-CLK) -> Net-(U1-V+)
- U38 pad 10: unconnected-(U38-GND-Pad10) -> Net-(U1-GND)
- U38 pad 11: Net-(U38-CLK) -> Net-(U1-V+)
- U38 pad 20: Net-(U38-CLK) -> Net-(U1-V+)
- U39 pad 1: Net-(U39-GND) -> Net-(U1-GND)
- U39 pad 10: Net-(U39-GND) -> Net-(U1-GND)
- U39 pad 12: unconnected-(U39-Q7-Pad12) -> Net-(U18-Point_(0)_/_Line_(1)_Sel)
- U39 pad 20: unconnected-(U39-V+-Pad20) -> Net-(U1-V+)
- U4 pad 11: Net-(U4-B0) -> Net-(U1-GND)
- U4 pad 15: Net-(U4-B0) -> Net-(U1-GND)
- U4 pad 16: Net-(U4-C_IN) -> Net-(U1-V+)
- U4 pad 2: Net-(U4-B0) -> Net-(U1-GND)
- U4 pad 6: Net-(U4-B0) -> Net-(U1-GND)
- U4 pad 7: Net-(U4-C_IN) -> Net-(U1-V+)
- U4 pad 8: Net-(U4-B0) -> Net-(U1-GND)
- U40 pad 1: Net-(U40-GND) -> Net-(U1-GND)
- U40 pad 10: Net-(U40-GND) -> Net-(U1-GND)
- U40 pad 20: unconnected-(U40-V+-Pad20) -> Net-(U1-V+)
- U41 pad 1: Net-(U41-GND) -> Net-(U1-GND)
- U41 pad 10: Net-(U41-GND) -> Net-(U1-GND)
- U41 pad 20: unconnected-(U41-V+-Pad20) -> Net-(U1-V+)
- U42 pad 14: unconnected-(U42-V+-Pad14) -> Net-(U1-V+)
- U42 pad 7: unconnected-(U42-GND-Pad7) -> Net-(U1-GND)
- U43 pad 14: unconnected-(U43-V+-Pad14) -> Net-(U1-V+)
- U43 pad 7: unconnected-(U43-GND-Pad7) -> Net-(U1-GND)
- U44 pad 10: Net-(U32-WR#) -> Net-(U117-O4)
- U44 pad 12: Net-(U44-AGND) -> Net-(U1-GND)
- U44 pad 14: Net-(U44-AGND) -> Net-(U1-GND)
- U44 pad 15: Net-(U44-CLR#) -> Net-(U1-V+)
- U44 pad 16: Net-(U32-LDAC#) -> Net-(U113-O4)
- U44 pad 17: Net-(U44-AGND) -> Net-(U1-GND)
- U44 pad 19: Net-(U44-AGND) -> Net-(U1-GND)
- U44 pad 22: Net-(U44-AGND) -> Net-(U1-GND)
- U44 pad 23: Net-(U44-CLR#) -> Net-(U1-V+)
- U44 pad 8: Net-(U32-A0) -> Net-(U117-O5)
- U44 pad 9: Net-(U32-A0) -> Net-(U117-O5)
- U45 pad 10: unconnected-(U45-GND-Pad10) -> Net-(U1-GND)
- U45 pad 11: Net-(U45-CLK) -> Net-(U1-V+)
- U45 pad 20: Net-(U45-CLK) -> Net-(U1-V+)
- U46 pad 14: unconnected-(U46-V+-Pad14) -> Net-(U1-V+)
- U46 pad 7: unconnected-(U46-GND-Pad7) -> Net-(U1-GND)
- U47 pad 14: unconnected-(U47-V+-Pad14) -> Net-(U1-V+)
- U47 pad 3: Net-(U47-1Q) -> Net-(U34-Reset)
- U47 pad 7: unconnected-(U47-GND-Pad7) -> Net-(U1-GND)
- U48 pad 11: Net-(U48-B0) -> Net-(U1-GND)
- U48 pad 15: Net-(U48-B0) -> Net-(U1-GND)
- U48 pad 16: Net-(U48-A0) -> Net-(U1-V+)
- U48 pad 2: Net-(U48-B0) -> Net-(U1-GND)
- U48 pad 5: Net-(U48-A0) -> Net-(U1-V+)
- U48 pad 6: Net-(U48-B0) -> Net-(U1-GND)
- U48 pad 7: Net-(U48-A0) -> Net-(U1-V+)
- U48 pad 8: Net-(U48-B0) -> Net-(U1-GND)
- U49 pad 11: Net-(U49-B0) -> Net-(U1-GND)
- U49 pad 15: Net-(U49-B0) -> Net-(U1-GND)
- U49 pad 16: unconnected-(U49-V+-Pad16) -> Net-(U1-V+)
- U49 pad 2: Net-(U49-B0) -> Net-(U1-GND)
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
Commit message: About to change bus loading
Parts:
- moved U129 444.9 mm to (420.2, 303.4)
- moved U18 430.1 mm to (484.6, 85.6)
- moved U32 428.5 mm to (433.3, 65.9), turned to 90 degrees
- moved U96 423.8 mm to (484.6, 117.8), turned to -90 degrees
- moved U119 417.8 mm to (482.4, 124.2)
- moved U44 412.0 mm to (433.2, 86.8), turned to 90 degrees
- moved U112 407.3 mm to (437.7, 303.4)
- moved U51 395.3 mm to (433.2, 112.3), turned to 90 degrees
- moved U72 391.6 mm to (473.4, 168.2)
- moved U120 388.9 mm to (448.7, 161.4)
- moved U54 387.4 mm to (476.8, 214.6), turned to -90 degrees
- moved U117 383.3 mm to (432.2, 161.4)
- moved U52 380.2 mm to (433.3, 136.8), turned to 90 degrees
- moved U62 376.4 mm to (469.1, 214.6), turned to -90 degrees
- moved U116 373.1 mm to (411.0, 161.1)
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Connections:
- U100 pad 10: unconnected-(U100-4A-Pad10) -> Net-(U1-GND)
- U100 pad 12: unconnected-(U100-3B-Pad12) -> Net-(U1-GND)
- U100 pad 13: unconnected-(U100-3A-Pad13) -> Net-(U1-GND)
- U100 pad 9: unconnected-(U100-4B-Pad9) -> Net-(U1-GND)
- U115 pad 1: unconnected-(U115-1A-Pad1) -> Net-(U114-0Q)
- U115 pad 10: Net-(U115-4A) -> Net-(U1-GND)
- U115 pad 11: Net-(U114-0Q#) -> unconnected-(U115-3Q-Pad11)
- U115 pad 12: Net-(U115-3B) -> Net-(U1-GND)
- U115 pad 13: Net-(U115-3A) -> Net-(U1-GND)
- U115 pad 14: Net-(U1-V+) -> Net-(U1-GND)
- U115 pad 2: Net-(U1-GND) -> Net-(U115-1B)
- U115 pad 3: Net-(U1-GND) -> Net-(U115-1Q)
- U115 pad 4: unconnected-(U115-2A-Pad4) -> Net-(U114-0Q#)
- U115 pad 5: Net-(U1-GND) -> Net-(U115-1B)
- U115 pad 6: Net-(U1-GND) -> Net-(U115-2Q)
- U115 pad 7: Net-(U1-GND) -> Net-(U1-V+)
- U115 pad 8: Net-(U114-0Q) -> unconnected-(U115-4Q-Pad8)
- U115 pad 9: Net-(U115-3B) -> Net-(U1-GND)
- U116 pad 1: Net-(U115-4A) -> Net-(U115-1Q)
- U116 pad 5: Net-(U115-3A) -> Net-(U115-2Q)
- U26 pad 3: Net-(U115-3B) -> Net-(U115-1B)
- U35 pad 1: Net-(U35-OE#) -> Net-(U104-3A)
- U36 pad 22: Net-(U36-OE#) -> Net-(U104-3A)
- U37 pad 1: Net-(U36-OE#) -> Net-(U104-3A)
- U38 pad 1: Net-(U36-OE#) -> Net-(U104-3A)
- U45 pad 1: Net-(U35-OE#) -> Net-(U104-3A)
- U61 pad 10: unconnected-(U61-4A-Pad10) -> Net-(U1-GND)
- U61 pad 9: unconnected-(U61-4B-Pad9) -> Net-(U1-GND)
- U69 pad 10: unconnected-(U69-4A-Pad10) -> Net-(U1-GND)
- U69 pad 9: unconnected-(U69-4B-Pad9) -> Net-(U1-GND)
Routing:
- net Net-(U1-GND): track 0.00 -> 4111.5 mm, vias 0 -> 17
- net Net-(U1-V+): track 0.00 -> 3217.4 mm, vias 0 -> 29
- net Net-(U102-0CLK): track 0.00 -> 789.3 mm, vias 0 -> 6
- net /SpriteData4: track 0.00 -> 610.5 mm, vias 0 -> 6
- net /SpriteData3: track 0.00 -> 522.8 mm, vias 0 -> 9
- net /SpriteData7: track 0.00 -> 472.0 mm, vias 0 -> 4
- net /VectorAddress11: track 0.00 -> 471.1 mm, vias 0 -> 6
- net Net-(U104-3A): track 0.00 -> 445.2 mm, vias 0 -> 6
- net /SpriteData2: track 0.00 -> 431.4 mm, vias 0 -> 9
- net Net-(U124-1A): track 0.00 -> 418.8 mm, vias 0 -> 4
- net Net-(U121-Q2): track 0.00 -> 414.5 mm, vias 0 -> 4
- net Net-(U10-OE#): track 0.00 -> 414.2 mm, vias 0 -> 3
- net Net-(U22-B2): track 0.00 -> 391.8 mm, vias 0 -> 4
- net Net-(U106-4A): track 0.00 -> 389.8 mm, vias 0 -> 6
- net /VectorAddress14: track 0.00 -> 387.9 mm, vias 0 -> 3
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Other:
- board outline added: 422 x 303.5 mm
- board text added: "CRT POWER CONNECT"
- board text added: "END UPDATE CONFIG"
- board text added: "X0 Y0 X1 Y1 LINE DONE BEAM ON POINT / LINE UPDATE V0 UPTADE V1 GND +5V"

Commit message: Vector thingy almost completely verified except math and DAC stuff
Parts:
- added U13: ~, Package_DIP:DIP-20_W7.62mm, F.Cu at (477.8, 285.6)
- added U139: ~, Package_DIP:DIP-20_W7.62mm, F.Cu at (499.3, 285.6)
- added U140: ~, Package_DIP:DIP-20_W7.62mm, F.Cu at (510.1, 285.6)
- added U141: ~, Package_DIP:DIP-20_W7.62mm, F.Cu at (520.9, 285.6)
- added U15: ~, Package_DIP:DIP-20_W7.62mm, F.Cu at (488.5, 285.6)
- added U31: ~, Package_DIP:DIP-14_W7.62mm, F.Cu at (467.0, 312.6)
- added U8: ~, Package_DIP:DIP-20_W7.62mm, F.Cu at (467.0, 285.6)
Connections:
- U100 pad 10: Net-(U1-GND) -> Net-(U100-4A)
- U100 pad 11: unconnected-(U100-3Q-Pad11) -> Net-(U100-3Q)
- U100 pad 12: Net-(U1-GND) -> Net-(U100-3B)
- U100 pad 13: Net-(U1-GND) -> Net-(U100-3A)
- U100 pad 2: Net-(U100-1B) -> /7
- U100 pad 4: Net-(U100-2A) -> Net-(U1-GND)
- U100 pad 5: Net-(U100-1B) -> Net-(U1-GND)
- U100 pad 6: Net-(U100-2Q) -> unconnected-(U100-2Q-Pad6)
- U100 pad 8: unconnected-(U100-4Q-Pad8) -> Net-(U100-4Q)
- U100 pad 9: Net-(U1-GND) -> Net-(U100-4B)
- U101 pad 10: Net-(U100-1B) -> unconnected-(U101-Q2-Pad10)
- U101 pad 2: Net-(U101-0B) -> Net-(U100-1A)
- U101 pad 4: Net-(U10-CLK) -> Net-(U100-3A)
- U101 pad 5: Net-(U100-1Q) -> Net-(U100-4A)
- U101 pad 6: Net-(U100-2Q) -> Net-(U101-1B)
- U101 pad 8: Net-(U101-2A) -> Net-(U1-GND)
- U101 pad 9: Net-(U101-2B) -> Net-(U1-GND)
- U105 pad 10: Net-(U105-2A) -> Net-(U10-D7)
- U105 pad 4: Net-(U105-2A) -> Net-(U10-D7)
- U115 pad 10: Net-(U1-GND) -> Net-(U110-OUT)
- U115 pad 11: unconnected-(U115-3Q-Pad11) -> Net-(U100-4B)
- U115 pad 12: Net-(U1-GND) -> Net-(U115-3B)
- U115 pad 13: Net-(U1-GND) -> Net-(U108-OUT)
- U115 pad 8: unconnected-(U115-4Q-Pad8) -> Net-(U100-3B)
- U115 pad 9: Net-(U1-GND) -> Net-(U115-4B)
- U120 pad 10: unconnected-(U120-Q2-Pad10) -> Net-(U120-Q2)
- U120 pad 11: unconnected-(U120-Q3-Pad11) -> Net-(U120-Q3)
- U120 pad 12: Net-(U1-GND) -> Net-(U120-3A)
- U120 pad 13: Net-(U1-GND) -> Net-(U120-3B)
- U120 pad 8: Net-(U1-GND) -> Net-(U120-2A)
- U120 pad 9: Net-(U1-GND) -> Net-(U120-2B)
- U127 pad 11: Net-(U127-I4) -> Net-(U120-2B)
- U130 pad 4: Net-(U130-2A) -> Net-(U120-2A)
- U130 pad 5: Net-(U127-I4) -> Net-(U120-2B)
- U130 pad 6: Net-(U130-2Q) -> Net-(U120-3A)
- U130 pad 8: Net-(U130-4Q) -> Net-(U120-3B)
- U132 pad 1: Net-(U127-I4) -> Net-(U120-2B)
- U136 pad 10: unconnected-(U136-O4-Pad10) -> Net-(U115-4B)
- U136 pad 11: Net-(U1-GND) -> Net-(U110-OUT)
- U136 pad 8: unconnected-(U136-03-Pad8) -> Net-(U115-3B)
- U136 pad 9: Net-(U1-GND) -> Net-(U108-OUT)
- U16 pad 11: Net-(U101-2A) -> Net-(U100-1Q)
- U16 pad 12: Net-(U16-Q7) -> unconnected-(U16-Q7-Pad12)
- U16 pad 13: Net-(U16-Q6) -> /SpriteMemAddr14
- U16 pad 14: Net-(U16-Q5) -> /SpriteMemAddr13
- U16 pad 15: Net-(U16-Q4) -> /SpriteMemAddr12
- U16 pad 16: Net-(U16-Q3) -> /SpriteMemAddr11
- U16 pad 17: Net-(U16-Q2) -> unconnected-(U16-Q2-Pad17)
- U16 pad 18: Net-(U16-Q1) -> unconnected-(U16-Q1-Pad18)
- U16 pad 19: Net-(U16-Q0) -> unconnected-(U16-Q0-Pad19)
- U48 pad 12: Net-(U16-Q3) -> Net-(U141-Q3)
- U48 pad 14: Net-(U16-Q2) -> Net-(U141-Q2)
- U48 pad 3: Net-(U16-Q1) -> Net-(U141-Q1)
- U49 pad 12: Net-(U16-Q7) -> Net-(U141-Q7)
- U49 pad 14: Net-(U16-Q6) -> Net-(U141-Q6)
- U49 pad 3: Net-(U16-Q5) -> Net-(U141-Q5)
- U49 pad 5: Net-(U16-Q4) -> Net-(U141-Q4)
- U5 pad 1: Net-(U31-OE#) -> Net-(U15-OE#)
- U5 pad 11: Net-(U10-CLK) -> Net-(U100-3Q)
- U50 pad 5: Net-(U105-2A) -> Net-(U10-D7)
- U58 pad 1: Net-(U16-Q0) -> Net-(U141-Q0)
- U58 pad 6: Net-(U31-OE#) -> Net-(U15-OE#)
- U59 pad 1: Net-(U16-Q0) -> Net-(U141-Q0)
- U59 pad 10: Net-(U16-Q0) -> Net-(U141-Q0)
- U59 pad 13: Net-(U16-Q0) -> Net-(U141-Q0)
- U59 pad 4: Net-(U16-Q0) -> Net-(U141-Q0)
- U6 pad 11: Net-(U101-0B) -> Net-(U100-1A)
- U61 pad 1: Net-(U16-Q0) -> Net-(U141-Q0)
- U61 pad 13: Net-(U16-Q0) -> Net-(U141-Q0)
- U61 pad 4: Net-(U16-Q0) -> Net-(U141-Q0)
- U68 pad 1: Net-(U16-Q0) -> Net-(U141-Q0)
- U68 pad 10: Net-(U16-Q0) -> Net-(U141-Q0)
- U68 pad 13: Net-(U16-Q0) -> Net-(U141-Q0)
- U68 pad 4: Net-(U16-Q0) -> Net-(U141-Q0)
- U69 pad 1: Net-(U16-Q0) -> Net-(U141-Q0)
- U69 pad 13: Net-(U16-Q0) -> Net-(U141-Q0)
- U69 pad 4: Net-(U16-Q0) -> Net-(U141-Q0)
- U7 pad 1: Net-(U1-GND) -> Net-(U15-OE#)
- U7 pad 11: Net-(U10-CLK) -> Net-(U100-3Q)
- U7 pad 12: Net-(U105-2A) -> unconnected-(U7-Q7-Pad12)
- U7 pad 13: /SpriteMemAddr14 -> unconnected-(U7-Q6-Pad13)
- U7 pad 14: /SpriteMemAddr13 -> unconnected-(U7-Q5-Pad14)
- U7 pad 15: /SpriteMemAddr12 -> unconnected-(U7-Q4-Pad15)
- U7 pad 16: /SpriteMemAddr11 -> unconnected-(U7-Q3-Pad16)
- U7 pad 17: Net-(U31-D2) -> /SpriteMemAddr2
- U7 pad 18: Net-(U31-D1) -> /SpriteMemAddr1
- U7 pad 19: Net-(U31-D0) -> /SpriteMemAddr0
- U73 pad 14: Net-(U130-2A) -> Net-(U120-2A)
- U73 pad 8: Net-(U127-I4) -> Net-(U120-2B)
- U79 pad 1: Net-(U130-2A) -> Net-(U120-2A)
- U80 pad 1: Net-(U127-I4) -> Net-(U120-2B)
- U82 pad 1: Net-(U130-2A) -> Net-(U120-2A)
- U83 pad 1: Net-(U131-Q0) -> Net-(U120-Q2)
- U84 pad 1: Net-(U131-Q1) -> Net-(U120-Q3)
- U95 pad 14: Net-(U127-I4) -> Net-(U120-2B)
- U95 pad 7: Net-(U130-2A) -> Net-(U120-2A)
- U97 pad 11: Net-(U101-2B) -> Net-(U8-CLK)
- U97 pad 6: Net-(U101-0B) -> Net-(U100-1A)
- U97 pad 8: Net-(U101-2A) -> Net-(U139-CLK)
- U98 pad 4: Net-(U100-1A) -> Net-(U100-4A)
- U98 pad 8: Net-(U100-2A) -> Net-(U101-1B)
- U99 pad 1: Net-(U100-1A) -> Net-(U100-4A)
- U99 pad 2: Net-(U101-2B) -> Net-(U8-CLK)
- U99 pad 8: Net-(U100-2A) -> Net-(U101-1B)
- U99 pad 9: Net-(U101-2A) -> Net-(U139-CLK)
Routing:
- net Net-(U1-GND): track 4111.5 -> 0.00 mm, vias 17 -> 0
- net Net-(U1-V+): track 3217.4 -> 0.00 mm, vias 29 -> 0
- net Net-(U102-0CLK): track 789.3 -> 0.00 mm, vias 6 -> 0
- net /SpriteData4: track 610.5 -> 0.00 mm, vias 6 -> 0
- net /SpriteData3: track 522.8 -> 0.00 mm, vias 9 -> 0
- net /SpriteData7: track 472.0 -> 0.00 mm, vias 4 -> 0
- net /VectorAddress11: track 471.1 -> 0.00 mm, vias 6 -> 0
- net Net-(U104-3A): track 445.2 -> 0.00 mm, vias 6 -> 0
- net /SpriteData2: track 431.4 -> 0.00 mm, vias 9 -> 0
- net Net-(U124-1A): track 418.8 -> 0.00 mm, vias 4 -> 0
- net Net-(U121-Q2): track 414.5 -> 0.00 mm, vias 4 -> 0
- net Net-(U10-OE#): track 414.2 -> 0.00 mm, vias 3 -> 0
- net Net-(U22-B2): track 391.8 -> 0.00 mm, vias 4 -> 0
- net Net-(U106-4A): track 389.8 -> 0.00 mm, vias 6 -> 0
- net /VectorAddress14: track 387.9 -> 0.00 mm, vias 3 -> 0
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Other:
- board size 422 x 303.5 mm -> 463.5 x 303.5 mm
