File: kicad/vector_digital_controller/vector_digital_controller.kicad_pcb (KiCad board)
At the start: 2 copper layers, 463.5 x 303.5 mm, 161 parts

Commit message: Vector graphics board finished
Parts:
- removed U13, U15, U31, U8 (x2): ~, Package_DIP:DIP-20_W7.62mm
- removed U131: ~, Package_DIP:DIP-14_W7.62mm
- removed U28: ~, Package_DIP:DIP-16_W7.62mm
- added U421: ~, Package_DIP:DIP-16_W7.62mm, F.Cu at (333.8, 189.7)
- added U425: ~, Package_DIP:DIP-20_W7.62mm, F.Cu at (188.4, 70.9)
- moved U423 406.5 mm to (158.0, 48.5)
- moved U139 366.1 mm to (218.2, 51.1)
- moved U140 357.4 mm to (240.5, 51.1)
- moved U424 350.4 mm to (171.7, 115.1)
- moved U141 338.0 mm to (245.4, 89.7), turned to -90 degrees
- moved U420 334.4 mm to (201.0, 115.0)
- moved U30 165.6 mm to (387.0, 262.9), turned to -90 degrees
- moved U58 158.9 mm to (376.4, 194.5)
- moved U132 132.3 mm to (438.4, 272.5)
- moved U113 127.8 mm to (460.5, 304.5)
- moved U61 87.3 mm to (330.7, 125.8)
- moved U68 83.6 mm to (358.2, 125.4)
- moved U69 75.8 mm to (352.7, 194.9)
- moved U67 75.6 mm to (365.5, 158.0)
- moved U7 73.7 mm to (178.3, 58.1)
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- renumbered U15 to U420, U38 to U422, U31 to U423, U13 to U424
Connections:
- U58 pad 11: Net-(U58-I4) -> Net-(U19-CLK)
- U75 pad 3: Net-(U58-I4) -> Net-(U421-Reset)
Routing:
- net Net-(U1-GND): track 0.00 -> 4295.1 mm, vias 0 -> 21
- net Net-(U1-V+): track 0.00 -> 3225.9 mm, vias 0 -> 28
- net Net-(U102-0CLK): track 0.00 -> 790.3 mm, vias 0 -> 6
- net /SpriteData7: track 0.00 -> 565.2 mm, vias 0 -> 3
- net Net-(U18-Point_(0)_/_Line_(1)_Sel): track 0.00 -> 551.3 mm, vias 0 -> 2
- net Net-(U10-D7): track 0.00 -> 523.7 mm, vias 0 -> 2
- net Net-(U106-4A): track 0.00 -> 501.0 mm, vias 0 -> 5
- net Net-(U114-1CLK): track 0.00 -> 495.6 mm, vias 0 -> 4
- net Net-(U102-1CLK): track 0.00 -> 488.2 mm, vias 0 -> 3
- net Net-(U100-3B): track 0.00 -> 483.7 mm, vias 0 -> 1
- net Net-(U113-I3): track 0.00 -> 467.4 mm
- net Net-(U100-4B): track 0.00 -> 461.7 mm, vias 0 -> 2
- net Net-(U124-1A): track 0.00 -> 455.4 mm, vias 0 -> 4
- net /VectorAddress12: track 0.00 -> 449.3 mm, vias 0 -> 5
- net /VectorAddress14: track 0.00 -> 440.2 mm, vias 0 -> 3
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Other:
- board size 463.5 x 303.5 mm -> 428.5 x 293 mm
- board text added: "CRT VECTOR GRAPHICS INTERFACE DESIGNED JAN 2026 WITH KICAD BY HADRIAN WARD"
