File: kicad/boards_version_2/call_stack_v2/call_stack.kicad_sch (KiCad schematic)
At the start: 27 parts

Commit message: 2 circuits verified
Parts:
- removed U1: ~, Connector_PinHeader_2.54mm:PinHeader_1x24_P2.54mm_Vertical, symbol custom_symbol_lib:control_unit_to_call_stack
- removed U12, U13, U14, U15, U16, U17, U18, U19, U20, U23: ~, custom_footprint_library:jumper, symbol custom_symbol_lib:jumper
- removed U21: ~, Package_DIP:DIP-14_W7.62mm, symbol custom_symbol_lib:6xNOT
- removed U22: ~, Package_DIP:DIP-14_W7.62mm, symbol custom_symbol_lib:quad_and
- removed U24, U26, U27: ~, Package_DIP:DIP-14_W7.62mm, symbol custom_symbol_lib:dual_latch
- removed U25: ~, Package_DIP:DIP-14_W7.62mm, symbol custom_symbol_lib:quad_OR
- removed U6, U7, U8, U9: ~, Package_DIP:DIP-20_W7.62mm, symbol custom_symbol_lib:rising_edge_8_bit_latch
- added U1, U17: ~, Package_DIP:DIP-14_W7.62mm, symbol custom_symbol_lib:dual_latch
- added U12, U13, U14, U15, U18: ~, custom_footprint_library:jumper_v2_gnd_debug_footprint, symbol custom_symbol_lib:jumper_v2_gnd_debug
- added U6: ~, Connector_PinHeader_2.54mm:PinHeader_1x22_P2.54mm_Vertical, symbol custom_symbol_lib:call_stack_v2
- added U7: ~, Package_DIP:DIP-14_W7.62mm, symbol custom_symbol_lib:quad_and
- added U8: ~, Package_DIP:DIP-14_W7.62mm, symbol custom_symbol_lib:quad_OR
- added U9: ~, Package_DIP:DIP-14_W7.62mm, symbol custom_symbol_lib:6xNOT
Connections:
- net at U10.16 (V+), U11.20 (V+), U2.16 (V+)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: now also U1.14 (V+), U17.14 (V+), U6.2 (+5V), U7.14 (V+), U8.14 (V+), U9.14 (V+)
- net at U10.8 (GND), U11.1 (OE#), U11.10 (GND)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: now also U1.10 (1RESET), U1.4 (0RESET), U1.6 (0SET), U1.7 (GND), U1.8 (1SET), U12.2 (GND), U13.2 (GND), U14.2 (GND), U15.2 (GND), U17.10 (1RESET), U17.4 (0RESET), U17.6 (0SET), U17.7 (GND), U17.8 (1SET), U18.2 (GND), U6.1 (GND), U7.1 (1A), U7.2 (1B), U7.4 (2A), U7.5 (2B), U7.7 (GND), U8.1 (0A), U8.12 (3A), U8.13 (3B), U8.2 (0B), U8.7 (GND), U9.11 (I4), U9.13 (I5), U9.7 (GND), U9.9 (I3)
- net at U11.11 (CLK): now also U13.3 (OUT)
- net at U4.19 (D7): now also U6.6 (Data_0)
- net at U4.18 (D6): now also U6.7 (Data_1)
- net at U4.17 (D5): now also U6.8 (Data_2)
- net at U4.16 (D4): now also U6.9 (Data_3)
- net at U4.15 (D3): now also U6.10 (Data_4)
- net at U4.13 (D2): now also U6.11 (Data_5)
- net at U4.12 (D1): now also U6.12 (Data_6)
- net at U4.11 (D0): now also U6.13 (Data_7)
- net at U10.11 (B3), U10.15 (B2), U10.2 (B1)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: now also U18.3 (OUT)
- net at U4.22 (OE#), U5.22 (OE#): now also U9.4 (O1)
- net at U4.27 (WE#), U5.27 (WE#): now also U9.6 (O2)
- net at U3.11 (CLK): now also U12.3 (OUT)
- net at U5.11 (D0): now also U6.21 (Data_15)
- net at U5.12 (D1): now also U6.20 (Data_14)
- net at U5.13 (D2): now also U6.19 (Data_13)
- net at U5.15 (D3): now also U6.18 (Data_12)
- net at U5.16 (D4): now also U6.17 (Data_11)
- net at U5.17 (D5): now also U6.16 (Data_10)
- net at U5.18 (D6): now also U6.15 (Data_9)
- net at U5.19 (D7): now also U6.14 (Data_8)
- new net: U17.11 (1CLK), U17.3 (0CLK), U6.22 (CLK), U9.1 (I0)
- new net: U1.11 (1CLK), U1.3 (0CLK), U9.2 (O0)
- new net: U14.3 (OUT), U9.3 (I1)
- new net: U15.3 (OUT), U9.5 (I2)
- new net: U1.13 (1Q), U17.9 (1D), U18.1 (IN), U8.6 (1B)
- new net: U15.1 (IN), U7.11 (3Q)
- new net: U13.1 (IN), U8.10 (Q2)
- new net: U1.1 (0Q), U17.5 (0D), U7.9 (4B), U8.8 (2A)
- new net: U1.5 (0D), U6.5 (Push), U8.5 (1A)
- new net: U1.9 (1D), U14.1 (IN), U6.4 (Pop_&_OE)
- new net: U12.1 (IN), U8.4 (Q1)
- new net: U17.13 (1Q), U8.9 (2B)
- new net: U17.1 (0Q), U7.10 (4A)
- new net: U6.3 (Enable), U7.12 (3B)
- new net: U7.13 (3A), U7.8 (4Q)
- no-connect marks 10 -> 12
Other:
- note added: "Falling"
- note added: "G0"
- note added: "G1"
- note added: "G2"
- note added: "G3"
- note added: "G4"
- note added: "Rising"
- note added: "read#"
- note added: "write#"
- note removed: "2 (B CLK) Push sequence 1 (A CLK)"
- note removed: "Decrement (A CLK)"
- note removed: "Pop (!B)"
- note removed: "Pre adder latch CLK (A CLK)"
- note removed: "Pre adder latch CLK (B CLK)"
- moved on the sheet: U4

Commit message: Debug figured out and work on ctrl unit main
Parts:
- removed U12, U13, U14, U15, U18: ~, custom_footprint_library:jumper_v2_gnd_debug_footprint, symbol custom_symbol_lib:jumper_v2_gnd_debug
- added U12, U13, U14, U15, U20: ~, custom_footprint_library:jumper_v2_gnd_footprint, symbol custom_symbol_lib:jumer_v2_gnd
- added U16: ~, Package_DIP:DIP-20_W7.62mm, symbol custom_symbol_lib:8_bit_transparent_latch
- added U19: ~, Connector_PinHeader_2.54mm:PinHeader_1x05_P2.54mm_Vertical, symbol custom_symbol_lib:debug_v2_call_stack
Connections:
- net at U1.10 (1RESET), U1.4 (0RESET), U1.6 (0SET)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: now also U12.2 (GND), U13.2 (GND), U14.2 (GND), U15.2 (GND), U16.1 (OE#), U16.10 (GND), U16.7 (D5), U16.8 (D6), U16.9 (D7), U20.2 (GND)
- net at U1.14 (V+), U10.16 (V+), U11.20 (V+)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: now also U16.11 (CLK), U16.20 (V+)
- net at U9.3 (I1): now also U14.3 (OUT)
- net at U9.5 (I2): now also U15.3 (OUT)
- net at U1.13 (1Q), U17.9 (1D), U8.6 (1B): now also U16.2 (D0), U20.1 (IN)
- net at U10.11 (B3), U10.15 (B2), U10.2 (B1)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: now also U20.3 (OUT)
- net at U7.11 (3Q): now also U15.1 (IN), U16.6 (D4)
- net at U11.11 (CLK): now also U13.3 (OUT)
- net at U3.11 (CLK): now also U12.3 (OUT)
- net at U8.10 (Q2): now also U13.1 (IN), U16.4 (D2)
- net at U1.9 (1D), U6.4 (Pop_&_OE): now also U14.1 (IN), U16.5 (D3)
- net at U8.4 (Q1): now also U12.1 (IN), U16.3 (D1)
- new net: U16.19 (Q0), U19.1 (Pointer_++(0)_/_--_(1))
- new net: U16.18 (Q1), U19.2 (Pre-adder_latch_CLK)
- new net: U16.17 (Q2), U19.3 (Post-adder_latch_CLK)
- new net: U16.16 (Q3), U19.4 (Read)
- new net: U16.15 (Q4), U19.5 (Write)
- no-connect marks 12 -> 15
Other:
- moved on the sheet: U1, U17, U7, U8, U9
