File: kicad/boards_version_2/control_unit_v2/control_unit.kicad_sch (KiCad schematic)
At the start: 53 parts

Commit message: Debug figured out and work on ctrl unit main
Parts:
- removed D1, D2, D3, D4: LED, LED_THT:LED_D4.0mm, symbol Device:LED
- removed U1: ~, Connector_PinHeader_2.54mm:PinHeader_1x23_P2.54mm_Vertical, symbol custom_symbol_lib:bus_edge_connector
- removed U10: ~, Package_DIP:DIP-16_W7.62mm, symbol custom_symbol_lib:2x4_bit_multiplexer
- removed U11: ~, Connector_PinHeader_2.54mm:PinHeader_1x23_P2.54mm_Horizontal, symbol custom_symbol_lib:control_unit_central_timing_interface
- removed U12, U16: ~, Package_DIP:DIP-14_W7.62mm, symbol custom_symbol_lib:quad_and
- removed U14: ~, Package_DIP:DIP-14_W7.62mm, symbol custom_symbol_lib:quad_OR
- removed U17: ~, Connector_PinHeader_2.54mm:PinHeader_1x39_P2.54mm_Vertical, symbol custom_symbol_lib:prog_mem_interface_read
- removed U2: ~, Connector_PinHeader_2.54mm:PinHeader_1x11_P2.54mm_Vertical, symbol custom_symbol_lib:bus_arbiter_control_unit_connection
- removed U20: ~, Package_DIP:DIP-14_W7.62mm, symbol custom_symbol_lib:6xNOT
- removed U23, U25: ~, custom_footprint_library:jumper, symbol custom_symbol_lib:jumper
- removed U26: ~, Connector_PinHeader_2.54mm:PinHeader_1x25_P2.54mm_Vertical, symbol custom_symbol_lib:gpram_instruction_load_interface
- removed U27, U28, U8: ~, Package_DIP:DIP-20_W7.62mm, symbol custom_symbol_lib:rising_edge_8_bit_latch
- removed U3: ~, Connector_PinHeader_2.54mm:PinHeader_1x24_P2.54mm_Vertical, symbol custom_symbol_lib:control_unit_to_call_stack
- removed U4: ~, Package_DIP:DIP-14_W7.62mm, symbol custom_symbol_lib:dual_latch
- added J1: Conn_01x01_Pin, Connector_Pin:Pin_D1.3mm_L11.0mm, symbol Connector:Conn_01x01_Pin
- added R1, R23, R24, R25, R26, R27, R28, R29, R30, R31, R32: 10k, custom_footprint_library:0.4_pitch_resistor, symbol Device:R
- added U1: ~, Connector_PinHeader_2.54mm:PinHeader_1x34_P2.54mm_Vertical, symbol custom_symbol_lib:prog_mem_read_bus_v2
- added U10, U12, U14, U16, U20, U23, U25, U33, U4: ~, Package_DIP:DIP-20_W7.62mm, symbol custom_symbol_lib:rising_edge_8_bit_latch
- added U11: ~, Connector_PinHeader_2.54mm:PinHeader_1x27_P2.54mm_Vertical, symbol custom_symbol_lib:bus_v2
- added U17: ~, Connector_PinHeader_2.54mm:PinHeader_1x30_P2.54mm_Vertical, symbol custom_symbol_lib:sequencer_v2
- added U2: ~, symbol custom_symbol_lib:ctrl_unit_bus_controls_v2
- added U26, U36: ~, Package_DIP:DIP-20_W7.62mm, symbol custom_symbol_lib:8_bit_transparent_latch
- added U27, U8: ~, Package_DIP:DIP-14_W7.62mm, symbol custom_symbol_lib:quad_OR
- added U28, U29, U30: ~, Package_DIP:DIP-14_W7.62mm, symbol custom_symbol_lib:quad_and
- added U3: ~, Connector_PinHeader_2.54mm:PinHeader_1x22_P2.54mm_Vertical, symbol custom_symbol_lib:call_stack_v2
- added U31: ~, Package_DIP:DIP-14_W7.62mm, symbol custom_symbol_lib:6xNOT
- added U32: ~, Package_DIP:DIP-14_W7.62mm, symbol custom_symbol_lib:dual_latch
- added U34, U37, U38: ~, custom_footprint_library:jumper_v2_gnd_footprint, symbol custom_symbol_lib:jumer_v2_gnd
- added U35: ~, Connector_PinHeader_2.54mm:PinHeader_2x04_P2.54mm_Vertical, symbol custom_symbol_lib:debug_v2_control_unit_main
Connections:
- net at R10.1, R11.1, R12.1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: no longer U13.16 (V+), U15.16 (V+), U18.16 (V+), U19.20 (V+), U21.16 (V+), U21.6 (B0), U24.20 (V+), U5.20 (V+), U6.20 (V+), U9.20 (V+)
- net at R11.2, U24.17 (Q2), U6.4 (D2)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: now also U1.6 (A2), U16.17 (Q2), U3.8 (Data_2)
- net at R10.2, U24.16 (Q3), U6.5 (D3)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: now also U1.7 (A3), U16.16 (Q3), U3.9 (Data_3)
- net at R9.2, U24.15 (Q4), U6.6 (D4)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: now also U1.8 (A4), U16.15 (Q4), U3.10 (Data_4)
- net at R8.2, U24.14 (Q5), U6.7 (D5)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: now also U1.9 (A5), U16.14 (Q5), U3.11 (Data_5)
- net at R4.2, U24.13 (Q6), U6.8 (D6)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: now also U1.10 (A6), U16.13 (Q6), U3.12 (Data_6)
- net at R14.2, U24.12 (Q7), U6.9 (D7)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: now also U1.11 (A7), U16.12 (Q7), U3.13 (Data_7)
- net at R15.2, U19.19 (Q0), U5.19 (Q0)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: now also R16.2, R17.2, R18.2, R19.2, R20.2, R21.2, R22.2, U19.12 (Q7), U19.13 (Q6), U19.14 (Q5), U19.15 (Q4), U19.16 (Q3), U19.17 (Q2), U19.18 (Q1), U5.12 (Q7), U5.13 (Q6), U5.14 (Q5), U5.15 (Q4), U5.16 (Q3), U5.17 (Q2), U5.18 (Q1), U6.11 (CLK), U9.11 (CLK), U9.3 (D1), U9.4 (D2), U9.5 (D3), U9.6 (D4), U9.7 (D5), U9.8 (D6), U9.9 (D7), U1.12 (A8), U1.13 (A9), U1.14 (A10), U1.15 (A11), U1.16 (A12), U1.17 (A13), U1.18 (A14), U17.10 (PC_MSB), U20.12 (Q7), U20.13 (Q6), U20.14 (Q5), U20.15 (Q4), U20.16 (Q3), U20.17 (Q2), U20.18 (Q1), U20.19 (Q0), U3.14 (Data_8), U3.15 (Data_9), U3.16 (Data_10), U3.17 (Data_11), U3.18 (Data_12), U3.19 (Data_13), U3.20 (Data_14), U3.21 (Data_15), U36.7 (D5)
- net at U13.11 (B3), U13.15 (B2), U13.2 (B1)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: no longer R2.2, R3.2, R5.2, R6.2, R7.2
- net at U22.1 (0): now also R28.2, U12.15 (Q4), U17.9 (Instruction_bit_4), U26.2 (D0), U36.6 (D4)
- net at U22.2 (1): now also R27.2, U12.14 (Q5), U26.3 (D1)
- net at U22.3 (2): now also R26.2, U12.13 (Q6), U26.4 (D2)
- net at U22.4 (3): now also R25.2, U12.12 (Q7), U26.5 (D3)
- net at R13.2, U24.19 (Q0), U6.2 (D0)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: now also U1.4 (A0), U16.19 (Q0), U3.6 (Data_0)
- net at R12.2, U24.18 (Q1), U6.3 (D1)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: now also U1.5 (A1), U16.18 (Q1), U3.7 (Data_1)
- net at U5.1 (OE#): no longer U7.1 (OE#)
- net at U5.2 (D0), U7.2 (D0): now also U11.20 (D0), U16.2 (D0), U20.2 (D0), U23.19 (Q0), U23.2 (D0), U25.19 (Q0), U25.2 (D0), U26.19 (Q0), U32.5 (0D)
- net at U5.3 (D1), U7.3 (D1): now also U11.21 (D1), U16.3 (D1), U20.3 (D1), U23.18 (Q1), U23.3 (D1), U25.18 (Q1), U25.3 (D1), U26.18 (Q1)
- net at U5.4 (D2), U7.4 (D2): now also U11.22 (D2), U16.4 (D2), U20.4 (D2), U23.17 (Q2), U23.4 (D2), U25.17 (Q2), U25.4 (D2), U26.17 (Q2)
- net at U5.5 (D3), U7.5 (D3): now also U11.23 (D3), U16.5 (D3), U20.5 (D3), U23.16 (Q3), U23.5 (D3), U25.16 (Q3), U25.5 (D3), U26.16 (Q3)
- net at U5.6 (D4), U7.6 (D4): now also U11.24 (D4), U16.6 (D4), U20.6 (D4), U23.15 (Q4), U23.6 (D4), U25.15 (Q4), U25.6 (D4), U26.15 (Q4)
- net at U5.7 (D5), U7.7 (D5): now also U11.25 (D5), U16.7 (D5), U20.7 (D5), U23.14 (Q5), U23.7 (D5), U25.14 (Q5), U25.7 (D5), U26.14 (Q5)
- net at U5.8 (D6), U7.8 (D6): now also U11.26 (D6), U16.8 (D6), U20.8 (D6), U23.13 (Q6), U23.8 (D6), U25.13 (Q6), U25.8 (D6), U26.13 (Q6)
- net at U5.9 (D7), U7.9 (D7): now also U11.27 (D7), U16.9 (D7), U20.9 (D7), U23.12 (Q7), U23.9 (D7), U25.12 (Q7), U25.9 (D7), U26.12 (Q7)
- net at R5.1: now also R2.1, R3.1, R6.1, R7.1, R1.1, R23.1, R24.1, R25.1, R26.1, R27.1, R29.1, R31.1, U11.1 (GND)
- new net: U12.1 (OE#), U14.1 (OE#)
- new net: U12.11 (CLK), U14.11 (CLK)
- new net: R29.2, U12.16 (Q3)
- new net: R30.2, U12.17 (Q2)
- new net: R31.2, U12.18 (Q1)
- new net: R32.2, U12.19 (Q0)
- new net: U12.2 (D0), U4.19 (Q0)
- new net: U12.3 (D1), U4.18 (Q1)
- new net: U12.4 (D2), U4.17 (Q2)
- new net: U12.5 (D3), U4.16 (Q3)
- new net: U12.6 (D4), U4.15 (Q4)
- new net: U12.7 (D5), U4.14 (Q5)
- new net: U12.8 (D6), U4.13 (Q6)
- new net: U12.9 (D7), U4.12 (Q7)
- new net: R3.2, U14.14 (Q5), U2.9 (RX_A1)
- new net: U1.19 (D0), U4.2 (D0)
- new net: U1.2 (Instruction_load_possible), U38.1 (IN)
- new net: U1.20 (D1), U4.3 (D1)
- new net: U1.21 (D2), U4.4 (D2)
- new net: U1.22 (D3), U4.5 (D3)
- new net: U1.23 (D4), U4.6 (D4)
- new net: U1.24 (D5), U4.7 (D5)
- new net: U1.25 (D6), U4.8 (D6)
- new net: U1.26 (D7), U4.9 (D7)
- new net: U1.27 (D8), U10.2 (D0)
- new net: U1.28 (D9), U10.3 (D1)
- new net: U1.29 (D10), U10.4 (D2)
- new net: U1.30 (D11), U10.5 (D3)
- new net: U1.31 (D12), U10.6 (D4)
- new net: U1.32 (D13), U10.7 (D5)
- new net: U1.33 (D14), U10.8 (D6)
- new net: U1.34 (D15), U10.9 (D7)
- new net: U32.1 (0Q), U34.1 (IN), U36.2 (D0)
- new net: U32.10 (1RESET), U32.11 (1CLK), U32.4 (0RESET), U32.6 (0SET), U32.7 (GND), U32.8 (1SET), U32.9 (1D), U34.2 (GND)
- new net: U17.3 (GOTO_Decider), U34.3 (OUT)
- new net: U17.7 (Opcode_(3-bit)_1), U29.11 (3Q), U36.4 (D2)
- new net: U17.8 (Opcode_(3-bit)_2), U29.8 (4Q), U36.5 (D3)
- new net: U32.3 (0CLK), U33.13 (Q6)
- new net: R2.2, U14.13 (Q6), U2.10 (RX_A2)
- new net: R1.2, U14.12 (Q7), U2.11 (RX_A4)
- new net: U2.12 (RX_A4), U30.6 (2Q)
- new net: U17.2 (Bus_move_done), U2.2 (Move_done)
- new net: R24.2, U14.19 (Q0), U2.3 (TX_A0), U26.6 (D4)
- new net: R23.2, U14.18 (Q1), U2.4 (TX_A1), U26.7 (D5)
- new net: R7.2, U14.17 (Q2), U2.5 (TX_A2), U26.8 (D6)
- new net: R6.2, U14.16 (Q3), U2.6 (TX_A3), U26.9 (D7)
- new net: U2.7 (TX_A4), U30.3 (1Q)
- new net: R5.2, U14.15 (Q4), U2.8 (RX_A0)
- new net: R28.1, R30.1, R32.1, U11.2 (+5V)
- new net: U11.3 (CLK), U17.4 (CLK)
- new net: U11.4 (Enable), U17.5 (Enable)
- new net: U11.6 (Start_-edge), U17.11 (Start_-edge)
- new net: U13.16 (V+), U15.16 (V+), U18.16 (V+), U19.20 (V+), U21.16 (V+), U21.6 (B0), U24.20 (V+), U6.20 (V+), U9.20 (V+)
- new net: U17.6 (Opcode_(3-bit)_0), U36.3 (D1), U8.11 (Q3)
- new net: U17.1 (Instruction_load_possible), U36.9 (D7), U38.3 (OUT)
- new net: U17.12 (Interrupt), U37.3 (OUT)
- new net: U16.20 (V+), U17.29 (+5V), U20.20 (V+), U23.20 (V+), U25.20 (V+)
- new net: U17.30 (GND), U20.10 (GND), U23.10 (GND), U37.2 (GND), U38.2 (GND)
- new net: U20.11 (CLK), U23.11 (CLK)
- new net: U35.1 (GOTO_Decider), U36.19 (Q0)
- new net: U35.2 (Opcode_(3-bit)_0), U36.18 (Q1)
- new net: U35.3 (Opcode_(3-bit)_1), U36.17 (Q2)
- new net: U35.4 (Opcode_(3-bit)_2), U36.16 (Q3)
- new net: U35.5 (Instruction_bit_4), U36.15 (Q4)
- new net: U35.6 (PC_MSB), U36.14 (Q5)
- new net: U35.7 (Interrupt), U36.13 (Q6)
- new net: U35.8 (Instruction_load_possible), U36.12 (Q7)
- new net: U16.10 (GND), U25.10 (GND)
- new net: U16.11 (CLK), U25.11 (CLK)
- new net: U10.1 (OE#), U10.10 (GND)
- new net: U10.12 (Q7), U14.9 (D7)
- new net: U10.13 (Q6), U14.8 (D6)
- new net: U10.14 (Q5), U14.7 (D5)
- new net: U10.15 (Q4), U14.6 (D4)
- new net: U10.16 (Q3), U14.5 (D3)
- new net: U10.17 (Q2), U14.4 (D2)
- new net: U10.18 (Q1), U14.3 (D1)
- new net: U10.19 (Q0), U14.2 (D0)
- new net: U36.1 (OE#), U36.10 (GND)
- new net: U36.11 (CLK), U36.20 (V+)
- new net: J1.1 (Pin_1), U36.8 (D6), U37.1 (IN)
- new net: U4.1 (OE#), U4.10 (GND)
- no-connect marks 13 -> 4
Other:
- note added: "Falling"
- note added: "G0"
- note added: "G1"
- note added: "G10"
- note added: "G11"
- note added: "G12"
- note added: "G13"
- note added: "G14"
- note added: "G15"
- note added: "G16"
- note added: "G17"
- note added: "G18"
- note added: "G2"
- note added: "G3"
- note added: "G4"
- note added: "G5"
- note added: "G6"
- note added: "G8"
- note added: "G9"
- note added: "INT-GOTO-A"
- note added: "INT-GOTO-B"
- note added: "Instruction final"
- note added: "Its pretty"
- note added: "Latch 7"
- note added: "PC and accessories"
- note added: "Pull up/down resistors to set the instruction to 0x0015 to call the interrupt handler"
- note added: "WRITE instruction -> Bus gate"
- note removed: "CALL STACK OE"
- note removed: "GOTO OE ->"
- note removed: "Instruction Lower"
- note removed: "Instruction Upper"
- note removed: "Pointer math"
- note removed: "Prog read done"
- moved on the sheet: R10, R11, R12, R13, R14, R15, R16, R17, R18, R19, R20, R21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

Commit message: Control unit main schematic verified
Parts:
- removed U14, U16: ~, Package_DIP:DIP-20_W7.62mm, symbol custom_symbol_lib:rising_edge_8_bit_latch
- removed U21: ~, Package_DIP:DIP-16_W7.62mm, symbol custom_symbol_lib:4bit_adder
- added R33, R34, R35, R36, R37: 10k, custom_footprint_library:0.4_pitch_resistor, symbol Device:R
- added U14: ~, Package_DIP:DIP-16_W7.62mm, symbol custom_symbol_lib:4bit_adder
- added U16: ~, Package_DIP:DIP-20_W7.62mm, symbol custom_symbol_lib:8_bit_transparent_latch
- added U39: ~, Package_DIP:DIP-14_W7.62mm, symbol custom_symbol_lib:6xNOT
- added U40, U41: ~, Package_DIP:DIP-20_W7.62mm, symbol custom_symbol_lib:rising_edge_8_bit_latch
Connections:
- net at R1.1, R2.1, R23.1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: now also U10.10 (GND), U12.10 (GND), U13.11 (B3), U13.15 (B2), U13.2 (B1), U13.6 (B0), U13.8 (GND), U15.11 (B3), U15.15 (B2), U15.2 (B1), U15.6 (B0), U15.8 (GND), U17.30 (GND), U18.11 (B3), U18.15 (B2), U18.2 (B1), U18.6 (B0), U18.8 (GND), U19.10 (GND), U20.10 (GND), U23.10 (GND), U24.1 (OE#), U24.10 (GND), U25.10 (GND), U26.10 (GND), U27.12 (3A), U27.13 (3B), U27.5 (1A), U27.6 (1B), U27.7 (GND), U27.8 (2A), U27.9 (2B), U28.7 (GND), U29.7 (GND), U3.1 (GND), U30.10 (4A), U30.12 (3B), U30.13 (3A), U30.7 (GND), U30.9 (4B), U31.7 (GND), U32.10 (1RESET), U32.11 (1CLK), U32.4 (0RESET), U32.6 (0SET), U32.7 (GND), U32.8 (1SET), U32.9 (1D), U33.1 (OE#), U33.10 (GND), U34.2 (GND), U36.1 (OE#), U36.10 (GND), U37.2 (GND), U38.2 (GND), U4.1 (OE#), U4.10 (GND), U5.10 (GND), U6.1 (OE#), U6.10 (GND), U7.10 (GND), U8.7 (GND), U9.10 (GND), R35.1, R36.1, R37.1, U14.11 (B3), U14.15 (B2), U14.2 (B1), U14.7 (C_IN), U14.8 (GND), U16.10 (GND), U39.11 (I4), U39.7 (GND), U39.9 (I3), U40.10 (GND), U41.1 (OE#), U41.10 (GND)
- net at U12.1 (OE#): now also U10.1 (OE#), U39.12 (O5)
- net at U12.11 (CLK): now also U10.11 (CLK), U17.24 (Instruction_post_latch_clk)
- net at R29.2, U12.16 (Q3): now also U29.1 (1A), U30.1 (1A), U30.4 (2A), U31.3 (I1)
- net at R30.2, U12.17 (Q2): now also U29.9 (4B)
- net at R31.2, U12.18 (Q1): now also U27.2 (0B), U28.9 (4B), U29.12 (3B)
- net at R32.2, U12.19 (Q0): now also U27.1 (0A), U28.10 (4A), U29.5 (2B), U31.5 (I2)
- net at U12.20 (V+): now also R10.1, R11.1, R12.1, R13.1, R14.1, R15.1, R16.1, R17.1, R18.1, R19.1, R20.1, R21.1, R22.1, R28.1, R30.1, R32.1, R4.1, R8.1, R9.1, U10.20 (V+), U11.2 (+5V), U13.16 (V+), U15.16 (V+), U17.29 (+5V), U18.16 (V+), U19.20 (V+), U20.20 (V+), U23.20 (V+), U24.20 (V+), U25.20 (V+), U26.11 (CLK), U26.20 (V+), U27.14 (V+), U28.14 (V+), U29.14 (V+), U3.2 (+5V), U30.14 (V+), U31.14 (V+), U32.14 (V+), U33.20 (V+), U36.11 (CLK), U36.20 (V+), U4.20 (V+), U5.20 (V+), U6.20 (V+), U7.20 (V+), U8.14 (V+), U9.20 (V+), R33.1, R34.1, U14.16 (V+), U16.11 (CLK), U16.20 (V+), U16.7 (D5), U16.8 (D6), U16.9 (D7), U39.14 (V+), U40.20 (V+), U41.20 (V+)
- net at R3.2, U2.9 (RX_A1): now also U10.14 (Q5)
- net at U1.1 (Read_source(0=flash_1=RAM)): now also U17.25 (RAM_Read)
- net at R4.2, U1.10 (A6), U3.12 (Data_6)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: now also U19.13 (Q6), U40.13 (Q6), U41.8 (D6); no longer U24.13 (Q6), U6.8 (D6)
- net at R14.2, U1.11 (A7), U3.13 (Data_7)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: now also U19.12 (Q7), U40.12 (Q7), U41.9 (D7); no longer U24.12 (Q7), U6.9 (D7)
- net at U1.2 (Instruction_load_possible), U38.1 (IN): now also U36.9 (D7)
- net at U1.27 (D8): now also U24.2 (D0); no longer U10.2 (D0)
- net at U1.28 (D9): now also U24.3 (D1); no longer U10.3 (D1)
- net at U1.29 (D10): now also U24.4 (D2); no longer U10.4 (D2)
- net at U1.3 (RAM_LSB): now also U17.14 (RAM_LSB)
- net at U1.30 (D11): now also U24.5 (D3); no longer U10.5 (D3)
- net at U1.31 (D12): now also U24.6 (D4); no longer U10.6 (D4)
- net at U1.32 (D13): now also U24.7 (D5); no longer U10.7 (D5)
- net at U1.33 (D14): now also U24.8 (D6); no longer U10.8 (D6)
- net at U1.34 (D15): now also U24.9 (D7); no longer U10.9 (D7)
- net at R13.2, U1.4 (A0), U3.6 (Data_0)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: now also U19.19 (Q0), U40.19 (Q0), U41.2 (D0); no longer U24.19 (Q0), U6.2 (D0)
- net at R12.2, U1.5 (A1), U3.7 (Data_1)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: now also U19.18 (Q1), U40.18 (Q1), U41.3 (D1); no longer U24.18 (Q1), U6.3 (D1)
- net at R11.2, U1.6 (A2), U3.8 (Data_2)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: now also U19.17 (Q2), U40.17 (Q2), U41.4 (D2); no longer U24.17 (Q2), U6.4 (D2)
- net at R10.2, U1.7 (A3), U3.9 (Data_3)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: now also U19.16 (Q3), U40.16 (Q3), U41.5 (D3); no longer U24.16 (Q3), U6.5 (D3)
- net at R9.2, U1.8 (A4), U3.10 (Data_4)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: now also U19.15 (Q4), U40.15 (Q4), U41.6 (D4); no longer U24.15 (Q4), U6.6 (D4)
- net at R8.2, U1.9 (A5), U3.11 (Data_5)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: now also U19.14 (Q5), U40.14 (Q5), U41.7 (D5); no longer U24.14 (Q5), U6.7 (D5)
- net at U29.10 (4A): now also U29.13 (3A), U29.4 (2A), U31.4 (O1)
- net at U29.2 (1B): now also U28.8 (4Q)
- net at U29.3 (1Q): now also U8.12 (3A)
- net at U29.6 (2Q): now also U8.13 (3B)
- net at U11.20 (D0), U20.2 (D0), U23.19 (Q0)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: now also U40.2 (D0)
- net at U2.1 (Move): now also U17.13 (Bus_move)
- net at R2.2, U2.10 (RX_A2): now also U10.13 (Q6)
- net at R1.2, U2.11 (RX_A4): now also U10.12 (Q7)
- net at R24.2, U26.6 (D4): now also U10.19 (Q0), U16.2 (D0); no longer U2.3 (TX_A0)
- net at R23.2, U26.7 (D5): now also U10.18 (Q1), U16.3 (D1); no longer U2.4 (TX_A1)
- net at R7.2, U26.8 (D6): now also U10.17 (Q2), U16.4 (D2); no longer U2.5 (TX_A2)
- net at R6.2, U26.9 (D7): now also U10.16 (Q3), U16.5 (D3); no longer U2.6 (TX_A3)
- net at U2.7 (TX_A4): now also R37.2, U16.15 (Q4); no longer U30.3 (1Q)
- net at R5.2, U2.8 (RX_A0): now also U10.15 (Q4)
- net at U11.10 (RX_Extend_(from_controller)): now also U28.12 (3B), U28.2 (1B), U28.5 (2B)
- net at U11.11 (TX_0): now also U33.9 (D7), U8.8 (2A)
- net at U11.12 (TX_1): now also U33.6 (D4), U8.1 (0A)
- net at U11.13 (TX_2): now also U33.7 (D5), U8.5 (1A)
- net at U11.15 (RX_0): now also U33.2 (D0)
- net at U11.16 (RX_1): now also U33.3 (D1)
- net at U11.17 (RX_2): now also U33.4 (D2)
- net at U11.18 (RX_3): now also U33.5 (D3)
- net at U11.19 (Fault): now also U17.20 (Halt)
- net at U11.21 (D1), U20.3 (D1), U23.18 (Q1)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: now also U40.3 (D1)
- net at U11.22 (D2), U20.4 (D2), U23.17 (Q2)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: now also U40.4 (D2)
- net at U11.23 (D3), U20.5 (D3), U23.16 (Q3)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: now also U40.5 (D3)
- net at U11.24 (D4), U20.6 (D4), U23.15 (Q4)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: now also U40.6 (D4)
- net at U11.25 (D5), U20.7 (D5), U23.14 (Q5)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: now also U40.7 (D5)
- net at U11.26 (D6), U20.8 (D6), U23.13 (Q6)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: now also U40.8 (D6)
- net at U11.27 (D7), U20.9 (D7), U23.12 (Q7)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: now also U40.9 (D7)
- net at U11.3 (CLK), U17.4 (CLK): now also U3.22 (CLK), U31.1 (I0)
- net at U11.4 (Enable), U17.5 (Enable): now also U3.3 (Enable)
- net at U5.1 (OE#): now also U7.1 (OE#), U39.2 (O0)
- net at U5.11 (CLK): now also U33.16 (Q3)
- net at U31.10 (O4): now also U23.1 (OE#)
- net at U31.11 (I4): now also U8.4 (Q1)
- net at U31.12 (O5): now also U25.1 (OE#)
- net at U31.13 (I5): now also U8.3 (Q0)
- net at U31.2 (O0): now also U33.11 (CLK)
- net at U31.6 (O2): now also U30.2 (1B)
- net at U31.8 (03): now also U26.1 (OE#)
- net at U31.9 (I3): now also U8.10 (Q2)
- net at U7.11 (CLK): now also U33.17 (Q2)
- net at U19.1 (OE#): now also U9.1 (OE#), U39.6 (O2); no longer U24.1 (OE#)
- net at U19.11 (CLK): now also U17.18 (Post-adder_latch_CLK), U9.11 (CLK); no longer U24.11 (CLK)
- net at U18.4 (Σ0): now also U19.6 (D4); no longer U24.6 (D4)
- net at U18.1 (Σ1): now also U19.7 (D5); no longer U24.7 (D5)
- net at U18.13 (Σ2): now also U19.8 (D6); no longer U24.8 (D6)
- net at U18.10 (Σ3): now also U19.9 (D7); no longer U24.9 (D7)
- net at U17.6 (Opcode_(3-bit)_0), U36.3 (D1), U8.11 (Q3): now also U16.1 (OE#)
- net at U8.2 (0B): now also U28.3 (1Q)
- net at U8.6 (1B): now also U28.6 (2Q)
- net at U8.9 (2B): now also U28.11 (3Q)
- net at U17.1 (Instruction_load_possible), U38.3 (OUT): no longer U36.9 (D7)
- net at U17.15 (INT-GOTO_latches_OE): now also U39.1 (I0)
- net at U17.16 (GOTO_latches_OE): now also U39.3 (I1)
- net at U17.17 (Post-adder_latch_OE): now also U39.5 (I2)
- net at U17.19 (Pre-adder_latch_CLK): now also U6.11 (CLK), U41.11 (CLK)
- net at U17.21 (Instruction++): now also U14.6 (B0)
- net at U17.22 (Instruction_pre-latch_A_clk): now also U4.11 (CLK)
- net at U17.23 (Instruction_pre-latch_B_clk): now also U24.11 (CLK)
- net at U17.26 (Call_stack_Pop_&_OE): now also U3.4 (Pop_&_OE)
- net at U17.27 (Call_stack_Push): now also U3.5 (Push)
- net at U17.28 (Instruction_post-latch_OE): now also U39.13 (I5)
- net at U15.1 (Σ1): now also U9.3 (D1); no longer U19.3 (D1)
- net at U15.10 (Σ3): now also U9.5 (D3); no longer U19.5 (D3)
- net at U9.16 (Q3): now also R18.2, U1.15 (A11), U20.16 (Q3), U3.17 (Data_11), U5.16 (Q3), U6.5 (D3); no longer U15.12 (A3)
- net at U15.13 (Σ2): now also U9.4 (D2); no longer U19.4 (D2)
- net at U9.17 (Q2): now also R17.2, U1.14 (A10), U20.17 (Q2), U3.16 (Data_10), U5.17 (Q2), U6.4 (D2); no longer U15.14 (A2)
- net at U9.18 (Q1): now also R16.2, U1.13 (A9), U20.18 (Q1), U3.15 (Data_9), U5.18 (Q1), U6.3 (D1); no longer U15.3 (A1)
- net at U15.4 (Σ0): now also U9.2 (D0); no longer U19.2 (D0)
- net at U9.19 (Q0): now also R15.2, U1.12 (A8), U20.19 (Q0), U3.14 (Data_8), U5.19 (Q0), U6.2 (D0); no longer U15.5 (A0)
- net at U20.1 (OE#): now also U39.4 (O1), U40.1 (OE#)
- net at U20.11 (CLK), U23.11 (CLK): now also U33.18 (Q1)
- net at U27.3 (Q0): now also U30.5 (2B)
- net at U25.11 (CLK): now also U33.19 (Q0), U40.11 (CLK)
- net at U28.1 (1A): now also U33.15 (Q4)
- net at U28.13 (3A): now also U33.12 (Q7)
- net at U28.4 (2A): now also U33.14 (Q5)
- net at U6.12 (Q7): now also U13.12 (A3); no longer U18.12 (A3)
- net at U6.13 (Q6): now also U13.14 (A2); no longer U18.14 (A2)
- net at U6.14 (Q5): now also U13.3 (A1); no longer U18.3 (A1)
- net at U6.15 (Q4): now also U13.5 (A0); no longer U18.5 (A0)
- net at U18.7 (C_IN): now also U14.9 (C_OUT)
- net at U13.1 (Σ1): now also U9.7 (D5); no longer U19.7 (D5)
- net at U13.10 (Σ3): now also U9.9 (D7); no longer U19.9 (D7)
- net at U9.12 (Q7): now also R22.2, U17.10 (PC_MSB), U20.12 (Q7), U3.21 (Data_15), U36.7 (D5), U5.12 (Q7), U6.9 (D7); no longer U13.12 (A3)
- net at U13.13 (Σ2): now also U9.8 (D6); no longer U19.8 (D6)
- net at U9.13 (Q6): now also R21.2, U1.18 (A14), U20.13 (Q6), U3.20 (Data_14), U5.13 (Q6), U6.8 (D6); no longer U13.14 (A2)
- net at U9.14 (Q5): now also R20.2, U1.17 (A13), U20.14 (Q5), U3.19 (Data_13), U5.14 (Q5), U6.7 (D5); no longer U13.3 (A1)
- net at U13.4 (Σ0): now also U9.6 (D4); no longer U19.6 (D4)
- net at U9.15 (Q4): now also R19.2, U1.16 (A12), U20.15 (Q4), U3.18 (Data_12), U5.15 (Q4), U6.6 (D4); no longer U13.5 (A0)
- net at U6.16 (Q3): now also U15.12 (A3)
- net at U6.17 (Q2): now also U15.14 (A2)
- net at U6.18 (Q1): now also U15.3 (A1)
- net at U6.19 (Q0): now also U15.5 (A0)
- net at U33.8 (D6): now also U2.13 (Bus_RX_GOTO_decider)
- new net: R33.2, U16.19 (Q0), U2.3 (TX_A0)
- new net: R34.2, U16.18 (Q1), U2.4 (TX_A1)
- new net: R35.2, U16.17 (Q2), U2.5 (TX_A2)
- new net: R36.2, U16.16 (Q3), U2.6 (TX_A3)
- new net: U10.2 (D0), U24.19 (Q0)
- new net: U10.3 (D1), U24.18 (Q1)
- new net: U10.4 (D2), U24.17 (Q2)
- new net: U10.5 (D3), U24.16 (Q3)
- new net: U10.6 (D4), U24.15 (Q4)
- new net: U10.7 (D5), U24.14 (Q5)
- new net: U10.8 (D6), U24.13 (Q6)
- new net: U10.9 (D7), U24.12 (Q7)
- new net: U16.6 (D4), U30.3 (1Q)
- new net: U18.12 (A3), U41.12 (Q7)
- new net: U18.14 (A2), U41.13 (Q6)
- new net: U18.3 (A1), U41.14 (Q5)
- new net: U18.5 (A0), U41.15 (Q4)
- new net: U14.12 (A3), U41.16 (Q3)
- new net: U14.14 (A2), U41.17 (Q2)
- new net: U14.3 (A1), U41.18 (Q1)
- new net: U14.5 (A0), U41.19 (Q0)
- new net: U14.1 (Σ1), U19.3 (D1)
- new net: U14.10 (Σ3), U19.5 (D3)
- new net: U14.13 (Σ2), U19.4 (D2)
- new net: U14.4 (Σ0), U19.2 (D0)
- no-connect marks 4 -> 19
Other:
- note added: "Bus TX Addr override for WRITE"
- note added: "GOTO-A OE -> Bus"
- note added: "GOTO-B OE -> Bus"
- note added: "INT-GOTO OE#"
- moved on the sheet: J1, R1, R2, R23, R24, R25, R26, R27, R28, R29, R3, R30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
