File: kicad/boards_version_2/gpram_v2/gpram.kicad_sch (KiCad schematic)
At the start: 68 parts

Commit message: Work mostly on bus
Parts:
- removed R1, R2, R3, R4, R5, R6, R7, R8: 10k, custom_footprint_library:0.4_pitch_resistor, symbol Device:R
- removed U1: ~, Connector_PinHeader_2.54mm:PinHeader_1x23_P2.54mm_Vertical, symbol custom_symbol_lib:bus_edge_connector
- removed U36, U42: ~, Package_DIP:DIP-14_W7.62mm, symbol custom_symbol_lib:quad_and
- removed U38, U41: ~, Package_DIP:DIP-14_W7.62mm, symbol custom_symbol_lib:quad_OR
- removed U39, U40: ~, Package_DIP:DIP-20_W7.62mm, symbol custom_symbol_lib:rising_edge_8_bit_latch
- removed U47: ~, Package_DIP:DIP-14_W7.62mm, symbol custom_symbol_lib:6xNOT
- added U9: ~, Connector_PinHeader_2.54mm:PinHeader_1x27_P2.54mm_Vertical, symbol custom_symbol_lib:bus_v2
Connections:
- net at U10.1 (OE#), U10.10 (GND), U11.11 (B3)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: no longer R9.1, U35.7 (GND), U35.8 (2A), U35.9 (2B), U4.10 (1RESET), U4.4 (0RESET), U4.6 (0SET), U4.7 (GND), U4.8 (1SET), U43.2 (GND), U44.7 (GND), U46.12 (3B), U46.13 (3A), U46.7 (GND)
- net at U14.2 (D0), U15.2 (D0), U16.19 (Q0)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: now also U9.20 (D0)
- net at U10.20 (V+), U11.16 (V+), U12.16 (V+)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: no longer U35.14 (V+), U37.14 (V+), U4.14 (V+), U44.14 (V+), U46.14 (V+)
- net at U14.3 (D1), U15.3 (D1), U16.18 (Q1)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: now also U9.21 (D1)
- net at U14.4 (D2), U15.4 (D2), U16.17 (Q2)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: now also U9.22 (D2)
- net at U14.5 (D3), U15.5 (D3), U16.16 (Q3)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: now also U9.23 (D3)
- net at U14.6 (D4), U15.6 (D4), U16.15 (Q4)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: now also U9.24 (D4)
- net at U14.7 (D5), U15.7 (D5), U16.14 (Q5)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: now also U9.25 (D5)
- net at U14.8 (D6), U15.8 (D6), U16.13 (Q6)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: now also U9.26 (D6)
- net at U14.9 (D7), U15.9 (D7), U16.12 (Q7)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: now also U9.27 (D7)
- net at U22.1 (IN), U23.1 (IN): no longer U37.4 (2A)
- net at U34.13 (I5), U37.9 (4B): no longer U35.12 (3A)
- new net: U4.10 (1RESET), U4.4 (0RESET), U4.6 (0SET), U4.7 (GND), U4.8 (1SET), U44.7 (GND), U46.12 (3B), U46.13 (3A), U46.7 (GND)
- new net: U4.14 (V+), U44.14 (V+), U46.14 (V+)
- new net: U35.7 (GND), U35.8 (2A), U35.9 (2B)
- no-connect marks 19 -> 5
Other:
- note added: "KEEP THIS FOR V2"
- note added: "RX Connections GPRAM-ADDR-B GPRAM-ADDR-A GPRAM-INC-ADDR GPRAM TX Connections: GPRAM-ADDR-B GPRAM-ADDR-A GPRAM-INC-ADDR GPRAM"
- note removed: "GPRAM-ADDR-B GPRAM-ADDR-A GPRAM-INC-ADDR GPRAM"
- note removed: "Write addr Write Read addr Read"
