File: kicad/boards_version_2/bus_v2/bus.kicad_sch (KiCad schematic)
At the start: 48 parts, among them J1 Barrel_Jack, U29 L7805

Commit message: Bus sequencer kicad verified
Parts:
- removed R1, R10, R11, R13, R14, R2, R3, R4, R5, R6, R7, R8, R9: 1k, custom_footprint_library:0.4_pitch_resistor, symbol Device:R
- removed U1: ~, Connector_PinHeader_2.54mm:PinHeader_1x11_P2.54mm_Vertical, symbol custom_symbol_lib:bus_arbiter_control_unit_connection
- removed U10, U11, U12, U13: ~, Package_DIP:DIP-16_W7.62mm, symbol custom_symbol_lib:3_to_8_demultiplexer
- removed U14, U28, U31: ~, Package_DIP:DIP-14_W7.62mm, symbol custom_symbol_lib:dual_latch
- removed U15: ~, Package_DIP:DIP-20_W7.62mm, symbol custom_symbol_lib:rising_edge_8_bit_latch
- removed U16, U30: ~, Package_DIP:DIP-14_W7.62mm, symbol custom_symbol_lib:quad_and
- removed U17, U18, U19, U20, U21, U22, U26, U27, U32, U33: ~, custom_footprint_library:jumper, symbol custom_symbol_lib:jumper
- removed U2, U24, U3, U4, U5, U6, U7: ~, Connector_PinHeader_2.54mm:PinHeader_1x23_P2.54mm_Vertical, symbol custom_symbol_lib:bus_edge_connector
- removed U23: ~, Package_DIP:DIP-14_W7.62mm, symbol custom_symbol_lib:6xNOT
- removed U25, U8: ~, Package_DIP:DIP-14_W7.62mm, symbol custom_symbol_lib:dual_4_input_OR
- removed U29: L7805, Package_TO_SOT_THT:TO-220-3_Vertical, symbol Regulator_Linear:L7805
- removed U34: ~, Connector_PinHeader_2.54mm:PinHeader_1x07_P2.54mm_Vertical, symbol custom_symbol_lib:bus_to_startup_ctrl
- removed U9: ~, Package_DIP:DIP-14_W7.62mm, symbol custom_symbol_lib:quad_OR
- added U1, U2, U3, U4, U5, U6, U7: ~, Connector_PinHeader_2.54mm:PinHeader_1x27_P2.54mm_Vertical, symbol custom_symbol_lib:bus_v2
- added U29: ~, symbol custom_symbol_lib:ctrl_unit_bus_controls_v2
- added U8: ~, Package_DIP:DIP-20_W7.62mm, symbol custom_symbol_lib:rising_edge_8_bit_latch
Connections:
- new net: U1.27 (D7), U2.27 (D7), U3.27 (D7), U4.27 (D7), U5.27 (D7), U6.27 (D7), U7.27 (D7), U8.12 (Q7), U8.9 (D7)
- new net: U1.26 (D6), U2.26 (D6), U3.26 (D6), U4.26 (D6), U5.26 (D6), U6.26 (D6), U7.26 (D6), U8.13 (Q6), U8.8 (D6)
- new net: U1.25 (D5), U2.25 (D5), U3.25 (D5), U4.25 (D5), U5.25 (D5), U6.25 (D5), U7.25 (D5), U8.14 (Q5), U8.7 (D5)
- new net: U1.24 (D4), U2.24 (D4), U3.24 (D4), U4.24 (D4), U5.24 (D4), U6.24 (D4), U7.24 (D4), U8.15 (Q4), U8.6 (D4)
- new net: U1.23 (D3), U2.23 (D3), U3.23 (D3), U4.23 (D3), U5.23 (D3), U6.23 (D3), U7.23 (D3), U8.16 (Q3), U8.5 (D3)
- new net: U1.22 (D2), U2.22 (D2), U3.22 (D2), U4.22 (D2), U5.22 (D2), U6.22 (D2), U7.22 (D2), U8.17 (Q2), U8.4 (D2)
- new net: U1.21 (D1), U2.21 (D1), U3.21 (D1), U4.21 (D1), U5.21 (D1), U6.21 (D1), U7.21 (D1), U8.18 (Q1), U8.3 (D1)
- new net: U1.20 (D0), U2.20 (D0), U3.20 (D0), U4.20 (D0), U5.20 (D0), U6.20 (D0), U7.20 (D0), U8.19 (Q0), U8.2 (D0)
- no-connect marks 42 -> 0
Other:
- note removed: "1 0"
- note removed: "10 9"
- note removed: "10 9 8 7"
- note removed: "11 8"
- note removed: "13 12 1"
- note removed: "14 3 2"
- note removed: "15 11"
- note removed: "2"
- note removed: "3"
- note removed: "6 5 4"
- note removed: "7 6 5 4"
- note removed: "ALU"
- note removed: "Clock"
- note removed: "Control unit"
- note removed: "Extra"
- note removed: "GPRAM controller"
- note removed: "I/O"
- note removed: "Read address"
- note removed: "Stack controller"
- note removed: "Write address"

Commit message: Work mostly on bus
Parts:
- removed J1: Barrel_Jack, Connector_BarrelJack:BarrelJack_Horizontal, symbol Connector:Barrel_Jack
- added D1, D10, D11, D12, D13, D14, D15, D16, D17, D18, D19, D2, D20, D21, D22, D23, D24, D25, D26, D27, D28, D29, D3, D30, D31, D32, D33, D34, D35, D36, D37, D38, D39, D4, D40, D41, D42, D43, D44, D45, D46, D47, D48, D49, D5, D50, D51, D52, D53, D54, D55, D56, D6, D7, D8, D9: LED, LED_THT:LED_D3.0mm, symbol Device:LED
- added R1, R10, R11, R12, R13, R14, R15, R16, R17, R18, R19, R2, R20, R21, R22, R23, R24, R25, R26, R27, R28, R29, R3, R30, R31, R32, R33, R34, R35, R36, R37, R38, R39, R4, R40, R41, R42, R43, R44, R45, R46, R47, R48, R49, R5, R50, R51, R52, R53, R54, R55, R56, R6, R7, R8, R9: 5K, symbol Device:R
- added U10, U11, U12, U13, U14, U15, U16: ~, Connector_PinHeader_2.54mm:PinHeader_1x27_P2.54mm_Vertical, symbol custom_symbol_lib:bus_v2
- added U17, U18, U19, U20, U21, U22, U23, U24: ~, Package_DIP:DIP-16_W7.62mm, symbol custom_symbol_lib:3_to_8_demultiplexer
- added U25: ~, Package_DIP:DIP-14_W7.62mm, symbol custom_symbol_lib:6xNOT
- added U26, U27, U28, U30, U31, U32, U33, U34, U47, U49: ~, Package_DIP:DIP-14_W7.62mm, symbol custom_symbol_lib:dual_4_input_OR
- added U35: ~, Connector_PinHeader_2.54mm:PinHeader_2x04_P2.54mm_Vertical, symbol custom_symbol_lib:debug_v2_bus
- added U36, U38, U39, U40, U41, U42, U43, U45: ~, custom_footprint_library:jumper_v2_gnd_footprint, symbol custom_symbol_lib:jumer_v2_gnd
- added U37: ~, Package_DIP:DIP-20_W7.62mm, symbol custom_symbol_lib:8_bit_transparent_latch
- added U44: ~, symbol custom_symbol_lib:starter_v2
- added U46: ~, Connector_PinHeader_2.54mm:PinHeader_1x05_P2.54mm_Vertical, symbol custom_symbol_lib:control_panel_v2
- added U9: ~, Connector_PinHeader_2.54mm:PinHeader_1x12_P2.54mm_Vertical, symbol custom_symbol_lib:bus_sequencer_v2
Connections:
- net at U8.1 (OE#): now also U25.2 (O0)
- net at U8.10 (GND): now also U1.1 (GND), U2.1 (GND), U3.1 (GND), U4.1 (GND), U5.1 (GND), U6.1 (GND), U7.1 (GND), R1.2, R10.2, R11.2, R12.2, R13.2, R14.2, R15.2, R16.2, R17.2, R18.2, R19.2, R2.2, R20.2, R21.2, R22.2, R23.2, R24.2, R25.2, R26.2, R27.2, R28.2, R29.2, R3.2, R30.2, R31.2, R32.2, R33.2, R34.2, R35.2, R36.2, R37.2, R38.2, R39.2, R4.2, R40.2, R41.2, R42.2, R43.2, R44.2, R45.2, R46.2, R47.2, R48.2, R49.2, R5.2, R50.2, R51.2, R52.2, R53.2, R54.2, R55.2, R56.2, R6.2, R7.2, R8.2, R9.2, U10.1 (GND), U11.1 (GND), U12.1 (GND), U13.1 (GND), U14.1 (GND), U15.1 (GND), U16.1 (GND), U25.13 (I5), U25.7 (GND), U26.7 (GND), U27.11 (B2), U27.12 (B3), U27.7 (GND), U28.7 (GND), U30.11 (B2), U30.12 (B3), U30.7 (GND), U31.7 (GND), U33.7 (GND), U34.7 (GND), U36.2 (GND), U37.1 (OE#), U37.10 (GND), U38.2 (GND), U39.2 (GND), U40.2 (GND), U41.2 (GND), U42.2 (GND), U43.2 (GND), U44.1 (GND), U45.2 (GND), U46.1 (GND), U47.7 (GND), U49.7 (GND), U9.2 (GND)
- net at U8.11 (CLK): now also U40.3 (OUT)
- net at U1.27 (D7), U2.27 (D7), U3.27 (D7)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: now also U10.27 (D7), U11.27 (D7), U12.27 (D7), U13.27 (D7), U14.27 (D7), U15.27 (D7), U16.27 (D7)
- net at U1.26 (D6), U2.26 (D6), U3.26 (D6)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: now also U10.26 (D6), U11.26 (D6), U12.26 (D6), U13.26 (D6), U14.26 (D6), U15.26 (D6), U16.26 (D6)
- net at U1.25 (D5), U2.25 (D5), U3.25 (D5)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: now also U10.25 (D5), U11.25 (D5), U12.25 (D5), U13.25 (D5), U14.25 (D5), U15.25 (D5), U16.25 (D5)
- net at U1.24 (D4), U2.24 (D4), U3.24 (D4)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: now also U10.24 (D4), U11.24 (D4), U12.24 (D4), U13.24 (D4), U14.24 (D4), U15.24 (D4), U16.24 (D4)
- net at U1.23 (D3), U2.23 (D3), U3.23 (D3)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: now also U10.23 (D3), U11.23 (D3), U12.23 (D3), U13.23 (D3), U14.23 (D3), U15.23 (D3), U16.23 (D3)
- net at U1.22 (D2), U2.22 (D2), U3.22 (D2)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: now also U10.22 (D2), U11.22 (D2), U12.22 (D2), U13.22 (D2), U14.22 (D2), U15.22 (D2), U16.22 (D2)
- net at U1.21 (D1), U2.21 (D1), U3.21 (D1)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: now also U10.21 (D1), U11.21 (D1), U12.21 (D1), U13.21 (D1), U14.21 (D1), U15.21 (D1), U16.21 (D1)
- net at U1.20 (D0), U2.20 (D0), U3.20 (D0)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: now also U10.20 (D0), U11.20 (D0), U12.20 (D0), U13.20 (D0), U14.20 (D0), U15.20 (D0), U16.20 (D0)
- net at U8.20 (V+): now also U1.2 (+5V), U2.2 (+5V), U3.2 (+5V), U4.2 (+5V), U5.2 (+5V), U6.2 (+5V), U7.2 (+5V), U10.2 (+5V), U11.2 (+5V), U12.2 (+5V), U13.2 (+5V), U14.2 (+5V), U15.2 (+5V), U16.2 (+5V), U25.14 (V+), U26.14 (V+), U27.14 (V+), U28.14 (V+), U30.14 (V+), U31.14 (V+), U32.14 (V+), U33.14 (V+), U34.14 (V+), U37.11 (CLK), U37.20 (V+), U44.2 (+5V), U46.2 (+5V), U47.14 (V+), U49.14 (V+), U9.1 (+5V)
- net at U4.10 (RX_Extend_(from_controller)): now also U1.10 (RX_Extend_(from_controller)), U2.10 (RX_Extend_(from_controller)), U3.10 (RX_Extend_(from_controller)), U5.10 (RX_Extend_(from_controller)), U6.10 (RX_Extend_(from_controller)), U7.10 (RX_Extend_(from_controller)), U10.10 (RX_Extend_(from_controller)), U11.10 (RX_Extend_(from_controller)), U12.10 (RX_Extend_(from_controller)), U13.10 (RX_Extend_(from_controller)), U14.10 (RX_Extend_(from_controller)), U15.10 (RX_Extend_(from_controller)), U16.10 (RX_Extend_(from_controller)), U43.3 (OUT)
- net at U4.19 (Fault): now also D13.2 (A), U26.5 (A3)
- net at U4.3 (CLK): now also U1.3 (CLK), U2.3 (CLK), U3.3 (CLK), U5.3 (CLK), U6.3 (CLK), U7.3 (CLK), U10.3 (CLK), U11.3 (CLK), U12.3 (CLK), U13.3 (CLK), U14.3 (CLK), U15.3 (CLK), U16.3 (CLK), U44.4 (CLK), U46.4 (CLK), U9.4 (CLK)
- net at U4.4 (Enable): now also U1.4 (Enable), U2.4 (Enable), U3.4 (Enable), U5.4 (Enable), U6.4 (Enable), U7.4 (Enable), U10.4 (Enable), U11.4 (Enable), U12.4 (Enable), U13.4 (Enable), U14.4 (Enable), U15.4 (Enable), U16.4 (Enable), U45.3 (OUT), U9.3 (Enable)
- net at U4.5 (Start_+edge): now also U1.5 (Start_+edge), U2.5 (Start_+edge), U3.5 (Start_+edge), U5.5 (Start_+edge), U6.5 (Start_+edge), U7.5 (Start_+edge), U10.5 (Start_+edge), U11.5 (Start_+edge), U12.5 (Start_+edge), U13.5 (Start_+edge), U14.5 (Start_+edge), U15.5 (Start_+edge), U16.5 (Start_+edge), U44.5 (Start_+edge)
- net at U4.6 (Start_-edge): now also U1.6 (Start_-edge), U2.6 (Start_-edge), U3.6 (Start_-edge), U5.6 (Start_-edge), U6.6 (Start_-edge), U7.6 (Start_-edge), U10.6 (Start_-edge), U11.6 (Start_-edge), U12.6 (Start_-edge), U13.6 (Start_-edge), U14.6 (Start_-edge), U15.6 (Start_-edge), U16.6 (Start_-edge), U44.6 (Start_-edge)
- net at U4.7 (TX_Ready): now also D16.2 (A), U33.5 (A3)
- net at U4.8 (RX_not_ready): now also D15.2 (A), U31.5 (A3)
- net at U4.9 (RX_Extend_(to_controller)): now also D14.2 (A), U28.5 (A3)
- net at U2.19 (Fault): now also D5.2 (A), U26.3 (A1)
- net at U2.7 (TX_Ready): now also D8.2 (A), U33.3 (A1)
- net at U2.8 (RX_not_ready): now also D7.2 (A), U31.3 (A1)
- net at U2.9 (RX_Extend_(to_controller)): now also D6.2 (A), U28.3 (A1)
- net at U29.1 (Move): now also U17.6 (E1), U25.5 (I2), U9.5 (Move/TX)
- net at U29.10 (RX_A2): now also U21.3 (A2), U22.3 (A2), U23.3 (A2), U24.3 (A2)
- net at U29.11 (RX_A4): now also U21.4 (E2#), U22.6 (E1), U23.4 (E2#), U24.6 (E1)
- net at U29.12 (RX_A4): now also U21.5 (E3#), U22.4 (E2#), U23.6 (E1), U25.11 (I4)
- net at U29.2 (Move_done): now also U42.3 (OUT)
- net at U29.3 (TX_A0): now also U17.1 (A0), U18.1 (A0), U19.1 (A0), U20.1 (A0)
- net at U29.4 (TX_A1): now also U17.2 (A1), U18.2 (A1), U19.2 (A1), U20.2 (A1)
- net at U29.5 (TX_A2): now also U17.3 (A2), U18.3 (A2), U19.3 (A2), U20.3 (A2)
- net at U29.6 (TX_A3): now also U17.4 (E2#), U18.6 (E1), U19.4 (E2#), U20.6 (E1)
- net at U29.7 (TX_A4): now also U17.5 (E3#), U18.4 (E2#), U19.6 (E1), U25.3 (I1)
- net at U29.8 (RX_A0): now also U21.1 (A0), U22.1 (A0), U23.1 (A0), U24.1 (A0)
- net at U29.9 (RX_A1): now also U21.2 (A1), U22.2 (A1), U23.2 (A1), U24.2 (A1)
- net at U1.19 (Fault): now also D1.2 (A), U26.2 (A0)
- net at U1.7 (TX_Ready): now also D4.2 (A), U33.2 (A0)
- net at U1.8 (RX_not_ready): now also D3.2 (A), U31.2 (A0)
- net at U1.9 (RX_Extend_(to_controller)): now also D2.2 (A), U28.2 (A0)
- net at U5.19 (Fault): now also D17.2 (A), U26.9 (B0)
- net at U5.7 (TX_Ready): now also D20.2 (A), U33.9 (B0)
- net at U5.8 (RX_not_ready): now also D19.2 (A), U31.9 (B0)
- net at U5.9 (RX_Extend_(to_controller)): now also D18.2 (A), U28.9 (B0)
- net at U7.19 (Fault): now also D25.2 (A), U26.11 (B2)
- net at U7.7 (TX_Ready): now also D28.2 (A), U33.11 (B2)
- net at U7.8 (RX_not_ready): now also D27.2 (A), U31.11 (B2)
- net at U7.9 (RX_Extend_(to_controller)): now also D26.2 (A), U28.11 (B2)
- net at U6.19 (Fault): now also D21.2 (A), U26.10 (B1)
- net at U6.7 (TX_Ready): now also D24.2 (A), U33.10 (B1)
- net at U6.8 (RX_not_ready): now also D23.2 (A), U31.10 (B1)
- net at U6.9 (RX_Extend_(to_controller)): now also D22.2 (A), U28.10 (B1)
- net at U3.19 (Fault): now also D9.2 (A), U26.4 (A2)
- net at U3.7 (TX_Ready): now also D12.2 (A), U33.4 (A2)
- net at U3.8 (RX_not_ready): now also D11.2 (A), U31.4 (A2)
- net at U3.9 (RX_Extend_(to_controller)): now also D10.2 (A), U28.4 (A2)
- new net: D39.1 (K), R39.1
- new net: D39.2 (A), U12.8 (RX_not_ready), U32.3 (A1)
- new net: D18.1 (K), R18.1
- new net: D42.1 (K), R42.1
- new net: D42.2 (A), U13.9 (RX_Extend_(to_controller)), U30.4 (A2)
- new net: D38.1 (K), R38.1
- new net: D38.2 (A), U12.9 (RX_Extend_(to_controller)), U30.3 (A1)
- new net: D47.1 (K), R47.1
- new net: D47.2 (A), U14.8 (RX_not_ready), U32.5 (A3)
- new net: U25.1 (I0), U41.3 (OUT)
- new net: U24.4 (E2#), U25.10 (O4)
- new net: U20.4 (E2#), U25.4 (O1)
- new net: U18.5 (E3#), U19.5 (E3#), U20.5 (E3#), U25.6 (O2)
- new net: U22.5 (E3#), U23.5 (E3#), U24.5 (E3#), U25.8 (03)
- new net: U21.6 (E1), U25.9 (I3), U36.3 (OUT), U9.6 (TX_ready/OE)
- new net: U37.9 (D7), U44.3 (Enable_out), U45.1 (IN)
- new net: U44.7 (Enable_in_debounced), U46.3 (Enable_to_starter)
- new net: D10.1 (K), R10.1
- new net: D3.1 (K), R3.1
- new net: D33.2 (A), U11.19 (Fault), U27.2 (A0)
- new net: D36.2 (A), U11.7 (TX_Ready), U34.2 (A0)
- new net: D35.2 (A), U11.8 (RX_not_ready), U32.2 (A0)
- new net: D34.2 (A), U11.9 (RX_Extend_(to_controller)), U30.2 (A0)
- new net: U17.16 (V+), U18.16 (V+), U19.16 (V+), U20.16 (V+), U21.16 (V+), U22.16 (V+), U23.16 (V+), U24.16 (V+)
- new net: U17.8 (GND), U18.8 (GND), U19.8 (GND), U20.8 (GND), U21.8 (GND), U22.8 (GND), U23.8 (GND), U24.8 (GND)
- new net: U37.5 (D3), U40.1 (IN), U9.9 (Bus_save_CLK)
- new net: D41.1 (K), R41.1
- new net: D41.2 (A), U13.19 (Fault), U27.4 (A2)
- new net: D29.1 (K), R29.1
- new net: D29.2 (A), U10.19 (Fault), U26.12 (B3)
- new net: U34.1 (OA), U49.4 (A2)
- new net: D56.2 (A), U16.7 (TX_Ready), U34.10 (B1)
- new net: U34.13 (OB), U49.5 (A3)
- new net: D40.2 (A), U12.7 (TX_Ready), U34.3 (A1)
- new net: D44.2 (A), U13.7 (TX_Ready), U34.4 (A2)
- new net: D48.2 (A), U14.7 (TX_Ready), U34.5 (A3)
- new net: D52.2 (A), U15.7 (TX_Ready), U34.9 (B0)
- new net: D33.1 (K), R33.1
- new net: D27.1 (K), R27.1
- new net: D37.1 (K), R37.1
- new net: D37.2 (A), U12.19 (Fault), U27.3 (A1)
- new net: D49.1 (K), R49.1
- new net: D49.2 (A), U15.19 (Fault), U27.9 (B0)
- new net: D9.1 (K), R9.1
- new net: D35.1 (K), R35.1
- new net: D56.1 (K), R56.1
- new net: D32.1 (K), R32.1
- new net: D55.1 (K), R55.1
- new net: D45.2 (A), U14.19 (Fault), U27.5 (A3)
- new net: D46.2 (A), U14.9 (RX_Extend_(to_controller)), U30.5 (A3)
- new net: D17.1 (K), R17.1
- new net: D4.1 (K), R4.1
- new net: D15.1 (K), R15.1
- new net: D5.1 (K), R5.1
- new net: D7.1 (K), R7.1
- new net: D23.1 (K), R23.1
- new net: D25.1 (K), R25.1
- new net: U37.3 (D1), U38.1 (IN), U49.13 (OB)
- new net: U38.3 (OUT), U9.7 (RX_not_ready)
- new net: D48.1 (K), R48.1
- new net: D22.1 (K), R22.1
- new net: U37.7 (D5), U42.1 (IN), U9.11 (Move_done)
- new net: D45.1 (K), R45.1
- new net: D20.1 (K), R20.1
- new net: D32.2 (A), U10.7 (TX_Ready), U33.12 (B3)
- new net: D31.2 (A), U10.8 (RX_not_ready), U31.12 (B3)
- new net: D30.2 (A), U10.9 (RX_Extend_(to_controller)), U28.12 (B3)
- new net: D19.1 (K), R19.1
- new net: D40.1 (K), R40.1
- new net: D11.1 (K), R11.1
- new net: D26.1 (K), R26.1
- new net: D50.1 (K), R50.1
- new net: D46.1 (K), R46.1
- new net: D16.1 (K), R16.1
- new net: D28.1 (K), R28.1
- new net: D31.1 (K), R31.1
- new net: D12.1 (K), R12.1
- new net: D54.1 (K), R54.1
- new net: U37.6 (D4), U41.1 (IN), U9.10 (Bus_save_OE)
- new net: U37.8 (D6), U43.1 (IN), U9.12 (RX_extend_from_controller)
- new net: U39.3 (OUT), U9.8 (RX_extend_to_controller)
- new net: D13.1 (K), R13.1
- new net: D53.1 (K), R53.1
- new net: D43.1 (K), R43.1
- new net: D34.1 (K), R34.1
- new net: U27.1 (OA), U47.11 (B2)
- new net: D53.2 (A), U16.19 (Fault), U27.10 (B1)
- new net: U27.13 (OB), U47.12 (B3)
- new net: D21.1 (K), R21.1
- new net: D51.2 (A), U15.8 (RX_not_ready), U32.9 (B0)
- new net: D50.2 (A), U15.9 (RX_Extend_(to_controller)), U30.9 (B0)
- new net: U30.1 (OA), U47.4 (A2)
- new net: D54.2 (A), U16.9 (RX_Extend_(to_controller)), U30.10 (B1)
- new net: U30.13 (OB), U47.5 (A3)
- new net: D52.1 (K), R52.1
- new net: U31.1 (OA), U49.9 (B0)
- new net: U31.13 (OB), U49.10 (B1)
- new net: D36.1 (K), R36.1
- new net: U32.1 (OA), U49.11 (B2)
- new net: D55.2 (A), U16.8 (RX_not_ready), U32.10 (B1)
- new net: U32.11 (B2), U32.12 (B3), U32.7 (GND)
- new net: U32.13 (OB), U49.12 (B3)
- new net: D43.2 (A), U13.8 (RX_not_ready), U32.4 (A2)
- new net: D1.1 (K), R1.1
- new net: D24.1 (K), R24.1
- new net: D44.1 (K), R44.1
- new net: U36.1 (IN), U37.2 (D0), U49.1 (OA)
- new net: U33.1 (OA), U49.2 (A0)
- new net: U33.13 (OB), U49.3 (A1)
- new net: D8.1 (K), R8.1
- new net: U37.4 (D2), U39.1 (IN), U47.1 (OA)
- new net: U26.13 (OB), U47.10 (B1)
- new net: U46.5 (Fault), U47.13 (OB)
- new net: U28.1 (OA), U47.2 (A0)
- new net: U28.13 (OB), U47.3 (A1)
- new net: U26.1 (OA), U47.9 (B0)
- new net: D30.1 (K), R30.1
- new net: D6.1 (K), R6.1
- new net: D14.1 (K), R14.1
- new net: U35.8 (Enable), U37.12 (Q7)
- new net: U35.7 (RX_extend_from_controller), U37.13 (Q6)
- new net: U35.6 (Move_done), U37.14 (Q5)
- new net: U35.5 (Bus_save_OE), U37.15 (Q4)
- new net: U35.4 (Bus_save_CLK), U37.16 (Q3)
- new net: U35.3 (RX_extend_to_controller), U37.17 (Q2)
- new net: U35.2 (RX_not_ready), U37.18 (Q1)
- new net: U35.1 (TX_Ready/OE/RX), U37.19 (Q0)
- new net: D2.1 (K), R2.1
- new net: D51.1 (K), R51.1
- no-connect marks 0 -> 1
Other:
- note added: "!Bus save OE"
- note added: "!RX"
- note added: "!RX A4"
- note added: "!TX"
- note added: "!TX A4"
- note added: "0 - 7"
- note added: "16 - 23"
- note added: "24 - 31"
- note added: "8 - 15"
- note added: "ALU"
- note added: "Control unit main board"
- note added: "Expansion slot 0"
- note added: "Expansion slot 1"
- note added: "Expansion slot 2"
- note added: "Expansion slot 3"
- note added: "Fault"
- note added: "GPRAM Sequencer & address"
- note added: "GPRAM Shared memory"
- note added: "I/O Controller (horizontal, to the side)"
- note added: "Interrupt handler data/main"
- note added: "Program memory"
- note added: "RX Decoders"
- note added: "RX Extend to controller"
- note added: "RX not ready"
- note added: "Stack data/main"
- note added: "TX Decoders"
- note added: "TX Ready"
- note added: "Timers"
- note added: "Vector digital board"
- moved on the sheet: U1, U2, U3, U4, U5, U6, U7, U8

Commit message: Work on bus
Parts:
- added J1, J4: Conn_01x16, symbol Connector_Generic:Conn_01x16
- added J2: Conn_01x15, symbol Connector_Generic:Conn_01x15
- added J3: Conn_01x06, symbol Connector_Generic:Conn_01x06
Connections:
- net at U11.15 (RX_0): now also U23.13 (Y2)
- net at U11.16 (RX_1): now also U23.12 (Y3)
- net at U11.17 (RX_2): now also U23.11 (Y4)
- net at U11.18 (RX_3): now also U23.10 (Y5)
- net at U21.10 (Y5): now also U1.16 (RX_1)
- net at U21.11 (Y4): now also U1.15 (RX_0)
- net at U21.12 (Y3): now also U5.16 (RX_1)
- net at U21.13 (Y2): now also U5.15 (RX_0)
- net at U21.14 (Y1): now also U6.15 (RX_0)
- net at U21.7 (Y7): now also U4.15 (RX_0)
- net at U21.9 (Y6): now also U29.13 (Bus_RX_GOTO_decider)
- net at U4.11 (TX_0): now also U17.11 (Y4)
- net at U4.12 (TX_1): now also U17.10 (Y5)
- net at U4.13 (TX_2): now also U17.9 (Y6)
- net at U4.14 (TX_3): now also U17.7 (Y7)
- net at U4.16 (RX_1): now also U22.15 (Y0)
- net at U4.17 (RX_2): now also U22.14 (Y1)
- net at U4.18 (RX_3): now also U22.13 (Y2)
- net at U12.11 (TX_0): now also U18.15 (Y0)
- net at U12.12 (TX_1): now also U18.12 (Y3)
- net at U12.15 (RX_0): now also U22.12 (Y3)
- net at U12.16 (RX_1): now also U22.7 (Y7)
- net at U18.10 (Y5): now also U7.12 (TX_1)
- net at U18.11 (Y4): now also U7.11 (TX_0)
- net at U18.13 (Y2): now also U10.12 (TX_1)
- net at U18.14 (Y1): now also U10.11 (TX_0)
- net at U18.7 (Y7): now also U1.12 (TX_1)
- net at U18.9 (Y6): now also U6.13 (TX_2)
- net at U14.11 (TX_0): now also J4.8 (Pin_8)
- net at U14.12 (TX_1): now also J4.7 (Pin_7)
- net at U14.13 (TX_2): now also J4.6 (Pin_6)
- net at U14.14 (TX_3): now also J4.5 (Pin_5)
- net at U14.15 (RX_0): now also J1.8 (Pin_8)
- net at U14.16 (RX_1): now also J1.7 (Pin_7)
- net at U14.17 (RX_2): now also J1.6 (Pin_6)
- net at U14.18 (RX_3): now also J1.5 (Pin_5)
- net at U10.15 (RX_0): now also U23.9 (Y6)
- net at U10.16 (RX_1): now also U23.7 (Y7)
- net at U10.17 (RX_2): now also U24.15 (Y0)
- net at U2.15 (RX_0): now also U24.14 (Y1)
- net at U19.10 (Y5): now also J2.5 (Pin_5)
- net at U19.11 (Y4): now also J2.4 (Pin_4)
- net at U19.12 (Y3): now also J2.3 (Pin_3)
- net at U19.13 (Y2): now also J2.2 (Pin_2)
- net at U19.14 (Y1): now also J2.1 (Pin_1)
- net at U19.15 (Y0): now also U1.13 (TX_2)
- net at U19.7 (Y7): now also J2.7 (Pin_7)
- net at U19.9 (Y6): now also J2.6 (Pin_6)
- net at U15.11 (TX_0): now also J4.12 (Pin_12)
- net at U15.12 (TX_1): now also J4.11 (Pin_11)
- net at U15.13 (TX_2): now also J4.10 (Pin_10)
- net at U15.14 (TX_3): now also J4.9 (Pin_9)
- net at U15.15 (RX_0): now also J1.12 (Pin_12)
- net at U15.16 (RX_1): now also J1.11 (Pin_11)
- net at U15.17 (RX_2): now also J1.10 (Pin_10)
- net at U15.18 (RX_3): now also J1.9 (Pin_9)
- net at U24.10 (Y5): now also J3.4 (Pin_4)
- net at U24.11 (Y4): now also J3.3 (Pin_3)
- net at U24.12 (Y3): now also J3.2 (Pin_2)
- net at U24.13 (Y2): now also J3.1 (Pin_1)
- net at U24.7 (Y7): now also J3.6 (Pin_6)
- net at U24.9 (Y6): now also J3.5 (Pin_5)
- net at U22.10 (Y5): now also U6.17 (RX_2)
- net at U22.11 (Y4): now also U6.16 (RX_1)
- net at U22.9 (Y6): now also U5.17 (RX_2)
- net at U16.11 (TX_0): now also J4.16 (Pin_16)
- net at U16.12 (TX_1): now also J4.15 (Pin_15)
- net at U16.13 (TX_2): now also J4.14 (Pin_14)
- net at U16.14 (TX_3): now also J4.13 (Pin_13)
- net at U16.15 (RX_0): now also J1.16 (Pin_16)
- net at U16.16 (RX_1): now also J1.15 (Pin_15)
- net at U16.17 (RX_2): now also J1.14 (Pin_14)
- net at U16.18 (RX_3): now also J1.13 (Pin_13)
- net at U23.14 (Y1): now also U1.18 (RX_3)
- net at U23.15 (Y0): now also U1.17 (RX_2)
- net at U13.11 (TX_0): now also J4.4 (Pin_4)
- net at U13.12 (TX_1): now also J4.3 (Pin_3)
- net at U13.13 (TX_2): now also J4.2 (Pin_2)
- net at U13.14 (TX_3): now also J4.1 (Pin_1)
- net at U13.15 (RX_0): now also J1.4 (Pin_4)
- net at U13.16 (RX_1): now also J1.3 (Pin_3)
- net at U13.17 (RX_2): now also J1.2 (Pin_2)
- net at U13.18 (RX_3): now also J1.1 (Pin_1)
- net at U17.12 (Y3): now also U1.11 (TX_0)
- net at U17.13 (Y2): now also U5.11 (TX_0)
- net at U17.14 (Y1): now also U6.12 (TX_1)
- net at U17.15 (Y0): now also U6.11 (TX_0)
- net at U20.10 (Y5): now also J2.13 (Pin_13)
- net at U20.11 (Y4): now also J2.12 (Pin_12)
- net at U20.12 (Y3): now also J2.11 (Pin_11)
- net at U20.13 (Y2): now also J2.10 (Pin_10)
- net at U20.14 (Y1): now also J2.9 (Pin_9)
- net at U20.15 (Y0): now also J2.8 (Pin_8)
- net at U20.7 (Y7): now also J2.15 (Pin_15)
- net at U20.9 (Y6): now also J2.14 (Pin_14)
- no-connect marks 1 -> 40
Other:
- note added: "Expansion RX"
- note added: "Expansion TX"
- note added: "RX outputs expansion"
- note added: "TX outputs expansion"

Commit message: Bus and starter verified
Connections:
- net at R1.2, R10.2, R11.2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: now also U17.8 (GND), U18.8 (GND), U19.8 (GND), U20.8 (GND), U21.8 (GND), U22.8 (GND), U23.8 (GND), U24.8 (GND), U32.11 (B2), U32.12 (B3), U32.7 (GND)
- net at U1.2 (+5V), U10.2 (+5V), U11.2 (+5V)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: now also U17.16 (V+), U18.16 (V+), U19.16 (V+), U20.16 (V+), U21.16 (V+), U22.16 (V+), U23.16 (V+), U24.16 (V+)
Changed lines of the file:
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@@
 	)
 	(junction
+		(at 226.06 142.24)
+		(diameter 0)
+		(color 0 0 0 0)
+	)
+	(junction
 		(at 417.83 264.16)
 		(diameter 0)
@@
 	)
 	(junction
+		(at 161.29 355.6)
+		(diameter 0)
+		(color 0 0 0 0)
+	)
+	(junction
 		(at 125.73 224.79)
 		(diameter 0)
@@
 	)
 	(junction
+		(at 161.29 341.63)
+		(diameter 0)
+		(color 0 0 0 0)
+	)
+	(junction
 		(at 110.49 224.79)
 		(diameter 0)
@@
 	)
 	(junction
+		(at 204.47 142.24)
+		(diameter 0)
+		(color 0 0 0 0)
+	)
+	(junction
 		(at 231.14 257.81)
 		(diameter 0)
@@
 	(wire
 		(pts
+			(xy 161.29 341.63) (xy 210.82 341.63)
+		)
+		(stroke
+			(width 0)
+			(type default)
+		)
+	)
+	(wire
+		(pts
 			(xy 661.67 288.29) (xy 702.31 288.29)
 		)
@@
 	(wire
 		(pts
+			(xy 204.47 142.24) (xy 204.47 123.19)
+		)
+		(stroke
+			(width 0)
+			(type default)
+		)
+	)
+	(wire
+		(pts
 			(xy 224.79 264.16) (xy 255.27 264.16)
 		)
@@
 	(wire
 		(pts
+			(xy 204.47 142.24) (xy 226.06 142.24)
+		)
+		(stroke
+			(width 0)
+			(type default)
+		)
+	)
+	(wire
+		(pts
 			(xy 283.21 443.23) (xy 231.14 443.23)
 		)
@@
 	(wire
 		(pts
-			(xy 204.47 163.83) (xy 204.47 123.19)
+			(xy 204.47 163.83) (xy 204.47 142.24)
 		)
 		(stroke
@@
 	(wire
 		(pts
+			(xy 161.29 358.14) (xy 161.29 355.6)
+		)
+		(stroke
+			(width 0)
+			(type default)
+		)
+	)
+	(wire
+		(pts
 			(xy 170.18 312.42) (xy 205.74 312.42)
 		)
@@
 		)
 		(stroke
+			(width 0)
+			(type default)
+		)
+	)
+	(wire
+		(pts
+			(xy 209.55 358.14) (xy 161.29 358.14)
+		)
+		(stroke
