File: kicad/boards_version_2/ALU_v2/ALU.kicad_sch (KiCad schematic)
At the start: 59 parts

Commit message: Work mostly on bus
Parts:
- removed U2: ~, Connector_PinHeader_2.54mm:PinHeader_1x23_P2.54mm_Vertical, symbol custom_symbol_lib:bus_edge_connector
- added U2: ~, Connector_PinHeader_2.54mm:PinHeader_1x27_P2.54mm_Vertical, symbol custom_symbol_lib:bus_v2
Connections:
- net at U10.7 (GND), U11.11 (I4), U11.7 (GND)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: no longer R1.1, R2.1, R3.1, R4.1, R5.1, U14.1 (OE#), U14.10 (GND), U46.2 (GND), U47.2 (GND), U48.2 (GND), U49.2 (GND), U50.1 (1A), U50.2 (1B), U50.4 (2A), U50.5 (2B), U50.7 (GND), U51.10 (1RESET), U51.11 (1CLK), U51.4 (0RESET), U51.6 (0SET), U51.7 (GND), U51.8 (1SET), U51.9 (1D), U52.1 (I0), U52.11 (I4), U52.3 (I1), U52.5 (I2), U52.7 (GND), U52.9 (I3), U53.12 (3B), U53.13 (3A), U53.7 (GND)
- net at U14.9 (D7), U16.12 (Q7), U17.12 (Q7)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: now also U2.27 (D7)
- net at U14.8 (D6), U16.13 (Q6), U17.13 (Q6)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: now also U2.26 (D6)
- net at U14.7 (D5), U16.14 (Q5), U17.14 (Q5)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: now also U2.25 (D5)
- net at U14.6 (D4), U16.15 (Q4), U17.15 (Q4)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: now also U2.24 (D4)
- net at U14.5 (D3), U16.16 (Q3), U17.16 (Q3)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: now also U2.23 (D3)
- net at U14.4 (D2), U16.17 (Q2), U17.17 (Q2)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: now also U2.22 (D2)
- net at U14.3 (D1), U16.18 (Q1), U17.18 (Q1)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: now also U2.21 (D1)
- net at U14.2 (D0), U16.19 (Q0), U17.19 (Q0)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: now also U2.20 (D0)
- new net: R1.1, R2.1, R3.1, R4.1, R5.1, U14.1 (OE#), U14.10 (GND), U46.2 (GND), U47.2 (GND), U48.2 (GND), U49.2 (GND), U50.1 (1A), U50.2 (1B), U50.4 (2A), U50.5 (2B), U50.7 (GND), U51.10 (1RESET), U51.11 (1CLK), U51.4 (0RESET), U51.6 (0SET), U51.7 (GND), U51.8 (1SET), U51.9 (1D), U52.1 (I0), U52.11 (I4), U52.3 (I1), U52.5 (I2), U52.7 (GND), U52.9 (I3), U53.12 (3B), U53.13 (3A), U53.7 (GND)
- no-connect marks 42 -> 37
Other:
- note added: "RX Addresses: 0. ALU-A 1. ALU-B 2. ALU-C-IN TX Addresses: 0. ALU"
- note removed: "ALU - - -"
- note removed: "ALU-A ALU-B ALU-C-IN -"

Commit message: ALU v2 verified
Parts:
- removed R1, R2, R3, R4, R5: 10k, custom_footprint_library:0.4_pitch_resistor, symbol Device:R
- removed U12: ~, Package_DIP:DIP-14_W7.62mm, symbol custom_symbol_lib:2x_4_input_AND
- removed U14: ~, Package_DIP:DIP-20_W7.62mm, symbol custom_symbol_lib:rising_edge_8_bit_latch
- removed U15: ~, Package_DIP:DIP-16_W7.62mm, symbol custom_symbol_lib:4bit_adder
- removed U19, U52: ~, Package_DIP:DIP-14_W7.62mm, symbol custom_symbol_lib:6xNOT
- removed U23: ~, Package_DIP:DIP-14_W7.62mm, symbol custom_symbol_lib:quad_OR
- removed U3: ~, Connector_PinHeader_2.54mm:PinHeader_1x30_P2.54mm_Horizontal, symbol custom_symbol_lib:ALU_extension
- removed U42, U53, U54: ~, Package_DIP:DIP-14_W7.62mm, symbol custom_symbol_lib:quad_and
- removed U46, U47, U48, U49: ~, custom_footprint_library:jumper, symbol custom_symbol_lib:jumper
- removed U51: ~, Package_DIP:DIP-14_W7.62mm, symbol custom_symbol_lib:dual_latch
- removed U6: ~, Package_DIP:DIP-20_W7.62mm, symbol custom_symbol_lib:8_bit_transparent_latch
- added U12, U46, U6: ~, Package_DIP:DIP-20_W7.62mm, symbol custom_symbol_lib:rising_edge_8_bit_latch
- added U14, U42: ~, Package_DIP:DIP-14_W7.62mm, symbol custom_symbol_lib:quad_OR
- added U15, U19: ~, Package_DIP:DIP-14_W7.62mm, symbol custom_symbol_lib:quad_and
- added U23, U49: ~, Package_DIP:DIP-14_W7.62mm, symbol custom_symbol_lib:6xNOT
- added U3: ~, Connector_PinHeader_2.54mm:PinHeader_2x20_P2.54mm_Vertical, symbol custom_symbol_lib:alu_extension_v2
- added U47: ~, Package_DIP:DIP-16_W7.62mm, symbol custom_symbol_lib:4bit_adder
- added U48: ~, Package_DIP:DIP-14_W7.62mm, symbol custom_symbol_lib:dual_4_input_OR
Connections:
- net at U24.1 (1A), U27.1 (1A), U30.4 (D0)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: now also U14.1 (0A), U23.1 (I0), U3.1 (A0), U47.5 (A0); no longer U13.5 (A0), U18.1 (I0), U21.1 (0A)
- net at U24.5 (2B), U27.6 (2B), U30.10 (A1)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: now also U14.6 (1B), U3.10 (B1), U47.2 (B1); no longer U13.2 (B1), U21.6 (1B)
- net at U24.12 (3B), U27.9 (3B), U30.9 (A2)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: now also U14.9 (2B), U3.11 (B2), U47.15 (B2); no longer U13.15 (B2), U21.9 (2B)
- net at U24.9 (4B), U27.13 (4B), U39.13 (4B)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: now also U14.13 (3B), U3.12 (B3), U47.11 (B3); no longer U13.11 (B3), U21.13 (3B)
- net at U28.2 (1B), U40.2 (1B), U45.6 (D4)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: now also U13.6 (B0), U21.2 (0B), U19.2 (1B), U3.13 (B4); no longer U25.2 (1B)
- net at U28.6 (2B), U40.6 (2B), U45.7 (D5)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: now also U13.2 (B1), U21.6 (1B), U19.5 (2B), U3.14 (B5); no longer U25.5 (2B)
- net at U28.9 (3B), U40.9 (3B), U45.8 (D6)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: now also U13.15 (B2), U21.9 (2B), U19.12 (3B), U3.15 (B6); no longer U25.12 (3B)
- net at U28.13 (4B), U40.13 (4B), U45.9 (D7)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: now also U13.11 (B3), U21.13 (3B), U19.9 (4B), U3.16 (B7); no longer U25.9 (4B)
- net at U24.4 (2A), U27.5 (2A), U30.12 (D7)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: now also U14.5 (1A), U23.3 (I1), U3.2 (A1), U47.3 (A1); no longer U13.3 (A1), U18.3 (I1), U21.5 (1A)
- net at U10.14 (V+), U11.14 (V+), U13.16 (V+)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: now also U2.2 (+5V), U12.20 (V+), U14.14 (V+), U15.14 (V+), U19.14 (V+), U23.14 (V+), U3.39 (V+), U42.14 (V+), U46.20 (V+), U47.16 (V+), U48.14 (V+), U49.14 (V+), U6.20 (V+)
- net at U24.13 (3A), U27.8 (3A), U30.13 (D6)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: now also U14.8 (2A), U23.5 (I2), U3.3 (A2), U47.14 (A2); no longer U13.14 (A2), U18.5 (I2), U21.8 (2A)
- net at U10.7 (GND), U11.7 (GND), U13.8 (GND)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: now also U18.11 (I4), U18.13 (I5), U18.5 (I2), U18.9 (I3), U2.1 (GND), U25.10 (4A), U25.12 (3B), U25.13 (3A), U25.4 (2A), U25.5 (2B), U25.9 (4B), U50.10 (4A), U50.12 (3B), U50.13 (3A), U50.7 (GND), U50.9 (4B), U12.1 (OE#), U12.10 (GND), U12.5 (D3), U12.6 (D4), U12.7 (D5), U12.8 (D6), U12.9 (D7), U14.7 (GND), U15.12 (3B), U15.13 (3A), U15.7 (GND), U19.7 (GND), U23.7 (GND), U3.40 (GND), U42.5 (1A), U42.6 (1B), U42.7 (GND), U46.1 (OE#), U46.10 (GND), U47.8 (GND), U48.2 (A0), U48.3 (A1), U48.7 (GND), U49.11 (I4), U49.13 (I5), U49.3 (I1), U49.5 (I2), U49.7 (GND), U49.9 (I3), U6.1 (OE#), U6.10 (GND), U6.6 (D4), U6.7 (D5), U6.8 (D6), U6.9 (D7); no longer U11.11 (I4)
- net at U24.10 (4A), U27.12 (4A), U30.14 (D5)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: now also U14.12 (3A), U23.9 (I3), U3.4 (A3), U47.12 (A3); no longer U13.12 (A3), U18.9 (I3), U21.12 (3A)
- net at U28.1 (1A), U30.15 (D4), U31.14 (D5)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: now also U13.5 (A0), U21.1 (0A), U19.1 (1A), U23.11 (I4), U3.5 (A4); no longer U18.11 (I4), U25.1 (1A)
- net at U28.5 (2A), U30.1 (D3), U31.15 (D4)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: now also U13.3 (A1), U21.5 (1A), U19.4 (2A), U23.13 (I5), U3.6 (A5); no longer U18.13 (I5), U25.4 (2A)
- net at U28.8 (3A), U30.2 (D2), U31.1 (D3)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: now also U13.14 (A2), U18.1 (I0), U21.8 (2A), U19.13 (3A), U3.7 (A6); no longer U25.13 (3A)
- net at U28.12 (4A), U30.3 (D1), U31.2 (D2)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: now also U13.12 (A3), U18.3 (I1), U21.12 (3A), U19.10 (4A), U3.8 (A7); no longer U25.10 (4A)
- net at U24.2 (1B), U27.2 (1B), U30.11 (A0)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: now also U14.2 (0B), U3.9 (B0), U47.6 (B0); no longer U13.6 (B0), U21.2 (0B)
- net at U2.10 (RX_Extend_(from_controller)): now also U15.9 (4B), U3.37 (RX_extend_half_cycle)
- net at U2.11 (TX_0): now also U50.2 (1B), U42.2 (0B), U6.5 (D3)
- net at U2.15 (RX_0): now also U6.2 (D0)
- net at U2.16 (RX_1): now also U6.3 (D1)
- net at U2.17 (RX_2): now also U6.4 (D2)
- net at U16.19 (Q0), U17.19 (Q0), U2.20 (D0)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: now also U3.24 (O0), U46.2 (D0)
- net at U16.18 (Q1), U17.18 (Q1), U2.21 (D1)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: now also U3.25 (O1), U46.3 (D1)
- net at U16.17 (Q2), U17.17 (Q2), U2.22 (D2)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: now also U3.26 (O2), U46.4 (D2)
- net at U16.16 (Q3), U17.16 (Q3), U2.23 (D3)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: now also U3.27 (O3), U46.5 (D3)
- net at U16.15 (Q4), U17.15 (Q4), U2.24 (D4)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: now also U3.28 (O4), U46.6 (D4)
- net at U16.14 (Q5), U17.14 (Q5), U2.25 (D5)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: now also U3.29 (O5), U46.7 (D5)
- net at U16.13 (Q6), U17.13 (Q6), U2.26 (D6)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: now also U3.30 (O6), U46.8 (D6)
- net at U16.12 (Q7), U17.12 (Q7), U2.27 (D7)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: now also U3.31 (O7), U46.9 (D7)
- net at U2.3 (CLK): now also U11.11 (I4), U12.11 (CLK), U3.36 (CLK)
- net at U2.4 (Enable): now also U15.5 (2B), U3.38 (Enable)
- net at U2.7 (TX_Ready): now also U42.10 (Q2)
- net at U10.10 (O4): now also U3.18 (S10#)
- net at U11.8 (03): now also U3.23 (S15#)
- net at U10.12 (O5): now also U3.19 (S11#)
- net at U11.2 (O0): now also U3.20 (S12#)
- net at U11.4 (O1): now also U3.21 (S13#)
- net at U11.6 (O2): now also U3.22 (S14#)
- net at U16.7 (D5): now also U13.1 (Σ1)
- net at U16.9 (D7): now also U13.10 (Σ3)
- net at U16.8 (D6): now also U13.13 (Σ2)
- net at U16.6 (D4): now also U13.4 (Σ0)
- net at U13.9 (C_OUT): now also U17.2 (D0)
- net at U26.6 (D4): now also U19.3 (1Q); no longer U25.3 (1Q)
- net at U26.7 (D5): now also U19.6 (2Q); no longer U25.6 (2Q)
- net at U26.8 (D6): now also U19.11 (3Q); no longer U25.11 (3Q)
- net at U26.9 (D7): now also U19.8 (4Q); no longer U25.8 (4Q)
- net at U4.11 (CLK): now also U12.2 (D0), U6.19 (Q0)
- net at U10.11 (I4), U8.13 (Y2): now also U48.5 (A3)
- net at U10.13 (I5), U8.12 (Y3): now also U48.4 (A2)
- net at U5.11 (CLK): now also U12.3 (D1), U6.18 (Q1)
- net at U13.7 (C_IN): now also U47.9 (C_OUT)
- net at U22.2 (D0): now also U14.3 (Q0); no longer U21.3 (Q0)
- net at U22.3 (D1): now also U14.4 (Q1); no longer U21.4 (Q1)
- net at U22.4 (D2): now also U14.10 (Q2); no longer U21.10 (Q2)
- net at U22.5 (D3): now also U14.11 (Q3); no longer U21.11 (Q3)
- net at U22.6 (D4): now also U21.3 (Q0)
- net at U22.7 (D5): now also U21.4 (Q1)
- net at U22.8 (D6): now also U21.10 (Q2)
- net at U22.9 (D7): now also U21.11 (Q3)
- net at U50.3 (1Q): now also U42.9 (2B)
- net at U50.6 (2Q): now also U42.8 (2A)
- net at U20.8 (D6): now also U18.2 (O0)
- net at U20.9 (D7): now also U18.4 (O1)
- net at U41.6 (1Q): now also U25.1 (1A)
- net at U41.8 (2Q): now also U25.2 (1B)
- net at U43.2 (D0): now also U25.3 (1Q)
- net at U16.3 (D1): now also U47.1 (Σ1); no longer U13.1 (Σ1)
- net at U16.5 (D3): now also U47.10 (Σ3); no longer U13.10 (Σ3)
- net at U16.4 (D2): now also U47.13 (Σ2); no longer U13.13 (Σ2)
- net at U16.2 (D0): now also U47.4 (Σ0); no longer U13.4 (Σ0)
- net at U11.13 (I5): now also U15.6 (2Q)
- net at U11.1 (I0), U8.11 (Y4): now also U48.9 (B0)
- net at U11.10 (O4): now also U6.11 (CLK)
- net at U11.3 (I1), U8.10 (Y5): now also U48.10 (B1)
- net at U11.5 (I2), U8.9 (Y6): now also U48.11 (B2)
- net at U11.9 (I3), U8.7 (Y7): now also U48.12 (B3)
- net at U20.6 (D4): now also U23.10 (O4); no longer U18.10 (O4)
- net at U20.7 (D5): now also U23.12 (O5); no longer U18.12 (O5)
- net at U20.2 (D0): now also U23.2 (O0); no longer U18.2 (O0)
- net at U20.3 (D1): now also U23.4 (O1); no longer U18.4 (O1)
- net at U20.4 (D2): now also U23.6 (O2); no longer U18.6 (O2)
- net at U20.5 (D3): now also U23.8 (03); no longer U18.8 (03)
- new net: U15.3 (1Q), U42.1 (0A)
- new net: U42.11 (Q3), U49.1 (I0), U50.4 (2A)
- new net: U42.12 (3A), U48.1 (OA)
- new net: U42.13 (3B), U48.13 (OB)
- new net: U15.4 (2A), U42.3 (Q0)
- new net: U15.10 (4A), U49.2 (O0), U50.1 (1A)
- new net: U3.17 (C0), U46.19 (Q0), U47.7 (C_IN)
- new net: U3.32 (TX_Ready), U50.5 (2B)
- new net: U12.19 (Q0), U3.33 (A_updated)
- new net: U12.18 (Q1), U3.34 (B_updated)
- new net: U12.17 (Q2), U3.35 (C_updated)
- new net: U12.4 (D2), U46.11 (CLK), U6.17 (Q2)
- new net: U15.1 (1A), U6.16 (Q3)
- new net: U15.2 (1B), U15.8 (4Q)
- no-connect marks 37 -> 49
Other:
- note added: "0 - Built-in"
- note added: "1 - Extension"
- note added: "Extension - TX Ready"
- note added: "Falling"
- note added: "G0"
- note added: "G1"
- note added: "G2 - Opcode decode EN"
- note added: "G3"
- note added: "Inverters for active low inputs"
- note added: "OE#"
- note added: "Opcode decoder"
- note added: "Opcode region extension"
- note added: "RX Extend enable only when built-in"
- note added: "Rising"
- note added: "TX Ready"
- note added: "TX ready select"
- moved on the sheet: U1, U2, U7, U8
